Commit message: removed robot_ prefix

File: src/map_server/models/rb_theron/rb_theron.urdf (robot description, URDF)
Before this commit: robot rb_theron, 32 links, 31 joints
Links:
- removed link robot_bottom_cover_link
- removed link robot_front_laser_base_link
- removed link robot_front_laser_link
- removed link robot_front_realsense_camera_camera_depth_frame
- removed link robot_front_realsense_camera_camera_depth_optical_frame
- removed link robot_front_realsense_camera_camera_fisheye_frame
- removed link robot_front_realsense_camera_camera_fisheye_optical_frame
- removed link robot_front_realsense_camera_camera_left_ir_frame
- removed link robot_front_realsense_camera_camera_left_ir_optical_frame
- removed link robot_front_realsense_camera_camera_link
- removed link robot_front_realsense_camera_camera_right_ir_frame
- removed link robot_front_realsense_camera_camera_right_ir_optical_frame
- removed link robot_front_rgbd_camera_depth_frame
- removed link robot_front_rgbd_camera_depth_optical_frame
- removed link robot_front_rgbd_camera_link
- removed link robot_front_rgbd_camera_rgb_frame
- removed link robot_front_rgbd_camera_rgb_optical_frame
- removed link robot_imu_link
- removed link robot_left_wheel_link
- removed link robot_leftcastorsupport
- removed link robot_leftcastorwheel
- removed link robot_leftrsupport
- removed link robot_leftsupport
- removed link robot_leftwheel
- removed link robot_right_wheel_link
- removed link robot_rightcastorsupport
- removed link robot_rightcastorwheel
- removed link robot_rightrsupport
- removed link robot_rightsupport
- removed link robot_rightwheel
- added link bottom_cover_link, mass 2.0; collision mesh filename=package://rb_theron/meshes/bases/mcq_prototype_bottom_cover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; visual mesh filename=package://rb_theron/meshes/bases/mcq_prototype_bottom_cover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
- added link front_laser_base_link, mass 0.67; collision mesh filename=package://robotnik_sensors/meshes/sick_nanoscan3.stl; visual mesh filename=package://robotnik_sensors/meshes/sick_nanoscan3.stl
- added link front_laser_link
- added link front_realsense_camera_camera_depth_frame
- added link front_realsense_camera_camera_depth_optical_frame
- added link front_realsense_camera_camera_fisheye_frame
- added link front_realsense_camera_camera_fisheye_optical_frame
- added link front_realsense_camera_camera_left_ir_frame
- added link front_realsense_camera_camera_left_ir_optical_frame
- added link front_realsense_camera_camera_link, mass 0.1; collision box size=0.025 0.1 0.025; visual mesh filename=package://robotnik_sensors/meshes/intel_r430.dae
- added link front_realsense_camera_camera_right_ir_frame
- added link front_realsense_camera_camera_right_ir_optical_frame
- added link front_rgbd_camera_depth_frame, mass 0.001
- added link front_rgbd_camera_depth_optical_frame, mass 0.001
- added link front_rgbd_camera_link, mass 0.001; collision mesh filename=package://robotnik_sensors/meshes/orbbec_astra.dae; visual mesh filename=package://robotnik_sensors/meshes/orbbec_astra.dae
- added link front_rgbd_camera_rgb_frame, mass 0.297
- added link front_rgbd_camera_rgb_optical_frame, mass 0.001
- added link imu_link, mass 0.05; collision box size=.001 .001 .001; visual box size=0.001 0.001 0.001
- added link left_wheel_link, mass 0.25; collision cylinder length=0.025 radius=0.0756; visual cylinder length=0.025 radius=0.0756
- added link leftcastorsupport, mass 1.5; collision mesh filename=package://rb_theron/meshes/wheels/mcq_prototype_base_castor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; visual mesh filename=package://rb_theron/meshes/wheels/mcq_prototype_base_castor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
- added link leftcastorwheel, mass 0.25; collision cylinder length=0.025 radius=0.05; visual cylinder length=0.025 radius=0.05
- added link leftrsupport, mass 1.5; collision mesh filename=package://rb_theron/meshes/rocker/mcq_prototype_rocker_l.dae; visual mesh filename=package://rb_theron/meshes/rocker/mcq_prototype_rocker_l.dae
- added link leftsupport, mass 1.5; collision mesh filename=package://rb_theron/meshes/wheels/mcq_prototype_base_castor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; visual mesh filename=package://rb_theron/meshes/wheels/mcq_prototype_base_castor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
- added link leftwheel, mass 0.25; collision cylinder length=0.025 radius=0.05; visual cylinder length=0.025 radius=0.05
- added link right_wheel_link, mass 0.25; collision cylinder length=0.025 radius=0.0756; visual cylinder length=0.025 radius=0.0756
- added link rightcastorsupport, mass 1.5; collision mesh filename=package://rb_theron/meshes/wheels/mcq_prototype_base_castor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; visual mesh filename=package://rb_theron/meshes/wheels/mcq_prototype_base_castor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
- added link rightcastorwheel, mass 0.25; collision cylinder length=0.025 radius=0.05; visual cylinder length=0.025 radius=0.05
- added link rightrsupport, mass 1.5; collision mesh filename=package://rb_theron/meshes/rocker/mcq_prototype_rocker_r.dae; visual mesh filename=package://rb_theron/meshes/rocker/mcq_prototype_rocker_r.dae
- added link rightsupport, mass 1.5; collision mesh filename=package://rb_theron/meshes/wheels/mcq_prototype_base_castor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; visual mesh filename=package://rb_theron/meshes/wheels/mcq_prototype_base_castor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
- added link rightwheel, mass 0.25; collision cylinder length=0.025 radius=0.05; visual cylinder length=0.025 radius=0.05
Joints:
- removed joint robot_bottom_cover_joint
- removed joint robot_front_laser_base_joint
- removed joint robot_front_laser_joint
- removed joint robot_front_realsense_camera_camera_depth_joint
- removed joint robot_front_realsense_camera_camera_depth_optical_joint
- removed joint robot_front_realsense_camera_camera_fisheye_joint
- removed joint robot_front_realsense_camera_camera_fisheye_optical_joint
- removed joint robot_front_realsense_camera_camera_joint
- removed joint robot_front_realsense_camera_camera_left_ir_joint
- removed joint robot_front_realsense_camera_camera_left_ir_optical_joint
- removed joint robot_front_realsense_camera_camera_right_ir_joint
- removed joint robot_front_realsense_camera_camera_right_ir_optical_joint
- removed joint robot_front_rgbd_camera_depth_joint
- removed joint robot_front_rgbd_camera_depth_optical_joint
- removed joint robot_front_rgbd_camera_joint
- removed joint robot_front_rgbd_camera_rgb_joint
- removed joint robot_front_rgbd_camera_rgb_optical_joint
- removed joint robot_imu_joint
- removed joint robot_left_wheel_joint
- removed joint robot_leftcastorjoint_support
- removed joint robot_leftcastorjoint_wheel
- removed joint robot_leftjoint_rsupport
- removed joint robot_leftjoint_support
- removed joint robot_leftjoint_wheel
- removed joint robot_right_wheel_joint
- removed joint robot_rightcastorjoint_support
- removed joint robot_rightcastorjoint_wheel
- removed joint robot_rightjoint_rsupport
- removed joint robot_rightjoint_support
- removed joint robot_rightjoint_wheel
- added joint bottom_cover_joint: type fixed, parent base_link, child bottom_cover_link, origin xyz=0 0 0 rpy=0 0 0
- added joint front_laser_base_joint: type fixed, parent base_link, child front_laser_base_link, origin xyz=0.250 0.0 0.1643 rpy=0 3.1416 3.1416
- added joint front_laser_joint: type fixed, parent front_laser_base_link, child front_laser_link, origin xyz=0.0 0 0.0505 rpy=0 0 0
- added joint front_realsense_camera_camera_depth_joint: type fixed, parent front_realsense_camera_camera_link, child front_realsense_camera_camera_depth_frame, origin xyz=0.0 -0.0115 0.0 rpy=0 0 0
- added joint front_realsense_camera_camera_depth_optical_joint: type fixed, parent front_realsense_camera_camera_depth_frame, child front_realsense_camera_camera_depth_optical_frame, origin xyz=0 0 0 rpy=-1.57079632679 0 -1.57079632679
- added joint front_realsense_camera_camera_fisheye_joint: type fixed, parent front_realsense_camera_camera_depth_frame, child front_realsense_camera_camera_fisheye_frame, origin xyz=0 0.044 0 rpy=0 0 0
- added joint front_realsense_camera_camera_fisheye_optical_joint: type fixed, parent front_realsense_camera_camera_fisheye_frame, child front_realsense_camera_camera_fisheye_optical_frame, origin xyz=0 0 0 rpy=-1.57079632679 0 -1.57079632679
- added joint front_realsense_camera_camera_joint: type fixed, parent base_link, child front_realsense_camera_camera_link, origin xyz=0.3305 0.0 0.1468 rpy=0 0 0
- added joint front_realsense_camera_camera_left_ir_joint: type fixed, parent front_realsense_camera_camera_depth_frame, child front_realsense_camera_camera_left_ir_frame, origin xyz=0 -0.021 0 rpy=0 0 0
- added joint front_realsense_camera_camera_left_ir_optical_joint: type fixed, parent front_realsense_camera_camera_left_ir_frame, child front_realsense_camera_camera_left_ir_optical_frame, origin xyz=0 0 0 rpy=-1.57079632679 0 -1.57079632679
- added joint front_realsense_camera_camera_right_ir_joint: type fixed, parent front_realsense_camera_camera_depth_frame, child front_realsense_camera_camera_right_ir_frame, origin xyz=0 0.029 0 rpy=0 0 0
- added joint front_realsense_camera_camera_right_ir_optical_joint: type fixed, parent front_realsense_camera_camera_right_ir_frame, child front_realsense_camera_camera_right_ir_optical_frame, origin xyz=0 0 0 rpy=-1.57079632679 0 -1.57079632679
- added joint front_rgbd_camera_depth_joint: type fixed, parent front_rgbd_camera_link, child front_rgbd_camera_depth_frame, origin xyz=0.0 0.0375 0.0150 rpy=0 0 0
- added joint front_rgbd_camera_depth_optical_joint: type fixed, parent front_rgbd_camera_depth_frame, child front_rgbd_camera_depth_optical_frame, origin xyz=0 0 0 rpy=-1.57079632679 0 -1.57079632679
- added joint front_rgbd_camera_joint: type fixed, parent base_link, child front_rgbd_camera_link, origin xyz=0.3305 0.0 0.1898 rpy=0 0 0
- added joint front_rgbd_camera_rgb_joint: type fixed, parent front_rgbd_camera_link, child front_rgbd_camera_rgb_frame, origin xyz=0.0 0.0125 0.0150 rpy=0.0 0.0 0.0
- added joint front_rgbd_camera_rgb_optical_joint: type fixed, parent front_rgbd_camera_rgb_frame, child front_rgbd_camera_rgb_optical_frame, origin xyz=0.0 0.0 0.0 rpy=-1.57079632679 0 -1.57079632679
- added joint imu_joint: type fixed, parent base_link, child imu_link, origin xyz=-0.1975 0.0 0.1598 rpy=0 0 0, axis 1 0 0
- added joint left_wheel_joint: type continuous, parent leftrsupport, child left_wheel_link, origin xyz=-0.1175 0.079 -0.0428 rpy=0 0 0, axis 0 1 0, limit effort=100 velocity=100
- added joint leftcastorjoint_support: type continuous, parent leftrsupport, child leftcastorsupport, origin xyz=0.1175 0.01 0.002 rpy=0 0 0, axis 0 0 1, limit effort=100 velocity=100
- added joint leftcastorjoint_wheel: type continuous, parent leftcastorsupport, child leftcastorwheel, origin xyz=-0.033 0.0 -0.071 rpy=0 0 0, axis 0 1 0, limit effort=100 velocity=100
- added joint leftjoint_rsupport: type revolute, parent base_link, child leftrsupport, origin xyz=0.1175 0.1725 0.0428 rpy=0 0 0, axis 0 1 0, limit lower=-0.5 upper=0.5 effort=100 velocity=100
- added joint leftjoint_support: type continuous, parent base_link, child leftsupport, origin xyz=-0.235 0.1725 0.0428 rpy=0 0 0, axis 0 0 1, limit effort=100 velocity=100
- added joint leftjoint_wheel: type continuous, parent leftsupport, child leftwheel, origin xyz=-0.033 0.0 -0.071 rpy=0 0 0, axis 0 1 0, limit effort=100 velocity=100
- added joint right_wheel_joint: type continuous, parent rightrsupport, child right_wheel_link, origin xyz=-0.1175 -0.079 -0.0428 rpy=0 0 0, axis 0 1 0, limit effort=100 velocity=100
- added joint rightcastorjoint_support: type continuous, parent rightrsupport, child rightcastorsupport, origin xyz=0.1175 0.01 0.002 rpy=0 0 0, axis 0 0 1, limit effort=100 velocity=100
- added joint rightcastorjoint_wheel: type continuous, parent rightcastorsupport, child rightcastorwheel, origin xyz=-0.033 0.0 -0.071 rpy=0 0 0, axis 0 1 0, limit effort=100 velocity=100
- added joint rightjoint_rsupport: type revolute, parent base_link, child rightrsupport, origin xyz=0.1175 -0.1725 0.0428 rpy=0 0 0, axis 0 1 0, limit lower=-0.5 upper=0.5 effort=100 velocity=100
- added joint rightjoint_support: type continuous, parent base_link, child rightsupport, origin xyz=-0.235 -0.1725 0.0428 rpy=0 0 0, axis 0 0 1, limit effort=100 velocity=100
- added joint rightjoint_wheel: type continuous, parent rightsupport, child rightwheel, origin xyz=-0.033 0.0 -0.071 rpy=0 0 0, axis 0 1 0, limit effort=100 velocity=100

Commit message: Cleaned up sensor files and added top laser sensor visualization to rb_theron

File: src/map_server/models/rb_theron/rb_theron.urdf (robot description, URDF)
Before this commit: robot rb_theron, 32 links, 31 joints
Links:
- added link top_laser_base_link, mass 0.67; collision mesh filename=package://robotnik_sensors/meshes/sensors/sick_nanoscan3.dae; visual mesh filename=package://robotnik_sensors/meshes/sensors/sick_nanoscan3.dae
- added link top_laser_link
- link front_laser_base_link: geometry collision mesh filename=package://robotnik_sensors/meshes/sick_nanoscan3.dae; visual mesh filename=package://robotnik_sensors/meshes/sick_nanoscan3.dae
Joints:
- added joint top_laser_base_joint: type fixed, parent base_link, child top_laser_base_link, origin xyz=0.250 0.0 0.2896 rpy=0 0 0
- added joint top_laser_joint: type fixed, parent top_laser_base_link, child top_laser_link, origin xyz=0.0 0 0.0505 rpy=0 0 0

Commit message: Fixed urdf to find all .dae files including wheels

File: src/map_server/models/rb_theron/rb_theron.urdf (robot description, URDF)
Before this commit: robot rb_theron, 34 links, 33 joints
Links:
- link base_link: geometry collision mesh filename=meshes/bases/theron_base.stl; visual mesh filename=meshes/bases/theron_base.stl
- link bottom_cover_link: geometry collision mesh filename=meshes/bases/mcq_prototype_bottom_cover.dae; visual mesh filename=meshes/bases/mcq_prototype_bottom_cover.dae
- link front_laser_base_link: geometry collision mesh filename=meshes/sensors/sick_nanoscan3.dae; visual mesh filename=meshes/sensors/sick_nanoscan3.dae
- link front_realsense_camera_camera_link: geometry collision box size=0.025 0.1 0.025; visual mesh filename=meshes/sensors/intel_r430.dae
- link front_rgbd_camera_link: geometry collision mesh filename=meshes/sensors/orbbec_astra.dae; visual mesh filename=meshes/sensors/orbbec_astra.dae
- link leftcastorsupport: geometry collision mesh filename=meshes/wheels/mcq_prototype_base_castor.dae; visual mesh filename=meshes/wheels/mcq_prototype_base_castor.dae
- link leftrsupport: geometry collision mesh filename=meshes/rocker/mcq_prototype_rocker_l.dae; visual mesh filename=meshes/rocker/mcq_prototype_rocker_l.dae
- link leftsupport: geometry collision mesh filename=meshes/wheels/mcq_prototype_base_castor.dae; visual mesh filename=meshes/wheels/mcq_prototype_base_castor.dae
- link rightcastorsupport: geometry collision mesh filename=meshes/wheels/mcq_prototype_base_castor.dae; visual mesh filename=meshes/wheels/mcq_prototype_base_castor.dae
- link rightrsupport: geometry collision mesh filename=meshes/rocker/mcq_prototype_rocker_r.dae; visual mesh filename=meshes/rocker/mcq_prototype_rocker_r.dae
- link rightsupport: geometry collision mesh filename=meshes/wheels/mcq_prototype_base_castor.dae; visual mesh filename=meshes/wheels/mcq_prototype_base_castor.dae
- link top_laser_base_link: geometry collision mesh filename=meshes/sensors/sick_nanoscan3.dae; visual mesh filename=meshes/sensors/sick_nanoscan3.dae

Commit message: Fix position of rightcastorjoint_support

File: src/map_server/models/rb_theron/rb_theron.urdf (robot description, URDF)
Before this commit: robot rb_theron, 34 links, 33 joints
Joints:
- joint rightcastorjoint_support: origin xyz=0.1175 0.01 0.002 rpy=0 0 0 -> xyz=0.1175 -0.01 0.002 rpy=0 0 0

Commit message: Major Fix for rb_theron model

File: src/map_server/models/rb_theron/rb_theron.urdf (robot description, URDF)
Before this commit: robot rb_theron, 34 links, 33 joints
Joints:
- joint front_laser_joint: origin xyz=0.0 0 0.0505 rpy=0 0 0 -> xyz=0.0 0.0 0.0505 rpy=3.14159265359 0 0
