Commit message: Fixing frame displacement for camera

File: src/simulation/tiplu_world/models/rb_theron/rb_theron.urdf (robot description, URDF)
Before this commit: robot rb_theron, 34 links, 33 joints
Joints:
- joint front_rgbd_camera_depth_joint: origin xyz=0.0 0.0375 0.0150 rpy=0 0 0 -> xyz=0.0 0.0 0.0 rpy=0 0 0
- joint front_rgbd_camera_joint: origin xyz=0.3305 0.0 0.1898 rpy=0 0 0 -> xyz=0.25 0 0.265 rpy=0 0 0
- joint front_rgbd_camera_rgb_joint: origin xyz=0.0 0.0125 0.0150 rpy=0.0 0.0 0.0 -> xyz=0.0 0.0 0.0 rpy=0.0 0.0 0.0
