Commit message: small fix for intel_430 collision origin

File: src/ros2/robot_description/robotnik_sensors/urdf/intel_r430.urdf.xacro (robot description, xacro)
@@ -43,5 +43,5 @@
       </visual>
       <collision>
-        <origin xyz="${-r430_cam_depth/2} 0.0 0.0" rpy="0 0 0"/>
+        <origin xyz="0 ${-r430_cam_mount_from_center_offset} 0" rpy="0 0 0"/>
         <geometry>
         <box size="${r430_cam_depth} ${r430_cam_width} ${r430_cam_height}"/>

Commit message: Fixing camera positions for now - not sure if this is the final solution.

File: src/ros2/robot_description/robotnik_sensors/urdf/intel_r430.urdf.xacro (robot description, xacro)
@@ -30,7 +30,7 @@
       <xacro:insert_block name="origin" />
       <parent link="${parent}"/>
-      <child link="${prefix}_camera_link" />
-    </joint>
-    <link name="${prefix}_camera_link">
+      <child link="${prefix}_link" />
+    </joint>
+    <link name="${prefix}_link">
       <visual>
         <!-- origin xyz="0 ${-r430_cam_mount_from_center_offset} ${r430_cam_height/2}" rpy="${M_PI/2} 0 ${M_PI/2}"/ -->
@@ -63,5 +63,5 @@
     <joint name="${prefix}_camera_depth_joint" type="fixed">
       <origin xyz="${r430_cam_depth_px} ${r430_cam_depth_py} ${r430_cam_depth_pz}" rpy="0 0 0"/>
-      <parent link="${prefix}_camera_link"/>
+      <parent link="${prefix}_link"/>
       <child link="${prefix}_camera_depth_frame" />
     </joint>
@@ -123,7 +123,6 @@
   <xacro:macro name="sensor_r430_gazebo">
     <!-- gazebo reference="${prefix}_rgb_base_link" -->
-    <gazebo reference="${sensor_link_name}_color_link">
+    <gazebo reference="${prefix}_link">
       <sensor name="${prefix}_color_link" type="camera">
-				<pose relative_to='${sensor_link_name}_color_link'>-0.1 0 0 0 0 0</pose>
 				<topic>${prefix_topic}/color</topic>
         <camera name="r430">
@@ -148,8 +147,5 @@
         <visualize>1</visualize>
       </sensor>
-    </gazebo>
-    <gazebo reference="${prefix}_camera_link">
       <sensor name="${prefix}_ired1" type="camera">
-      <pose relative_to='${prefix}_camera_depth_frame'>-0.2 0 0 0 0 0</pose>
       <topic>${prefix_topic}/${prefix}/ired1</topic>
         <camera name="r430">
@@ -175,5 +171,4 @@
       </sensor>
       <sensor name="${prefix}_ired2" type="camera">
-        <pose relative_to='${prefix}_camera_depth_frame'>0.2 0 0 0 0 0</pose>
         <topic>${prefix_topic}/${prefix}/ired2</topic>
         <camera name="r430">
@@ -198,8 +193,5 @@
         <visualize>0</visualize>
       </sensor>
-    </gazebo>
-    <gazebo reference="${sensor_link_name}_depth_link">
       <sensor name="${prefix}_depth_link" type="depth">
-        <pose relative_to='${sensor_link_name}_depth_link'>0.1 0 0 0 0 0</pose>
         <topic>${prefix_topic}/${prefix}/depth</topic>
         <camera name="r430">

Commit message: fixed point cloud data rotation

File: src/ros2/robot_description/robotnik_sensors/urdf/intel_r430.urdf.xacro (robot description, xacro)
@@ -68,5 +68,5 @@
     <link name="${prefix}_camera_depth_frame"/>
     <joint name="${prefix}_camera_depth_optical_joint" type="fixed">
-      <origin xyz="0 0 0" rpy="${-M_PI/2} 0 ${-M_PI/2}" />
+      <origin xyz="0 0 0" rpy="0 0 0" />
       <parent link="${prefix}_camera_depth_frame" />
       <child link="${sensor_link_name}_depth_link" />
@@ -213,5 +213,5 @@
         <always_on>1</always_on>
         <update_rate>15</update_rate>
-        <visualize>0</visualize>
+        <visualize>1</visualize>
       </sensor>
     </gazebo>
