Commit message: Updating moveit2_drawer package and moveit_launch

File: src/ros2/simulation_ignition/moveit2_drawer/config/rb_theron.ros2_control.xacro (robot description, xacro)
@@ -8,8 +8,15 @@
                 <plugin>mock_components/GenericSystem</plugin>
             </hardware>
-            <joint name="top_drawer_joint">
+            <joint name="first_drawer_joint">
                 <command_interface name="position"/>
                 <state_interface name="position">
-                  <param name="initial_value">${initial_positions['top_drawer_joint']}</param>
+                  <param name="initial_value">${initial_positions['first_drawer_joint']}</param>
+                </state_interface>
+                <state_interface name="velocity"/>
+            </joint>
+            <joint name="second_drawer_joint">
+                <command_interface name="position"/>
+                <state_interface name="position">
+                  <param name="initial_value">${initial_positions['second_drawer_joint']}</param>
                 </state_interface>
                 <state_interface name="velocity"/>

Commit message: moveit2 can now actuate all 5 drawers of the robot

File: src/ros2/simulation_ignition/moveit2_drawer/config/rb_theron.ros2_control.xacro (robot description, xacro)
@@ -8,15 +8,36 @@
                 <plugin>mock_components/GenericSystem</plugin>
             </hardware>
-            <joint name="first_drawer_joint">
+            <joint name="drawer_1_joint">
                 <command_interface name="position"/>
                 <state_interface name="position">
-                  <param name="initial_value">${initial_positions['first_drawer_joint']}</param>
+                  <param name="initial_value">${initial_positions['drawer_1_joint']}</param>
                 </state_interface>
                 <state_interface name="velocity"/>
             </joint>
-            <joint name="second_drawer_joint">
+            <joint name="drawer_2_joint">
                 <command_interface name="position"/>
                 <state_interface name="position">
-                  <param name="initial_value">${initial_positions['second_drawer_joint']}</param>
+                  <param name="initial_value">${initial_positions['drawer_2_joint']}</param>
+                </state_interface>
+                <state_interface name="velocity"/>
+            </joint>
+            <joint name="drawer_3_joint">
+                <command_interface name="position"/>
+                <state_interface name="position">
+                  <param name="initial_value">${initial_positions['drawer_3_joint']}</param>
+                </state_interface>
+                <state_interface name="velocity"/>
+            </joint>
+            <joint name="drawer_4_joint">
+                <command_interface name="position"/>
+                <state_interface name="position">
+                  <param name="initial_value">${initial_positions['drawer_4_joint']}</param>
+                </state_interface>
+                <state_interface name="velocity"/>
+            </joint>
+            <joint name="drawer_5_joint">
+                <command_interface name="position"/>
+                <state_interface name="position">
+                  <param name="initial_value">${initial_positions['drawer_5_joint']}</param>
                 </state_interface>
                 <state_interface name="velocity"/>
