Commit message: Completely removed Gazebo-Classic

File: src/ros2/simulation/moveit2_drawer/config/rb_theron.ros2_control.xacro (robot description, xacro)
@@ -3,17 +3,41 @@
     <xacro:macro name="rb_theron_ros2_control" params="name initial_positions_file">
         <xacro:property name="initial_positions" value="${load_yaml(initial_positions_file)['initial_positions']}"/>
-        <plugin filename="libgazebo_ros2_control.so" name="gazebo_ros2_control">
-				<robot_sim_type>gazebo_ros2_control/GazeboSystem</robot_sim_type>
-				<parameters>$(find moveit2_drawer)/config/ros2_controllers.yaml</parameters>
-        </plugin>
         <ros2_control name="${name}" type="system">
             <hardware>
                 <!-- By default, set up controllers for simulation. This won't work on real hardware -->
-                <plugin>gazebo_ros2_control/GazeboSystem</plugin>
+                <plugin>mock_components/GenericSystem</plugin>
             </hardware>
-            <joint name="top_drawer_joint">
+            <joint name="drawer_1_joint">
                 <command_interface name="position"/>
                 <state_interface name="position">
-                  <param name="initial_value">${initial_positions['top_drawer_joint']}</param>
+                  <param name="initial_value">${initial_positions['drawer_1_joint']}</param>
+                </state_interface>
+                <state_interface name="velocity"/>
+            </joint>
+            <joint name="drawer_2_joint">
+                <command_interface name="position"/>
+                <state_interface name="position">
+                  <param name="initial_value">${initial_positions['drawer_2_joint']}</param>
+                </state_interface>
+                <state_interface name="velocity"/>
+            </joint>
+            <joint name="drawer_3_joint">
+                <command_interface name="position"/>
+                <state_interface name="position">
+                  <param name="initial_value">${initial_positions['drawer_3_joint']}</param>
+                </state_interface>
+                <state_interface name="velocity"/>
+            </joint>
+            <joint name="drawer_4_joint">
+                <command_interface name="position"/>
+                <state_interface name="position">
+                  <param name="initial_value">${initial_positions['drawer_4_joint']}</param>
+                </state_interface>
+                <state_interface name="velocity"/>
+            </joint>
+            <joint name="drawer_5_joint">
+                <command_interface name="position"/>
+                <state_interface name="position">
+                  <param name="initial_value">${initial_positions['drawer_5_joint']}</param>
                 </state_interface>
                 <state_interface name="velocity"/>
