Commit message: Adding hook for gripper

File: src/ros2/robot_description/rb_theron_common/rb_theron_description/urdf/door_opening_mechanism/door_opening_gripper.urdf.xacro (robot description, xacro)
@@ -1,14 +1,16 @@
 <?xml version="1.0"?>
 <robot name="door_opening_gripper" xmlns:xacro="http://www.ros.org/wiki/xacro">
-    <xacro:macro name="box_inertia_robot" params="m x y z">
-        <inertia  ixx="${m*(y*y+z*z)/12}" ixy = "0" ixz = "0"
-                iyy="${m*(x*x+z*z)/12}" iyz = "0"
-                izz="${m*(x*x+z*z)/12}" />
-    </xacro:macro>
     <xacro:macro name="door_opening_gripper" params="prefix parent *origin">
-    <!-- <xacro:include filename="$(find rb_theron_description)/urdf/door_opening_mechanism/alu_profile.urdf.xacro" /> -->
-    <xacro:alu_profile prefix="${prefix}" suffix="gripper" parent="${parent}" x="0.03" y="0.03" z="0.3" r="0" g="1" b="0">
-        <xacro:insert_block name="origin" />
-	</xacro:alu_profile>
+        <xacro:include filename="$(find rb_theron_description)/urdf/door_opening_mechanism/alu_profile.urdf.xacro" />
+        <xacro:alu_profile prefix="${prefix}" suffix="gripper" parent="${parent}" x="0.03" y="0.03" z="0.3" r="0" g="1" b="0">
+            <xacro:insert_block name="origin" />
+        </xacro:alu_profile>
+        <xacro:include filename="$(find rb_theron_description)/urdf/door_opening_mechanism/hook.urdf.xacro" />
+        <xacro:hook prefix="${prefix}" suffix="left_hook" parent="${prefix}alu_profile_link_gripper" r="0" g="0" b="1">
+            <origin xyz="-0.045 -0.01 0.13" rpy="0 0 0"/>
+        </xacro:hook>
+        <xacro:hook prefix="${prefix}" suffix="right_hook" parent="${prefix}alu_profile_link_gripper" r="0" g="0" b="1">
+            <origin xyz="-0.045 -0.01 -0.13" rpy="0 0 0"/>
+        </xacro:hook>
     </xacro:macro>
 </robot>

File: src/ros2/robot_description/rb_theron_common/rb_theron_description/urdf/door_opening_mechanism/door_opening_mechanism.urdf.xacro (robot description, xacro)
@@ -7,4 +7,8 @@
     </xacro:macro>
     <xacro:macro name="door_opening_mechanism" params="prefix parent *origin hq">
+    <!-- Please mind: We might need to set the settings for the mass extremly low, because there
+    is an issue, that if there is too much load on the theron base, it would be able to drive
+    properly, because this makes some of the wheels lose contact to the ground and
+    therefore steering of the rb_theron becomes impossible. -->
     <xacro:property name="door_opening_mechanism_base_link" value="${prefix}door_opening_mechanism_base_link" />
     <joint name="${prefix}door_opening_mechanism_joint" type="fixed">
@@ -50,11 +54,7 @@
     <link name="${prefix}door_opening_mechanism_link_y_axis_rail">
         <inertial>
-            <!-- Mass should actually not be zero, but there is an issue, that if there is too much load on the theron base,
-            it would be able to drive properly, because this makes some of the wheels lose contact to the ground and
-            therefore steering of the rb_theron becomes impossible.
-            The mass of a 30 mm x 30 mm Aluprofile from item is m = 1.26 kg/m -->
-            <mass value="5" />
-            <origin xyz="0 0 0" />
-            <xacro:box_inertia_robot m="5" x="0.06" y="0.06" z="0.56"/>
+            <mass value="2.64" />
+            <origin xyz="0 0 0" />
+            <xacro:box_inertia_robot m="2.64" x="0.06" y="0.06" z="0.56"/>
         </inertial>
         <visual>
@@ -103,8 +103,5 @@
     <link name="${prefix}door_opening_mechanism_link_y_axis_slide">
         <inertial>
-            <!-- Mass should actually not be zero, but there is an issue, that if there is too much load on the theron base,
-            it would be able to drive properly, because this makes some of the wheels lose contact to the ground and
-            therefore steering of the rb_theron becomes impossible.
-            The mass of the 550mm norelem Zahnradantrieb is 2.34kg (rail) + 0.3kg (slide) -->
+            <!-- The mass of the 550mm norelem Zahnradantrieb is 2.34kg (rail) + 0.3kg (slide) -->
             <mass value="2.64" />
             <origin xyz="0 0 0" />
