Commit message: Creating basic_joint urdf

File: src/ros2/robot_description/rb_theron_common/rb_theron_description/urdf/door_opening_mechanism/basic_box.urdf.xacro (robot description, xacro)
@@ -6,5 +6,5 @@
                 izz="${m*(x*x+z*z)/12}" />
     </xacro:macro>
-    <xacro:macro name="basic_box" params="parent joint_name link_name *origin m x y z r g b">
+    <xacro:macro name="basic_box" params="parent joint_name link_name m x y z r g b *origin">
     <joint name="${joint_name}" type="fixed" >
         <parent link="${parent}" />

File: src/ros2/robot_description/rb_theron_common/rb_theron_description/urdf/door_opening_mechanism/door_opening_mechanism.urdf.xacro (robot description, xacro)
@@ -7,227 +7,159 @@
     </xacro:macro>
     <xacro:macro name="door_opening_mechanism" params="prefix parent *origin hq">
-    <!-- Please mind: We might need to set the settings for the mass extremly low, because there
-    is an issue, that if there is too much load on the theron base, it would be able to drive
-    properly, because this makes some of the wheels lose contact to the ground and
-    therefore steering of the rb_theron becomes impossible. -->
-    <xacro:property name="door_opening_mechanism_base_link" value="${prefix}door_opening_mechanism_base_link" />
-    <joint name="${prefix}door_opening_mechanism_joint" type="fixed">
-        <parent link="${parent}"/>
-        <child link="${door_opening_mechanism_base_link}"/>
-        <xacro:insert_block name="origin" />
-    </joint>
-    <!-- Base link -->
-    <link name="${door_opening_mechanism_base_link}">
-        <visual>
-          <origin xyz="0 0 0" rpy="0 0 0" />
-          <geometry>
-            <box size="0.001 0.001 0.001" />
-          </geometry>
-        </visual>
-        <collision>
-          <origin xyz="0 0 0" rpy="0 0 0" />
-          <geometry>
-            <box size="0.001 0.001 0.001" />
-          </geometry>
-        </collision>
-    </link>
-    <!-- Aluprofile frame -->
-    <xacro:include filename="$(find rb_theron_description)/urdf/door_opening_mechanism/alu_profile.urdf.xacro" />
-    <xacro:alu_profile prefix="${prefix}" suffix="bottom" parent="${door_opening_mechanism_base_link}" x="0.03" y="0.03" z="0.46" r="0.1" g="0.1" b="0.1" >
-		<origin xyz="0 0 0" rpy="1.57079632679 0 0"/>
-	</xacro:alu_profile>
-	<xacro:alu_profile prefix="${prefix}" suffix="left" parent="${door_opening_mechanism_base_link}" x="0.03" y="0.03" z="1.0" r="0.1" g="0.1" b="0.1" >
-		<origin xyz="0 -0.245 0.515" rpy="0 0 0"/>
-	</xacro:alu_profile>
-	<xacro:alu_profile prefix="${prefix}" suffix="right" parent="${door_opening_mechanism_base_link}" x="0.03" y="0.03" z="1.0" r="0.1" g="0.1" b="0.1" >
-		<origin xyz="0 +0.245 0.515" rpy="0 0 0"/>
-	</xacro:alu_profile>
-    <xacro:alu_profile prefix="${prefix}" suffix="top" parent="${door_opening_mechanism_base_link}" x="0.03" y="0.03" z="0.52" r="0.1" g="0.1" b="0.1" >
-		<origin xyz="0 0 1.03" rpy="1.57079632679 0 0"/>
-	</xacro:alu_profile>
-    <xacro:include filename="$(find rb_theron_description)/urdf/door_opening_mechanism/basic_box.urdf.xacro" />
-    <xacro:basic_box
-        parent="${door_opening_mechanism_base_link}"
-        joint_name="${prefix}door_opening_mechanism_joint_y_axis_rail"
-        link_name="${prefix}door_opening_mechanism_link_y_axis_rail"
-        m="2.64"
-        x="0.06"
-        y="0.06"
-        z="0.56"
-        r="1"
-        g="0"
-        b="0">
-        <origin xyz="-0.015 0.2 0.55" rpy="0 0 0"/>
-    </xacro:basic_box>
-    <joint name="${prefix}door_opening_mechanism_joint_y_axis_slide" type="prismatic" >
-        <axis xyz="0 1 0" />
-        <parent link="${prefix}alu_profile_link_right" />
-        <child link="${prefix}door_opening_mechanism_link_y_axis_slide" />
-        <origin xyz="-0.075 -0.225 -0.1" rpy="1.57079632679 0 0"/>
-        <limit lower="-0.05" upper="0.25" effort="100" velocity="100" />
-        <dynamics damping="0.1" friction="0.3"/>
-    </joint>
-    <gazebo>
-        <plugin filename="libgz-sim-joint-position-controller-system.so" name="gz::sim::systems::JointPositionController">
-            <joint_name>${prefix}door_opening_mechanism_joint_y_axis_slide</joint_name>
-            <p_gain>50000.0</p_gain>
-            <i_gain>1000</i_gain>
-            <d_gain>5000</d_gain>
-            <i_max>200</i_max>
-            <i_min>-200</i_min>
-            <cmd_max>1000</cmd_max>
-            <cmd_min>-1000</cmd_min>
-        </plugin>
-    </gazebo>
-    <link name="${prefix}door_opening_mechanism_link_y_axis_slide">
-        <inertial>
-            <!-- The mass of the 550mm norelem Zahnradantrieb is 2.34kg (rail) + 0.3kg (slide) -->
-            <mass value="2.64" />
-            <origin xyz="0 0 0" />
-            <xacro:box_inertia_robot m="2.64" x="0.06" y="0.06" z="0.55"/>
-        </inertial>
-        <visual>
-            <origin xyz="0 0 0" rpy="0 0 0"/>
+        <!-- Element imports -->
+        <xacro:include filename="$(find rb_theron_description)/urdf/door_opening_mechanism/alu_profile.urdf.xacro" />
+        <xacro:include filename="$(find rb_theron_description)/urdf/door_opening_mechanism/basic_box.urdf.xacro" />
+        <xacro:include filename="$(find rb_theron_description)/urdf/door_opening_mechanism/basic_joint.urdf.xacro" />
+        <!-- Please mind: We might need to set the settings for the mass extremly low, because there
+        is an issue, that if there is too much load on the theron base, it would be able to drive
+        properly, because this makes some of the wheels lose contact to the ground and
+        therefore steering of the rb_theron becomes impossible. -->
+        <xacro:property name="door_opening_mechanism_base_link" value="${prefix}door_opening_mechanism_base_link" />
+        <joint name="${prefix}door_opening_mechanism_joint" type="fixed">
+            <parent link="${parent}"/>
+            <child link="${door_opening_mechanism_base_link}"/>
+            <xacro:insert_block name="origin" />
+        </joint>
+        <!-- Base link -->
+        <link name="${door_opening_mechanism_base_link}">
+            <visual>
+            <origin xyz="0 0 0" rpy="0 0 0" />
             <geometry>
-                <box size="0.06 0.06 0.56"/>
+                <box size="0.001 0.001 0.001" />
             </geometry>
-        </visual>
-        <collision>
-            <origin xyz="0 0 0" rpy="0 0 0"/>
+            </visual>
+            <collision>
+            <origin xyz="0 0 0" rpy="0 0 0" />
             <geometry>
-                <box size="0.06 0.06 0.56"/>
+                <box size="0.001 0.001 0.001" />
             </geometry>
-        </collision>
-    </link>
-    <gazebo reference="${prefix}door_opening_mechanism_link_y_axis_slide">
-        <visual>
-            <material>
-                <!-- RGBA -->
-                <ambient>1 1 0 1</ambient>
-                <diffuse>1 1 0 1</diffuse>
-                <specular>1 1 0 1</specular>
-            </material>
-        </visual>
-    </gazebo>
-    <joint name="${prefix}door_opening_mechanism_joint_x_axis_slide" type="prismatic" >
-        <axis xyz="0 0 1" />
-        <parent link="${prefix}door_opening_mechanism_link_y_axis_slide" />
-        <child link="${prefix}door_opening_mechanism_link_x_axis_slide" />
-        <origin xyz="-0.04 0 0" rpy="0 0 1.57079632679"/>
-        <limit lower="-0.175" upper="0.20" effort="100" velocity="100" />
-        <dynamics damping="0.1" friction="0.3"/>
-    </joint>
-    <gazebo>
-        <plugin filename="libgz-sim-joint-position-controller-system.so" name="gz::sim::systems::JointPositionController">
-            <joint_name>${prefix}door_opening_mechanism_joint_x_axis_slide</joint_name>
-            <p_gain>50000.0</p_gain>
-            <i_gain>100</i_gain>
-            <d_gain>5000</d_gain>
-            <i_max>200</i_max>
-            <i_min>-200</i_min>
-        </plugin>
-    </gazebo>
-    <link name="${prefix}door_opening_mechanism_link_x_axis_slide">
-        <inertial>
-            <!-- Mass should actually not be zero, but there is an issue, that if there is too much load on the theron base,
-            it would be able to drive properly, because this makes some of the wheels lose contact to the ground and
-            therefore steering of the rb_theron becomes impossible.
-            The mass of a 30 mm x 30 mm Aluprofile from item is m = 1.26 kg/m -->
-            <mass value="1" />
-            <origin xyz="0 0 0" />
-            <xacro:box_inertia_robot m="1" x="0.065" y="0.015" z="0.175"/>
-        </inertial>
-        <visual>
-            <origin xyz="0 0 0" rpy="0 0 0"/>
-            <geometry>
-                <box size="0.065 0.015 0.175"/>
-            </geometry>
-        </visual>
-        <collision>
-            <origin xyz="0 0 0" rpy="0 0 0"/>
-            <geometry>
-                <box size="0.065 0.015 0.175"/>
-            </geometry>
-        </collision>
-    </link>
-    <gazebo reference="${prefix}door_opening_mechanism_link_x_axis_slide">
-        <visual>
-            <material>
-                <!-- RGBA -->
-                <ambient>1 1 1 1</ambient>
-                <diffuse>1 1 1 1</diffuse>
-                <specular>1 1 1 1</specular>
-            </material>
-        </visual>
-    </gazebo>
-    <xacro:basic_box
-        parent="${prefix}door_opening_mechanism_link_x_axis_slide"
-        joint_name="${prefix}door_opening_mechanism_joint_x_axis_slide_screwing"
-        link_name="${prefix}door_opening_mechanism_link_x_slide_screwing"
-        m="1"
-        x="0.073"
-        y="0.015"
-        z="0.175"
-        r="1"
-        g="1"
-        b="1">
-        <origin xyz="0.038 -0.027 0" rpy="0 0 1.57079632679"/>
-    </xacro:basic_box>
-    <joint name="${prefix}door_opening_mechanism_joint_tilting_hook" type="revolute" >
-        <axis xyz="1 0 0" />
-        <parent link="${prefix}door_opening_mechanism_link_x_slide_screwing" />
-        <child link="${prefix}door_opening_mechanism_link_tilting_hook" />
-        <origin xyz="0 -0.025 0" rpy="0 1.57079632679 0"/>
-        <limit lower="0" upper="1.6" effort="100" velocity="100" />
-        <dynamics damping="0.1" friction="0.3"/>
-    </joint>
-    <gazebo>
-        <plugin filename="libgz-sim-joint-position-controller-system.so" name="gz::sim::systems::JointPositionController">
-            <joint_name>${prefix}door_opening_mechanism_joint_tilting_hook</joint_name>
-            <p_gain>500.0</p_gain>
-            <i_gain>1000</i_gain>
-            <d_gain>10</d_gain>
-            <i_max>200</i_max>
-            <i_min>-200</i_min>
-        </plugin>
-    </gazebo>
-    <link name="${prefix}door_opening_mechanism_link_tilting_hook">
-        <inertial>
-            <!-- Mass should actually not be zero, but there is an issue, that if there is too much load on the theron base,
-            it would be able to drive properly, because this makes some of the wheels lose contact to the ground and
-            therefore steering of the rb_theron becomes impossible.
-            The mass of a 30 mm x 30 mm Aluprofile from item is m = 1.26 kg/m -->
-            <mass value="0.2" />
-            <origin xyz="0 0 0.1" />
-            <xacro:box_inertia_robot m="0.2" x="0.03" y="0.03" z="0.2"/>
-        </inertial>
-        <visual>
-            <origin xyz="0 0 0.1" rpy="0 0 0"/>
-            <geometry>
-                <box size="0.03 0.03 0.2"/>
-            </geometry>
-        </visual>
-        <collision>
-            <origin xyz="0 0 0.1" rpy="0 0 0"/>
-            <geometry>
-                <box size="0.03 0.03 0.2"/>
-            </geometry>
-        </collision>
-    </link>
-    <gazebo reference="${prefix}door_opening_mechanism_link_tilting_hook">
-        <visual>
-            <material>
-                <!-- RGBA -->
-                <ambient>0 1 0 1</ambient>
-                <diffuse>0 1 0 1</diffuse>
-                <specular>0 1 0 1</specular>
-            </material>
-        </visual>
-    </gazebo>
-    <!-- Gripper -->
-    <xacro:include filename="$(find rb_theron_description)/urdf/door_opening_mechanism/door_opening_gripper.urdf.xacro" />
-    <xacro:door_opening_gripper prefix="${prefix}" parent="${prefix}door_opening_mechanism_link_tilting_hook" >
-		<origin xyz="0 0 0.215" rpy="0 1.57079632679 0"/>
-	</xacro:door_opening_gripper>
+            </collision>
+        </link>
+        <!-- Aluprofile frame -->
+        <xacro:alu_profile prefix="${prefix}" suffix="bottom" parent="${door_opening_mechanism_base_link}" x="0.03" y="0.03" z="0.46" r="0.1" g="0.1" b="0.1" >
+            <origin xyz="0 0 0" rpy="1.57079632679 0 0"/>
+        </xacro:alu_profile>
+        <xacro:alu_profile prefix="${prefix}" suffix="left" parent="${door_opening_mechanism_base_link}" x="0.03" y="0.03" z="1.0" r="0.1" g="0.1" b="0.1" >
+            <origin xyz="0 -0.245 0.515" rpy="0 0 0"/>
+        </xacro:alu_profile>
+        <xacro:alu_profile prefix="${prefix}" suffix="right" parent="${door_opening_mechanism_base_link}" x="0.03" y="0.03" z="1.0" r="0.1" g="0.1" b="0.1" >
+            <origin xyz="0 +0.245 0.515" rpy="0 0 0"/>
+        </xacro:alu_profile>
+        <xacro:alu_profile prefix="${prefix}" suffix="top" parent="${door_opening_mechanism_base_link}" x="0.03" y="0.03" z="0.52" r="0.1" g="0.1" b="0.1" >
+            <origin xyz="0 0 1.03" rpy="1.57079632679 0 0"/>
+        </xacro:alu_profile>
+        <!-- Door opening mechanism -->
+        <xacro:basic_box
+            parent="${door_opening_mechanism_base_link}"
+            joint_name="${prefix}door_opening_mechanism_joint_y_axis_rail"
+            link_name="${prefix}door_opening_mechanism_link_y_axis_rail"
+            m="2.64"
+            x="0.06"
+            y="0.06"
+            z="0.56"
+            r="0"
+            g="1"
+            b="0">
+            <origin xyz="-0.015 0.2 0.55" rpy="0 0 0"/>
+        </xacro:basic_box>
+        <xacro:basic_joint
+            parent="${prefix}alu_profile_link_right"
+            joint_name="${prefix}door_opening_mechanism_joint_y_axis_slide"
+            joint_type="prismatic"
+            axis_x="0"
+            axis_y="1"
+            axis_z="0"
+            lower_limit="-0.05"
+            upper_limit="0.25"
+            damping="0.1"
+            friction="0.3"
+            p_gain="50000"
+            i_gain="1000"
+            d_gain="5000"
+            link_name="${prefix}door_opening_mechanism_link_y_axis_slide"
+            link_origin_x="0.0"
+            link_origin_y="0.0"
+            link_origin_z="0.0"
+            m="2.64"
+            x="0.06"
+            y="0.06"
+            z="0.55"
+            r="1"
+            g="0"
+            b="0">
+            <origin xyz="-0.075 -0.225 -0.1" rpy="1.57079632679 0 0"/>
+        </xacro:basic_joint>
+        <xacro:basic_joint
+            parent="${prefix}door_opening_mechanism_link_y_axis_slide"
+            joint_name="${prefix}door_opening_mechanism_joint_x_axis_slide"
+            joint_type="prismatic"
+            axis_x="0"
+            axis_y="0"
+            axis_z="1"
+            lower_limit="-0.175"
+            upper_limit="0.20"
+            damping="0.1"
+            friction="0.3"
+            p_gain="50000"
+            i_gain="100"
+            d_gain="5000"
+            link_name="${prefix}door_opening_mechanism_link_x_axis_slide"
+            link_origin_x="0.0"
+            link_origin_y="0.0"
+            link_origin_z="0.0"
+            m="1"
+            x="0.065"
+            y="0.015"
+            z="0.175"
+            r="1"
+            g="1"
+            b="1">
+            <origin xyz="-0.04 0 0" rpy="0 0 1.57079632679"/>
+        </xacro:basic_joint>
+        <xacro:basic_box
+            parent="${prefix}door_opening_mechanism_link_x_axis_slide"
+            joint_name="${prefix}door_opening_mechanism_joint_x_axis_slide_screwing"
+            link_name="${prefix}door_opening_mechanism_link_x_slide_screwing"
+            m="1"
+            x="0.073"
+            y="0.015"
+            z="0.175"
+            r="1"
+            g="1"
+            b="1">
+            <origin xyz="0.038 -0.027 0" rpy="0 0 1.57079632679"/>
+        </xacro:basic_box>
+        <xacro:basic_joint
+            parent="${prefix}door_opening_mechanism_link_x_slide_screwing"
+            joint_name="${prefix}door_opening_mechanism_joint_tilting_hook"
+            joint_type="revolute"
+            axis_x="1"
+            axis_y="0"
+            axis_z="0"
+            lower_limit="0"
+            upper_limit="1.6"
+            damping="0.1"
+            friction="0.3"
+            p_gain="500"
+            i_gain="1000"
+            d_gain="10"
+            link_name="${prefix}door_opening_mechanism_link_tilting_hook"
+            link_origin_x="0.0"
+            link_origin_y="0.0"
+            link_origin_z="0.1"
+            m="0.2"
+            x="0.03"
+            y="0.03"
+            z="0.2"
+            r="0"
+            g="1"
+            b="0">
+            <origin xyz="0 -0.025 0" rpy="0 1.57079632679 0"/>
+        </xacro:basic_joint>
+        <!-- Gripper -->
+        <xacro:include filename="$(find rb_theron_description)/urdf/door_opening_mechanism/door_opening_gripper.urdf.xacro" />
+        <xacro:door_opening_gripper prefix="${prefix}" parent="${prefix}door_opening_mechanism_link_tilting_hook" >
+            <origin xyz="0 0 0.215" rpy="0 1.57079632679 0"/>
+        </xacro:door_opening_gripper>
     </xacro:macro>
 </robot>

File: src/ros2/robot_description/rb_theron_common/rb_theron_description/urdf/door_opening_mechanism/hook.urdf.xacro (robot description, xacro)
@@ -8,8 +8,28 @@
     <xacro:macro name="hook" params="prefix suffix parent *origin r g b">
     <xacro:include filename="$(find rb_theron_description)/urdf/door_opening_mechanism/basic_box.urdf.xacro" />
-    <xacro:basic_box parent="${prefix}${parent}" joint_name="${prefix}hook_joint_${suffix}" link_name="${prefix}hook_base_link_${suffix}" m="0.1" x="0.06" y="0.01" z="0.04" r="0" g="0" b="1">
+    <xacro:basic_box
+        parent="${prefix}${parent}"
+        joint_name="${prefix}hook_joint_${suffix}"
+        link_name="${prefix}hook_base_link_${suffix}"
+        m="0.1"
+        x="0.06"
+        y="0.01"
+        z="0.04"
+        r="0"
+        g="0"
+        b="1">
         <xacro:insert_block name="origin" />
     </xacro:basic_box>
-    <xacro:basic_box parent="${prefix}hook_base_link_${suffix}" joint_name="${prefix}hook_joint_front_side_${suffix}" link_name="${prefix}hook_front_side_link_${suffix}" m="0.1" x="0.008" y="0.03" z="0.04" r="0" g="0" b="1">
+    <xacro:basic_box
+        parent="${prefix}hook_base_link_${suffix}"
+        joint_name="${prefix}hook_joint_front_side_${suffix}"
+        link_name="${prefix}hook_front_side_link_${suffix}"
+        m="0.1"
+        x="0.008"
+        y="0.03"
+        z="0.04"
+        r="0"
+        g="0"
+        b="1">
         <origin xyz="-0.026 0.02 0" rpy="0 0 0"/>
     </xacro:basic_box>
