Commit message: For now we need to reduce the mass of the cage, drawer and door opening, otherwise rb_theron cant drive properly

File: src/ros2/robot_description/rb_theron_common/rb_theron_description/urdf/door_opening_mechanism/door_opening_mechanism.urdf.xacro (robot description, xacro)
@@ -15,5 +15,8 @@
     <link name="${prefix}door_opening_mechanism_link">
         <inertial>
-            <mass value="25.0" />
+            <!-- Mass should actually not be zero, but there is an issue, that if there is too much load on the theron base,
+            it would be able to drive properly, because this makes some of the wheels lose contact to the ground and
+            therefore steering of the rb_theron becomes impossible -->
+            <mass value="0.0" />
             <origin xyz="0 0 0" />
             <xacro:box_inertia_robot m="100" x="0.25" y="0.25" z="1.55"/>

File: src/ros2/robot_description/rb_theron_common/rb_theron_description/urdf/drawer/drawer.urdf.xacro (robot description, xacro)
@@ -8,5 +8,8 @@
     <xacro:property name="drawer_size_x" value="0.45" />
     <xacro:property name="drawer_size_y" value="0.358" />
-    <xacro:property name="drawer_mass" value="1.5" />
+    <!-- Mass should actually not be that small, but there is an issue, that if there is too much load on the theron base,
+      it would be able to drive properly, because this makes some of the wheels lose contact to the ground and
+      therefore steering of the rb_theron becomes impossible -->
+    <xacro:property name="drawer_mass" value="0.1" />
     <xacro:property name="drawer_offset_x" value="0.0" />
     <xacro:property name="drawer_offset_y" value="0.0" />

File: src/ros2/robot_description/rb_theron_common/rb_theron_description/urdf/module_cage/module_cage.urdf.xacro (robot description, xacro)
@@ -15,5 +15,8 @@
   <link name="${prefix}module_cage_link">
     <inertial>
-      <mass value="25.0" />
+      <!-- Mass should actually not be zero, but there is an issue, that if there is too much load on the theron base,
+      it would be able to drive properly, because this makes some of the wheels lose contact to the ground and
+      therefore steering of the rb_theron becomes impossible -->
+      <mass value="0.0" />
       <origin xyz="0 0 0" />
       <xacro:box_inertia_robot m="10" x="0.25" y="0.25" z="1.55"/>

Commit message: Adding third joint - WIP

File: src/ros2/robot_description/rb_theron_common/rb_theron_description/urdf/door_opening_mechanism/door_opening_mechanism.urdf.xacro (robot description, xacro)
@@ -63,7 +63,4 @@
                 <box size="0.06 0.06 0.56"/>
             </geometry>
-            <material name="darkgrey">
-                <color rgba="0.1 0.1 0.1 1"/>
-            </material>
         </visual>
         <collision>
@@ -74,4 +71,14 @@
         </collision>
     </link>
+    <gazebo reference="${prefix}door_opening_mechanism_link_y_axis_rail">
+        <visual>
+            <material>
+                <!-- RGBA -->
+                <ambient>1 0 0 1</ambient>
+                <diffuse>1 0 0 1</diffuse>
+                <specular>1 0 0 1</specular>
+            </material>
+        </visual>
+    </gazebo>
     <joint name="${prefix}door_opening_mechanism_joint_y_axis_slide" type="prismatic" >
         <axis xyz="0 1 0" />
@@ -81,4 +88,14 @@
         <limit lower="0.0" upper="0.25" effort="100" velocity="100" />
     </joint>
+    <gazebo>
+        <plugin filename="libgz-sim-joint-position-controller-system.so" name="gz::sim::systems::JointPositionController">
+            <joint_name>${prefix}door_opening_mechanism_joint_y_axis_slide</joint_name>
+            <p_gain>50000.0</p_gain>
+            <i_gain>100</i_gain>
+            <d_gain>1000</d_gain>
+            <i_max>200</i_max>
+            <i_min>-200</i_min>
+        </plugin>
+    </gazebo>
     <link name="${prefix}door_opening_mechanism_link_y_axis_slide">
         <inertial>
@@ -96,22 +113,39 @@
                 <box size="0.06 0.06 0.56"/>
             </geometry>
-            <material name="darkgrey">
-                <color rgba="0.1 0.1 0.1 1"/>
-            </material>
-        </visual>
-        <collision>
-            <origin xyz="0 0 0" rpy="0 0 0"/>
-            <geometry>
-                <box size="0.06 0.06 0.56"/>
-            </geometry>
-        </collision>
-    </link>
+        </visual>
+        <collision>
+            <origin xyz="0 0 0" rpy="0 0 0"/>
+            <geometry>
+                <box size="0.06 0.06 0.56"/>
+            </geometry>
+        </collision>
+    </link>
+    <gazebo reference="${prefix}door_opening_mechanism_link_y_axis_slide">
+        <visual>
+            <material>
+                <!-- RGBA -->
+                <ambient>1 1 0 1</ambient>
+                <diffuse>1 1 0 1</diffuse>
+                <specular>1 1 0 1</specular>
+            </material>
+        </visual>
+    </gazebo>
     <joint name="${prefix}door_opening_mechanism_joint_x_axis_slide" type="prismatic" >
-        <axis xyz="1 0 0" />
+        <axis xyz="0 0 1" />
         <parent link="${prefix}door_opening_mechanism_link_y_axis_slide" />
         <child link="${prefix}door_opening_mechanism_link_x_axis_slide" />
         <origin xyz="-0.04 0 0" rpy="0 0 1.57079632679"/>
-        <limit lower="0.0" upper="0.25" effort="100" velocity="100" />
-    </joint>
+        <limit lower="-0.25" upper="0.25" effort="100" velocity="100" />
+    </joint>
+    <gazebo>
+        <plugin filename="libgz-sim-joint-position-controller-system.so" name="gz::sim::systems::JointPositionController">
+            <joint_name>${prefix}door_opening_mechanism_joint_x_axis_slide</joint_name>
+            <p_gain>50000.0</p_gain>
+            <i_gain>100</i_gain>
+            <d_gain>1000</d_gain>
+            <i_max>200</i_max>
+            <i_min>-200</i_min>
+        </plugin>
+    </gazebo>
     <link name="${prefix}door_opening_mechanism_link_x_axis_slide">
         <inertial>
@@ -122,16 +156,16 @@
             <mass value="5" />
             <origin xyz="0 0 0" />
-            <xacro:box_inertia_robot m="5" x="0.06" y="0.015" z="0.175"/>
-        </inertial>
-        <visual>
-            <origin xyz="0 0 0" rpy="0 0 0"/>
-            <geometry>
-                <box size="0.06 0.015 0.175"/>
-            </geometry>
-        </visual>
-        <collision>
-            <origin xyz="0 0 0" rpy="0 0 0"/>
-            <geometry>
-                <box size="0.06 0.015 0.175"/>
+            <xacro:box_inertia_robot m="5" x="0.065" y="0.015" z="0.175"/>
+        </inertial>
+        <visual>
+            <origin xyz="0 0 0" rpy="0 0 0"/>
+            <geometry>
+                <box size="0.065 0.015 0.175"/>
+            </geometry>
+        </visual>
+        <collision>
+            <origin xyz="0 0 0" rpy="0 0 0"/>
+            <geometry>
+                <box size="0.065 0.015 0.175"/>
             </geometry>
         </collision>
@@ -147,4 +181,93 @@
         </visual>
     </gazebo>
+    <joint name="${prefix}door_opening_mechanism_joint_x_axis_slide_screwing" type="fixed" >
+        <axis xyz="1 0 0" />
+        <parent link="${prefix}door_opening_mechanism_link_x_axis_slide" />
+        <child link="${prefix}door_opening_mechanism_link_x_slide_screwing" />
+        <origin xyz="0.038 -0.032 0" rpy="0 0 1.57079632679"/>
+    </joint>
+    <link name="${prefix}door_opening_mechanism_link_x_slide_screwing">
+        <inertial>
+            <!-- Mass should actually not be zero, but there is an issue, that if there is too much load on the theron base,
+            it would be able to drive properly, because this makes some of the wheels lose contact to the ground and
+            therefore steering of the rb_theron becomes impossible.
+            The mass of a 30 mm x 30 mm Aluprofile from item is m = 1.26 kg/m -->
+            <mass value="5" />
+            <origin xyz="0 0 0" />
+            <xacro:box_inertia_robot m="5" x="0.08" y="0.015" z="0.175"/>
+        </inertial>
+        <visual>
+            <origin xyz="0 0 0" rpy="0 0 0"/>
+            <geometry>
+                <box size="0.08 0.015 0.175"/>
+            </geometry>
+        </visual>
+        <collision>
+            <origin xyz="0 0 0" rpy="0 0 0"/>
+            <geometry>
+                <box size="0.08 0.015 0.175"/>
+            </geometry>
+        </collision>
+    </link>
+    <gazebo reference="${prefix}door_opening_mechanism_link_x_slide_screwing">
+        <visual>
+            <material>
+                <!-- RGBA -->
+                <ambient>1 1 1 1</ambient>
+                <diffuse>1 1 1 1</diffuse>
+                <specular>1 1 1 1</specular>
+            </material>
+        </visual>
+    </gazebo>
+    <joint name="${prefix}door_opening_mechanism_joint_tilting_hook" type="revolute" >
+        <axis xyz="1 0 0" />
+        <parent link="${prefix}door_opening_mechanism_link_x_slide_screwing" />
+        <child link="${prefix}door_opening_mechanism_link_tilting_hook" />
+        <origin xyz="0 -0.025 0" rpy="0 1.57079632679 0"/>
+        <limit lower="0" upper="1.6" effort="100" velocity="100" />
+    </joint>
+    <gazebo>
+        <plugin filename="libgz-sim-joint-position-controller-system.so" name="gz::sim::systems::JointPositionController">
+            <joint_name>${prefix}door_opening_mechanism_joint_tilting_hook</joint_name>
+            <p_gain>50000.0</p_gain>
+            <i_gain>100</i_gain>
+            <d_gain>1000</d_gain>
+            <i_max>200</i_max>
+            <i_min>-200</i_min>
+        </plugin>
+    </gazebo>
+    <link name="${prefix}door_opening_mechanism_link_tilting_hook">
+        <inertial>
+            <!-- Mass should actually not be zero, but there is an issue, that if there is too much load on the theron base,
+            it would be able to drive properly, because this makes some of the wheels lose contact to the ground and
+            therefore steering of the rb_theron becomes impossible.
+            The mass of a 30 mm x 30 mm Aluprofile from item is m = 1.26 kg/m -->
+            <mass value="5" />
+            <origin xyz="0 0 0.1" />
+            <xacro:box_inertia_robot m="5" x="0.03" y="0.03" z="0.2"/>
+        </inertial>
+        <visual>
+            <origin xyz="0 0 0.1" rpy="0 0 0"/>
+            <geometry>
+                <box size="0.03 0.03 0.2"/>
+            </geometry>
+        </visual>
+        <collision>
+            <origin xyz="0 0 0.1" rpy="0 0 0"/>
+            <geometry>
+                <box size="0.03 0.03 0.2"/>
+            </geometry>
+        </collision>
+    </link>
+    <gazebo reference="${prefix}door_opening_mechanism_link_tilting_hook">
+        <visual>
+            <material>
+                <!-- RGBA -->
+                <ambient>1 0 1 1</ambient>
+                <diffuse>1 0 1 1</diffuse>
+                <specular>1 0 1 1</specular>
+            </material>
+        </visual>
+    </gazebo>
     </xacro:macro>
 </robot>

Commit message: Modifying masses and PID controller to an acceptable behaviour for now

File: src/ros2/robot_description/rb_theron_common/rb_theron_description/urdf/door_opening_mechanism/door_opening_mechanism.urdf.xacro (robot description, xacro)
@@ -86,5 +86,6 @@
         <child link="${prefix}door_opening_mechanism_link_y_axis_slide" />
         <origin xyz="-0.075 -0.225 -0.1" rpy="1.57079632679 0 0"/>
-        <limit lower="0.0" upper="0.25" effort="100" velocity="100" />
+        <limit lower="-0.25" upper="0.25" effort="100" velocity="100" />
+        <dynamics damping="0.1" friction="0.3"/>
     </joint>
     <gazebo>
@@ -92,8 +93,10 @@
             <joint_name>${prefix}door_opening_mechanism_joint_y_axis_slide</joint_name>
             <p_gain>50000.0</p_gain>
-            <i_gain>100</i_gain>
-            <d_gain>1000</d_gain>
+            <i_gain>1000</i_gain>
+            <d_gain>5000</d_gain>
             <i_max>200</i_max>
             <i_min>-200</i_min>
+            <cmd_max>1000</cmd_max>
+            <cmd_min>-1000</cmd_min>
         </plugin>
     </gazebo>
@@ -103,8 +106,8 @@
             it would be able to drive properly, because this makes some of the wheels lose contact to the ground and
             therefore steering of the rb_theron becomes impossible.
-            The mass of a 30 mm x 30 mm Aluprofile from item is m = 1.26 kg/m -->
-            <mass value="5" />
-            <origin xyz="0 0 0" />
-            <xacro:box_inertia_robot m="5" x="0.06" y="0.06" z="0.55"/>
+            The mass of the 550mm norelem Zahnradantrieb is 2.34kg (rail) + 0.3kg (slide) -->
+            <mass value="2.64" />
+            <origin xyz="0 0 0" />
+            <xacro:box_inertia_robot m="2.64" x="0.06" y="0.06" z="0.55"/>
         </inertial>
         <visual>
@@ -137,4 +140,5 @@
         <origin xyz="-0.04 0 0" rpy="0 0 1.57079632679"/>
         <limit lower="-0.25" upper="0.25" effort="100" velocity="100" />
+        <dynamics damping="0.1" friction="0.3"/>
     </joint>
     <gazebo>
@@ -143,5 +147,5 @@
             <p_gain>50000.0</p_gain>
             <i_gain>100</i_gain>
-            <d_gain>1000</d_gain>
+            <d_gain>5000</d_gain>
             <i_max>200</i_max>
             <i_min>-200</i_min>
@@ -154,7 +158,7 @@
             therefore steering of the rb_theron becomes impossible.
             The mass of a 30 mm x 30 mm Aluprofile from item is m = 1.26 kg/m -->
-            <mass value="5" />
-            <origin xyz="0 0 0" />
-            <xacro:box_inertia_robot m="5" x="0.065" y="0.015" z="0.175"/>
+            <mass value="1" />
+            <origin xyz="0 0 0" />
+            <xacro:box_inertia_robot m="1" x="0.065" y="0.015" z="0.175"/>
         </inertial>
         <visual>
@@ -193,7 +197,7 @@
             therefore steering of the rb_theron becomes impossible.
             The mass of a 30 mm x 30 mm Aluprofile from item is m = 1.26 kg/m -->
-            <mass value="5" />
-            <origin xyz="0 0 0" />
-            <xacro:box_inertia_robot m="5" x="0.08" y="0.015" z="0.175"/>
+            <mass value="1" />
+            <origin xyz="0 0 0" />
+            <xacro:box_inertia_robot m="1" x="0.08" y="0.015" z="0.175"/>
         </inertial>
         <visual>
@@ -226,13 +230,14 @@
         <origin xyz="0 -0.025 0" rpy="0 1.57079632679 0"/>
         <limit lower="0" upper="1.6" effort="100" velocity="100" />
+        <dynamics damping="0.1" friction="0.3"/>
     </joint>
     <gazebo>
         <plugin filename="libgz-sim-joint-position-controller-system.so" name="gz::sim::systems::JointPositionController">
             <joint_name>${prefix}door_opening_mechanism_joint_tilting_hook</joint_name>
-            <p_gain>50000.0</p_gain>
-            <i_gain>100</i_gain>
-            <d_gain>1000</d_gain>
-            <i_max>200</i_max>
-            <i_min>-200</i_min>
+            <p_gain>5000.0</p_gain>
+            <i_gain>10000</i_gain>
+            <d_gain></d_gain>
+            <i_max>2000</i_max>
+            <i_min>-2000</i_min>
         </plugin>
     </gazebo>
@@ -243,7 +248,7 @@
             therefore steering of the rb_theron becomes impossible.
             The mass of a 30 mm x 30 mm Aluprofile from item is m = 1.26 kg/m -->
-            <mass value="5" />
+            <mass value="0.2" />
             <origin xyz="0 0 0.1" />
-            <xacro:box_inertia_robot m="5" x="0.03" y="0.03" z="0.2"/>
+            <xacro:box_inertia_robot m="0.2" x="0.03" y="0.03" z="0.2"/>
         </inertial>
         <visual>

Commit message: First draft for the gripper

File: src/ros2/robot_description/rb_theron_common/rb_theron_description/urdf/door_opening_mechanism/door_opening_mechanism.urdf.xacro (robot description, xacro)
@@ -275,4 +275,9 @@
         </visual>
     </gazebo>
+    <!-- Gripper -->
+    <xacro:include filename="$(find rb_theron_description)/urdf/door_opening_mechanism/door_opening_gripper.urdf.xacro" />
+    <xacro:door_opening_gripper prefix="${prefix}" parent="${prefix}door_opening_mechanism_link_tilting_hook" >
+		<origin xyz="0 0 0.215" rpy="0 1.57079632679 0"/>
+	</xacro:door_opening_gripper>
     </xacro:macro>
 </robot>

Commit message: Adjusting limits for joints and gazebo_controller_manager works for now for door opening mechanism in super simple way

File: src/ros2/robot_description/rb_theron_common/rb_theron_description/urdf/door_opening_mechanism/door_opening_mechanism.urdf.xacro (robot description, xacro)
@@ -86,5 +86,5 @@
         <child link="${prefix}door_opening_mechanism_link_y_axis_slide" />
         <origin xyz="-0.075 -0.225 -0.1" rpy="1.57079632679 0 0"/>
-        <limit lower="-0.25" upper="0.25" effort="100" velocity="100" />
+        <limit lower="-0.05" upper="0.25" effort="100" velocity="100" />
         <dynamics damping="0.1" friction="0.3"/>
     </joint>
@@ -139,5 +139,5 @@
         <child link="${prefix}door_opening_mechanism_link_x_axis_slide" />
         <origin xyz="-0.04 0 0" rpy="0 0 1.57079632679"/>
-        <limit lower="-0.25" upper="0.25" effort="100" velocity="100" />
+        <limit lower="-0.175" upper="0.20" effort="100" velocity="100" />
         <dynamics damping="0.1" friction="0.3"/>
     </joint>
@@ -189,26 +189,22 @@
         <parent link="${prefix}door_opening_mechanism_link_x_axis_slide" />
         <child link="${prefix}door_opening_mechanism_link_x_slide_screwing" />
-        <origin xyz="0.038 -0.032 0" rpy="0 0 1.57079632679"/>
+        <origin xyz="0.038 -0.027 0" rpy="0 0 1.57079632679"/>
     </joint>
     <link name="${prefix}door_opening_mechanism_link_x_slide_screwing">
         <inertial>
-            <!-- Mass should actually not be zero, but there is an issue, that if there is too much load on the theron base,
-            it would be able to drive properly, because this makes some of the wheels lose contact to the ground and
-            therefore steering of the rb_theron becomes impossible.
-            The mass of a 30 mm x 30 mm Aluprofile from item is m = 1.26 kg/m -->
             <mass value="1" />
             <origin xyz="0 0 0" />
-            <xacro:box_inertia_robot m="1" x="0.08" y="0.015" z="0.175"/>
-        </inertial>
-        <visual>
-            <origin xyz="0 0 0" rpy="0 0 0"/>
-            <geometry>
-                <box size="0.08 0.015 0.175"/>
-            </geometry>
-        </visual>
-        <collision>
-            <origin xyz="0 0 0" rpy="0 0 0"/>
-            <geometry>
-                <box size="0.08 0.015 0.175"/>
+            <xacro:box_inertia_robot m="1" x="0.073" y="0.015" z="0.175"/>
+        </inertial>
+        <visual>
+            <origin xyz="0 0 0" rpy="0 0 0"/>
+            <geometry>
+                <box size="0.073 0.015 0.175"/>
+            </geometry>
+        </visual>
+        <collision>
+            <origin xyz="0 0 0" rpy="0 0 0"/>
+            <geometry>
+                <box size="0.073 0.015 0.175"/>
             </geometry>
         </collision>
