Commit message: Adding simple box urdf

File: src/ros2/robot_description/rb_theron_common/rb_theron_description/urdf/door_opening_mechanism/door_opening_mechanism.urdf.xacro (robot description, xacro)
@@ -46,39 +46,18 @@
 		<origin xyz="0 0 1.03" rpy="1.57079632679 0 0"/>
 	</xacro:alu_profile>
-    <!-- Door opening mechanism -->
-    <joint name="${prefix}door_opening_mechanism_joint_y_axis_rail" type="fixed" >
-        <parent link="${door_opening_mechanism_base_link}" />
-        <child link="${prefix}door_opening_mechanism_link_y_axis_rail" />
+    <xacro:include filename="$(find rb_theron_description)/urdf/door_opening_mechanism/basic_box.urdf.xacro" />
+    <xacro:basic_box
+        parent="${door_opening_mechanism_base_link}"
+        joint_name="${prefix}door_opening_mechanism_joint_y_axis_rail"
+        link_name="${prefix}door_opening_mechanism_link_y_axis_rail"
+        m="2.64"
+        x="0.06"
+        y="0.06"
+        z="0.56"
+        r="1"
+        g="0"
+        b="0">
         <origin xyz="-0.015 0.2 0.55" rpy="0 0 0"/>
-    </joint>
-    <link name="${prefix}door_opening_mechanism_link_y_axis_rail">
-        <inertial>
-            <mass value="2.64" />
-            <origin xyz="0 0 0" />
-            <xacro:box_inertia_robot m="2.64" x="0.06" y="0.06" z="0.56"/>
-        </inertial>
-        <visual>
-            <origin xyz="0 0 0" rpy="0 0 0" />
-            <geometry>
-                <box size="0.06 0.06 0.56"/>
-            </geometry>
-        </visual>
-        <collision>
-            <origin xyz="0 0 0" rpy="0 0 0" />
-            <geometry>
-                <box size="0.06 0.06 0.56"/>
-            </geometry>
-        </collision>
-    </link>
-    <gazebo reference="${prefix}door_opening_mechanism_link_y_axis_rail">
-        <visual>
-            <material>
-                <!-- RGBA -->
-                <ambient>1 0 0 1</ambient>
-                <diffuse>1 0 0 1</diffuse>
-                <specular>1 0 0 1</specular>
-            </material>
-        </visual>
-    </gazebo>
+    </xacro:basic_box>
     <joint name="${prefix}door_opening_mechanism_joint_y_axis_slide" type="prismatic" >
         <axis xyz="0 1 0" />
@@ -182,39 +161,17 @@
         </visual>
     </gazebo>
-    <joint name="${prefix}door_opening_mechanism_joint_x_axis_slide_screwing" type="fixed" >
-        <axis xyz="1 0 0" />
-        <parent link="${prefix}door_opening_mechanism_link_x_axis_slide" />
-        <child link="${prefix}door_opening_mechanism_link_x_slide_screwing" />
+    <xacro:basic_box
+        parent="${prefix}door_opening_mechanism_link_x_axis_slide"
+        joint_name="${prefix}door_opening_mechanism_joint_x_axis_slide_screwing"
+        link_name="${prefix}door_opening_mechanism_link_x_slide_screwing"
+        m="1"
+        x="0.073"
+        y="0.015"
+        z="0.175"
+        r="1"
+        g="1"
+        b="1">
         <origin xyz="0.038 -0.027 0" rpy="0 0 1.57079632679"/>
-    </joint>
-    <link name="${prefix}door_opening_mechanism_link_x_slide_screwing">
-        <inertial>
-            <mass value="1" />
-            <origin xyz="0 0 0" />
-            <xacro:box_inertia_robot m="1" x="0.073" y="0.015" z="0.175"/>
-        </inertial>
-        <visual>
-            <origin xyz="0 0 0" rpy="0 0 0"/>
-            <geometry>
-                <box size="0.073 0.015 0.175"/>
-            </geometry>
-        </visual>
-        <collision>
-            <origin xyz="0 0 0" rpy="0 0 0"/>
-            <geometry>
-                <box size="0.073 0.015 0.175"/>
-            </geometry>
-        </collision>
-    </link>
-    <gazebo reference="${prefix}door_opening_mechanism_link_x_slide_screwing">
-        <visual>
-            <material>
-                <!-- RGBA -->
-                <ambient>1 1 1 1</ambient>
-                <diffuse>1 1 1 1</diffuse>
-                <specular>1 1 1 1</specular>
-            </material>
-        </visual>
-    </gazebo>
+    </xacro:basic_box>
     <joint name="${prefix}door_opening_mechanism_joint_tilting_hook" type="revolute" >
         <axis xyz="1 0 0" />

File: src/ros2/robot_description/rb_theron_common/rb_theron_description/urdf/door_opening_mechanism/hook.urdf.xacro (robot description, xacro)
@@ -7,72 +7,11 @@
     </xacro:macro>
     <xacro:macro name="hook" params="prefix suffix parent *origin r g b">
-    <joint name="${prefix}hook_joint_${suffix}" type="fixed" >
-        <parent link="${parent}" />
-        <child link="${prefix}hook_base_link_${suffix}" />
+    <xacro:include filename="$(find rb_theron_description)/urdf/door_opening_mechanism/basic_box.urdf.xacro" />
+    <xacro:basic_box parent="${prefix}${parent}" joint_name="${prefix}hook_joint_${suffix}" link_name="${prefix}hook_base_link_${suffix}" m="0.1" x="0.06" y="0.01" z="0.04" r="0" g="0" b="1">
         <xacro:insert_block name="origin" />
-    </joint>
-    <link name="${prefix}hook_base_link_${suffix}">
-        <inertial>
-            <mass value="0.1" />
-            <origin xyz="0 0 0" />
-            <xacro:box_inertia_robot m="0.1" x="0.06" y="0.01" z="0.04"/>
-        </inertial>
-        <visual>
-            <origin xyz="0 0 0" rpy="0 0 0" />
-            <geometry>
-                <box size="0.06 0.01 0.04"/>
-            </geometry>
-        </visual>
-        <collision>
-            <origin xyz="0 0 0" rpy="0 0 0" />
-            <geometry>
-                <box size="0.06 0.01 0.04"/>
-            </geometry>
-        </collision>
-    </link>
-    <gazebo reference="${prefix}hook_base_link_${suffix}">
-        <visual>
-            <material>
-                <!-- RGBA -->
-                <ambient>${r} ${g} ${b} 1</ambient>
-                <diffuse>${r} ${g} ${b} 1</diffuse>
-                <specular>${r} ${g} ${b} 1</specular>
-            </material>
-        </visual>
-    </gazebo>
-    <joint name="${prefix}hook_joint_front_side_${suffix}" type="fixed" >
-        <parent link="${prefix}hook_base_link_${suffix}" />
-        <child link="${prefix}hook_front_side_link_${suffix}" />
+    </xacro:basic_box>
+    <xacro:basic_box parent="${prefix}hook_base_link_${suffix}" joint_name="${prefix}hook_joint_front_side_${suffix}" link_name="${prefix}hook_front_side_link_${suffix}" m="0.1" x="0.008" y="0.03" z="0.04" r="0" g="0" b="1">
         <origin xyz="-0.026 0.02 0" rpy="0 0 0"/>
-    </joint>
-    <link name="${prefix}hook_front_side_link_${suffix}">
-        <inertial>
-            <mass value="0.1" />
-            <origin xyz="0 0 0" />
-            <xacro:box_inertia_robot m="0.1" x="0.008" y="0.03" z="0.04"/>
-        </inertial>
-        <visual>
-            <origin xyz="0 0 0" rpy="0 0 0" />
-            <geometry>
-                <box size="0.008 0.03 0.04"/>
-            </geometry>
-        </visual>
-        <collision>
-            <origin xyz="0 0 0" rpy="0 0 0" />
-            <geometry>
-                <box size="0.008 0.03 0.04"/>
-            </geometry>
-        </collision>
-    </link>
-    <gazebo reference="${prefix}hook_front_side_link_${suffix}">
-        <visual>
-            <material>
-                <!-- RGBA -->
-                <ambient>${r} ${g} ${b} 1</ambient>
-                <diffuse>${r} ${g} ${b} 1</diffuse>
-                <specular>${r} ${g} ${b} 1</specular>
-            </material>
-        </visual>
-    </gazebo>
+    </xacro:basic_box>
     </xacro:macro>
 </robot>

Commit message: More links for the hook

File: src/ros2/robot_description/rb_theron_common/rb_theron_description/urdf/door_opening_mechanism/door_opening_mechanism.urdf.xacro (robot description, xacro)
@@ -15,25 +15,19 @@
         properly, because this makes some of the wheels lose contact to the ground and
         therefore steering of the rb_theron becomes impossible. -->
+        <!-- Base link -->
         <xacro:property name="door_opening_mechanism_base_link" value="${prefix}door_opening_mechanism_base_link" />
-        <joint name="${prefix}door_opening_mechanism_joint" type="fixed">
-            <parent link="${parent}"/>
-            <child link="${door_opening_mechanism_base_link}"/>
+        <xacro:basic_box
+            parent="${parent}"
+            joint_name="${prefix}door_opening_mechanism_joint"
+            link_name="${door_opening_mechanism_base_link}"
+            m="0.001"
+            x="0.001"
+            y="0.001"
+            z="0.001"
+            r="0"
+            g="1"
+            b="1">
             <xacro:insert_block name="origin" />
-        </joint>
-        <!-- Base link -->
-        <link name="${door_opening_mechanism_base_link}">
-            <visual>
-            <origin xyz="0 0 0" rpy="0 0 0" />
-            <geometry>
-                <box size="0.001 0.001 0.001" />
-            </geometry>
-            </visual>
-            <collision>
-            <origin xyz="0 0 0" rpy="0 0 0" />
-            <geometry>
-                <box size="0.001 0.001 0.001" />
-            </geometry>
-            </collision>
-        </link>
+        </xacro:basic_box>
         <!-- Aluprofile frame -->
         <xacro:alu_profile prefix="${prefix}" suffix="bottom" parent="${door_opening_mechanism_base_link}" x="0.03" y="0.03" z="0.46" r="0.1" g="0.1" b="0.1" >
@@ -60,5 +54,5 @@
             r="0"
             g="1"
-            b="0">
+            b="1">
             <origin xyz="-0.015 0.2 0.55" rpy="0 0 0"/>
         </xacro:basic_box>

File: src/ros2/robot_description/rb_theron_common/rb_theron_description/urdf/door_opening_mechanism/hook.urdf.xacro (robot description, xacro)
@@ -24,5 +24,5 @@
         parent="${prefix}hook_base_link_${suffix}"
         joint_name="${prefix}hook_joint_front_side_${suffix}"
-        link_name="${prefix}hook_front_side_link_${suffix}"
+        link_name="${prefix}hook_link_front_side_${suffix}"
         m="0.1"
         x="0.008"
@@ -34,4 +34,17 @@
         <origin xyz="-0.026 0.02 0" rpy="0 0 0"/>
     </xacro:basic_box>
+    <xacro:basic_box
+        parent="${prefix}hook_base_link_${suffix}"
+        joint_name="${prefix}hook_joint_back_side_${suffix}"
+        link_name="${prefix}hook_link_back_side_${suffix}"
+        m="0.1"
+        x="0.008"
+        y="0.03"
+        z="0.04"
+        r="0"
+        g="0"
+        b="1">
+        <origin xyz="+0.026 0.02 0" rpy="0 0 0"/>
+    </xacro:basic_box>
     </xacro:macro>
 </robot>

Commit message: temporary commit: turned the door openenmechanisim up

File: src/ros2/robot_description/rb_theron_common/rb_theron_description/urdf/door_opening_mechanism/door_opening_mechanism.urdf.xacro (robot description, xacro)
@@ -149,5 +149,5 @@
             g="1"
             b="0">
-            <origin xyz="0 -0.025 0" rpy="0 1.57079632679 0"/>
+            <origin xyz="0 -0.025 0" rpy="1.57079632679 1.57079632679 0"/>
         </xacro:basic_joint>
         <!-- Gripper -->

Commit message: Resetting the roll value to the correct angle for now

File: src/ros2/robot_description/rb_theron_common/rb_theron_description/urdf/door_opening_mechanism/door_opening_mechanism.urdf.xacro (robot description, xacro)
@@ -149,6 +149,6 @@
             g="1"
             b="0">
-            <!-- TODO the default value for roll was changed from 0 to pi/2. Revert this change when the mechanism is working -->
-            <origin xyz="0 -0.025 0" rpy="1.57079632679 1.57079632679 0"/>
+            <!-- The default value for roll can be changed from 0 to pi/2 to position the arm upwards to get it out of the way -->
+            <origin xyz="0 -0.025 0" rpy="0 1.57079632679 0"/>
         </xacro:basic_joint>
         <!-- Gripper -->

Commit message: feat: add rotating arm and freely rotating hook

File: src/ros2/robot_description/rb_theron_common/rb_theron_description/urdf/door_opening_mechanism/door_opening_mechanism.urdf.xacro (robot description, xacro)
@@ -125,8 +125,13 @@
         </xacro:basic_box>
         <!-- Tilting arm -->
-        <xacro:include filename="$(find rb_theron_description)/urdf/door_opening_mechanism/arm_variations/tilting_arm.urdf.xacro" />
+        <!-- <xacro:include filename="$(find rb_theron_description)/urdf/door_opening_mechanism/arm_variations/tilting_arm.urdf.xacro" />
         <xacro:tilting_arm prefix="${prefix}" parent="${prefix}door_opening_mechanism_link_x_slide_screwing" >
             <origin xyz="0 -0.025 0" rpy="0 1.57079632679 0"/>
-        </xacro:tilting_arm>
+        </xacro:tilting_arm> -->
+        <!-- Rotating arm -->
+        <xacro:include filename="$(find rb_theron_description)/urdf/door_opening_mechanism/arm_variations/rotating_arm.urdf.xacro" />
+        <xacro:rotating_arm prefix="${prefix}" parent="${prefix}door_opening_mechanism_link_x_slide_screwing" arm_length="0.3" >
+            <origin xyz="0.05 -0.025 0" rpy="0 0 1.57079632679"/>
+        </xacro:rotating_arm>
     </xacro:macro>
 </robot>

Commit message: refactor: reorganizes axis for door opening mechanism

File: src/ros2/robot_description/rb_theron_common/rb_theron_description/urdf/door_opening_mechanism/door_opening_mechanism.urdf.xacro (robot description, xacro)
@@ -62,6 +62,6 @@
             joint_type="prismatic"
             axis_x="0"
-            axis_y="1"
-            axis_z="0"
+            axis_y="0"
+            axis_z="1"
             lower_limit="-0.05"
             upper_limit="0.25"
@@ -75,10 +75,10 @@
             m="2.64"
             x="0.06"
-            y="0.06"
-            z="0.55"
+            y="0.55"
+            z="0.06"
             r="1"
             g="0"
             b="0">
-            <origin xyz="-0.075 -0.225 -0.1" rpy="1.57079632679 0 0"/>
+            <origin xyz="-0.075 -0.225 -0.1" rpy="0 0 0"/>
         </xacro:basic_joint>
         <xacro:basic_joint
@@ -105,5 +105,5 @@
             g="1"
             b="1">
-            <origin xyz="-0.04 0 0" rpy="0 0 1.57079632679"/>
+            <origin xyz="-0.04 0 0" rpy="1.57079632679 4.71238898038 0"/>
         </xacro:basic_joint>
         <xacro:basic_box

Commit message: fix: moving x-axis slide a little bit to the side

File: src/ros2/robot_description/rb_theron_common/rb_theron_description/urdf/door_opening_mechanism/door_opening_mechanism.urdf.xacro (robot description, xacro)
@@ -115,5 +115,5 @@
             g="1"
             b="1">
-            <origin xyz="-0.032 0 0" rpy="1.57079632679 4.71238898038 0"/>
+            <origin xyz="-0.032 0.15 0" rpy="1.57079632679 4.71238898038 0"/>
         </xacro:basic_joint>
         <xacro:basic_box

Commit message: chore: slightly changes position of y-axis

File: src/ros2/robot_description/rb_theron_common/rb_theron_description/urdf/door_opening_mechanism/door_opening_mechanism.urdf.xacro (robot description, xacro)
@@ -85,5 +85,5 @@
             g="0"
             b="0">
-            <origin xyz="-0.075 -0.225 -0.1" rpy="0 0 0"/>
+            <origin xyz="-0.075 -0.225 0.0" rpy="0 0 0"/>
         </xacro:basic_joint>
         <xacro:basic_joint
