Commit message: minor fix for origin of module cage

File: src/ros2/robot_description/rb_theron_common/rb_theron_description/urdf/module_cage/module_cage.urdf.xacro (robot description, xacro)
@@ -21,5 +21,5 @@
     <visual>
       <xacro:if value="${hq}">
-        <origin xyz="0 0 0" rpy="0 0 0" />
+        <origin xyz="0.5 0.0 -0.8" rpy="0 0 1.57" />
         <geometry>
           <mesh filename="$(find rb_theron_description)/meshes/module_cage/module_cage.stl" scale="0.001 0.001 0.001"/>

Commit message: Fixing cage mass

File: src/ros2/robot_description/rb_theron_common/rb_theron_description/urdf/module_cage/module_cage.urdf.xacro (robot description, xacro)
@@ -15,10 +15,7 @@
   <link name="${prefix}module_cage_link">
     <inertial>
-      <!-- Mass should actually not be zero, but there is an issue, that if there is too much load on the theron base,
-      it would be able to drive properly, because this makes some of the wheels lose contact to the ground and
-      therefore steering of the rb_theron becomes impossible -->
-      <mass value="0.0" />
+      <mass value="8.0" />
       <origin xyz="0 0 0" />
-      <xacro:box_inertia_robot m="10" x="0.25" y="0.25" z="1.55"/>
+      <xacro:box_inertia_robot m="8" x="0.25" y="0.25" z="1.55"/>
     </inertial>
     <visual>
