Commit message: creating directory moveit2_ressources and moveit configs for simple door opening mechanism

File: src/ros2/robot_description/rb_theron_common/rb_theron_description/robots/robot_door_opening_mechanism.urdf.xacro (robot description, xacro)
@@ -42,3 +42,7 @@
 		<origin xyz="0 0 0.1" rpy="0 0 0"/>
 	</xacro:door_opening_mechanism>
+  <plugin
+    filename="libgz-sim-joint-state-publisher-system"
+    name="gz::sim::systems::JointStatePublisher">
+  </plugin>
 </robot>

File: src/ros2/simulation/moveit2_ressources/moveit2_door_opening_mechanism/config/rb_theron.ros2_control.xacro (robot description, xacro)
@@ -15,18 +15,4 @@
                 <state_interface name="velocity"/>
             </joint>
-            <joint name="door_opening_mechanism_joint_x_axis_slide">
-                <command_interface name="position"/>
-                <state_interface name="position">
-                  <param name="initial_value">${initial_positions['door_opening_mechanism_joint_x_axis_slide']}</param>
-                </state_interface>
-                <state_interface name="velocity"/>
-            </joint>
-            <joint name="door_opening_mechanism_joint_tilting_hook">
-                <command_interface name="position"/>
-                <state_interface name="position">
-                  <param name="initial_value">${initial_positions['door_opening_mechanism_joint_tilting_hook']}</param>
-                </state_interface>
-                <state_interface name="velocity"/>
-            </joint>
         </ros2_control>
     </xacro:macro>

Commit message: More testing

File: src/ros2/robot_description/rb_theron_common/rb_theron_description/robots/robot_door_opening_mechanism.urdf.xacro (robot description, xacro)
@@ -7,6 +7,6 @@
                 izz="${m*(x*x+z*z)/12}" />
     </xacro:macro>
-    <!-- BASE_LINK -->
-    <link name="base_link">
+    <!-- base_footprint -->
+    <link name="base_footprint">
       <inertial>
         <mass value="45" />
@@ -27,5 +27,5 @@
       </collision>
     </link>
-    <gazebo reference="base_link">
+    <gazebo reference="base_footprint">
         <visual>
             <material>
@@ -38,8 +38,8 @@
     </gazebo>
 	<!-- ROBAST Door Opening Mechanism -->
-	<xacro:include filename="$(find rb_theron_description)/urdf/door_opening_mechanism/door_opening_mechanism.urdf.xacro" />
-	<xacro:door_opening_mechanism prefix="" parent="base_link" hq="false" >
+	<xacro:include filename="$(find rb_theron_description)/urdf/simple_mechanism/simple_mechanism.urdf.xacro" />
+	<xacro:simple_mechanism prefix="" parent="base_footprint" hq="false" >
 		<origin xyz="0 0 0.1" rpy="0 0 0"/>
-	</xacro:door_opening_mechanism>
+	</xacro:simple_mechanism>
   <plugin
     filename="libgz-sim-joint-state-publisher-system"

File: src/ros2/simulation/moveit2_ressources/moveit2_simple_mechanism/config/rb_theron.ros2_control.xacro (robot description, xacro)
@@ -8,8 +8,8 @@
                 <plugin>mock_components/GenericSystem</plugin>
             </hardware>
-            <joint name="door_opening_mechanism_joint_y_axis_slide">
+            <joint name="joint_1">
                 <command_interface name="position"/>
                 <state_interface name="position">
-                  <param name="initial_value">${initial_positions['door_opening_mechanism_joint_y_axis_slide']}</param>
+                  <param name="initial_value">${initial_positions['joint_1']}</param>
                 </state_interface>
                 <state_interface name="velocity"/>
