Commit message: fix: adds missing arg `model_door_opening_mechanism`

File: src/ros2/robot_description/rb_theron_common/rb_theron_description/robots/rb_theron_arm.urdf.xacro (robot description, xacro)
@@ -22,20 +22,15 @@
 	<xacro:arg name="ros2_control_hardware_type_positon_joint" default="mock_components" />
 	<xacro:arg name="ros_distro" default="humble" />
-	<!-- Whether the position joint should be modeled as a prismatic joint or just as a fixed joint -->
+	<!-- Whether the robot should have a door opening mechanism -->
+	<xacro:arg name="model_door_opening_mechanism" default="true" />
+	<!-- Whether the position joint should be modeled as a fixed joint, a prismatic joint or a planar joint -->
 	<xacro:arg name="model_position_joint" default="fixed" />
 	<xacro:property name="model_position_joint_prop" value="$(arg model_position_joint)"/>
-	<!-- If we model the position joint, the sensors need be placed in the base_link frame,
-	otherwise they should be placed in the base_footprint frame -->
-	<xacro:if value="${model_position_joint_prop == 'prismatic'}">
-		<xacro:property name="sensor_base_frame" value="base_link" />
+	<xacro:if value="${publish_bf}">
+		<xacro:property name="sensor_base_frame" value="base_footprint"/>
 	</xacro:if>
-	<xacro:if value="${model_position_joint_prop == 'fixed'}">
-		<xacro:if value="${publish_bf}">
-			<xacro:property name="sensor_base_frame" value="base_footprint" />
-		</xacro:if>
-		<xacro:unless value="${publish_bf}">
-			<xacro:property name="sensor_base_frame" value="base_link" />
-		</xacro:unless>
-	</xacro:if>
+	<xacro:unless value="${publish_bf}">
+		<xacro:property name="sensor_base_frame" value="base_link"/>
+	</xacro:unless>
     <xacro:include filename="$(find rb_theron_description)/urdf/bases/theron_base.urdf.xacro" />
     <xacro:include filename="$(find rb_theron_description)/urdf/inertia.urdf.xacro" />
@@ -44,4 +39,5 @@
       publish_bf="${publish_bf}"
       model_position_joint="$(arg model_position_joint)"
+	  model_door_opening_mechanism="$(arg model_door_opening_mechanism)"
       ros2_control_hardware_type_positon_joint="$(arg ros2_control_hardware_type_positon_joint)"
       hq="${hq}"

Commit message: feat: first attempt to run moveit_real_world without namespace

File: src/ros2/robot_description/rb_theron_common/rb_theron_description/robots/rb_theron_arm.urdf.xacro (robot description, xacro)
@@ -22,18 +22,7 @@
 	<xacro:arg name="ros2_control_hardware_type_positon_joint" default="mock_components" />
 	<xacro:arg name="ros_distro" default="humble" />
-	<!-- Whether the robot should have a door opening mechanism -->
-	<xacro:arg name="model_door_opening_mechanism" default="true" />
-	<!-- Whether the position joint should be modeled as a fixed joint, a prismatic joint or a planar joint -->
-	<xacro:arg name="model_position_joint" default="fixed" />
-	<xacro:property name="model_position_joint_prop" value="$(arg model_position_joint)"/>
-	<xacro:if value="${publish_bf}">
-		<xacro:property name="sensor_base_frame" value="base_footprint"/>
-	</xacro:if>
-	<xacro:unless value="${publish_bf}">
-		<xacro:property name="sensor_base_frame" value="base_link"/>
-	</xacro:unless>
     <xacro:include filename="$(find rb_theron_description)/urdf/bases/theron_base.urdf.xacro" />
     <xacro:include filename="$(find rb_theron_description)/urdf/inertia.urdf.xacro" />
-    <xacro:theron_base
+    <!-- <xacro:theron_base
       prefix="$(arg prefix)"
       publish_bf="${publish_bf}"
@@ -42,10 +31,15 @@
       ros2_control_hardware_type_positon_joint="$(arg ros2_control_hardware_type_positon_joint)"
       hq="${hq}"
-    />
+    /> -->
+	<xacro:include filename="$(find rb_theron_description)/urdf/door_opening_mechanism/ros2_control/position_ros2_control.urdf.xacro" />
+	<xacro:position_ros2_control
+		ros2_control_hardware_type_positon_joint="${ros2_control_hardware_type_positon_joint}"
+		ros_distro="${ros_distro}">
+	</xacro:position_ros2_control>
 	<!-- ROBAST Door Opening Mechanism -->
 	<xacro:include filename="$(find rb_theron_description)/urdf/door_opening_mechanism/door_opening_mechanism.urdf.xacro" />
 	<xacro:door_opening_mechanism
 	    prefix="$(arg prefix)"
-		parent="$(arg prefix)base_link"
+		parent="$(arg prefix)robot/base_link"
 		ros2_control_hardware_type="$(arg ros2_control_hardware_type)"
 		ros_distro="$(arg ros_distro)"

Commit message: fix: some smaller fixes to get `moveit_real_world` running after latest changes

File: src/ros2/robot_description/rb_theron_common/rb_theron_description/robots/rb_theron_arm.urdf.xacro (robot description, xacro)
@@ -34,7 +34,26 @@
 	<xacro:include filename="$(find rb_theron_description)/urdf/door_opening_mechanism/ros2_control/position_ros2_control.urdf.xacro" />
 	<xacro:position_ros2_control
-		ros2_control_hardware_type_positon_joint="${ros2_control_hardware_type_positon_joint}"
-		ros_distro="${ros_distro}">
+		ros2_control_hardware_type_positon_joint="$(arg ros2_control_hardware_type_positon_joint)"
+		ros_distro="$(arg ros_distro)">
 	</xacro:position_ros2_control>
+	<link name="$(arg prefix)robot/base_link">
+		<inertial>
+		<mass value="0.01" />
+		<origin xyz="0.0 0.0 0.0" />
+		<xacro:solid_cuboid_inertia m="0.01" w="0.001" h="0.001" d="0.001" />
+		</inertial>
+		<visual>
+		<origin xyz="0 0 0.01" rpy="0 0 0" />
+		<geometry>
+			<box size="0.001 0.001 0.001" />
+		</geometry>
+		</visual>
+		<collision>
+		<origin xyz="0 0 0.01" rpy="0 0 0" />
+		<geometry>
+			<box size="0.001 0.001 0.001" />
+		</geometry>
+		</collision>
+	</link>
 	<!-- ROBAST Door Opening Mechanism -->
 	<xacro:include filename="$(find rb_theron_description)/urdf/door_opening_mechanism/door_opening_mechanism.urdf.xacro" />

Commit message: feat: uses `robot` for `prefix` argument for real life

File: src/ros2/robot_description/rb_theron_common/rb_theron_description/robots/rb_theron_arm.urdf.xacro (robot description, xacro)
@@ -4,6 +4,4 @@
 	<!-- This is only used for MoveitStudio -->
 	<xacro:attribute name="web_ui_gripper" value="package://rb_theron_description/urdf/door_opening_mechanism/components/hook.urdf" />
-	<!-- Import differential base elements -->
-	<xacro:include filename="$(find rb_theron_description)/robots/rb_theron_base.urdf.xacro" />
 	<xacro:property name="PI" value="3.1415926535897931"/>
 	<!-- Flag to determine if the base_footprint should be published or not -->
@@ -22,14 +20,6 @@
 	<xacro:arg name="ros2_control_hardware_type_positon_joint" default="mock_components" />
 	<xacro:arg name="ros_distro" default="humble" />
-    <xacro:include filename="$(find rb_theron_description)/urdf/bases/theron_base.urdf.xacro" />
     <xacro:include filename="$(find rb_theron_description)/urdf/inertia.urdf.xacro" />
-    <!-- <xacro:theron_base
-      prefix="$(arg prefix)"
-      publish_bf="${publish_bf}"
-      model_position_joint="$(arg model_position_joint)"
-	  model_door_opening_mechanism="$(arg model_door_opening_mechanism)"
-      ros2_control_hardware_type_positon_joint="$(arg ros2_control_hardware_type_positon_joint)"
-      hq="${hq}"
-    /> -->
+	<!-- We add the ros2_control for the position joint here to launch the hardware interface for the position joint -->
 	<xacro:include filename="$(find rb_theron_description)/urdf/door_opening_mechanism/ros2_control/position_ros2_control.urdf.xacro" />
 	<xacro:position_ros2_control
@@ -37,5 +27,5 @@
 		ros_distro="$(arg ros_distro)">
 	</xacro:position_ros2_control>
-	<link name="$(arg prefix)robot/base_link">
+	<link name="$(arg prefix)base_link">
 		<inertial>
 		<mass value="0.01" />
@@ -60,5 +50,5 @@
 	<xacro:door_opening_mechanism
 	    prefix="$(arg prefix)"
-		parent="$(arg prefix)robot/base_link"
+		parent="$(arg prefix)base_link"
 		ros2_control_hardware_type="$(arg ros2_control_hardware_type)"
 		ros_distro="$(arg ros_distro)"

File: src/ros2/robot_description/rb_theron_common/rb_theron_description/urdf/bases/theron_base.urdf.xacro (robot description, xacro)
@@ -30,5 +30,5 @@
           <axis xyz="-1 0 0" />
           <origin xyz="0 0 0" rpy="0 0 0" />
-          <parent link="base_footprint"/>
+          <parent link="${prefix}base_footprint"/>
           <child link="${prefix}base_link"/>
           <limit lower="-1" upper="1" effort="1000" velocity="100" />
@@ -37,5 +37,5 @@
       <!-- Planar position joint -->
       <xacro:if value="${model_position_joint == 'planar'}">
-        <link name="odom">
+        <link name="${prefix}odom">
           <inertial>
             <mass value="0.01" />
@@ -58,5 +58,5 @@
         <joint name="position" type="planar">
           <origin rpy="0 0 0" xyz="0 0 0"/>
-          <parent link="odom"/>
+          <parent link="${prefix}odom"/>
           <child link="${prefix}base_footprint"/>
         </joint>
