Commit message: First draft for adding drawer

File: src/ros2/robot_description/rb_theron_common/rb_theron_description/robots/rb_theron.urdf.xacro (robot description, xacro)
@@ -101,3 +101,8 @@
 		<origin xyz="0.35 -0.0 -0.075" rpy="0 0 1.570796326794896619"/>
 	</xacro:module_cage> -->
+	<!-- ROBAST Drawer -->
+	<xacro:include filename="$(find rb_theron_description)/urdf/drawer/drawer.urdf.xacro" />
+	<xacro:drawer prefix="$(arg prefix)first" parent="$(arg prefix)base_link">
+		<origin xyz="0.0 0.0 0.3" rpy="0 0 0"/>
+	</xacro:drawer>
 </robot>

Commit message: Preparing theron urdf collisions to be readable by moveit

File: src/ros2/robot_description/rb_theron_common/rb_theron_description/robots/rb_theron.urdf.xacro (robot description, xacro)
@@ -97,12 +97,12 @@
 	<xacro:depthai_camera camera_name = "$(arg camera_name)" parent = "$(arg prefix)base_link" camera_model = "$(arg camera_model)" base_frame = "$(arg base_frame)" cam_pos_x = "$(arg cam_pos_x)" cam_pos_y = "$(arg cam_pos_y)" cam_pos_z = "$(arg cam_pos_z)" cam_roll = "$(arg cam_roll)" cam_pitch = "$(arg cam_pitch)" cam_yaw = "$(arg cam_yaw)"/>
 	<!-- ROBAST Module Cage -->
-	<!-- <xacro:include filename="$(find rb_theron_description)/urdf/module_cage/module_cage.urdf.xacro" />
+	<xacro:include filename="$(find rb_theron_description)/urdf/module_cage/module_cage.urdf.xacro" />
 	<xacro:module_cage prefix="$(arg prefix)module_cage" parent="$(arg prefix)base_link">
 		<origin xyz="0.35 -0.0 -0.075" rpy="0 0 1.570796326794896619"/>
-	</xacro:module_cage> -->
+	</xacro:module_cage>
 	<!-- ROBAST Drawer -->
 	<xacro:include filename="$(find rb_theron_description)/urdf/drawer/drawer.urdf.xacro" />
 	<xacro:drawer prefix="$(arg prefix)first" parent="$(arg prefix)base_link">
-		<origin xyz="0.0 0.0 0.3" rpy="0 0 0"/>
+		<origin xyz="0.105 0.0 0.3" rpy="0 0 0"/>
 	</xacro:drawer>
 </robot>

File: src/ros2/robot_description/rb_theron_common/rb_theron_description/urdf/bases/theron_base.urdf.xacro (robot description, xacro)
@@ -54,6 +54,6 @@
         <origin xyz="0 0 0" rpy="0 0 0 " />
         <geometry>
-          <!--box size="0.390 0.240 0.165"/-->
-          <mesh filename="$(find rb_theron_description)/meshes/bases/theron_base.stl"/>
+          <box size="0.390 0.240 0.165"/>
+          <!-- <mesh filename="$(find rb_theron_description)/meshes/bases/theron_base.stl"/> -->
         </geometry>
       </collision>
@@ -82,7 +82,8 @@
       </visual>
       <collision>
-        <origin xyz="0 0 0" rpy="0 0 0 " />
+        <origin xyz="0 0 0.2" rpy="0 0 0" />
         <geometry>
-          <mesh filename="$(find rb_theron_description)/meshes/bases/mcq_prototype_bottom_cover.dae"/>
+          <box size="0.655 0.54 0.02"/>
+          <!-- <mesh filename="$(find rb_theron_description)/meshes/bases/mcq_prototype_bottom_cover.dae"/> -->
         </geometry>
       </collision>

File: src/ros2/robot_description/rb_theron_common/rb_theron_description/urdf/module_cage/module_cage.urdf.xacro (robot description, xacro)
@@ -20,9 +20,10 @@
       </inertial>
       <visual>
-        <origin xyz="0 0 0" rpy="0 0 0" />
-		  		<!-- in this case change origin -->
+	  <origin xyz="0 ${0.655-0.167} 0.8" rpy="0 0 1.57" />
+        <!-- <origin xyz="0 0 0" rpy="0 0 0" /> -->
           <geometry>
             <!-- <box size="0.25 0.25 1.55"/> -->
-            <mesh filename="$(find rb_theron_description)/meshes/module_cage/module_cage.stl" scale="0.001 0.001 0.001"/>
+	    <box size="0.03 0.43 1.05"/>
+            <!-- <mesh filename="$(find rb_theron_description)/meshes/module_cage/module_cage.stl" scale="0.001 0.001 0.001"/> -->
           </geometry>
         <material name="darkgrey">
@@ -31,33 +32,11 @@
       </visual>
       <collision>
-        <origin xyz="0 0 0" rpy="0 0 0 " />
+        <origin xyz="0 ${0.655-0.167} 0.8" rpy="0 0 1.57" />
         <geometry>
-          <!-- <box size="0.25 0.25 1.55"/> -->
-          <mesh filename="$(find rb_theron_description)/meshes/module_cage/module_cage.stl" scale="0.001 0.001 0.001"/>
+          <box size="0.03 0.43 1.05"/>
+          <!-- <mesh filename="$(find rb_theron_description)/meshes/module_cage/module_cage.stl" scale="0.001 0.001 0.001"/> -->
         </geometry>
       </collision>
     </link>
-    <!-- <gazebo reference="${prefix}pole_link">
-			<mu1 value="100.0"/>
-			<mu2 value="100.0"/>
-			<kp value="500000.0" />
-			<kd value="1.0" />
-			<material>Gazebo/Yellow</material>
-			<turnGravityOff>false</turnGravityOff> -->
-			<!--kp>500000.0</kp>
-			<kd>10.0</kd>
-			<mu1>10</mu1>
-			<mu2>10</mu2>
-			<fdir1>1 0 0</fdir1-->
-			<!--minDepth>0.001</minDepth-->
-			<!--material>Gazebo/Black</material-->
-			<!--mu1 value="10"/>
-			<mu2 value="5"/>
-			<kp value="500000.0" />
-			<kd value="10.0" />
-			<fdir1 value="1 0 0"/>
-			<material>Gazebo/Yellow</material>
-			<turnGravityOff>false</turnGravityOff-->
-		<!-- </gazebo> -->
   </xacro:macro>
 </robot>

File: src/ros2/robot_description/rb_theron_common/rb_theron_description/urdf/rocker/mcq_prototype_rocker.urdf.xacro (robot description, xacro)
@@ -36,5 +36,5 @@
           <xacro:if value="${reflect}">
             <geometry>
-	          <mesh filename="$(find rb_theron_description)/meshes/rocker/mcq_prototype_rocker_r.dae" />
+	            <mesh filename="$(find rb_theron_description)/meshes/rocker/mcq_prototype_rocker_r.dae" />
             </geometry>
           </xacro:if>
@@ -49,10 +49,12 @@
           <xacro:if value="${reflect}">
             <geometry>
-	          <mesh filename="$(find rb_theron_description)/meshes/rocker/mcq_prototype_rocker_r.dae" />
+              <box size="0.2 0.022 0.01" />
+	            <!-- <mesh filename="$(find rb_theron_description)/meshes/rocker/mcq_prototype_rocker_r.dae" /> -->
             </geometry>
           </xacro:if>
           <xacro:unless value="${reflect}">
             <geometry>
-              <mesh filename="$(find rb_theron_description)/meshes/rocker/mcq_prototype_rocker_l.dae" />
+                <box size="0.2 0.022 0.01" />
+                <!-- <mesh filename="$(find rb_theron_description)/meshes/rocker/mcq_prototype_rocker_l.dae" /> -->
             </geometry>
 		  </xacro:unless>

File: src/ros2/robot_description/rb_theron_common/rb_theron_description/urdf/wheels/castor.urdf.xacro (robot description, xacro)
@@ -39,5 +39,6 @@
         <origin xyz="0 0 0" rpy="0 0 0" />
           <geometry>
-	       <mesh filename="$(find rb_theron_description)/meshes/wheels/mcq_prototype_base_castor.dae" />
+            <box size="0.022 0.022 0.01" />
+	          <!-- <mesh filename="$(find rb_theron_description)/meshes/wheels/mcq_prototype_base_castor.dae" /> -->
           </geometry>
       </collision>

File: src/ros2/robot_description/robotnik_sensors/urdf/rs_bpearl.urdf.xacro (robot description, xacro)
@@ -22,5 +22,6 @@
         <origin xyz="0 0 0" rpy="0 0 0"/>
         <geometry>
-          <mesh filename="$(find robotnik_sensors)/meshes/rs_bpearl.stl" />
+          <cylinder radius="0.10" length="0.11"/>
+          <!-- <mesh filename="$(find robotnik_sensors)/meshes/rs_bpearl.stl" /> -->
         </geometry>
       </collision>

File: src/ros2/robot_description/robotnik_sensors/urdf/sick_nanoscan3.urdf.xacro (robot description, xacro)
@@ -13,6 +13,6 @@
 				<geometry>
 					<!--<box size="0.106 0.094 0.152"/>-->
-					<!--<cylinder radius="0.058" length="0.152"/>-->
-					<mesh filename="$(find robotnik_sensors)/meshes/sick_nanoscan3.stl"/>
+					<cylinder radius="0.058" length="0.152"/>
+					<!-- <mesh filename="$(find robotnik_sensors)/meshes/sick_nanoscan3.stl"/> -->
 				</geometry>
 			</collision>

Commit message: Extended support for hq (high quality) flag to create a complete low quality model of the theron for moveit

File: src/ros2/robot_description/rb_theron_common/rb_theron_description/robots/rb_theron.urdf.xacro (robot description, xacro)
@@ -33,5 +33,5 @@
 	<xacro:property name="wheel_offset_z" value="0.015" />
 	<!-- Flag to select the high or low quality model -->
-	<xacro:property name="hq" value="true" />
+	<xacro:property name="hq" value="false" />
 	<!-- *************** -->
 	<!-- Robots Elements -->
@@ -61,8 +61,8 @@
 	<!-- TODO: Should be sensor_intel_d435, but this one isn't migrated to ros2 yet -->
 	<!-- TODO: Moved 0.01 in x, otherwise the camera is still inside the robot -->
-	<xacro:sensor_r430 prefix="$(arg prefix)front_realsense_camera" parent="$(arg prefix)base_link" prefix_topic="front_realsense_camera">
+	<xacro:sensor_r430 prefix="$(arg prefix)front_realsense_camera" parent="$(arg prefix)base_link" prefix_topic="front_realsense_camera" hq="${hq}">
 		<origin xyz="0.3305 0.0 0.1468" rpy="0 0 0"/>
 	</xacro:sensor_r430>
-	<xacro:sensor_r430 prefix="$(arg prefix)back_realsense_camera" parent="$(arg prefix)base_link" prefix_topic="back_realsense_camera">
+	<xacro:sensor_r430 prefix="$(arg prefix)back_realsense_camera" parent="$(arg prefix)base_link" prefix_topic="back_realsense_camera" hq="${hq}">
 		<origin xyz="-0.3305 0.0 0.1468" rpy="0 0 3.1416"/>
 	</xacro:sensor_r430>
@@ -74,5 +74,5 @@
 		<origin xyz="-0.1975 0.0 0.1598" rpy="0 0 0"/>
 	</xacro:sensor_imu_hector>
-	<xacro:sensor_sick_nanoscan3 prefix="$(arg prefix)front_laser" parent="$(arg prefix)base_link" prefix_topic="front_laser" min_angle="-1.9507619" max_angle="1.9507619">
+	<xacro:sensor_sick_nanoscan3 prefix="$(arg prefix)front_laser" parent="$(arg prefix)base_link" prefix_topic="front_laser" hq="${hq}" min_angle="-1.9507619" max_angle="1.9507619">
 		<origin xyz="0.250 0.0 0.1643" rpy="0 3.1416 3.1416"/>
 	</xacro:sensor_sick_nanoscan3>
@@ -80,5 +80,5 @@
 		<origin xyz="0.214 0.0 0.275" rpy="-1.57079632679 0 -0.23"/>
 	</xacro:sensor_rs_lidar_16>-->
-	<xacro:sensor_rs_bpearl prefix="$(arg prefix)top_laser"  parent="$(arg prefix)base_link" prefix_topic="top_laser" range_min="0.1" range_max="90" hfov="360" samples="1200" vfov="90.0" lasers="32" fps="15" gpu="false">
+	<xacro:sensor_rs_bpearl prefix="$(arg prefix)top_laser"  parent="$(arg prefix)base_link" prefix_topic="top_laser" hq="${hq}" range_min="0.1" range_max="90" hfov="360" samples="1200" vfov="90.0" lasers="32" fps="15" gpu="false">
             <origin xyz="0.28 -0.159 1.22" rpy="-1.570796326795 0 -1.570796326795"/>
         </xacro:sensor_rs_bpearl>
@@ -95,5 +95,5 @@
 	<xacro:arg name="cam_pitch"     default="0.0" />
 	<xacro:arg name="cam_yaw"       default="0.0" />
-	<xacro:depthai_camera camera_name = "$(arg camera_name)" parent = "$(arg prefix)base_link" camera_model = "$(arg camera_model)" base_frame = "$(arg base_frame)" cam_pos_x = "$(arg cam_pos_x)" cam_pos_y = "$(arg cam_pos_y)" cam_pos_z = "$(arg cam_pos_z)" cam_roll = "$(arg cam_roll)" cam_pitch = "$(arg cam_pitch)" cam_yaw = "$(arg cam_yaw)"/>
+	<!-- <xacro:depthai_camera camera_name = "$(arg camera_name)" parent = "$(arg prefix)base_link" camera_model = "$(arg camera_model)" base_frame = "$(arg base_frame)" cam_pos_x = "$(arg cam_pos_x)" cam_pos_y = "$(arg cam_pos_y)" cam_pos_z = "$(arg cam_pos_z)" cam_roll = "$(arg cam_roll)" cam_pitch = "$(arg cam_pitch)" cam_yaw = "$(arg cam_yaw)"/> -->
 	<!-- ROBAST Module Cage -->
 	<xacro:include filename="$(find rb_theron_description)/urdf/module_cage/module_cage.urdf.xacro" />

File: src/ros2/robot_description/rb_theron_common/rb_theron_description/urdf/bases/theron_base.urdf.xacro (robot description, xacro)
@@ -35,6 +35,6 @@
       </inertial>
       <visual>
-        <origin xyz="0 0 0" rpy="0 0 0" />
         <xacro:if value="${hq}">
+          <origin xyz="0 0 0" rpy="0 0 0" />
           <geometry>
             <mesh filename="$(find rb_theron_description)/meshes/bases/theron_base.stl"/>
@@ -42,7 +42,7 @@
         </xacro:if>
         <xacro:unless value="${hq}">
-		  <!-- in this case change origin -->
+          <origin xyz="0 0 0.05" rpy="0 0 0" />
           <geometry>
-            <box size="0.700 0.600 0.350"/>
+            <box size="0.390 0.240 0.165"/>
           </geometry>
         </xacro:unless>
@@ -52,5 +52,5 @@
       </visual>
       <collision>
-        <origin xyz="0 0 0" rpy="0 0 0 " />
+        <origin xyz="0 0 0.05" rpy="0 0 0 " />
         <geometry>
           <box size="0.390 0.240 0.165"/>
@@ -66,6 +66,6 @@
       </inertial>
       <visual>
-        <origin xyz="0 0 0" rpy="0 0 0" />
         <xacro:if value="${hq}">
+          <origin xyz="0 0 0" rpy="0 0 0"/>
           <geometry>
             <mesh filename="$(find rb_theron_description)/meshes/bases/mcq_prototype_bottom_cover.dae"/>
@@ -73,6 +73,7 @@
         </xacro:if>
         <xacro:unless value="${hq}">
+          <origin xyz="0 0 0.2" rpy="0 0 0"/>
           <geometry>
-            <box size="0.700 0.600 0.350"/>
+            <box size="0.655 0.54 0.02"/>
           </geometry>
         </xacro:unless>

File: src/ros2/robot_description/rb_theron_common/rb_theron_description/urdf/rocker/mcq_prototype_rocker.urdf.xacro (robot description, xacro)
@@ -35,13 +35,27 @@
         <origin xyz="0 0 0" rpy="0 0 0" />
           <xacro:if value="${reflect}">
-            <geometry>
-	            <mesh filename="$(find rb_theron_description)/meshes/rocker/mcq_prototype_rocker_r.dae" />
-            </geometry>
+            <xacro:if value="${hq}">
+	            <geometry>
+                <mesh filename="$(find rb_theron_description)/meshes/rocker/mcq_prototype_rocker_r.stl" />
+              </geometry>
+            </xacro:if>
+            <xacro:unless value="${hq}">
+              <geometry>
+                <box size="0.2 0.022 0.01" />
+              </geometry>
+            </xacro:unless>
           </xacro:if>
           <xacro:unless value="${reflect}">
-            <geometry>
-              <mesh filename="$(find rb_theron_description)/meshes/rocker/mcq_prototype_rocker_l.dae" />
-            </geometry>
-		  </xacro:unless>
+            <xacro:if value="${hq}">
+              <geometry>
+                <mesh filename="$(find rb_theron_description)/meshes/rocker/mcq_prototype_rocker_l.stl" />
+              </geometry>
+            </xacro:if>
+            <xacro:unless value="${hq}">
+              <geometry>
+                <box size="0.2 0.022 0.01" />
+              </geometry>
+            </xacro:unless>
+		      </xacro:unless>
       </visual>
       <collision>
@@ -98,6 +112,4 @@
 			</joint>
 		</ros2_control>
-	<!-- Flag to select the high or low quality model -->
-	<xacro:property name="hq" value="true" />
     <xacro:property name="wheel_offset_x" value="-0.1175" />
     <xacro:if value="${reflect}">
@@ -123,20 +135,4 @@
 		<origin xyz="${caster_offset_x} ${caster_offset_y} ${caster_offset_z}" rpy="0 0 0"/>
 	</xacro:caster>
-    <!-- gazebo reference="${prefix}support">
-			<mu1 value="5.0"/>
-			<mu2 value="0.5"/>
-			<kp value="10000000.0" />
-			<kd value="1.0" />
-			<fdir1 value="1 0 0"/>
-      <turnGravityOff>false</turnGravityOff>
-    </gazebo>
-     <gazebo reference="${prefix}_wheel">
-			<mu1 value="5.0"/>
-			<mu2 value="0.5"/>
-			<kp value="10000000.0" />
-			<kd value="1.0" />
-			<fdir1 value="1 0 0"/>
-      <turnGravityOff>false</turnGravityOff>
-    </gazebo -->
  </xacro:macro>
 </robot>

File: src/ros2/robot_description/rb_theron_common/rb_theron_description/urdf/wheels/castor.urdf.xacro (robot description, xacro)
@@ -32,7 +32,12 @@
       <visual>
         <origin xyz="0 0 0" rpy="0 0 0" />
-          <geometry>
-	       <mesh filename="$(find rb_theron_description)/meshes/wheels/mcq_prototype_base_castor.dae" />
-          </geometry>
+        <geometry>
+          <xacro:if value="${hq}">
+            <mesh filename="$(find rb_theron_description)/meshes/wheels/mcq_prototype_base_castor.dae" />
+          </xacro:if>
+          <xacro:unless value="${hq}">
+            <box size="0.022 0.022 0.01" />
+          </xacro:unless>
+        </geometry>
       </visual>
       <collision>

File: src/ros2/robot_description/robotnik_sensors/urdf/intel_r430.urdf.xacro (robot description, xacro)
@@ -19,5 +19,5 @@
   <xacro:property name="r430_cam_depth_py" value="-0.0115"/>
   <xacro:property name="r430_cam_depth_pz" value="0.0"/>
-  <xacro:macro name="sensor_r430" params="prefix parent prefix_topic:='front_rgbd_camera' *origin">
+  <xacro:macro name="sensor_r430" params="prefix parent prefix_topic:='front_rgbd_camera' hq *origin">
     <!-- camera body, with origin at bottom screw mount -->
     <joint name="${prefix}_camera_joint" type="fixed">
@@ -28,9 +28,13 @@
     <link name="${prefix}_camera_link">
       <visual>
-      <!-- origin xyz="0 ${-r430_cam_mount_from_center_offset} ${r430_cam_height/2}" rpy="${M_PI/2} 0 ${M_PI/2}"/ -->
-      <origin xyz="0 ${-r430_cam_mount_from_center_offset} 0" rpy="0 0 0"/>
+        <!-- origin xyz="0 ${-r430_cam_mount_from_center_offset} ${r430_cam_height/2}" rpy="${M_PI/2} 0 ${M_PI/2}"/ -->
+        <origin xyz="0 ${-r430_cam_mount_from_center_offset} 0" rpy="0 0 0"/>
         <geometry>
-          <!-- box size="${r430_cam_width} ${r430_cam_height} ${r430_cam_depth}"/ -->
-          <mesh filename="$(find robotnik_sensors)/meshes/intel_r430.dae" />
+          <xacro:if value="${hq}">
+            <mesh filename="$(find robotnik_sensors)/meshes/intel_r430.dae" />
+          </xacro:if>
+          <xacro:unless value="${hq}">
+            <box size="${r430_cam_depth} ${r430_cam_width} ${r430_cam_height} "/>
+          </xacro:unless>
         </geometry>
         <material name="aluminum">

File: src/ros2/robot_description/robotnik_sensors/urdf/rs_bpearl.urdf.xacro (robot description, xacro)
@@ -2,5 +2,5 @@
 <robot name="sensor_rs_bpearl" xmlns:xacro="http://wiki.ros.org/xacro">
   <xacro:property name="M_PI" value="3.1415926535897931" />
-  <xacro:macro name="sensor_rs_bpearl" params="prefix parent prefix_topic *origin range_min range_max hfov samples vfov lasers fps gpu:=true">
+  <xacro:macro name="sensor_rs_bpearl" params="prefix parent prefix_topic hq *origin range_min range_max hfov samples vfov lasers fps gpu:=true">
     <joint name="${prefix}_base_joint" type="fixed">
       <xacro:insert_block name="origin" />
@@ -10,8 +10,13 @@
     <link name="${prefix}_base_link">
       <visual>
-      <!-- origin xyz="0 0 0" rpy="0 0 1.5708"/ -->
-      <origin xyz="0 0 0" rpy="0 0 0"/>
+        <!-- origin xyz="0 0 0" rpy="0 0 1.5708"/ -->
+        <origin xyz="0 0 0" rpy="0 0 0"/>
         <geometry>
-          <mesh filename="$(find robotnik_sensors)/meshes/rs_bpearl.stl" />
+          <xacro:if value="${hq}">
+            <mesh filename="$(find robotnik_sensors)/meshes/rs_bpearl.stl" />
+          </xacro:if>
+          <xacro:unless value="${hq}">
+            <cylinder radius="0.10" length="0.11"/>
+          </xacro:unless>
         </geometry>
         <material name="blackgray_color">

File: src/ros2/robot_description/robotnik_sensors/urdf/sick_nanoscan3.urdf.xacro (robot description, xacro)
@@ -2,5 +2,5 @@
 <robot name="sensor_sick_nanoscan3"
 	xmlns:xacro="http://wiki.ros.org/xacro">
-	<xacro:macro name="sensor_sick_nanoscan3" params="prefix parent prefix_topic:='front_laser' *origin max_angle:=2.3998 min_angle:=-2.3998 gpu:=^|false">
+	<xacro:macro name="sensor_sick_nanoscan3" params="prefix parent prefix_topic:='front_laser' hq *origin max_angle:=2.3998 min_angle:=-2.3998 gpu:=^|false">
 		<joint name="${prefix}_base_joint" type="fixed">
 			<xacro:insert_block name="origin" />
@@ -13,5 +13,5 @@
 				<geometry>
 					<!--<box size="0.106 0.094 0.152"/>-->
-					<cylinder radius="0.058" length="0.152"/>
+					<cylinder radius="0.058" length="0.07"/>
 					<!-- <mesh filename="$(find robotnik_sensors)/meshes/sick_nanoscan3.stl"/> -->
 				</geometry>
@@ -19,7 +19,14 @@
 			<visual>
 				<origin xyz="0 0 0" rpy="0 0 0"/>
-				<geometry>
-					<mesh filename="$(find robotnik_sensors)/meshes/sick_nanoscan3.stl"/>
-				</geometry>
+				<xacro:if value="${hq}">
+					<geometry>
+						<mesh filename="$(find robotnik_sensors)/meshes/sick_nanoscan3.stl"/>
+					</geometry>
+				</xacro:if>
+				<xacro:unless value="${hq}">
+					<geometry>
+						<cylinder radius="0.058" length="0.07"/>
+					</geometry>
+				</xacro:unless>
 			</visual>
 			<inertial>

Commit message: Robot description commit

File: src/ros2/robot_description/rb_theron_common/rb_theron_description/robots/rb_theron.urdf.xacro (robot description, xacro)
@@ -41,7 +41,5 @@
 	<!-- this property is for the chassis -->
 	<!-- rbogie base -->
-	<xacro:theron_base prefix="$(arg prefix)" publish_bf="true" hq="${hq}" />
-	<!-- Gazebo ros control pluggins -->
-	<xacro:ros_control prefix="$(arg prefix)"/>
+	<xacro:theron_base prefix="$(arg prefix)" publish_bf="false" hq="${hq}" />
 	<xacro:gazebo_colors prefix="$(arg prefix)"/>
 	<!-- WHEELS -->
@@ -106,3 +104,5 @@
 		<origin xyz="0.105 0.0 0.3" rpy="0 0 0"/>
 	</xacro:drawer>
+	<!-- Gazebo ros control pluggins -->
+	<xacro:ros_control prefix="$(arg prefix)"/>
 </robot>

File: src/ros2/robot_description/rb_theron_common/rb_theron_description/urdf/common.gazebo.xacro (robot description, xacro)
@@ -7,5 +7,5 @@
 				<parameters>$(find rb_theron_description)/config/rb_theron_controller.yaml</parameters>
 			</plugin> -->
-			<plugin name="joint_state" filename="libgazebo_ros_joint_state_publisher.so">
+			<!-- <plugin name="joint_state" filename="libgazebo_ros_joint_state_publisher.so">
 				<ros>
 					<remapping>~/out:=joint_states</remapping>
@@ -25,5 +25,6 @@
 				<joint_name>$(arg prefix)leftjoint_wheel</joint_name>
 				<joint_name>$(arg prefix)rightjoint_wheel</joint_name>
-			</plugin>
+				<joint_name>top_drawer_joint</joint_name>
+			</plugin> -->
 			<plugin name="diff_drive" filename="libgazebo_ros_diff_drive.so">
 				<alwaysOn>1</alwaysOn>

File: src/ros2/robot_description/rb_theron_common/rb_theron_description/urdf/drawer/drawer.urdf.xacro (robot description, xacro)
@@ -46,4 +46,14 @@
                 <limit lower="0.0" upper="${0.95*drawer_size_y}" effort="100" velocity="100" />
         </joint>
+        <transmission name="${prefix}_drawer_joint">
+                <type>transmission_interface/SimpleTransmission</type>
+                <joint name="top_drawer_joint">
+                        <hardwareInterface>hardware_interface/EffortJointInterface</hardwareInterface>
+                </joint>
+                <actuator name="${prefix}_drawer_joint_motor">
+                        <mechanicalReduction>1</mechanicalReduction>
+                        <motorTorqueConstant>1</motorTorqueConstant>
+                </actuator>
+        </transmission>
 </xacro:macro>
 </robot>
