Commit message: commenting out cage and drawer for now. Using high quality model and base footprint.

File: src/ros2/robot_description/rb_theron_common/rb_theron_description/robots/rb_theron.urdf.xacro (robot description, xacro)
@@ -33,5 +33,5 @@
 	<xacro:property name="wheel_offset_z" value="0.015" />
 	<!-- Flag to select the high or low quality model -->
-	<xacro:property name="hq" value="false" />
+	<xacro:property name="hq" value="true" />
 	<!-- *************** -->
 	<!-- Robots Elements -->
@@ -41,5 +41,5 @@
 	<!-- this property is for the chassis -->
 	<!-- rbogie base -->
-	<xacro:theron_base prefix="$(arg prefix)" publish_bf="false" hq="${hq}" />
+	<xacro:theron_base prefix="$(arg prefix)" publish_bf="true" hq="${hq}" />
 	<xacro:gazebo_colors prefix="$(arg prefix)"/>
 	<!-- WHEELS -->
@@ -95,13 +95,13 @@
 	<!-- <xacro:depthai_camera camera_name = "$(arg camera_name)" parent = "$(arg prefix)base_link" camera_model = "$(arg camera_model)" base_frame = "$(arg base_frame)" cam_pos_x = "$(arg cam_pos_x)" cam_pos_y = "$(arg cam_pos_y)" cam_pos_z = "$(arg cam_pos_z)" cam_roll = "$(arg cam_roll)" cam_pitch = "$(arg cam_pitch)" cam_yaw = "$(arg cam_yaw)"/> -->
 	<!-- ROBAST Module Cage -->
-	<xacro:include filename="$(find rb_theron_description)/urdf/module_cage/module_cage.urdf.xacro" />
+	<!-- <xacro:include filename="$(find rb_theron_description)/urdf/module_cage/module_cage.urdf.xacro" />
 	<xacro:module_cage prefix="$(arg prefix)module_cage" parent="$(arg prefix)base_link">
 		<origin xyz="0.35 -0.0 -0.075" rpy="0 0 1.570796326794896619"/>
-	</xacro:module_cage>
+	</xacro:module_cage> -->
 	<!-- ROBAST Drawer -->
-	<xacro:include filename="$(find rb_theron_description)/urdf/drawer/drawer.urdf.xacro" />
+	<!-- <xacro:include filename="$(find rb_theron_description)/urdf/drawer/drawer.urdf.xacro" />
 	<xacro:drawer prefix="$(arg prefix)first" parent="$(arg prefix)base_link">
 		<origin xyz="0.105 0.0 0.3" rpy="0 0 0"/>
-	</xacro:drawer>
+	</xacro:drawer> -->
 	<!-- Gazebo ros control pluggins -->
 	<xacro:ros_control prefix="$(arg prefix)"/>

Commit message: Fixing tf for odom -> base_footprint

File: src/ros2/robot_description/rb_theron_common/rb_theron_description/robots/rb_theron.urdf.xacro (robot description, xacro)
@@ -34,4 +34,5 @@
 	<!-- Flag to select the high or low quality model -->
 	<xacro:property name="hq" value="true" />
+	<xacro:property name="publish_bf" value="true"/>
 	<!-- *************** -->
 	<!-- Robots Elements -->
@@ -41,5 +42,5 @@
 	<!-- this property is for the chassis -->
 	<!-- rbogie base -->
-	<xacro:theron_base prefix="$(arg prefix)" publish_bf="true" hq="${hq}" />
+	<xacro:theron_base prefix="$(arg prefix)" publish_bf="${publish_bf}" hq="${hq}" />
 	<xacro:gazebo_colors prefix="$(arg prefix)"/>
 	<!-- WHEELS -->
@@ -105,4 +106,4 @@
 	</xacro:drawer> -->
 	<!-- Gazebo ros control pluggins -->
-	<xacro:ros_control prefix="$(arg prefix)"/>
+	<xacro:ros_control prefix="$(arg prefix)" publish_bf="${publish_bf}"/>
 </robot>

File: src/ros2/robot_description/rb_theron_common/rb_theron_description/urdf/common.gazebo.xacro (robot description, xacro)
@@ -2,5 +2,5 @@
 <robot xmlns:xacro="http://www.ros.org/wiki/xacro">
 	<!-- ROS CONTROL GAZEBO PLUGIN -->
-	<xacro:macro name="ros_control" params="prefix">
+	<xacro:macro name="ros_control" params="prefix publish_bf">
 		<gazebo>
 			<!-- <plugin filename="libgazebo_ros2_control.so" name="gazebo_ros2_control">
@@ -20,4 +20,11 @@
 				<odom_publish_frequency>30</odom_publish_frequency>
 				<topic>cmd_vel</topic>
+				<frame_id>$(arg prefix)odom</frame_id>
+				<xacro:if value="${publish_bf}">
+					<child_frame_id>$(arg prefix)base_footprint</child_frame_id>
+				</xacro:if>
+				<xacro:unless value="${publish_bf}">
+					<child_frame_id>$(arg prefix)base_link</child_frame_id>
+				</xacro:unless>
 			</plugin>
 		</gazebo>

Commit message: Laser scan messages and joint states are now published by gazebo ign

File: src/ros2/robot_description/rb_theron_common/rb_theron_description/robots/rb_theron.urdf.xacro (robot description, xacro)
@@ -73,5 +73,5 @@
 		<origin xyz="-0.1975 0.0 0.1598" rpy="0 0 0"/>
 	</xacro:sensor_imu_hector>
-	<xacro:sensor_sick_nanoscan3 prefix="$(arg prefix)front_laser" parent="$(arg prefix)base_link" prefix_topic="front_laser" hq="${hq}" min_angle="-1.9507619" max_angle="1.9507619">
+	<xacro:sensor_sick_nanoscan3 prefix="$(arg prefix)front_laser" parent="$(arg prefix)base_link" prefix_topic="front_laser" hq="${hq}" min_angle="-1.9507619" max_angle="1.9507619" gpu="true">
 		<origin xyz="0.250 0.0 0.1643" rpy="0 3.1416 3.1416"/>
 	</xacro:sensor_sick_nanoscan3>

File: src/ros2/robot_description/robotnik_sensors/urdf/sick_nanoscan3.urdf.xacro (robot description, xacro)
@@ -49,9 +49,9 @@
 			<xacro:if value="${gpu}">
 				<xacro:property name="ray_type" value="gpu_ray" />
-				<xacro:property name="plugin_lib" value="libgz-sim-sensors-system.so" />
+				<xacro:property name="plugin_lib" value="gz-sim-sensors-system" />
 			</xacro:if>
 			<xacro:unless value="${gpu}">
 				<xacro:property name="ray_type" value="ray" />
-				<xacro:property name="plugin_lib" value="libgz-sim-sensors-system.so" />
+				<xacro:property name="plugin_lib" value="gz-sim-sensors-system" />
 			</xacro:unless>
 			<sensor type="${ray_type}" name="${prefix}_sensor">
@@ -59,5 +59,5 @@
 				<topic>${prefix_topic}/scan</topic>
 				<always_on>1</always_on>
-    				<visualize>true</visualize>
+    				<visualize>false</visualize>
 				<update_rate>12.5</update_rate>
 				<ray>

Commit message: rb_theron lidar plugin is now working

File: src/ros2/robot_description/rb_theron_common/rb_theron_description/robots/rb_theron.urdf.xacro (robot description, xacro)
@@ -34,5 +34,8 @@
 	<!-- Flag to select the high or low quality model -->
 	<xacro:property name="hq" value="true" />
-	<xacro:property name="publish_bf" value="true"/>
+	<!-- Flag to determine if the base_footprint should be published or not -->
+	<xacro:property name="publish_bf" value="false"/>
+	<!-- This name should match the "-name" argument we need to declare when spawing the robot into ign gazebo -->
+	<xacro:property name="robot_name" value="rb_theron"/>
 	<!-- *************** -->
 	<!-- Robots Elements -->
@@ -73,5 +76,5 @@
 		<origin xyz="-0.1975 0.0 0.1598" rpy="0 0 0"/>
 	</xacro:sensor_imu_hector>
-	<xacro:sensor_sick_nanoscan3 prefix="$(arg prefix)front_laser" parent="$(arg prefix)base_link" prefix_topic="front_laser" hq="${hq}" min_angle="-1.9507619" max_angle="1.9507619" gpu="true">
+	<xacro:sensor_sick_nanoscan3 prefix="$(arg prefix)front_laser" parent="$(arg prefix)base_link" publish_bf="${publish_bf}" robot_name="${robot_name}" prefix_topic="front_laser" hq="${hq}" min_angle="-1.9507619" max_angle="1.9507619" gpu="true">
 		<origin xyz="0.250 0.0 0.1643" rpy="0 3.1416 3.1416"/>
 	</xacro:sensor_sick_nanoscan3>

File: src/ros2/robot_description/robotnik_sensors/urdf/sick_nanoscan3.urdf.xacro (robot description, xacro)
@@ -2,5 +2,11 @@
 <robot name="sensor_sick_nanoscan3"
 	xmlns:xacro="http://wiki.ros.org/xacro">
-	<xacro:macro name="sensor_sick_nanoscan3" params="prefix parent prefix_topic:='front_laser' hq *origin max_angle:=2.3998 min_angle:=-2.3998 gpu:=^|false">
+	<xacro:macro name="sensor_sick_nanoscan3" params="prefix parent publish_bf robot_name prefix_topic:='front_laser' hq *origin max_angle:=2.3998 min_angle:=-2.3998 gpu:=^|false">
+		<xacro:if value="${publish_bf}">
+			<xacro:property name="sensor_link_name" value="${robot_name}/base_footprint/${prefix}_link" />
+		</xacro:if>
+		<xacro:unless value="${publish_bf}">
+			<xacro:property name="sensor_link_name" value="${robot_name}/base_link/${prefix}_link" />
+		</xacro:unless>
 		<joint name="${prefix}_base_joint" type="fixed">
 			<xacro:insert_block name="origin" />
@@ -38,13 +44,13 @@
 		<joint name="${prefix}_joint" type="fixed">
 			<parent link="${prefix}_base_link"/>
-			<child link="${prefix}_link"/>
+			<child link="${sensor_link_name}"/>
 			<origin xyz="0.0 0 0.0505" rpy="0 0 0"/>
 		</joint>
-		<link name="${prefix}_link" />
+		<link name="${sensor_link_name}" />
 		<!-- Sick sensor sensor for simulation -->
 		<xacro:sensor_sick_nanoscan3_gazebo />
 	</xacro:macro>
 	<xacro:macro name="sensor_sick_nanoscan3_gazebo">
-		<gazebo reference="${prefix}_link">
+		<gazebo reference="${sensor_link_name}">
 			<xacro:if value="${gpu}">
 				<xacro:property name="ray_type" value="gpu_ray" />
@@ -55,6 +61,6 @@
 				<xacro:property name="plugin_lib" value="gz-sim-sensors-system" />
 			</xacro:unless>
-			<sensor type="${ray_type}" name="${prefix}_sensor">
-				<pose relative_to='${prefix}_link'>0 0 0 0 0 0</pose>
+			<sensor type="${ray_type}" name="${prefix}_link">
+				<pose relative_to='${sensor_link_name}'>0 0 0 0 0 0</pose>
 				<topic>${prefix_topic}/scan</topic>
 				<always_on>1</always_on>

Commit message: rb_theron can now be navigated through ros / rviz

File: src/ros2/robot_description/rb_theron_common/rb_theron_description/robots/rb_theron.urdf.xacro (robot description, xacro)
@@ -35,5 +35,5 @@
 	<xacro:property name="hq" value="true" />
 	<!-- Flag to determine if the base_footprint should be published or not -->
-	<xacro:property name="publish_bf" value="false"/>
+	<xacro:property name="publish_bf" value="true"/>
 	<!-- This name should match the "-name" argument we need to declare when spawing the robot into ign gazebo -->
 	<xacro:property name="robot_name" value="rb_theron"/>

Commit message: including module cage and drawer to rb_theron.urdf and disabling hq model

File: src/ros2/robot_description/rb_theron_common/rb_theron_description/robots/rb_theron.urdf.xacro (robot description, xacro)
@@ -33,5 +33,5 @@
 	<xacro:property name="wheel_offset_z" value="0.015" />
 	<!-- Flag to select the high or low quality model -->
-	<xacro:property name="hq" value="true" />
+	<xacro:property name="hq" value="false" />
 	<!-- Flag to determine if the base_footprint should be published or not -->
 	<xacro:property name="publish_bf" value="true"/>
@@ -99,13 +99,13 @@
 	<!-- <xacro:depthai_camera camera_name = "$(arg camera_name)" parent = "$(arg prefix)base_link" camera_model = "$(arg camera_model)" base_frame = "$(arg base_frame)" cam_pos_x = "$(arg cam_pos_x)" cam_pos_y = "$(arg cam_pos_y)" cam_pos_z = "$(arg cam_pos_z)" cam_roll = "$(arg cam_roll)" cam_pitch = "$(arg cam_pitch)" cam_yaw = "$(arg cam_yaw)"/> -->
 	<!-- ROBAST Module Cage -->
-	<!-- <xacro:include filename="$(find rb_theron_description)/urdf/module_cage/module_cage.urdf.xacro" />
+	<xacro:include filename="$(find rb_theron_description)/urdf/module_cage/module_cage.urdf.xacro" />
 	<xacro:module_cage prefix="$(arg prefix)module_cage" parent="$(arg prefix)base_link">
 		<origin xyz="0.35 -0.0 -0.075" rpy="0 0 1.570796326794896619"/>
-	</xacro:module_cage> -->
+	</xacro:module_cage>
 	<!-- ROBAST Drawer -->
-	<!-- <xacro:include filename="$(find rb_theron_description)/urdf/drawer/drawer.urdf.xacro" />
+	<xacro:include filename="$(find rb_theron_description)/urdf/drawer/drawer.urdf.xacro" />
 	<xacro:drawer prefix="$(arg prefix)first" parent="$(arg prefix)base_link">
 		<origin xyz="0.105 0.0 0.3" rpy="0 0 0"/>
-	</xacro:drawer> -->
+	</xacro:drawer>
 	<!-- Gazebo ros control pluggins -->
 	<xacro:ros_control prefix="$(arg prefix)" publish_bf="${publish_bf}"/>

Commit message: Realsense r430 in ignition

File: src/ros2/robot_description/rb_theron_common/rb_theron_description/robots/rb_theron.urdf.xacro (robot description, xacro)
@@ -88,4 +88,9 @@
 		<origin xyz="-0.250 0.0 0.1643" rpy="0 3.1416 0"/>
 	</xacro:sensor_sick_nanoscan3> -->
+	<gazebo>
+		<plugin name="gz::sim::systems::Sensors" filename="gz-sim-sensors-system">
+			<render_engine>ogre2</render_engine>
+		</plugin>
+	</gazebo>
 	<xacro:arg name="camera_name"   default="oak" />
 	<xacro:arg name="camera_model"  default="OAK-D-LITE" />

File: src/ros2/robot_description/robotnik_sensors/urdf/intel_r430.urdf.xacro (robot description, xacro)
@@ -4,6 +4,6 @@
   <!-- The following values are approximate, and the camera node
    publishing TF values with actual calibrated camera extrinsic values -->
-  <xacro:property name="r430_cam_depth_to_left_ir_offset" value="-0.021"/>
-  <xacro:property name="r430_cam_depth_to_right_ir_offset" value="0.029"/>
+    <xacro:property name="r430_cam_depth_to_left_ir_offset" value="-0.021"/>
+    <xacro:property name="r430_cam_depth_to_right_ir_offset" value="0.029"/>
   <xacro:property name="r430_cam_depth_to_fisheye_offset" value="0.044"/>
   <!-- The following values model the aluminum peripherial case for the
@@ -107,86 +107,131 @@
     <link name="${prefix}_camera_fisheye_optical_frame"/>
     <!-- RGBD sensor for simulation, same as Kinect -->
-    <sensor_r430_gazebo/>
+    <xacro:sensor_r430_gazebo/>
   </xacro:macro>
   <xacro:macro name="sensor_r430_gazebo">
     <!-- gazebo reference="${prefix}_rgb_base_link" -->
     <gazebo reference="${prefix}_camera_link">
-      <!-- <sensor type="depth" name="${prefix}_depth_sensor">
-        <always_on>true</always_on>
-        <update_rate>15.0</update_rate>
-        <camera>
-          <horizontal_fov>${91.2*M_PI/180.0}</horizontal_fov>
-          <image>
-            <format>R8G8B8</format>
-            <width>640</width>
-            <height>480</height>
-          </image>
-          <clip>
-            <near>0.3</near>
-            <far>10.0</far>
-          </clip>
-        </camera>
-        <plugin name="${prefix}_controller" filename="libgazebo_ros_openni_kinect.so">
-          <cameraName>${prefix_topic}</cameraName>
-          <alwaysOn>true</alwaysOn>
-          <updateRate>10</updateRate>
-          <imageTopicName>rgb/image_raw</imageTopicName>
-          <depthImageTopicName>depth/image_raw</depthImageTopicName>
-          <pointCloudTopicName>depth/points</pointCloudTopicName>
-          <cameraInfoTopicName>rgb/camera_info</cameraInfoTopicName>
-          <depthImageCameraInfoTopicName>depth/camera_info</depthImageCameraInfoTopicName>
-          <frame_name>/${prefix}_camera_depth_optical_frame</frame_name>
-          <baseline>0.1</baseline>
-          <distortion_k1>0.0</distortion_k1>
-          <distortion_k2>0.0</distortion_k2>
-          <distortion_k3>0.0</distortion_k3>
-          <distortion_t1>0.0</distortion_t1>
-          <distortion_t2>0.0</distortion_t2>
-          <pointCloudCutoff>0.4</pointCloudCutoff>
-        </plugin>
-      </sensor> -->
-      <sensor type="depth" name="${prefix}_depth_sensor">
-          <!-- Set always_on only sensor, not on plugin -->
-          <always_on>true</always_on>
-          <!-- Set update_rate only sensor, not on plugin -->
-          <update_rate>15.0</update_rate>
-          <camera>
-            <horizontal_fov>${91.2*M_PI/180.0}</horizontal_fov>
-            <image>
-              <format>R8G8B8</format>
-              <width>640</width>
-              <height>480</height>
-            </image>
-            <clip>
-              <near>0.3</near>
-              <far>10.0</far>
-            </clip>
-          </camera>
-          <plugin name="${prefix}_controller" filename="libgazebo_ros_camera.so">
-            <!-- Change namespace, camera name and topics so:
-                 * Raw images are published to: /custom_ns/custom_camera/custom_image
-                 * Depth images are published to: /custom_ns/custom_camera/custom_image_depth
-                 * Raw image camera info is published to: /custom_ns/custom_camera/custom_info_raw
-                 * Depth image camera info is published to: /custom_ns/custom_camera/custom_info_depth
-                 * Point cloud is published to: /custom_ns/custom_camera/custom_points
-            -->
-            <ros>
-              <argument>image_raw:=custom_image</argument>
-              <argument>image_depth:=custom_image_depth</argument>
-              <argument>camera_info:=custom_info_raw</argument>
-              <argument>camera_info_depth:=custom_info_depth</argument>
-              <argument>points:=custom_points</argument>
-            </ros>
-            <!-- Set camera name. If empty, defaults to sensor name (i.e. "sensor_name") -->
-            <!-- <camera_name>${prefix}_camera</camera_name> -->
-            <!-- Set TF frame name. If empty, defaults to link name (i.e. "link_name") -->
-            <frame_name>${prefix}_camera_depth_optical_frame</frame_name>
-            <hack_baseline>0.1</hack_baseline>
-            <!-- No need to repeat distortion parameters or to set autoDistortion -->
-             <min_depth>0.4</min_depth>
-             <max_depth>10.0</max_depth>
-          </plugin>
-        </sensor>
+      <sensor name="${prefix}_color" type="camera">
+				<pose relative_to='${prefix}_camera_depth_frame'>-0.1 0 0 0 0 0</pose>
+				<topic>${prefix_topic}/color</topic>
+        			<camera name="r430">
+          				<horizontal_fov>1.2112585008840648</horizontal_fov>
+          				<image>
+            					<width>640</width>
+            					<height>480</height>
+            					<format>RGB_INT8</format>
+          				</image>
+          				<clip>
+            					<near>0.1</near>
+            					<far>100</far>
+          				</clip>
+    		      			<noise>
+            					<type>gaussian</type>
+            					<mean>0.0</mean>
+            					<stddev>0.007</stddev>
+          				</noise>
+        			</camera>
+        			<always_on>1</always_on>
+        			<update_rate>30</update_rate>
+        			<visualize>1</visualize>
+      			</sensor>
+            <sensor name="${prefix}_ired1" type="camera">
+            <pose relative_to='${prefix}_camera_depth_frame'>-0.2 0 0 0 0 0</pose>
+				    <topic>${prefix_topic}/${prefix}/ired1</topic>
+              <camera name="r430">
+                <horizontal_fov>${91.2*M_PI/180.0}</horizontal_fov>
+                <image>
+                  <width>640</width>
+                  <height>480</height>
+                  <format>L_INT8</format>
+                </image>
+                <clip>
+                  <near>0.3</near>
+                  <far>10.0</far>
+                </clip>
+                <noise>
+                  <type>gaussian</type>
+                  <mean>0.0</mean>
+                  <stddev>0.05</stddev>
+                </noise>
+              </camera>
+              <always_on>1</always_on>
+              <update_rate>90</update_rate>
+              <visualize>0</visualize>
+            </sensor>
+            <sensor name="${prefix}_ired2" type="camera">
+               <pose relative_to='${prefix}_camera_depth_frame'>0.2 0 0 0 0 0</pose>
+            		<topic>${prefix_topic}/${prefix}/ired2</topic>
+                <camera name="r430">
+                  <horizontal_fov>1.4870205226991688</horizontal_fov>
+                  <image>
+                    <width>640</width>
+                    <height>480</height>
+                    <format>L_INT8</format>
+                  </image>
+                  <clip>
+                    <near>0.3</near>
+                    <far>10.0</far>
+                  </clip>
+                  <noise>
+                    <type>gaussian</type>
+                    <mean>0.0</mean>
+                    <stddev>0.05</stddev>
+                  </noise>
+                </camera>
+                <always_on>1</always_on>
+                <update_rate>90</update_rate>
+                <visualize>0</visualize>
+              </sensor>
+              <sensor name="${prefix}_depth" type="depth">
+                <pose relative_to='${prefix}_camera_depth_frame'>0.1 0 0 0 0 0</pose>
+            		<topic>${prefix_topic}/${prefix}/depth</topic>
+                <camera name="r430">
+                 <horizontal_fov>${91.2*M_PI/180.0}</horizontal_fov>
+                 <image>
+                   <width>640</width>
+                   <height>480</height>
+                 </image>
+                 <clip>
+                   <near>0.3</near>
+                   <far>10.0</far>
+                 </clip>
+                 <noise>
+                   <type>gaussian</type>
+                   <mean>0.0</mean>
+                   <stddev>0.100</stddev>
+                 </noise>
+                </camera>
+                <always_on>1</always_on>
+                <update_rate>15</update_rate>
+                <visualize>0</visualize>
+              </sensor>
     </gazebo>
+    <!-- <gazebo>
+      <plugin filename="librealsense_gazebo_plugin.so" name="r430">
+        <prefix>r430_</prefix>
+        <depthUpdateRate>10</depthUpdateRate>
+        <colorUpdateRate>10</colorUpdateRate>
+        <infraredUpdateRate>10</infraredUpdateRate>
+        <depthTopicName>depth/image_raw</depthTopicName>
+        <depthCameraInfoTopicName>depth/camera_info</depthCameraInfoTopicName>
+        <colorTopicName>color/image_raw</colorTopicName>
+        <colorCameraInfoTopicName>color/camera_info</colorCameraInfoTopicName>
+        <infrared1TopicName>infra1/image_raw</infrared1TopicName>
+        <infrared1CameraInfoTopicName>infra1/camera_info</infrared1CameraInfoTopicName>
+        <infrared2TopicName>infra2/image_raw</infrared2TopicName>
+        <infrared2CameraInfoTopicName>infra2/camera_info</infrared2CameraInfoTopicName>
+        <colorOpticalframeName>r430_color_optical_frame</colorOpticalframeName>
+        <depthOpticalframeName>r430_depth_optical_frame</depthOpticalframeName>
+        <infrared1OpticalframeName>r430_infrared1_optical_frame</infrared1OpticalframeName>
+        <infrared2OpticalframeName>r430_infrared2_optical_frame</infrared2OpticalframeName>
+        <rangeMinDepth>0.2</rangeMinDepth>
+        <rangeMaxDepth>10.0</rangeMaxDepth>
+        <pointCloud>false</pointCloud>
+        <pointCloudTopicName>depth/color/points</pointCloudTopicName>
+        <pointCloudCutoff>0.25</pointCloudCutoff>
+        <pointCloudCutoffMax>9.0</pointCloudCutoffMax>
+      </plugin>
+    </gazebo> -->
   </xacro:macro>
 </robot>

File: src/ros2/robot_description/robotnik_sensors/urdf/sick_nanoscan3.urdf.xacro (robot description, xacro)
@@ -61,5 +61,5 @@
 				<xacro:property name="plugin_lib" value="gz-sim-sensors-system" />
 			</xacro:unless>
-			<sensor type="${ray_type}" name="${prefix}_link">
+			<sensor type="${ray_type}" name="${prefix}_Ray">
 				<pose relative_to='${sensor_link_name}'>0 0 0 0 0 0</pose>
 				<topic>${prefix_topic}/scan</topic>
@@ -93,7 +93,4 @@
 					</noise>
 				</ray>
-				<plugin name="gz::sim::systems::Sensors" filename="${plugin_lib}">
-					<render_engine>ogre2</render_engine>
-				</plugin>
 			</sensor>
 		</gazebo>
