Commit message: RSBPerl in Ignition

File: src/ros2/robot_description/rb_theron_common/rb_theron_description/robots/rb_theron.urdf.xacro (robot description, xacro)
@@ -82,7 +82,7 @@
 		<origin xyz="0.214 0.0 0.275" rpy="-1.57079632679 0 -0.23"/>
 	</xacro:sensor_rs_lidar_16>-->
-	<!-- <xacro:sensor_rs_bpearl prefix="$(arg prefix)top_laser"  parent="$(arg prefix)base_link" prefix_topic="top_laser" hq="${hq}" range_min="0.1" range_max="90" hfov="360" samples="1200" vfov="90.0" lasers="32" fps="15" gpu="false">
+	<xacro:sensor_rs_bpearl prefix="$(arg prefix)top_laser"  parent="$(arg prefix)base_link" prefix_topic="top_laser" hq="${hq}" range_min="0.1" range_max="90" hfov="360" samples="1200" vfov="90.0" lasers="32" fps="15" gpu="false">
             <origin xyz="0.28 -0.159 1.22" rpy="-1.570796326795 0 -1.570796326795"/>
-        </xacro:sensor_rs_bpearl> -->
+        </xacro:sensor_rs_bpearl>
 	<!-- <xacro:sensor_sick_nanoscan3 prefix="$(arg prefix)back_laser" parent="$(arg prefix)base_link" prefix_topic="back_laser" min_angle="-1.8107619" max_angle="1.8107619">
 		<origin xyz="-0.250 0.0 0.1643" rpy="0 3.1416 0"/>

File: src/ros2/robot_description/robotnik_sensors/urdf/rs_bpearl.urdf.xacro (robot description, xacro)
@@ -66,46 +66,34 @@
         </material>
       </visual>
-      <xacro:if value="${gpu}">
-        <!-- Using GPU needs: https://github.com/RobotnikAutomation/velodyne_simulator -->
-        <xacro:property name="ray_type" value="gpu_ray" />
-        <xacro:property name="plugin_lib" value="libGazeboRosVelodyneLaser.so" />
-      </xacro:if>
-      <xacro:unless value="${gpu}">
-        <xacro:property name="ray_type" value="ray" />
-        <xacro:property name="plugin_lib" value="libGazeboRosVelodyneLaser.so" />
-      </xacro:unless>
-        <sensor type="${ray_type}" name="${prefix}_sensor">
-          <pose>0 0 0 0 0 0.0</pose>
-          <visualize>false</visualize>
-          <update_rate>${fps}</update_rate>
-          <ray>
-            <scan>
-              <horizontal>
-				<!-- for a high quality simulation -->
-                <samples>${samples}</samples>
-                <min_angle>-${hfov/2*M_PI/180.0}</min_angle>
-                <max_angle>${hfov/2*M_PI/180.0}</max_angle>
-              </horizontal>
-              <vertical>
-                <samples>${lasers}</samples>
-                <min_angle>-${5*M_PI/180.0}</min_angle>  <!-- bpearl has 90 degrees of vertical field of view-->
-                <max_angle> ${(vfov-5)*M_PI/180.0}</max_angle>
-              </vertical>
-            </scan>
-            <range>
-              <min>${range_min}</min>
-              <max>${range_max}</max>
-              <resolution>0.01</resolution>
-            </range>
-            <noise>
-              <type>none</type>
-            </noise>
-          </ray>
-          <plugin name="${prefix}_controller" filename="${plugin_lib}">
-            <topicName>${prefix_topic}/points</topicName>
-            <frame_name>${prefix}_link</frame_name>
-            <gaussianNoise>0.008</gaussianNoise>
-          </plugin>
-        </sensor>
+                        <sensor name='gpu_lidar' type='gpu_lidar'>
+                                <visualize>true</visualize>
+                                <update_rate>10</update_rate>
+                                <ray>
+                                        <scan>
+                                                <horizontal>
+                                                        <samples>440</samples>
+                                                        <resolution>1</resolution>
+                                                        <min_angle>0</min_angle>
+							                                          <max_angle>1.570796326795</max_angle>
+                                                </horizontal>
+                                                <vertical>
+                                                        <samples>32</samples>
+                                                        <resolution>1</resolution>
+                                                        <min_angle>-3.14159265359</min_angle> <!-- -180° -->
+                                                        <max_angle>3.14159265359</max_angle> <!-- +180° -->
+                                                </vertical>
+                                        </scan>
+                                        <range>
+                                                <min>0.3</min>
+                                                <max>131</max>
+                                                <resolution>0.001</resolution>
+                                        </range>
+                                        <noise>
+                                                <type>gaussian</type>
+                                                <mean>0</mean>
+                                                <stddev>0</stddev>
+                                        </noise>
+                                </ray>
+                        </sensor>
     </gazebo>
   </xacro:macro>

Commit message: Rbpearl lidar data is now visible in ros2

File: src/ros2/robot_description/rb_theron_common/rb_theron_description/robots/rb_theron.urdf.xacro (robot description, xacro)
@@ -82,5 +82,5 @@
 		<origin xyz="0.214 0.0 0.275" rpy="-1.57079632679 0 -0.23"/>
 	</xacro:sensor_rs_lidar_16>-->
-	<xacro:sensor_rs_bpearl prefix="$(arg prefix)top_laser"  parent="$(arg prefix)base_link" prefix_topic="top_laser" hq="${hq}" range_min="0.1" range_max="90" hfov="360" samples="1200" vfov="90.0" lasers="32" fps="15" gpu="false">
+	<xacro:sensor_rs_bpearl prefix="$(arg prefix)top_laser"  parent="$(arg prefix)base_link" publish_bf="${publish_bf}" robot_name="${robot_name}" prefix_topic="top_laser" hq="${hq}" range_min="0.1" range_max="90" hfov="360" samples="1200" vfov="90.0" lasers="32" fps="15" gpu="false">
             <origin xyz="0.28 -0.159 1.22" rpy="-1.570796326795 0 -1.570796326795"/>
         </xacro:sensor_rs_bpearl>

File: src/ros2/robot_description/robotnik_sensors/urdf/rs_bpearl.urdf.xacro (robot description, xacro)
@@ -2,5 +2,11 @@
 <robot name="sensor_rs_bpearl" xmlns:xacro="http://wiki.ros.org/xacro">
   <xacro:property name="M_PI" value="3.1415926535897931" />
-  <xacro:macro name="sensor_rs_bpearl" params="prefix parent prefix_topic hq *origin range_min range_max hfov samples vfov lasers fps gpu:=true">
+  <xacro:macro name="sensor_rs_bpearl" params="prefix parent publish_bf robot_name prefix_topic hq *origin range_min range_max hfov samples vfov lasers fps gpu:=true">
+    <xacro:if value="${publish_bf}">
+			<xacro:property name="sensor_link_name" value="${robot_name}/base_footprint/${prefix}_link" />
+		</xacro:if>
+		<xacro:unless value="${publish_bf}">
+			<xacro:property name="sensor_link_name" value="${robot_name}/base_link/${prefix}_link" />
+		</xacro:unless>
     <joint name="${prefix}_base_joint" type="fixed">
       <xacro:insert_block name="origin" />
@@ -40,12 +46,12 @@
     <joint name="${prefix}_joint" type="fixed">
       <parent link="${prefix}_base_link"/>
-      <child link="${prefix}_link" />
+      <child link="${sensor_link_name}"/>
       <origin xyz="0 0 0.09427" rpy="0 0 0"/>
     </joint>
-    <link name="${prefix}_link"/>
-  <xacro:sensor_rs_bpearl_gazebo range_min="${range_min}" range_max="${range_max}" hfov="${hfov}" samples="${samples}" vfov="${vfov}" lasers="${lasers}" fps="${fps}" gpu="${gpu}"/>
+    <link name="${sensor_link_name}" />
+    <xacro:sensor_rs_bpearl_gazebo range_min="${range_min}" range_max="${range_max}" hfov="${hfov}" samples="${samples}" vfov="${vfov}" lasers="${lasers}" fps="${fps}" gpu="${gpu}"/>
   </xacro:macro>
   <xacro:macro name="sensor_rs_bpearl_gazebo" params="range_min range_max hfov samples vfov lasers fps gpu">
-    <gazebo reference="${prefix}_base_link">
+    <gazebo reference="${sensor_link_name}">
       <visual>
         <material>
@@ -57,5 +63,5 @@
       </visual>
     </gazebo>
-    <gazebo reference="${prefix}_link">
+    <gazebo reference="${sensor_link_name}">
       <visual>
         <material>
@@ -66,5 +72,6 @@
         </material>
       </visual>
-      <sensor name='gpu_lidar' type='gpu_lidar'>
+      <sensor name='${prefix}_link' type='gpu_lidar'>
+        <pose relative_to='${sensor_link_name}'>0 0 0 0 0 0</pose>
         <visualize>true</visualize>
         <topic>bpearl_laser/scan</topic>

Commit message: Further modifying intel_r430 to make sensor data being attached to the correct frame

File: src/ros2/robot_description/rb_theron_common/rb_theron_description/robots/rb_theron.urdf.xacro (robot description, xacro)
@@ -63,8 +63,8 @@
 	<!-- TODO: Should be sensor_intel_d435, but this one isn't migrated to ros2 yet -->
 	<!-- TODO: Moved 0.01 in x, otherwise the camera is still inside the robot -->
-	<xacro:sensor_r430 prefix="$(arg prefix)front_realsense_camera" parent="$(arg prefix)base_link" prefix_topic="front_realsense_camera" hq="${hq}">
+	<xacro:sensor_r430 prefix="$(arg prefix)front_realsense_camera" parent="$(arg prefix)base_link" publish_bf="${publish_bf}" robot_name="${robot_name}" prefix_topic="front_realsense_camera" hq="${hq}">
 		<origin xyz="0.3305 0.0 0.1468" rpy="0 0 0"/>
 	</xacro:sensor_r430>
-	<xacro:sensor_r430 prefix="$(arg prefix)back_realsense_camera" parent="$(arg prefix)base_link" prefix_topic="back_realsense_camera" hq="${hq}">
+	<xacro:sensor_r430 prefix="$(arg prefix)back_realsense_camera" parent="$(arg prefix)base_link" publish_bf="${publish_bf}" robot_name="${robot_name}" prefix_topic="back_realsense_camera" hq="${hq}">
 		<origin xyz="-0.3305 0.0 0.1468" rpy="0 0 3.1416"/>
 	</xacro:sensor_r430>

File: src/ros2/robot_description/robotnik_sensors/urdf/intel_r430.urdf.xacro (robot description, xacro)
@@ -19,5 +19,11 @@
   <xacro:property name="r430_cam_depth_py" value="-0.0115"/>
   <xacro:property name="r430_cam_depth_pz" value="0.0"/>
-  <xacro:macro name="sensor_r430" params="prefix parent prefix_topic:='front_rgbd_camera' hq *origin">
+  <xacro:macro name="sensor_r430" params="prefix parent publish_bf robot_name prefix_topic:='front_rgbd_camera' hq *origin">
+    <xacro:if value="${publish_bf}">
+			<xacro:property name="sensor_link_name" value="${robot_name}/base_footprint/${prefix}" />
+		</xacro:if>
+		<xacro:unless value="${publish_bf}">
+			<xacro:property name="sensor_link_name" value="${robot_name}/base_link/${prefix}" />
+		</xacro:unless>
     <!-- camera body, with origin at bottom screw mount -->
     <joint name="${prefix}_camera_joint" type="fixed">
@@ -64,7 +70,13 @@
       <origin xyz="0 0 0" rpy="${-M_PI/2} 0 ${-M_PI/2}" />
       <parent link="${prefix}_camera_depth_frame" />
-      <child link="${prefix}_camera_depth_optical_frame" />
-    </joint>
-    <link name="${prefix}_camera_depth_optical_frame"/>
+      <child link="${sensor_link_name}_depth_link" />
+    </joint>
+    <link name="${sensor_link_name}_depth_link"/>
+    <joint name="${prefix}_camera_color_joint" type="fixed">
+      <origin xyz="0 0 0" rpy="${-M_PI/2} 0 ${-M_PI/2}" />
+      <parent link="${prefix}_camera_depth_frame" />
+      <child link="${sensor_link_name}_color_link" />
+    </joint>
+    <link name="${sensor_link_name}_color_link"/>
     <!-- camera left IR joints and links -->
     <joint name="${prefix}_camera_left_ir_joint" type="fixed">
@@ -111,100 +123,104 @@
   <xacro:macro name="sensor_r430_gazebo">
     <!-- gazebo reference="${prefix}_rgb_base_link" -->
+    <gazebo reference="${sensor_link_name}_color_link">
+      <sensor name="${prefix}_color_link" type="camera">
+				<pose relative_to='${sensor_link_name}_color_link'>-0.1 0 0 0 0 0</pose>
+				<topic>${prefix_topic}/color</topic>
+        <camera name="r430">
+            <horizontal_fov>1.2112585008840648</horizontal_fov>
+            <image>
+                <width>640</width>
+                <height>480</height>
+                <format>RGB_INT8</format>
+            </image>
+            <clip>
+                <near>0.1</near>
+                <far>100</far>
+            </clip>
+              <noise>
+                <type>gaussian</type>
+                <mean>0.0</mean>
+                <stddev>0.007</stddev>
+            </noise>
+        </camera>
+        <always_on>1</always_on>
+        <update_rate>30</update_rate>
+        <visualize>1</visualize>
+      </sensor>
+    </gazebo>
     <gazebo reference="${prefix}_camera_link">
-      <sensor name="${prefix}_color" type="camera">
-				<pose relative_to='${prefix}_camera_depth_frame'>-0.1 0 0 0 0 0</pose>
-				<topic>${prefix_topic}/color</topic>
-        			<camera name="r430">
-          				<horizontal_fov>1.2112585008840648</horizontal_fov>
-          				<image>
-            					<width>640</width>
-            					<height>480</height>
-            					<format>RGB_INT8</format>
-          				</image>
-          				<clip>
-            					<near>0.1</near>
-            					<far>100</far>
-          				</clip>
-    		      			<noise>
-            					<type>gaussian</type>
-            					<mean>0.0</mean>
-            					<stddev>0.007</stddev>
-          				</noise>
-        			</camera>
-        			<always_on>1</always_on>
-        			<update_rate>30</update_rate>
-        			<visualize>1</visualize>
-      			</sensor>
-            <sensor name="${prefix}_ired1" type="camera">
-            <pose relative_to='${prefix}_camera_depth_frame'>-0.2 0 0 0 0 0</pose>
-				    <topic>${prefix_topic}/${prefix}/ired1</topic>
-              <camera name="r430">
-                <horizontal_fov>${91.2*M_PI/180.0}</horizontal_fov>
-                <image>
-                  <width>640</width>
-                  <height>480</height>
-                  <format>L_INT8</format>
-                </image>
-                <clip>
-                  <near>0.3</near>
-                  <far>10.0</far>
-                </clip>
-                <noise>
-                  <type>gaussian</type>
-                  <mean>0.0</mean>
-                  <stddev>0.05</stddev>
-                </noise>
-              </camera>
-              <always_on>1</always_on>
-              <update_rate>90</update_rate>
-              <visualize>0</visualize>
-            </sensor>
-            <sensor name="${prefix}_ired2" type="camera">
-               <pose relative_to='${prefix}_camera_depth_frame'>0.2 0 0 0 0 0</pose>
-            		<topic>${prefix_topic}/${prefix}/ired2</topic>
-                <camera name="r430">
-                  <horizontal_fov>1.4870205226991688</horizontal_fov>
-                  <image>
-                    <width>640</width>
-                    <height>480</height>
-                    <format>L_INT8</format>
-                  </image>
-                  <clip>
-                    <near>0.3</near>
-                    <far>10.0</far>
-                  </clip>
-                  <noise>
-                    <type>gaussian</type>
-                    <mean>0.0</mean>
-                    <stddev>0.05</stddev>
-                  </noise>
-                </camera>
-                <always_on>1</always_on>
-                <update_rate>90</update_rate>
-                <visualize>0</visualize>
-              </sensor>
-              <sensor name="${prefix}_depth" type="depth">
-                <pose relative_to='${prefix}_camera_depth_frame'>0.1 0 0 0 0 0</pose>
-            		<topic>${prefix_topic}/${prefix}/depth</topic>
-                <camera name="r430">
-                 <horizontal_fov>${91.2*M_PI/180.0}</horizontal_fov>
-                 <image>
-                   <width>640</width>
-                   <height>480</height>
-                 </image>
-                 <clip>
-                   <near>0.3</near>
-                   <far>10.0</far>
-                 </clip>
-                 <noise>
-                   <type>gaussian</type>
-                   <mean>0.0</mean>
-                   <stddev>0.100</stddev>
-                 </noise>
-                </camera>
-                <always_on>1</always_on>
-                <update_rate>15</update_rate>
-                <visualize>0</visualize>
-              </sensor>
+      <sensor name="${prefix}_ired1" type="camera">
+      <pose relative_to='${prefix}_camera_depth_frame'>-0.2 0 0 0 0 0</pose>
+      <topic>${prefix_topic}/${prefix}/ired1</topic>
+        <camera name="r430">
+          <horizontal_fov>${91.2*M_PI/180.0}</horizontal_fov>
+          <image>
+            <width>640</width>
+            <height>480</height>
+            <format>L_INT8</format>
+          </image>
+          <clip>
+            <near>0.3</near>
+            <far>10.0</far>
+          </clip>
+          <noise>
+            <type>gaussian</type>
+            <mean>0.0</mean>
+            <stddev>0.05</stddev>
+          </noise>
+        </camera>
+        <always_on>1</always_on>
+        <update_rate>90</update_rate>
+        <visualize>0</visualize>
+      </sensor>
+      <sensor name="${prefix}_ired2" type="camera">
+        <pose relative_to='${prefix}_camera_depth_frame'>0.2 0 0 0 0 0</pose>
+        <topic>${prefix_topic}/${prefix}/ired2</topic>
+        <camera name="r430">
+          <horizontal_fov>1.4870205226991688</horizontal_fov>
+          <image>
+            <width>640</width>
+            <height>480</height>
+            <format>L_INT8</format>
+          </image>
+          <clip>
+            <near>0.3</near>
+            <far>10.0</far>
+          </clip>
+          <noise>
+            <type>gaussian</type>
+            <mean>0.0</mean>
+            <stddev>0.05</stddev>
+          </noise>
+        </camera>
+        <always_on>1</always_on>
+        <update_rate>90</update_rate>
+        <visualize>0</visualize>
+      </sensor>
+    </gazebo>
+    <gazebo reference="${sensor_link_name}_depth_link">
+      <sensor name="${prefix}_depth_link" type="depth">
+        <pose relative_to='${sensor_link_name}_depth_link'>0.1 0 0 0 0 0</pose>
+        <topic>${prefix_topic}/${prefix}/depth</topic>
+        <camera name="r430">
+          <horizontal_fov>${91.2*M_PI/180.0}</horizontal_fov>
+          <image>
+            <width>640</width>
+            <height>480</height>
+          </image>
+          <clip>
+            <near>0.3</near>
+            <far>10.0</far>
+          </clip>
+          <noise>
+            <type>gaussian</type>
+            <mean>0.0</mean>
+            <stddev>0.100</stddev>
+          </noise>
+        </camera>
+        <always_on>1</always_on>
+        <update_rate>15</update_rate>
+        <visualize>0</visualize>
+      </sensor>
     </gazebo>
     <!-- <gazebo>

Commit message: Adding second drawer

File: src/ros2/robot_description/rb_theron_common/rb_theron_description/robots/rb_theron.urdf.xacro (robot description, xacro)
@@ -113,4 +113,8 @@
 		<origin xyz="0.105 0.0 0.3" rpy="0 0 0"/>
 	</xacro:drawer>
+	<xacro:include filename="$(find rb_theron_description)/urdf/drawer/drawer.urdf.xacro" />
+	<xacro:drawer prefix="$(arg prefix)second" parent="$(arg prefix)base_link">
+		<origin xyz="0.105 0.0 0.5" rpy="0 0 0"/>
+	</xacro:drawer>
 	<!-- Gazebo ros control pluggins -->
 	<xacro:ros_control prefix="$(arg prefix)" publish_bf="${publish_bf}"/>

File: src/ros2/robot_description/rb_theron_common/rb_theron_description/urdf/drawer/drawer.urdf.xacro (robot description, xacro)
@@ -39,5 +39,5 @@
                 <turnGravityOff>false</turnGravityOff>
         </gazebo>
-        <joint name="top_drawer_joint" type="prismatic" >
+        <joint name="${prefix}_drawer_joint" type="prismatic" >
                 <axis xyz="1 0 0" />
                 <parent link="${parent}" />
@@ -48,5 +48,5 @@
         <gazebo>
                 <plugin filename="libignition-gazebo-joint-position-controller-system.so" name="ignition::gazebo::systems::JointPositionController">
-                        <joint_name>top_drawer_joint</joint_name>
+                        <joint_name>${prefix}_drawer_joint</joint_name>
                         <p_gain>50000.0</p_gain>
                         <i_gain>100</i_gain>
