Commit message: Adding more drawers and a placeholder door opening mechanism

File: src/ros2/robot_description/rb_theron_common/rb_theron_description/robots/rb_theron.urdf.xacro (robot description, xacro)
@@ -105,16 +105,29 @@
 	<!-- ROBAST Module Cage -->
 	<xacro:include filename="$(find rb_theron_description)/urdf/module_cage/module_cage.urdf.xacro" />
-	<xacro:module_cage prefix="$(arg prefix)module_cage" parent="$(arg prefix)base_link">
-		<origin xyz="0.35 -0.0 -0.075" rpy="0 0 1.570796326794896619"/>
+	<xacro:module_cage prefix="$(arg prefix)module_cage" parent="$(arg prefix)base_link" hq="${hq}" >
+		<origin xyz="-0.15 0.0 0.725" rpy="0 0 0"/>
 	</xacro:module_cage>
 	<!-- ROBAST Drawer -->
 	<xacro:include filename="$(find rb_theron_description)/urdf/drawer/drawer.urdf.xacro" />
-	<xacro:drawer prefix="$(arg prefix)first" parent="$(arg prefix)base_link">
-		<origin xyz="0.105 0.0 0.3" rpy="0 0 0"/>
+	<xacro:drawer prefix="$(arg prefix)" suffix="5" parent="$(arg prefix)base_link" drawer_size_z="0.28">
+		<origin xyz="0.125 0.0 0.42" rpy="0 0 0"/>
 	</xacro:drawer>
-	<xacro:include filename="$(find rb_theron_description)/urdf/drawer/drawer.urdf.xacro" />
-	<xacro:drawer prefix="$(arg prefix)second" parent="$(arg prefix)base_link">
-		<origin xyz="0.105 0.0 0.5" rpy="0 0 0"/>
+	<xacro:drawer prefix="$(arg prefix)" suffix="4" parent="$(arg prefix)base_link" drawer_size_z="0.18">
+		<origin xyz="0.125 0.0 0.67" rpy="0 0 0"/>
 	</xacro:drawer>
+	<xacro:drawer prefix="$(arg prefix)" suffix="3" parent="$(arg prefix)base_link" drawer_size_z="0.08">
+		<origin xyz="0.125 0.0 0.82" rpy="0 0 0"/>
+	</xacro:drawer>
+	<xacro:drawer prefix="$(arg prefix)" suffix="2" parent="$(arg prefix)base_link" drawer_size_z="0.08">
+		<origin xyz="0.125 0.0 0.92" rpy="0 0 0"/>
+	</xacro:drawer>
+	<xacro:drawer prefix="$(arg prefix)" suffix="1" parent="$(arg prefix)base_link" drawer_size_z="0.08">
+		<origin xyz="0.125 0.0 1.02" rpy="0 0 0"/>
+	</xacro:drawer>
+	<!-- ROBAST Door Opening Mechanism -->
+	<xacro:include filename="$(find rb_theron_description)/urdf/door_opening_mechanism/door_opening_mechanism.urdf.xacro" />
+	<xacro:door_opening_mechanism prefix="$(arg prefix)door_opening_mechanism" parent="$(arg prefix)base_link" hq="${hq}" >
+		<origin xyz="-0.3 0 0.725" rpy="0 0 0"/>
+	</xacro:door_opening_mechanism>
 	<!-- Gazebo ros control pluggins -->
 	<xacro:ros_control prefix="$(arg prefix)" publish_bf="${publish_bf}"/>

File: src/ros2/robot_description/rb_theron_common/rb_theron_description/urdf/drawer/drawer.urdf.xacro (robot description, xacro)
@@ -1,59 +1,58 @@
 <?xml version="1.0"?>
 <robot name="drawer" xmlns:xacro="http://www.ros.org/wiki/xacro">
-<xacro:macro name="box_inertia_robot" params="m x y z">
-	<inertia  ixx="${m*(y*y+z*z)/12}" ixy = "0" ixz = "0"
-			iyy="${m*(x*x+z*z)/12}" iyz = "0"
-			izz="${m*(x*x+z*z)/12}" />
-</xacro:macro>
-<xacro:property name="drawer_size_x" value="0.45" />
-<xacro:property name="drawer_size_y" value="0.358" />
-<xacro:property name="drawer_size_z" value="0.08" />
-<xacro:property name="drawer_mass" value="1.5" />
-<xacro:property name="drawer_offset_x" value="0.0" />
-<xacro:property name="drawer_offset_y" value="0.0" />
-<xacro:property name="drawer_offset_z" value="0.0" />
-<xacro:macro name="drawer" params="prefix parent *origin">
-        <link name="${prefix}_drawer">
-                <inertial>
-                        <mass value="${drawer_mass}" />
-                        <origin xyz="${drawer_offset_x} ${drawer_offset_y} ${drawer_offset_z}" />
-                        <xacro:box_inertia_robot m="${drawer_mass}" x="${drawer_size_x}" y="${drawer_size_y}" z="${drawer_size_z}"/>
-                </inertial>
-                <visual>
-                        <!-- visual origin is defined w.r.t. link local coordinate system -->
-                        <origin xyz="${drawer_offset_x} ${drawer_offset_y} ${drawer_offset_z}" rpy="0 0 0" />
-                        <geometry>
+    <xacro:macro name="box_inertia_robot" params="m x y z">
+        <inertia  ixx="${m*(y*y+z*z)/12}" ixy = "0" ixz = "0"
+                iyy="${m*(x*x+z*z)/12}" iyz = "0"
+                izz="${m*(x*x+z*z)/12}" />
+    </xacro:macro>
+    <xacro:property name="drawer_size_x" value="0.45" />
+    <xacro:property name="drawer_size_y" value="0.358" />
+    <xacro:property name="drawer_mass" value="1.5" />
+    <xacro:property name="drawer_offset_x" value="0.0" />
+    <xacro:property name="drawer_offset_y" value="0.0" />
+    <xacro:property name="drawer_offset_z" value="0.0" />
+    <xacro:macro name="drawer" params="prefix suffix parent *origin drawer_size_z">
+        <link name="${prefix}_drawer_${suffix}">
+            <inertial>
+                <mass value="${drawer_mass}" />
+                <origin xyz="${drawer_offset_x} ${drawer_offset_y} ${drawer_offset_z}" />
+                <xacro:box_inertia_robot m="${drawer_mass}" x="${drawer_size_x}" y="${drawer_size_y}" z="${drawer_size_z}"/>
+            </inertial>
+            <visual>
+                <!-- visual origin is defined w.r.t. link local coordinate system -->
+                <origin xyz="${drawer_offset_x} ${drawer_offset_y} ${drawer_offset_z}" rpy="0 0 0" />
+                <geometry>
+                    <box size="${drawer_size_x} ${drawer_size_y} ${drawer_size_z}" />
+                </geometry>
+            </visual>
+            <collision>
+                <!-- collision origin is defined w.r.t. link local coordinate system -->
+                <origin xyz="${drawer_offset_x} ${drawer_offset_y} ${drawer_offset_z}" rpy="0 0 0 " />
+                <geometry>
                         <box size="${drawer_size_x} ${drawer_size_y} ${drawer_size_z}" />
-                        </geometry>
-                </visual>
-                <collision>
-                        <!-- collision origin is defined w.r.t. link local coordinate system -->
-                        <origin xyz="${drawer_offset_x} ${drawer_offset_y} ${drawer_offset_z}" rpy="0 0 0 " />
-                        <geometry>
-                        <box size="${drawer_size_x} ${drawer_size_y} ${drawer_size_z}" />
-                        </geometry>
-                </collision>
+                </geometry>
+        </collision>
         </link>
-        <gazebo reference="${prefix}_drawer">
+        <gazebo reference="${prefix}_drawer_${suffix}">
                 <material>Gazebo/White</material>
                 <turnGravityOff>false</turnGravityOff>
         </gazebo>
-        <joint name="${prefix}_drawer_joint" type="prismatic" >
-                <axis xyz="1 0 0" />
-                <parent link="${parent}" />
-                <child link="${prefix}_drawer" />
-                <xacro:insert_block name="origin" />
-                <limit lower="0.0" upper="${0.95*drawer_size_y}" effort="100" velocity="100" />
+        <joint name="${prefix}_drawer_${suffix}_joint" type="prismatic" >
+            <axis xyz="1 0 0" />
+            <parent link="${parent}" />
+            <child link="${prefix}_drawer_${suffix}" />
+            <xacro:insert_block name="origin" />
+            <limit lower="0.0" upper="${0.95*drawer_size_y}" effort="100" velocity="100" />
         </joint>
         <gazebo>
-                <plugin filename="libignition-gazebo-joint-position-controller-system.so" name="ignition::gazebo::systems::JointPositionController">
-                        <joint_name>${prefix}_drawer_joint</joint_name>
-                        <p_gain>50000.0</p_gain>
-                        <i_gain>100</i_gain>
-                        <d_gain>1000</d_gain>
-                        <i_max>200</i_max>
-                        <i_min>-200</i_min>
-                </plugin>
+            <plugin filename="libignition-gazebo-joint-position-controller-system.so" name="ignition::gazebo::systems::JointPositionController">
+                <joint_name>${prefix}_drawer_${suffix}_joint</joint_name>
+                <p_gain>50000.0</p_gain>
+                <i_gain>100</i_gain>
+                <d_gain>1000</d_gain>
+                <i_max>200</i_max>
+                <i_min>-200</i_min>
+            </plugin>
         </gazebo>
-</xacro:macro>
+    </xacro:macro>
 </robot>

File: src/ros2/robot_description/rb_theron_common/rb_theron_description/urdf/module_cage/module_cage.urdf.xacro (robot description, xacro)
@@ -6,37 +6,42 @@
 			izz="${m*(x*x+z*z)/12}" />
 </xacro:macro>
-  <xacro:macro name="module_cage" params="prefix parent *origin">
-		<joint name="${prefix}module_cage_joint" type="fixed">
-			<parent link="${parent}"/>
-			<child link="${prefix}module_cage_link"/>
-			<xacro:insert_block name="origin" />
-		</joint>
-    <!-- BASE_LINK -->
-    <link name="${prefix}module_cage_link">
-      <inertial>
-        <mass value="10.0" />
-        <origin xyz="0 0 0" />
-	    <xacro:box_inertia_robot m="10" x="0.25" y="0.25" z="1.55"/>
-      </inertial>
-      <visual>
-	  <origin xyz="0 ${0.655-0.167} 0.8" rpy="0 0 1.57" />
-        <!-- <origin xyz="0 0 0" rpy="0 0 0" /> -->
-          <geometry>
-            <!-- <box size="0.25 0.25 1.55"/> -->
-	    <box size="0.03 0.43 1.05"/>
-            <!-- <mesh filename="$(find rb_theron_description)/meshes/module_cage/module_cage.stl" scale="0.001 0.001 0.001"/> -->
-          </geometry>
-        <material name="darkgrey">
-          <color rgba="0.1 0.1 0.1 1"/>
-        </material>
-      </visual>
-      <collision>
-        <origin xyz="0 ${0.655-0.167} 0.8" rpy="0 0 1.57" />
+<xacro:macro name="module_cage" params="prefix parent *origin hq">
+  <joint name="${prefix}module_cage_joint" type="fixed">
+    <parent link="${parent}"/>
+    <child link="${prefix}module_cage_link"/>
+    <xacro:insert_block name="origin" />
+  </joint>
+  <!-- BASE_LINK -->
+  <link name="${prefix}module_cage_link">
+    <inertial>
+      <mass value="25.0" />
+      <origin xyz="0 0 0" />
+      <xacro:box_inertia_robot m="10" x="0.25" y="0.25" z="1.55"/>
+    </inertial>
+    <visual>
+      <xacro:if value="${hq}">
+        <origin xyz="0 0 0" rpy="0 0 0" />
+        <geometry>
+          <mesh filename="$(find rb_theron_description)/meshes/module_cage/module_cage.stl" scale="0.001 0.001 0.001"/>
+        </geometry>
+      </xacro:if>
+      <xacro:unless value="${hq}">
+        <origin xyz="0 0 0" rpy="0 0 0" />
         <geometry>
           <box size="0.03 0.43 1.05"/>
-          <!-- <mesh filename="$(find rb_theron_description)/meshes/module_cage/module_cage.stl" scale="0.001 0.001 0.001"/> -->
         </geometry>
-      </collision>
-    </link>
-  </xacro:macro>
+      </xacro:unless>
+      <material name="darkgrey">
+        <color rgba="0.1 0.1 0.1 1"/>
+      </material>
+    </visual>
+    <collision>
+      <origin xyz="0 0 0" rpy="0 0 0" />
+      <geometry>
+        <box size="0.03 0.43 1.05"/>
+        <!-- <mesh filename="$(find rb_theron_description)/meshes/module_cage/module_cage.stl" scale="0.001 0.001 0.001"/> -->
+      </geometry>
+    </collision>
+  </link>
+</xacro:macro>
 </robot>

Commit message: minor fixes

File: src/ros2/robot_description/rb_theron_common/rb_theron_description/robots/rb_theron.urdf.xacro (robot description, xacro)
@@ -105,5 +105,5 @@
 	<!-- ROBAST Module Cage -->
 	<xacro:include filename="$(find rb_theron_description)/urdf/module_cage/module_cage.urdf.xacro" />
-	<xacro:module_cage prefix="$(arg prefix)module_cage" parent="$(arg prefix)base_link" hq="${hq}" >
+	<xacro:module_cage prefix="$(arg prefix)" parent="$(arg prefix)base_link" hq="${hq}" >
 		<origin xyz="-0.15 0.0 0.725" rpy="0 0 0"/>
 	</xacro:module_cage>

File: src/ros2/robot_description/rb_theron_common/rb_theron_description/urdf/drawer/drawer.urdf.xacro (robot description, xacro)
@@ -13,5 +13,5 @@
     <xacro:property name="drawer_offset_z" value="0.0" />
     <xacro:macro name="drawer" params="prefix suffix parent *origin drawer_size_z">
-        <link name="${prefix}_drawer_${suffix}">
+        <link name="${prefix}drawer_${suffix}">
             <inertial>
                 <mass value="${drawer_mass}" />
@@ -34,12 +34,12 @@
         </collision>
         </link>
-        <gazebo reference="${prefix}_drawer_${suffix}">
+        <gazebo reference="${prefix}drawer_${suffix}">
                 <material>Gazebo/White</material>
                 <turnGravityOff>false</turnGravityOff>
         </gazebo>
-        <joint name="${prefix}_drawer_${suffix}_joint" type="prismatic" >
+        <joint name="${prefix}drawer_${suffix}_joint" type="prismatic" >
             <axis xyz="1 0 0" />
             <parent link="${parent}" />
-            <child link="${prefix}_drawer_${suffix}" />
+            <child link="${prefix}drawer_${suffix}" />
             <xacro:insert_block name="origin" />
             <limit lower="0.0" upper="${0.95*drawer_size_y}" effort="100" velocity="100" />
@@ -47,5 +47,5 @@
         <gazebo>
             <plugin filename="libignition-gazebo-joint-position-controller-system.so" name="ignition::gazebo::systems::JointPositionController">
-                <joint_name>${prefix}_drawer_${suffix}_joint</joint_name>
+                <joint_name>${prefix}drawer_${suffix}_joint</joint_name>
                 <p_gain>50000.0</p_gain>
                 <i_gain>100</i_gain>

Commit message: First draft for alu frame of door opening mechanism

File: src/ros2/robot_description/rb_theron_common/rb_theron_description/robots/rb_theron.urdf.xacro (robot description, xacro)
@@ -127,6 +127,6 @@
 	<!-- ROBAST Door Opening Mechanism -->
 	<xacro:include filename="$(find rb_theron_description)/urdf/door_opening_mechanism/door_opening_mechanism.urdf.xacro" />
-	<xacro:door_opening_mechanism prefix="$(arg prefix)door_opening_mechanism" parent="$(arg prefix)base_link" hq="${hq}" >
-		<origin xyz="-0.3 0 0.725" rpy="0 0 0"/>
+	<xacro:door_opening_mechanism prefix="$(arg prefix)" parent="$(arg prefix)base_link" hq="${hq}" >
+		<origin xyz="-0.3 0 0.225" rpy="0 0 0"/>
 	</xacro:door_opening_mechanism>
 	<!-- Gazebo ros control pluggins -->

File: src/ros2/robot_description/rb_theron_common/rb_theron_description/urdf/door_opening_mechanism/door_opening_mechanism.urdf.xacro (robot description, xacro)
@@ -9,9 +9,9 @@
     <joint name="${prefix}door_opening_mechanism_joint" type="fixed">
         <parent link="${parent}"/>
-        <child link="${prefix}door_opening_mechanism_link"/>
+        <child link="${prefix}door_opening_mechanism_base_link"/>
         <xacro:insert_block name="origin" />
     </joint>
     <!-- BASE_LINK -->
-    <link name="${prefix}door_opening_mechanism_link">
+    <link name="${prefix}door_opening_mechanism_base_link">
         <inertial>
             <!-- Mass should actually not be zero, but there is an issue, that if there is too much load on the theron base,
@@ -23,16 +23,8 @@
         </inertial>
         <visual>
-            <xacro:if value="${hq}">
-                <origin xyz="0 0 0" rpy="0 0 0" />
-                <geometry>
-                <box size="0.03 0.43 1.05"/>
-                </geometry>
-            </xacro:if>
-            <xacro:unless value="${hq}">
-                <origin xyz="0 0 0" rpy="0 0 0" />
-                <geometry>
-                <box size="0.03 0.43 1.05"/>
-                </geometry>
-            </xacro:unless>
+            <origin xyz="0 0 0" rpy="0 0 0" />
+            <geometry>
+                <box size="0.03 0.46 0.03"/>
+            </geometry>
             <material name="darkgrey">
                 <color rgba="0.1 0.1 0.1 1"/>
@@ -42,8 +34,23 @@
             <origin xyz="0 0 0" rpy="0 0 0" />
             <geometry>
-                <box size="0.03 0.43 1.05"/>
+                <box size="0.03 0.46 0.03"/>
             </geometry>
         </collision>
     </link>
+    <!-- <joint name="${prefix}door_opening_mechanism_frame_joint_left" type="fixed">
+        <parent link="${prefix}door_opening_mechanism_base_link"/>
+        <child link="${prefix}door_opening_mechanism_frame_link_left"/>
+        <xacro:insert_block name="origin" />
+    </joint> -->
+    <xacro:include filename="$(find rb_theron_description)/urdf/door_opening_mechanism/alu_profile.urdf.xacro" />
+	<xacro:alu_profile prefix="$(arg prefix)" suffix="left" parent="${prefix}door_opening_mechanism_base_link" x="0.03" y="0.03" z="1.0" >
+		<origin xyz="0 -0.245 0.515" rpy="0 0 0"/>
+	</xacro:alu_profile>
+	<xacro:alu_profile prefix="$(arg prefix)" suffix="right" parent="${prefix}door_opening_mechanism_base_link" x="0.03" y="0.03" z="1.0" >
+		<origin xyz="0 +0.245 0.515" rpy="0 0 0"/>
+	</xacro:alu_profile>
+    <xacro:alu_profile prefix="$(arg prefix)" suffix="top" parent="${prefix}door_opening_mechanism_base_link" x="0.03" y="0.03" z="0.52" >
+		<origin xyz="0 0 1.03" rpy="1.5705 0 0"/>
+	</xacro:alu_profile>
     </xacro:macro>
 </robot>

Commit message: Fixing position for oak d camera and rs_bpearl after try and error with the real life robot

File: src/ros2/robot_description/rb_theron_common/rb_theron_description/robots/rb_theron.urdf.xacro (robot description, xacro)
@@ -83,5 +83,5 @@
 	</xacro:sensor_rs_lidar_16>-->
 	<xacro:sensor_rs_bpearl prefix="$(arg prefix)top_laser"  parent="$(arg prefix)base_link" publish_bf="${publish_bf}" robot_name="${robot_name}" prefix_topic="top_laser" hq="${hq}" range_min="0.1" range_max="90" hfov="360" samples="1800" vfov="90.0" lasers="32" fps="10" gpu="false">
-            <origin xyz="0.28 -0.159 1.22" rpy="-1.570796326795 0 -1.570796326795"/>
+            <origin xyz="0.16 -0.159 1.22" rpy="-1.570796326795 0 -1.570796326795"/>
         </xacro:sensor_rs_bpearl>
 	<!-- <xacro:sensor_sick_nanoscan3 prefix="$(arg prefix)back_laser" parent="$(arg prefix)base_link" prefix_topic="back_laser" min_angle="-1.8107619" max_angle="1.8107619">
@@ -96,5 +96,5 @@
 	<xacro:arg name="camera_model"  default="OAK-D-LITE" />
 	<xacro:arg name="base_frame"    default="oak-d_frame" />
-	<xacro:arg name="cam_pos_x"     default="0.347" />
+	<xacro:arg name="cam_pos_x"     default="0.287" />
 	<xacro:arg name="cam_pos_y"     default="-0.159" />
 	<xacro:arg name="cam_pos_z"     default="1.149" />
@@ -102,5 +102,5 @@
 	<xacro:arg name="cam_pitch"     default="0.0" />
 	<xacro:arg name="cam_yaw"       default="0.0" />
-	<!-- <xacro:depthai_camera camera_name = "$(arg camera_name)" parent = "$(arg prefix)base_link" camera_model = "$(arg camera_model)" base_frame = "$(arg base_frame)" cam_pos_x = "$(arg cam_pos_x)" cam_pos_y = "$(arg cam_pos_y)" cam_pos_z = "$(arg cam_pos_z)" cam_roll = "$(arg cam_roll)" cam_pitch = "$(arg cam_pitch)" cam_yaw = "$(arg cam_yaw)"/> -->
+	<xacro:depthai_camera camera_name = "$(arg camera_name)" parent = "$(arg prefix)base_link" camera_model = "$(arg camera_model)" base_frame = "$(arg base_frame)" cam_pos_x = "$(arg cam_pos_x)" cam_pos_y = "$(arg cam_pos_y)" cam_pos_z = "$(arg cam_pos_z)" cam_roll = "$(arg cam_roll)" cam_pitch = "$(arg cam_pitch)" cam_yaw = "$(arg cam_yaw)"/>
 	<!-- ROBAST Module Cage -->
 	<xacro:include filename="$(find rb_theron_description)/urdf/module_cage/module_cage.urdf.xacro" />
