Commit message: Extending the depthai_macro to generate data in gazebo

File: src/ros2/robot_description/rb_theron_common/rb_theron_description/robots/rb_theron.urdf.xacro (robot description, xacro)
@@ -93,14 +93,13 @@
 		</plugin>
 	</gazebo>
-	<xacro:arg name="camera_name"   default="oak" />
-	<xacro:arg name="camera_model"  default="OAK-D-LITE" />
-	<xacro:arg name="base_frame"    default="oak-d_frame" />
-	<xacro:arg name="cam_pos_x"     default="0.347" />
-	<xacro:arg name="cam_pos_y"     default="-0.159" />
-	<xacro:arg name="cam_pos_z"     default="1.149" />
-	<xacro:arg name="cam_roll"      default="0.0" />
-	<xacro:arg name="cam_pitch"     default="0.0" />
-	<xacro:arg name="cam_yaw"       default="0.0" />
-	<!-- <xacro:depthai_camera camera_name = "$(arg camera_name)" parent = "$(arg prefix)base_link" camera_model = "$(arg camera_model)" base_frame = "$(arg base_frame)" cam_pos_x = "$(arg cam_pos_x)" cam_pos_y = "$(arg cam_pos_y)" cam_pos_z = "$(arg cam_pos_z)" cam_roll = "$(arg cam_roll)" cam_pitch = "$(arg cam_pitch)" cam_yaw = "$(arg cam_yaw)"/> -->
+    <xacro:arg name="camera_model"  default="OAK-D-LITE" />
+    <xacro:arg name="base_frame"    default="oak-d_frame" />
+    <xacro:arg name="cam_pos_x"     default="0.287" />
+    <xacro:arg name="cam_pos_y"     default="-0.159" />
+    <xacro:arg name="cam_pos_z"     default="1.149" />
+    <xacro:arg name="cam_roll"      default="0.0" />
+    <xacro:arg name="cam_pitch"     default="0.0" />
+    <xacro:arg name="cam_yaw"       default="0.0" />
+    <xacro:depthai_camera prefix="$(arg prefix)front_top_oak_d_camera" parent="$(arg prefix)base_link" publish_bf="${publish_bf}" robot_name="${robot_name}" prefix_topic="front_top_oak_d_camera" camera_model = "$(arg camera_model)" base_frame = "$(arg base_frame)" cam_pos_x = "$(arg cam_pos_x)" cam_pos_y = "$(arg cam_pos_y)" cam_pos_z = "$(arg cam_pos_z)" cam_roll = "$(arg cam_roll)" cam_pitch = "$(arg cam_pitch)" cam_yaw = "$(arg cam_yaw)"/>
 	<!-- ROBAST Module Cage -->
 	<xacro:include filename="$(find rb_theron_description)/urdf/module_cage/module_cage.urdf.xacro" />

File: src/ros2/robot_description/robotnik_sensors/urdf/depthai_macro.urdf.xacro (robot description, xacro)
@@ -1,8 +1,14 @@
 <?xml version="1.0"?>
 <robot name="depthai_camera" xmlns:xacro="http://ros.org/wiki/xacro">
-<xacro:macro name="depthai_camera" params="camera_name camera_model parent base_frame
+<xacro:macro name="depthai_camera" params="prefix parent publish_bf robot_name prefix_topic camera_model base_frame
                                            cam_pos_x cam_pos_y cam_pos_z
                                            cam_roll cam_pitch cam_yaw
                                            r:=0.8 g:=0.8 b:=0.8 a:=0.8">
+    <xacro:if value="${publish_bf}">
+			<xacro:property name="sensor_link_name" value="${robot_name}/base_footprint/${prefix}" />
+		</xacro:if>
+		<xacro:unless value="${publish_bf}">
+			<xacro:property name="sensor_link_name" value="${robot_name}/base_link/${prefix}" />
+		</xacro:unless>
     <xacro:property name="M_PI"     value="3.1415926535897931" />
     <xacro:property name="model"    value="${camera_model}" />
@@ -22,11 +28,11 @@
     <!-- base_link of the sensor-->
     <link name="${base_frame}"/>
-    <joint name="${camera_name}_center_joint" type="fixed">
+    <joint name="${prefix}_center_joint" type="fixed">
         <parent link="${parent}"/>
         <child link="${base_frame}"/>
         <origin xyz="${cam_pos_x} ${cam_pos_y} ${cam_pos_z}" rpy="${cam_roll} ${cam_pitch} ${cam_yaw}" />
     </joint>
-<!-- device Center -->
-    <link name="${camera_name}_model_origin">
+    <!-- device Center -->
+    <link name="${prefix}_model_origin">
         <visual>
             <origin xyz="0 0 0" rpy="0 0 0"/>
@@ -39,57 +45,108 @@
         </visual>
     </link>
-    <joint name="${camera_name}_model_origin_joint" type="fixed">
+    <joint name="${prefix}_model_origin_joint" type="fixed">
         <parent link="${base_frame}"/>
-        <child link="${camera_name}_model_origin"/>
+        <child link="${prefix}_model_origin"/>
         <origin xyz="0 0 0" rpy="1.5708 0 1.5708" />
     </joint>
-<!-- IMU -->
+    <!-- IMU -->
     <xacro:if value="${has_imu}">
-        <link name="${camera_name}_imu_frame" />
-        <joint name="${camera_name}_imu_joint" type="fixed">
+        <link name="${prefix}_imu_frame" />
+        <joint name="${prefix}_imu_joint" type="fixed">
             <parent link="${base_frame}"/>
-            <child link="${camera_name}_imu_frame"/>
+            <child link="${prefix}_imu_frame"/>
             <origin xyz="${imu_offset_x} ${imu_offset_y} ${imu_offset_z}" rpy="${imu_r} ${imu_p} ${imu_y}" />
         </joint>
     </xacro:if>
-<!-- RGB Camera -->
-    <link name="${camera_name}_rgb_camera_frame" />
-    <joint name="${camera_name}_rgb_camera_joint" type="fixed">
+    <!-- RGB Camera -->
+    <link name="${prefix}_rgb_camera_frame" />
+    <joint name="${prefix}_rgb_camera_joint" type="fixed">
         <parent link="${base_frame}"/>
-        <child link="${camera_name}_rgb_camera_frame"/>
+        <child link="${prefix}_rgb_camera_frame"/>
         <origin xyz="0 0 0" rpy="0 0 0" />
     </joint>
-    <link name="${camera_name}_rgb_camera_optical_frame"/>
-    <joint name="${camera_name}_rgb_camera_optical_joint" type="fixed">
+    <link name="${sensor_link_name}_rgb_camera_optical_frame"/>
+    <joint name="${prefix}_rgb_camera_optical_joint" type="fixed">
         <origin xyz="0 0 0" rpy="-${M_PI/2} 0.0 -${M_PI/2}"/>
-        <parent link="${camera_name}_rgb_camera_frame"/>
-        <child link="${camera_name}_rgb_camera_optical_frame"/>
+        <parent link="${prefix}_rgb_camera_frame"/>
+        <child link="${sensor_link_name}_rgb_camera_optical_frame"/>
     </joint>
-<!-- Left Camera -->
-    <link name="${camera_name}_left_camera_frame" />
-    <joint name="${camera_name}_left_camera_joint" type="fixed">
+    <!-- Left Camera -->
+    <link name="${prefix}_left_camera_frame" />
+    <joint name="${prefix}_left_camera_joint" type="fixed">
         <parent link="${base_frame}"/>
-        <child link="${camera_name}_left_camera_frame"/>
+        <child link="${prefix}_left_camera_frame"/>
         <origin xyz="0 ${baseline/2} 0" rpy="0 0 0" />
     </joint>
-    <link name="${camera_name}_left_camera_optical_frame"/>
-    <joint name="${camera_name}_left_camera_optical_joint" type="fixed">
+    <link name="${prefix}_left_camera_optical_frame"/>
+    <joint name="${prefix}_left_camera_optical_joint" type="fixed">
         <origin xyz="0 0 0" rpy="-${M_PI/2} 0.0 -${M_PI/2}"/>
-        <parent link="${camera_name}_left_camera_frame"/>
-        <child link="${camera_name}_left_camera_optical_frame"/>
+        <parent link="${prefix}_left_camera_frame"/>
+        <child link="${prefix}_left_camera_optical_frame"/>
     </joint>
-<!-- right Camera -->
-    <link name="${camera_name}_right_camera_frame" />
-    <joint name="${camera_name}_right_camera_joint" type="fixed">
+    <!-- right Camera -->
+    <link name="${prefix}_right_camera_frame" />
+    <joint name="${prefix}_right_camera_joint" type="fixed">
         <parent link="${base_frame}"/>
-        <child link="${camera_name}_right_camera_frame"/>
+        <child link="${prefix}_right_camera_frame"/>
         <origin xyz="0 -${baseline/2} 0" rpy="0 0 0" />
     </joint>
-    <link name="${camera_name}_right_camera_optical_frame"/>
-    <joint name="${camera_name}_right_camera_optical_joint" type="fixed">
+    <link name="${sensor_link_name}_right_camera_optical_frame"/>
+    <joint name="${prefix}_right_camera_optical_joint" type="fixed">
         <origin xyz="0 0 0" rpy="-${M_PI/2} 0.0 -${M_PI/2}"/>
-        <parent link="${camera_name}_right_camera_frame"/>
-        <child link="${camera_name}_right_camera_optical_frame"/>
+        <parent link="${prefix}_right_camera_frame"/>
+        <child link="${sensor_link_name}_right_camera_optical_frame"/>
     </joint>
+    <xacro:sensor_depthai_gazebo/>
+</xacro:macro>
+  <xacro:macro name="sensor_depthai_gazebo">
+    <!-- gazebo reference="${prefix}_rgb_base_link" -->
+    <gazebo reference="${base_frame}">
+      <sensor name="${prefix}_rgb_camera_optical_frame" type="camera">
+				<topic>${prefix_topic}/color</topic>
+        <camera name="r430">
+            <horizontal_fov>1.2112585008840648</horizontal_fov>
+            <image>
+                <width>640</width>
+                <height>480</height>
+                <format>RGB_INT8</format>
+            </image>
+            <clip>
+                <near>0.1</near>
+                <far>100</far>
+            </clip>
+              <noise>
+                <type>gaussian</type>
+                <mean>0.0</mean>
+                <stddev>0.007</stddev>
+            </noise>
+        </camera>
+        <always_on>1</always_on>
+        <update_rate>30</update_rate>
+        <visualize>1</visualize>
+      </sensor>
+      <sensor name="${prefix}_right_camera_optical_frame" type="depth">
+        <topic>${prefix_topic}/${prefix}/depth</topic>
+        <camera name="r430">
+          <horizontal_fov>${91.2*M_PI/180.0}</horizontal_fov>
+          <image>
+            <width>640</width>
+            <height>480</height>
+          </image>
+          <clip>
+            <near>0.3</near>
+            <far>10.0</far>
+          </clip>
+          <noise>
+            <type>gaussian</type>
+            <mean>0.0</mean>
+            <stddev>0.010</stddev>
+          </noise>
+        </camera>
+        <always_on>1</always_on>
+        <update_rate>15</update_rate>
+        <visualize>1</visualize>
+      </sensor>
+    </gazebo>
 </xacro:macro>
 </robot>

Commit message: Add behaviour plugins, ROS package for door and handle detection and new door materials for simulation

File: src/ros2/robot_description/rb_theron_common/rb_theron_description/robots/rb_theron.urdf.xacro (robot description, xacro)
@@ -65,4 +65,7 @@
 	<xacro:sensor_r430 prefix="$(arg prefix)front_realsense_camera" parent="$(arg prefix)base_link" publish_bf="${publish_bf}" robot_name="${robot_name}" prefix_topic="front_realsense_camera" hq="${hq}">
 		<origin xyz="0.3305 0.0 0.1468" rpy="0 0 0"/>
+	</xacro:sensor_r430>
+	<xacro:sensor_r430 prefix="$(arg prefix)back_upper_realsense_camera" parent="$(arg prefix)base_link" publish_bf="${publish_bf}" robot_name="${robot_name}" prefix_topic="back_upper_realsense_camera" hq="${hq}">
+		<origin xyz="-0.3305 0.0 1.1468" rpy="0 0 3.1416"/>
 	</xacro:sensor_r430>
 	<xacro:sensor_r430 prefix="$(arg prefix)back_realsense_camera" parent="$(arg prefix)base_link" publish_bf="${publish_bf}" robot_name="${robot_name}" prefix_topic="back_realsense_camera" hq="${hq}">

Commit message: Modify BT plugin and position of OAK-D camera

File: src/ros2/robot_description/rb_theron_common/rb_theron_description/robots/rb_theron.urdf.xacro (robot description, xacro)
@@ -66,7 +66,4 @@
 		<origin xyz="0.3305 0.0 0.1468" rpy="0 0 0"/>
 	</xacro:sensor_r430>
-	<xacro:sensor_r430 prefix="$(arg prefix)back_upper_realsense_camera" parent="$(arg prefix)base_link" publish_bf="${publish_bf}" robot_name="${robot_name}" prefix_topic="back_upper_realsense_camera" hq="${hq}">
-		<origin xyz="-0.3305 0.0 1.1468" rpy="0 0 3.1416"/>
-	</xacro:sensor_r430>
 	<xacro:sensor_r430 prefix="$(arg prefix)back_realsense_camera" parent="$(arg prefix)base_link" publish_bf="${publish_bf}" robot_name="${robot_name}" prefix_topic="back_realsense_camera" hq="${hq}">
 		<origin xyz="-0.3305 0.0 0.1468" rpy="0 0 3.1416"/>
@@ -96,12 +93,12 @@
 		</plugin>
 	</gazebo>
-    <xacro:arg name="camera_model"  default="OAK-D-LITE" />
+    <xacro:arg name="camera_model"  default="OAK-D-POE" />
     <xacro:arg name="base_frame"    default="oak-d_frame" />
-    <xacro:arg name="cam_pos_x"     default="0.287" />
-    <xacro:arg name="cam_pos_y"     default="-0.159" />
-    <xacro:arg name="cam_pos_z"     default="1.149" />
+    <xacro:arg name="cam_pos_x"     default="-0.3305" />
+    <xacro:arg name="cam_pos_y"     default="0.0" />
+    <xacro:arg name="cam_pos_z"     default="1.1468" />
     <xacro:arg name="cam_roll"      default="0.0" />
     <xacro:arg name="cam_pitch"     default="0.0" />
-    <xacro:arg name="cam_yaw"       default="0.0" />
+    <xacro:arg name="cam_yaw"       default="3.1416" />
     <xacro:depthai_camera prefix="$(arg prefix)front_top_oak_d_camera" parent="$(arg prefix)base_link" publish_bf="${publish_bf}" robot_name="${robot_name}" prefix_topic="front_top_oak_d_camera" camera_model = "$(arg camera_model)" base_frame = "$(arg base_frame)" cam_pos_x = "$(arg cam_pos_x)" cam_pos_y = "$(arg cam_pos_y)" cam_pos_z = "$(arg cam_pos_z)" cam_roll = "$(arg cam_roll)" cam_pitch = "$(arg cam_pitch)" cam_yaw = "$(arg cam_yaw)"/>
 	<!-- ROBAST Module Cage -->

Commit message: Add front OAK-D camera to the simulation

File: src/ros2/robot_description/rb_theron_common/rb_theron_description/robots/rb_theron.urdf.xacro (robot description, xacro)
@@ -101,5 +101,6 @@
     <xacro:arg name="cam_pitch"     default="0.0" />
     <xacro:arg name="cam_yaw"       default="3.1416" />
-    <xacro:depthai_camera prefix="$(arg prefix)front_top_oak_d_camera" parent="$(arg prefix)base_link" publish_bf="${publish_bf}" robot_name="${robot_name}" prefix_topic="front_top_oak_d_camera" camera_model = "$(arg camera_model)" base_frame = "$(arg base_frame)" cam_pos_x = "$(arg cam_pos_x)" cam_pos_y = "$(arg cam_pos_y)" cam_pos_z = "$(arg cam_pos_z)" cam_roll = "$(arg cam_roll)" cam_pitch = "$(arg cam_pitch)" cam_yaw = "$(arg cam_yaw)"/>
+    <xacro:depthai_camera prefix="$(arg prefix)back_top_oak_d_camera" parent="$(arg prefix)base_link" publish_bf="${publish_bf}" robot_name="${robot_name}" prefix_topic="back_top_oak_d_camera" camera_model = "$(arg camera_model)" base_frame = "$(arg base_frame)" cam_pos_x = "$(arg cam_pos_x)" cam_pos_y = "$(arg cam_pos_y)" cam_pos_z = "$(arg cam_pos_z)" cam_roll = "$(arg cam_roll)" cam_pitch = "$(arg cam_pitch)" cam_yaw = "$(arg cam_yaw)"/>
+	<xacro:depthai_camera prefix="$(arg prefix)front_top_oak_d_camera" parent="$(arg prefix)base_link" publish_bf="${publish_bf}" robot_name="${robot_name}" prefix_topic="front_top_oak_d_camera" camera_model = "OAK-D-LITE" base_frame = "oak-dlite_frame" cam_pos_x = "0.3305" cam_pos_y = "0.0" cam_pos_z = "1.1468" cam_roll = "0.0" cam_pitch = "0.0" cam_yaw = "0.0"/>
 	<!-- ROBAST Module Cage -->
 	<xacro:include filename="$(find rb_theron_description)/urdf/module_cage/module_cage.urdf.xacro" />

File: src/ros2/robot_description/robotnik_sensors/urdf/depthai_macro.urdf.xacro (robot description, xacro)
@@ -94,5 +94,5 @@
     <link name="${sensor_link_name}_right_camera_optical_frame"/>
     <joint name="${prefix}_right_camera_optical_joint" type="fixed">
-        <origin xyz="0 0 0" rpy="-${M_PI/2} 0.0 -${M_PI/2}"/>
+        <origin xyz="0 0 0" rpy="0 0 0"/>
         <parent link="${prefix}_right_camera_frame"/>
         <child link="${sensor_link_name}_right_camera_optical_frame"/>
@@ -129,5 +129,5 @@
         <topic>${prefix_topic}/${prefix}/depth</topic>
         <camera name="r430">
-          <horizontal_fov>${91.2*M_PI/180.0}</horizontal_fov>
+          <horizontal_fov>${85.2*M_PI/180.0}</horizontal_fov>
           <image>
             <width>640</width>

Commit message: combining the topics from a robot in there own namespace

File: src/ros2/robot_description/rb_theron_common/rb_theron_description/robots/rb_theron.urdf.xacro (robot description, xacro)
@@ -42,4 +42,5 @@
 	<!-- *************** -->
 	<xacro:arg name="prefix" default=""/>
+	<xacro:arg name="topic_namespace" default=""/>
 	<!-- Here we create the robot elements using the xacro:macros imported at the beggining of this file -->
 	<!-- this property is for the chassis -->
@@ -63,8 +64,8 @@
 	<!-- TODO: Should be sensor_intel_d435, but this one isn't migrated to ros2 yet -->
 	<!-- TODO: Moved 0.01 in x, otherwise the camera is still inside the robot -->
-	<xacro:sensor_r430 prefix="$(arg prefix)front_realsense_camera" parent="$(arg prefix)base_link" publish_bf="${publish_bf}" robot_name="${robot_name}" prefix_topic="front_realsense_camera" hq="${hq}">
+	<xacro:sensor_r430 prefix="$(arg prefix)front_realsense_camera" parent="$(arg prefix)base_link" publish_bf="${publish_bf}" robot_name="${robot_name}" prefix_topic="$(arg topic_namespace)/front_realsense_camera" hq="${hq}">
 		<origin xyz="0.3305 0.0 0.1468" rpy="0 0 0"/>
 	</xacro:sensor_r430>
-	<xacro:sensor_r430 prefix="$(arg prefix)back_realsense_camera" parent="$(arg prefix)base_link" publish_bf="${publish_bf}" robot_name="${robot_name}" prefix_topic="back_realsense_camera" hq="${hq}">
+	<xacro:sensor_r430 prefix="$(arg prefix)back_realsense_camera" parent="$(arg prefix)base_link" publish_bf="${publish_bf}" robot_name="${robot_name}" prefix_topic="$(arg topic_namespace)/back_realsense_camera" hq="${hq}">
 		<origin xyz="-0.3305 0.0 0.1468" rpy="0 0 3.1416"/>
 	</xacro:sensor_r430>
@@ -73,8 +74,8 @@
 		<origin xyz="0.3305 0.0 0.1898" rpy="0 0 0"/>
 	</xacro:sensor_orbbec_astra -->
-	<xacro:sensor_imu_hector prefix="$(arg prefix)imu" parent="$(arg prefix)base_link">
+	<xacro:sensor_imu_hector prefix="$(arg prefix)imu" parent="$(arg prefix)base_link" prefix_topic="$(arg topic_namespace)/imu">
 		<origin xyz="-0.1975 0.0 0.1598" rpy="0 0 0"/>
 	</xacro:sensor_imu_hector>
-	<xacro:sensor_sick_nanoscan3 prefix="$(arg prefix)front_laser" parent="$(arg prefix)base_link" publish_bf="${publish_bf}" robot_name="${robot_name}" prefix_topic="front_laser" hq="${hq}" min_angle="-1.9507619" max_angle="1.9507619" gpu="true">
+	<xacro:sensor_sick_nanoscan3 prefix="$(arg prefix)front_laser" parent="$(arg prefix)base_link" publish_bf="${publish_bf}" robot_name="${robot_name}" prefix_topic="$(arg topic_namespace)/front_laser" hq="${hq}" min_angle="-1.9507619" max_angle="1.9507619" gpu="true">
 		<origin xyz="0.250 0.0 0.1643" rpy="0 3.1416 3.1416"/>
 	</xacro:sensor_sick_nanoscan3>
@@ -82,5 +83,5 @@
 		<origin xyz="0.214 0.0 0.275" rpy="-1.57079632679 0 -0.23"/>
 	</xacro:sensor_rs_lidar_16>-->
-	<xacro:sensor_rs_bpearl prefix="$(arg prefix)top_laser"  parent="$(arg prefix)base_link" publish_bf="${publish_bf}" robot_name="${robot_name}" prefix_topic="top_laser" hq="${hq}" range_min="0.1" range_max="90" hfov="360" samples="1200" vfov="90.0" lasers="32" fps="15" gpu="false">
+	<xacro:sensor_rs_bpearl prefix="$(arg prefix)top_laser"  parent="$(arg prefix)base_link" publish_bf="${publish_bf}" robot_name="${robot_name}" prefix_topic="$(arg topic_namespace)/top_laser" hq="${hq}" range_min="0.1" range_max="90" hfov="360" samples="1200" vfov="90.0" lasers="32" fps="15" gpu="false">
             <origin xyz="0.28 -0.159 1.22" rpy="-1.570796326795 0 -1.570796326795"/>
         </xacro:sensor_rs_bpearl>

File: src/ros2/robot_description/robotnik_sensors/urdf/imu_hector_plugin.urdf.xacro (robot description, xacro)
@@ -39,5 +39,5 @@
 				<update_rate>40</update_rate>
 				<visualize>true</visualize>
-				<topic>${prefix}/imu/data</topic>
+				<topic>${prefix_topic}/imu/data</topic>
 			</sensor>
 		</gazebo>

File: src/ros2/robot_description/robotnik_sensors/urdf/intel_r430.urdf.xacro (robot description, xacro)
@@ -21,8 +21,8 @@
   <xacro:macro name="sensor_r430" params="prefix parent publish_bf robot_name prefix_topic:='front_rgbd_camera' hq *origin">
     <xacro:if value="${publish_bf}">
-			<xacro:property name="sensor_link_name" value="${robot_name}/base_footprint/${prefix}" />
+		<xacro:property name="sensor_link_name" value="base_footprint/${prefix}" /> 	<!--"${robot_name}/base_footprint/${prefix}" /> -->
 		</xacro:if>
 		<xacro:unless value="${publish_bf}">
-			<xacro:property name="sensor_link_name" value="${robot_name}/base_link/${prefix}" />
+			<xacro:property name="sensor_link_name" value="base_link/${prefix}" />      <!-- value="${robot_name}/base_link/${prefix}"  -->
 		</xacro:unless>
     <!-- camera body, with origin at bottom screw mount -->
@@ -148,5 +148,5 @@
       </sensor>
       <sensor name="${prefix}_ired1" type="camera">
-      <topic>${prefix_topic}/${prefix}/ired1</topic>
+      <topic>/${prefix_topic}/${prefix}/ired1</topic>
         <camera name="r430">
           <horizontal_fov>${91.2*M_PI/180.0}</horizontal_fov>

File: src/ros2/robot_description/robotnik_sensors/urdf/rs_bpearl.urdf.xacro (robot description, xacro)
@@ -4,8 +4,8 @@
   <xacro:macro name="sensor_rs_bpearl" params="prefix parent publish_bf robot_name prefix_topic hq *origin range_min range_max hfov samples vfov lasers fps gpu:=true">
     <xacro:if value="${publish_bf}">
-			<xacro:property name="sensor_link_name" value="${robot_name}/base_footprint/${prefix}_link" />
+			<xacro:property name="sensor_link_name" value="base_footprint/${prefix}_link" /> <!-- value="${robot_name}/base_footprint/${prefix}_link" /> -->
 		</xacro:if>
 		<xacro:unless value="${publish_bf}">
-			<xacro:property name="sensor_link_name" value="${robot_name}/base_link/${prefix}_link" />
+			<xacro:property name="sensor_link_name" value="base_link/${prefix}_link" /> <!-- value="${robot_name}/base_link/${prefix}_link" /> -->
 		</xacro:unless>
     <joint name="${prefix}_base_joint" type="fixed">
@@ -74,5 +74,5 @@
       <sensor name='${prefix}_link' type='gpu_lidar'>
         <visualize>true</visualize>
-        <topic>bpearl_laser/scan</topic>
+        <topic>${prefix_topic}/bpearl_laser/scan</topic>
         <update_rate>10</update_rate>
         <ray>

File: src/ros2/robot_description/robotnik_sensors/urdf/sick_nanoscan3.urdf.xacro (robot description, xacro)
@@ -4,8 +4,8 @@
 	<xacro:macro name="sensor_sick_nanoscan3" params="prefix parent publish_bf robot_name prefix_topic:='front_laser' hq *origin max_angle:=2.3998 min_angle:=-2.3998 gpu:=^|false">
 		<xacro:if value="${publish_bf}">
-			<xacro:property name="sensor_link_name" value="${robot_name}/base_footprint/${prefix}_link" />
+			<xacro:property name="sensor_link_name" value="base_footprint/${prefix}_link" /><!-- value="${robot_name}/base_footprint/${prefix}_link" /> -->
 		</xacro:if>
 		<xacro:unless value="${publish_bf}">
-			<xacro:property name="sensor_link_name" value="${robot_name}/base_link/${prefix}_link" />
+			<xacro:property name="sensor_link_name" value="base_link/${prefix}_link" /> <!-- value="${robot_name}/base_link/${prefix}_link" /> -->
 		</xacro:unless>
 		<joint name="${prefix}_base_joint" type="fixed">
