Commit message: build a multi robot launch of the odom to Robot base translation. adjust the multistart launch of the simulation to he same structure

File: src/ros2/robot_description/rb_theron_common/rb_theron_description/robots/rb_theron.urdf.xacro (robot description, xacro)
@@ -132,4 +132,4 @@
 	</xacro:door_opening_mechanism>
 	<!-- Gazebo ros control pluggins -->
-	<xacro:ros_control prefix="$(arg prefix)" publish_bf="${publish_bf}"/>
+	<xacro:ros_control prefix="$(arg prefix)" publish_bf="${publish_bf}" namespace= "$(arg topic_namespace)" />
 </robot>

File: src/ros2/robot_description/rb_theron_common/rb_theron_description/urdf/common.gazebo.xacro (robot description, xacro)
@@ -2,5 +2,5 @@
 <robot xmlns:xacro="http://www.ros.org/wiki/xacro">
 	<!-- ROS CONTROL GAZEBO PLUGIN -->
-	<xacro:macro name="ros_control" params="prefix publish_bf">
+	<xacro:macro name="ros_control" params="prefix publish_bf namespace">
 		<gazebo>
 			<!-- <plugin filename="libgazebo_ros2_control.so" name="gazebo_ros2_control">
@@ -19,11 +19,11 @@
 				<wheel_radius>0.0762</wheel_radius>
 				<odom_publish_frequency>30</odom_publish_frequency>
-				<topic>cmd_vel</topic>
-				<frame_id>$(arg prefix)odom</frame_id>
+				<topic>${namespace}/cmd_vel</topic>
+				<frame_id>${namespace}/$(arg prefix)odom</frame_id>
 				<!-- There is no possiblity (as far as I know) to disable tf publishing of odom->base, so if you
 				don't want the tf to be published, you can just dump it into a different topic -->
 				<tf_topic>tf_dump</tf_topic>
 				<xacro:if value="${publish_bf}">
-					<child_frame_id>$(arg prefix)base_footprint</child_frame_id>
+					<child_frame_id>${namespace}/$(arg prefix)base_footprint</child_frame_id>
 				</xacro:if>
 				<xacro:unless value="${publish_bf}">

Commit message: fix sensor issues
sensor fix

File: src/ros2/robot_description/rb_theron_common/rb_theron_description/robots/rb_theron.urdf.xacro (robot description, xacro)
@@ -42,4 +42,5 @@
 	<!-- *************** -->
 	<xacro:arg name="prefix" default=""/>
+	<xacro:arg name="topic_namespace" default=""/>
 	<!-- Here we create the robot elements using the xacro:macros imported at the beggining of this file -->
 	<!-- this property is for the chassis -->
@@ -63,8 +64,8 @@
 	<!-- TODO: Should be sensor_intel_d435, but this one isn't migrated to ros2 yet -->
 	<!-- TODO: Moved 0.01 in x, otherwise the camera is still inside the robot -->
-	<xacro:sensor_r430 prefix="$(arg prefix)front_realsense_camera" parent="$(arg prefix)base_link" publish_bf="${publish_bf}" robot_name="${robot_name}" prefix_topic="front_realsense_camera" hq="${hq}">
+	<xacro:sensor_r430 prefix="$(arg prefix)front_realsense_camera" parent="$(arg prefix)base_link" publish_bf="${publish_bf}" robot_name="${robot_name}" prefix_topic="$(arg topic_namespace)/front_realsense_camera" hq="${hq}">
 		<origin xyz="0.3305 0.0 0.1468" rpy="0 0 0"/>
 	</xacro:sensor_r430>
-	<xacro:sensor_r430 prefix="$(arg prefix)back_realsense_camera" parent="$(arg prefix)base_link" publish_bf="${publish_bf}" robot_name="${robot_name}" prefix_topic="back_realsense_camera" hq="${hq}">
+	<xacro:sensor_r430 prefix="$(arg prefix)back_realsense_camera" parent="$(arg prefix)base_link" publish_bf="${publish_bf}" robot_name="${robot_name}" prefix_topic="$(arg topic_namespace)/back_realsense_camera" hq="${hq}">
 		<origin xyz="-0.3305 0.0 0.1468" rpy="0 0 3.1416"/>
 	</xacro:sensor_r430>
@@ -73,8 +74,8 @@
 		<origin xyz="0.3305 0.0 0.1898" rpy="0 0 0"/>
 	</xacro:sensor_orbbec_astra -->
-	<xacro:sensor_imu_hector prefix="$(arg prefix)imu" parent="$(arg prefix)base_link">
+	<xacro:sensor_imu_hector prefix="$(arg prefix)imu" parent="$(arg prefix)base_link" prefix_topic="$(arg topic_namespace)/imu">
 		<origin xyz="-0.1975 0.0 0.1598" rpy="0 0 0"/>
 	</xacro:sensor_imu_hector>
-	<xacro:sensor_sick_nanoscan3 prefix="$(arg prefix)front_laser" parent="$(arg prefix)base_link" publish_bf="${publish_bf}" robot_name="${robot_name}" prefix_topic="front_laser" hq="${hq}" min_angle="-1.9507619" max_angle="1.9507619" gpu="true">
+	<xacro:sensor_sick_nanoscan3 prefix="$(arg prefix)front_laser" parent="$(arg prefix)base_link" publish_bf="${publish_bf}" robot_name="${robot_name}" prefix_topic="$(arg topic_namespace)/front_laser" hq="${hq}" min_angle="-1.9507619" max_angle="1.9507619" gpu="true">
 		<origin xyz="0.250 0.0 0.1643" rpy="0 3.1416 3.1416"/>
 	</xacro:sensor_sick_nanoscan3>
@@ -82,5 +83,5 @@
 		<origin xyz="0.214 0.0 0.275" rpy="-1.57079632679 0 -0.23"/>
 	</xacro:sensor_rs_lidar_16>-->
-	<xacro:sensor_rs_bpearl prefix="$(arg prefix)top_laser"  parent="$(arg prefix)base_link" publish_bf="${publish_bf}" robot_name="${robot_name}" prefix_topic="top_laser" hq="${hq}" range_min="0.1" range_max="90" hfov="360" samples="1800" vfov="90.0" lasers="32" fps="10" gpu="false">
+	<xacro:sensor_rs_bpearl prefix="$(arg prefix)top_laser"  parent="$(arg prefix)base_link" publish_bf="${publish_bf}" robot_name="${robot_name}" prefix_topic="$(arg topic_namespace)/top_laser" hq="${hq}" range_min="0.1" range_max="90" hfov="360" samples="1800" vfov="90.0" lasers="32" fps="10" gpu="false">
             <origin xyz="0.28 -0.159 1.22" rpy="-1.570796326795 0 -1.570796326795"/>
         </xacro:sensor_rs_bpearl>
@@ -88,10 +89,5 @@
 		<origin xyz="-0.250 0.0 0.1643" rpy="0 3.1416 0"/>
 	</xacro:sensor_sick_nanoscan3> -->
-	<gazebo>
-		<plugin name="gz::sim::systems::Sensors" filename="libgz-sim-sensors-system.so">
-			<render_engine>ogre2</render_engine>
-		</plugin>
-	</gazebo>
-    <xacro:arg name="back_oak_d_camera_model"  default="OAK-D-POE" />
+	<xacro:arg name="back_oak_d_camera_model"  default="OAK-D-POE" />
     <xacro:arg name="back_oak_d_base_frame"    default="oak-d-s2-poe-base-frame" />
     <xacro:arg name="back_oak_d_pos_x"     	   default="-0.3305" />
@@ -139,4 +135,4 @@
 	</xacro:door_opening_mechanism>
 	<!-- Gazebo ros control pluggins -->
-	<xacro:ros_control prefix="$(arg prefix)" publish_bf="${publish_bf}"/>
+	<xacro:ros_control prefix="$(arg prefix)" publish_bf="${publish_bf}" namespace= "$(arg topic_namespace)" />
 </robot>

File: src/ros2/robot_description/robotnik_sensors/urdf/imu_hector_plugin.urdf.xacro (robot description, xacro)
@@ -1,10 +1,10 @@
 <?xml version="1.0"?>
 <robot name="sensor_imu" xmlns:xacro="http://wiki.ros.org/xacro">
-	<xacro:macro name="sensor_imu_hector" params="prefix topic:='imu/data' parent *origin">
+	<xacro:macro name="sensor_imu_hector" params="prefix prefix_topic topic:='imu/data' parent *origin">
 		<xacro:if value="${publish_bf}">
-			<xacro:property name="sensor_link_name" value="${robot_name}/base_footprint/${prefix}_link" />
+			<xacro:property name="sensor_link_name" value="base_footprint/${prefix}_link" />
 		</xacro:if>
 		<xacro:unless value="${publish_bf}">
-			<xacro:property name="sensor_link_name" value="${robot_name}/base_link/${prefix}_link" />
+			<xacro:property name="sensor_link_name" value="base_link/${prefix}_link" />
 		</xacro:unless>
 		<joint name="${prefix}_joint" type="fixed">

Commit message: changed front oak position as well as B-Pearl based on CAD and reallife testing

File: src/ros2/robot_description/rb_theron_common/rb_theron_description/robots/rb_theron.urdf.xacro (robot description, xacro)
@@ -69,5 +69,5 @@
 		<origin xyz="-0.3305 0.0 0.1468" rpy="0 0 3.1416"/>
 	</xacro:sensor_r430>
-  	<!-- TODO: Moved 0.01 in x, otherwise the camera is still inside the robot -->
+	<!-- TODO: Moved 0.01 in x, otherwise the camera is still inside the robot -->
 	<!--xacro:sensor_orbbec_astra prefix="$(arg prefix)front_rgbd_camera" parent="$(arg prefix)base_link" prefix_topic="front_rgbd_camera">
 		<origin xyz="0.3305 0.0 0.1898" rpy="0 0 0"/>
@@ -82,7 +82,8 @@
 		<origin xyz="0.214 0.0 0.275" rpy="-1.57079632679 0 -0.23"/>
 	</xacro:sensor_rs_lidar_16>-->
-	<xacro:sensor_rs_bpearl prefix="$(arg prefix)top_laser"  parent="$(arg prefix)base_link" publish_bf="${publish_bf}" robot_name="${robot_name}" prefix_topic="top_laser" hq="${hq}" range_min="0.1" range_max="90" hfov="360" samples="1800" vfov="90.0" lasers="32" fps="10" gpu="false">
-            <origin xyz="0.28 -0.159 1.22" rpy="-1.570796326795 0 -1.570796326795"/>
-        </xacro:sensor_rs_bpearl>
+	<xacro:sensor_rs_bpearl prefix="$(arg prefix)top_laser" parent="$(arg prefix)base_link" publish_bf="${publish_bf}" robot_name="${robot_name}" prefix_topic="top_laser" hq="${hq}" range_min="0.1" range_max="90" hfov="360" samples="1800" vfov="90.0" lasers="32" fps="10" gpu="false">
+		<origin xyz="0.17 -0.175 1.165" rpy="-1.570796326795 0 -1.570796326795"/>
+		<!-- positions of the b-pearl based on solid: xyz="0.333 -0.180 1.194" rpy="-1.570796326795 0 -1.570796326795" -->
+	</xacro:sensor_rs_bpearl>
 	<!-- <xacro:sensor_sick_nanoscan3 prefix="$(arg prefix)back_laser" parent="$(arg prefix)base_link" prefix_topic="back_laser" min_angle="-1.8107619" max_angle="1.8107619">
 		<origin xyz="-0.250 0.0 0.1643" rpy="0 3.1416 0"/>
@@ -93,25 +94,25 @@
 		</plugin>
 	</gazebo>
-    <xacro:arg name="back_oak_d_camera_model"  default="OAK-D-POE" />
-    <xacro:arg name="back_oak_d_base_frame"    default="oak-d-s2-poe-base-frame" />
-    <xacro:arg name="back_oak_d_pos_x"     	   default="-0.3305" />
-    <xacro:arg name="back_oak_d_pos_y"         default="0.0" />
-    <xacro:arg name="back_oak_d_pos_z"         default="1.1468" />
-    <xacro:arg name="back_oak_d_roll"          default="0.0" />
-    <xacro:arg name="back_oak_d_pitch"         default="0.0" />
-    <xacro:arg name="back_oak_d_yaw"           default="3.1416" />
-    <xacro:depthai_camera prefix="$(arg prefix)back_top_oak_d_camera" parent="$(arg prefix)base_link" publish_bf="${publish_bf}" robot_name="${robot_name}" prefix_topic="back_top_oak_d_camera" camera_model = "$(arg back_oak_d_camera_model)" base_frame = "$(arg back_oak_d_base_frame)" cam_pos_x = "$(arg back_oak_d_pos_x)" cam_pos_y = "$(arg back_oak_d_pos_y)" cam_pos_z = "$(arg back_oak_d_pos_z)" cam_roll = "$(arg back_oak_d_roll)" cam_pitch = "$(arg back_oak_d_pitch)" cam_yaw = "$(arg back_oak_d_yaw)"/>
-	<xacro:arg name="front_oak_d_camera_model"  default="OAK-D-S2" />
-    <xacro:arg name="front_oak_d_base_frame"    default="oak-d-s2-usb-base--frame" />
-    <xacro:arg name="front_oak_d_pos_x"         default="0.3305" />
-    <xacro:arg name="front_oak_d_pos_y"         default="0.0" />
-    <xacro:arg name="front_oak_d_pos_z"         default="1.1468" />
-    <xacro:arg name="front_oak_d_roll"          default="0.0" />
-    <xacro:arg name="front_oak_d_pitch"         default="0.0" />
-    <xacro:arg name="front_oak_d_yaw"           default="0.0" />
+	<xacro:arg name="back_oak_d_camera_model" default="OAK-D-POE" />
+	<xacro:arg name="back_oak_d_base_frame" default="oak-d-s2-poe-base-frame" />
+	<xacro:arg name="back_oak_d_pos_x" default="-0.3305" />
+	<xacro:arg name="back_oak_d_pos_y" default="0.0" />
+	<xacro:arg name="back_oak_d_pos_z" default="1.1468" />
+	<xacro:arg name="back_oak_d_roll" default="0.0" />
+	<xacro:arg name="back_oak_d_pitch" default="0.0" />
+	<xacro:arg name="back_oak_d_yaw" default="3.1416" />
+	<xacro:depthai_camera prefix="$(arg prefix)back_top_oak_d_camera" parent="$(arg prefix)base_link" publish_bf="${publish_bf}" robot_name="${robot_name}" prefix_topic="back_top_oak_d_camera" camera_model = "$(arg back_oak_d_camera_model)" base_frame = "$(arg back_oak_d_base_frame)" cam_pos_x = "$(arg back_oak_d_pos_x)" cam_pos_y = "$(arg back_oak_d_pos_y)" cam_pos_z = "$(arg back_oak_d_pos_z)" cam_roll = "$(arg back_oak_d_roll)" cam_pitch = "$(arg back_oak_d_pitch)" cam_yaw = "$(arg back_oak_d_yaw)"/>
+	<xacro:arg name="front_oak_d_camera_model" default="OAK-D-S2" />
+	<xacro:arg name="front_oak_d_base_frame" default="oak-d-s2-usb-base--frame" />
+	<xacro:arg name="front_oak_d_pos_x" default="0.317" />
+	<xacro:arg name="front_oak_d_pos_y" default="-0.197" />
+	<xacro:arg name="front_oak_d_pos_z" default="1.3044" />
+	<xacro:arg name="front_oak_d_roll" default="0.0" />
+	<xacro:arg name="front_oak_d_pitch" default="0.0" />
+	<xacro:arg name="front_oak_d_yaw" default="0.0" />
 	<xacro:depthai_camera prefix="$(arg prefix)front_top_oak_d_camera" parent="$(arg prefix)base_link" publish_bf="${publish_bf}" robot_name="${robot_name}" prefix_topic="front_top_oak_d_camera" camera_model = "$(arg front_oak_d_camera_model)" base_frame = "$(arg front_oak_d_base_frame)" cam_pos_x = "$(arg front_oak_d_pos_x)" cam_pos_y = "$(arg front_oak_d_pos_y)" cam_pos_z = "$(arg front_oak_d_pos_z)" cam_roll = "$(arg front_oak_d_roll)" cam_pitch = "$(arg front_oak_d_pitch)" cam_yaw = "$(arg front_oak_d_yaw)"/>
 	<!-- ROBAST Module Cage -->
 	<xacro:include filename="$(find rb_theron_description)/urdf/module_cage/module_cage.urdf.xacro" />
-	<xacro:module_cage prefix="$(arg prefix)" parent="$(arg prefix)base_link" hq="${hq}" >
+	<xacro:module_cage prefix="$(arg prefix)" parent="$(arg prefix)base_link" hq="${hq}">
 		<origin xyz="-0.15 0.0 0.725" rpy="0 0 0"/>
 	</xacro:module_cage>
@@ -135,5 +136,5 @@
 	<!-- ROBAST Door Opening Mechanism -->
 	<xacro:include filename="$(find rb_theron_description)/urdf/door_opening_mechanism/door_opening_mechanism.urdf.xacro" />
-	<xacro:door_opening_mechanism prefix="$(arg prefix)" parent="$(arg prefix)base_link" hq="${hq}" >
+	<xacro:door_opening_mechanism prefix="$(arg prefix)" parent="$(arg prefix)base_link" hq="${hq}">
 		<origin xyz="-0.3 0 0.225" rpy="0 0 0"/>
 	</xacro:door_opening_mechanism>

Commit message: Some test changes

File: src/ros2/robot_description/rb_theron_common/rb_theron_description/robots/rb_theron.urdf.xacro (robot description, xacro)
@@ -64,5 +64,5 @@
 	<!-- TODO: Moved 0.01 in x, otherwise the camera is still inside the robot -->
 	<xacro:sensor_r430 prefix="$(arg prefix)front_realsense_camera" parent="$(arg prefix)base_link" publish_bf="${publish_bf}" robot_name="${robot_name}" prefix_topic="front_realsense_camera" hq="${hq}">
-		<origin xyz="0.3305 0.0 0.1468" rpy="0 0 0"/>
+		<origin xyz="0.3305 0.0 1.1468" rpy="0 0 0"/>
 	</xacro:sensor_r430>
 	<xacro:sensor_r430 prefix="$(arg prefix)back_realsense_camera" parent="$(arg prefix)base_link" publish_bf="${publish_bf}" robot_name="${robot_name}" prefix_topic="back_realsense_camera" hq="${hq}">
@@ -93,22 +93,4 @@
 		</plugin>
 	</gazebo>
-    <xacro:arg name="back_oak_d_camera_model"  default="OAK-D-POE" />
-    <xacro:arg name="back_oak_d_base_frame"    default="oak-d-s2-poe-base-frame" />
-    <xacro:arg name="back_oak_d_pos_x"     	   default="-0.3305" />
-    <xacro:arg name="back_oak_d_pos_y"         default="0.0" />
-    <xacro:arg name="back_oak_d_pos_z"         default="1.1468" />
-    <xacro:arg name="back_oak_d_roll"          default="0.0" />
-    <xacro:arg name="back_oak_d_pitch"         default="0.0" />
-    <xacro:arg name="back_oak_d_yaw"           default="3.1416" />
-    <xacro:depthai_camera prefix="$(arg prefix)back_top_oak_d_camera" parent="$(arg prefix)base_link" publish_bf="${publish_bf}" robot_name="${robot_name}" prefix_topic="back_top_oak_d_camera" camera_model = "$(arg back_oak_d_camera_model)" base_frame = "$(arg back_oak_d_base_frame)" cam_pos_x = "$(arg back_oak_d_pos_x)" cam_pos_y = "$(arg back_oak_d_pos_y)" cam_pos_z = "$(arg back_oak_d_pos_z)" cam_roll = "$(arg back_oak_d_roll)" cam_pitch = "$(arg back_oak_d_pitch)" cam_yaw = "$(arg back_oak_d_yaw)"/>
-	<xacro:arg name="front_oak_d_camera_model"  default="OAK-D-S2" />
-    <xacro:arg name="front_oak_d_base_frame"    default="oak-d-s2-usb-base--frame" />
-    <xacro:arg name="front_oak_d_pos_x"         default="0.3305" />
-    <xacro:arg name="front_oak_d_pos_y"         default="0.0" />
-    <xacro:arg name="front_oak_d_pos_z"         default="1.1468" />
-    <xacro:arg name="front_oak_d_roll"          default="0.0" />
-    <xacro:arg name="front_oak_d_pitch"         default="0.0" />
-    <xacro:arg name="front_oak_d_yaw"           default="0.0" />
-	<xacro:depthai_camera prefix="$(arg prefix)front_top_oak_d_camera" parent="$(arg prefix)base_link" publish_bf="${publish_bf}" robot_name="${robot_name}" prefix_topic="front_top_oak_d_camera" camera_model = "$(arg front_oak_d_camera_model)" base_frame = "$(arg front_oak_d_base_frame)" cam_pos_x = "$(arg front_oak_d_pos_x)" cam_pos_y = "$(arg front_oak_d_pos_y)" cam_pos_z = "$(arg front_oak_d_pos_z)" cam_roll = "$(arg front_oak_d_roll)" cam_pitch = "$(arg front_oak_d_pitch)" cam_yaw = "$(arg front_oak_d_yaw)"/>
 	<!-- ROBAST Module Cage -->
 	<xacro:include filename="$(find rb_theron_description)/urdf/module_cage/module_cage.urdf.xacro" />

File: src/ros2/robot_description/robotnik_sensors/urdf/depthai_macro.urdf.xacro (robot description, xacro)
@@ -108,6 +108,6 @@
             <horizontal_fov>1.2112585008840648</horizontal_fov>
             <image>
-                <width>1280</width>
-                <height>720</height>
+                <width>640</width>
+                <height>480</height>
                 <format>RGB_INT8</format>
             </image>

File: src/ros2/robot_description/robotnik_sensors/urdf/intel_r430.urdf.xacro (robot description, xacro)
@@ -130,5 +130,5 @@
             <image>
                 <width>640</width>
-                <height>480</height>
+                <height>640</height>
                 <format>RGB_INT8</format>
             </image>

Commit message: Added door_handle detection for simulation

File: src/ros2/robot_description/rb_theron_common/rb_theron_description/robots/rb_theron.urdf.xacro (robot description, xacro)
@@ -64,10 +64,13 @@
 	<!-- TODO: Moved 0.01 in x, otherwise the camera is still inside the robot -->
 	<xacro:sensor_r430 prefix="$(arg prefix)front_realsense_camera" parent="$(arg prefix)base_link" publish_bf="${publish_bf}" robot_name="${robot_name}" prefix_topic="front_realsense_camera" hq="${hq}">
-		<origin xyz="0.3305 0.0 1.1468" rpy="0 0 0"/>
+		<origin xyz="0.3305 0.0 0.1468" rpy="0 0 0"/>
 	</xacro:sensor_r430>
 	<xacro:sensor_r430 prefix="$(arg prefix)back_realsense_camera" parent="$(arg prefix)base_link" publish_bf="${publish_bf}" robot_name="${robot_name}" prefix_topic="back_realsense_camera" hq="${hq}">
 		<origin xyz="-0.3305 0.0 0.1468" rpy="0 0 3.1416"/>
 	</xacro:sensor_r430>
-  	<!-- TODO: Moved 0.01 in x, otherwise the camera is still inside the robot -->
+	<xacro:sensor_r430 prefix="$(arg prefix)back_top_realsense_camera" parent="$(arg prefix)base_link" publish_bf="${publish_bf}" robot_name="${robot_name}" prefix_topic="back_top_realsense_camera" hq="${hq}">
+		<origin xyz="-0.3305 0.0 1.1468" rpy="0 0 3.1416"/>
+	</xacro:sensor_r430>
+	<!-- TODO: Moved 0.01 in x, otherwise the camera is still inside the robot -->
 	<!--xacro:sensor_orbbec_astra prefix="$(arg prefix)front_rgbd_camera" parent="$(arg prefix)base_link" prefix_topic="front_rgbd_camera">
 		<origin xyz="0.3305 0.0 0.1898" rpy="0 0 0"/>
@@ -82,7 +85,8 @@
 		<origin xyz="0.214 0.0 0.275" rpy="-1.57079632679 0 -0.23"/>
 	</xacro:sensor_rs_lidar_16>-->
-	<xacro:sensor_rs_bpearl prefix="$(arg prefix)top_laser"  parent="$(arg prefix)base_link" publish_bf="${publish_bf}" robot_name="${robot_name}" prefix_topic="top_laser" hq="${hq}" range_min="0.1" range_max="90" hfov="360" samples="1800" vfov="90.0" lasers="32" fps="10" gpu="false">
-            <origin xyz="0.28 -0.159 1.22" rpy="-1.570796326795 0 -1.570796326795"/>
-        </xacro:sensor_rs_bpearl>
+	<xacro:sensor_rs_bpearl prefix="$(arg prefix)top_laser" parent="$(arg prefix)base_link" publish_bf="${publish_bf}" robot_name="${robot_name}" prefix_topic="top_laser" hq="${hq}" range_min="0.1" range_max="90" hfov="360" samples="1800" vfov="90.0" lasers="32" fps="10" gpu="false">
+		<origin xyz="0.17 -0.175 1.165" rpy="-1.570796326795 0 -1.570796326795"/>
+		<!-- positions of the b-pearl based on solid: xyz="0.333 -0.180 1.194" rpy="-1.570796326795 0 -1.570796326795" -->
+	</xacro:sensor_rs_bpearl>
 	<!-- <xacro:sensor_sick_nanoscan3 prefix="$(arg prefix)back_laser" parent="$(arg prefix)base_link" prefix_topic="back_laser" min_angle="-1.8107619" max_angle="1.8107619">
 		<origin xyz="-0.250 0.0 0.1643" rpy="0 3.1416 0"/>
@@ -93,7 +97,16 @@
 		</plugin>
 	</gazebo>
+	<xacro:arg name="front_oak_d_camera_model" default="OAK-D-S2" />
+	<xacro:arg name="front_oak_d_base_frame" default="oak-d-s2-usb-base--frame" />
+	<xacro:arg name="front_oak_d_pos_x" default="0.317" />
+	<xacro:arg name="front_oak_d_pos_y" default="-0.197" />
+	<xacro:arg name="front_oak_d_pos_z" default="1.3044" />
+	<xacro:arg name="front_oak_d_roll" default="0.0" />
+	<xacro:arg name="front_oak_d_pitch" default="0.0" />
+	<xacro:arg name="front_oak_d_yaw" default="0.0" />
+	<xacro:depthai_camera prefix="$(arg prefix)front_top_oak_d_camera" parent="$(arg prefix)base_link" publish_bf="${publish_bf}" robot_name="${robot_name}" prefix_topic="front_top_oak_d_camera" camera_model = "$(arg front_oak_d_camera_model)" base_frame = "$(arg front_oak_d_base_frame)" cam_pos_x = "$(arg front_oak_d_pos_x)" cam_pos_y = "$(arg front_oak_d_pos_y)" cam_pos_z = "$(arg front_oak_d_pos_z)" cam_roll = "$(arg front_oak_d_roll)" cam_pitch = "$(arg front_oak_d_pitch)" cam_yaw = "$(arg front_oak_d_yaw)"/>
 	<!-- ROBAST Module Cage -->
 	<xacro:include filename="$(find rb_theron_description)/urdf/module_cage/module_cage.urdf.xacro" />
-	<xacro:module_cage prefix="$(arg prefix)" parent="$(arg prefix)base_link" hq="${hq}" >
+	<xacro:module_cage prefix="$(arg prefix)" parent="$(arg prefix)base_link" hq="${hq}">
 		<origin xyz="-0.15 0.0 0.725" rpy="0 0 0"/>
 	</xacro:module_cage>
@@ -117,5 +130,5 @@
 	<!-- ROBAST Door Opening Mechanism -->
 	<xacro:include filename="$(find rb_theron_description)/urdf/door_opening_mechanism/door_opening_mechanism.urdf.xacro" />
-	<xacro:door_opening_mechanism prefix="$(arg prefix)" parent="$(arg prefix)base_link" hq="${hq}" >
+	<xacro:door_opening_mechanism prefix="$(arg prefix)" parent="$(arg prefix)base_link" hq="${hq}">
 		<origin xyz="-0.3 0 0.225" rpy="0 0 0"/>
 	</xacro:door_opening_mechanism>

File: src/ros2/robot_description/robotnik_sensors/urdf/intel_r430.urdf.xacro (robot description, xacro)
@@ -130,5 +130,5 @@
             <image>
                 <width>640</width>
-                <height>640</height>
+                <height>480</height>
                 <format>RGB_INT8</format>
             </image>

Commit message: tmp

File: src/ros2/robot_description/rb_theron_common/rb_theron_description/robots/rb_theron.urdf.xacro (robot description, xacro)
@@ -83,5 +83,5 @@
 	</xacro:sensor_rs_lidar_16>-->
 	<xacro:sensor_rs_bpearl prefix="$(arg prefix)top_laser" parent="$(arg prefix)base_link" publish_bf="${publish_bf}" robot_name="${robot_name}" prefix_topic="top_laser" hq="${hq}" range_min="0.1" range_max="90" hfov="360" samples="1800" vfov="90.0" lasers="32" fps="10" gpu="false">
-		<origin xyz="0.17 -0.175 1.165" rpy="-1.570796326795 0 -1.570796326795"/>
+		<origin xyz="0.3 -0.175 1.165" rpy="-1.570796326795 0 -1.570796326795"/>
 		<!-- positions of the b-pearl based on solid: xyz="0.333 -0.180 1.194" rpy="-1.570796326795 0 -1.570796326795" -->
 	</xacro:sensor_rs_bpearl>
