Commit message: feat: humble works now with fortress and iron with garden

File: src/ros2/robot_description/rb_theron_common/rb_theron_description/robots/rb_theron.urdf.xacro (robot description, xacro)
@@ -34,4 +34,5 @@
 	-->
     <xacro:arg name="ros2_control_hardware_type" default="mock_components" />
+	<xacro:arg name="ros_distro" default="humble" />
 	<!-- *************** -->
 	<!-- Robots Elements -->
@@ -42,5 +43,6 @@
 	  hq="${hq}"
 	  publish_bf="${publish_bf}"
-	  ros2_control_hardware_type="$(arg ros2_control_hardware_type)">
+	  ros2_control_hardware_type="$(arg ros2_control_hardware_type)"
+	  ros_distro="$(arg ros_distro)">
 	</xacro:rb_theron_base>
 	<!-- Gazebo ros control pluggins -->
@@ -80,9 +82,4 @@
 		<origin xyz="-0.250 0.0 0.1643" rpy="0 3.1416 0"/>
 	</xacro:sensor_sick_nanoscan3> -->
-	<gazebo>
-		<plugin name="gz::sim::systems::Sensors" filename="libgz-sim-sensors-system.so">
-			<render_engine>ogre2</render_engine>
-		</plugin>
-	</gazebo>
 	<xacro:arg name="front_oak_d_camera_model" default="OAK-D-S2" />
 	<xacro:arg name="front_oak_d_base_frame" default="oak-d-s2-usb-base--frame" />
@@ -106,4 +103,5 @@
 		parent="$(arg prefix)base_link"
 		ros2_control_hardware_type="$(arg ros2_control_hardware_type)"
+		ros_distro="$(arg ros_distro)"
 		drawer_size_z="0.28">
 		<origin xyz="0.125 0.0 0.42" rpy="0 0 0"/>
@@ -114,4 +112,5 @@
 		parent="$(arg prefix)base_link"
 		ros2_control_hardware_type="$(arg ros2_control_hardware_type)"
+		ros_distro="$(arg ros_distro)"
 		drawer_size_z="0.18">
 		<origin xyz="0.125 0.0 0.67" rpy="0 0 0"/>
@@ -122,4 +121,5 @@
 		parent="$(arg prefix)base_link"
 		ros2_control_hardware_type="$(arg ros2_control_hardware_type)"
+		ros_distro="$(arg ros_distro)"
 		drawer_size_z="0.08">
 		<origin xyz="0.125 0.0 0.82" rpy="0 0 0"/>
@@ -130,4 +130,5 @@
 		parent="$(arg prefix)base_link"
 		ros2_control_hardware_type="$(arg ros2_control_hardware_type)"
+		ros_distro="$(arg ros_distro)"
 		drawer_size_z="0.08">
 		<origin xyz="0.125 0.0 0.92" rpy="0 0 0"/>
@@ -138,4 +139,5 @@
 		parent="$(arg prefix)base_link"
 		ros2_control_hardware_type="$(arg ros2_control_hardware_type)"
+		ros_distro="$(arg ros_distro)"
 		drawer_size_z="0.08">
 		<origin xyz="0.125 0.0 1.02" rpy="0 0 0"/>
@@ -147,8 +149,10 @@
 		parent="$(arg prefix)base_link"
 		ros2_control_hardware_type="$(arg ros2_control_hardware_type)"
+		ros_distro="$(arg ros_distro)"
 		hq="${hq}">
 		<origin xyz="-0.3 0 0.225" rpy="0 0 0"/>
 	</xacro:door_opening_mechanism>
-	<!-- Gazebo ros control pluggins -->
-	<xacro:ros_control prefix="$(arg prefix)" publish_bf="${publish_bf}"/>
+	<!-- Gazebo plugins -->
+	<xacro:ros_control ros_distro="$(arg ros_distro)"/>
+	<xacro:gazebo_sensor_plugins ros_distro="$(arg ros_distro)"/>
 </robot>

File: src/ros2/robot_description/rb_theron_common/rb_theron_description/robots/rb_theron_base.urdf.xacro (robot description, xacro)
@@ -20,5 +20,5 @@
   <!-- Robots Elements -->
   <!-- *************** -->
-  <xacro:macro name="rb_theron_base" params="prefix hq publish_bf ros2_control_hardware_type">
+  <xacro:macro name="rb_theron_base" params="prefix hq publish_bf ros2_control_hardware_type ros_distro">
     <xacro:theron_base prefix="${prefix}" publish_bf="${publish_bf}" hq="${hq}" />
     <xacro:gazebo_colors prefix="${prefix}"/>
@@ -28,4 +28,5 @@
       parent="${prefix}base_link"
       ros2_control_hardware_type="${ros2_control_hardware_type}"
+      ros_distro="${ros_distro}"
       hq="${hq}">
       <origin xyz="${wheel_offset_x} ${-wheel_offset_y} ${wheel_offset_z}" rpy="0 0 0"/>
@@ -35,4 +36,5 @@
       parent="${prefix}base_link"
       ros2_control_hardware_type="${ros2_control_hardware_type}"
+      ros_distro="${ros_distro}"
       hq="${hq}">
       <origin xyz="${wheel_offset_x} ${wheel_offset_y} ${wheel_offset_z}" rpy="0 0 0"/>
@@ -43,4 +45,5 @@
       parent="${prefix}base_link"
       ros2_control_hardware_type="${ros2_control_hardware_type}"
+      ros_distro="${ros_distro}"
       hq="${hq}">
       <origin xyz="0.235 0.1825 0.046" rpy="0 0 0"/>
@@ -50,4 +53,5 @@
       parent="${prefix}base_link"
       ros2_control_hardware_type="${ros2_control_hardware_type}"
+      ros_distro="${ros_distro}"
       hq="${hq}">
       <origin xyz="0.235 -0.1825 0.046" rpy="0 0 0"/>
@@ -57,4 +61,5 @@
       parent="${prefix}base_link"
       ros2_control_hardware_type="${ros2_control_hardware_type}"
+      ros_distro="${ros_distro}"
       hq="${hq}">
       <origin xyz="-0.235 0.1825 0.046" rpy="0 0 0"/>
@@ -64,4 +69,5 @@
       parent="${prefix}base_link"
       ros2_control_hardware_type="${ros2_control_hardware_type}"
+      ros_distro="${ros_distro}"
       hq="${hq}">
       <origin xyz="-0.235 -0.1825 0.046" rpy="0 0 0"/>

File: src/ros2/robot_description/rb_theron_common/rb_theron_description/urdf/common.gazebo.xacro (robot description, xacro)
@@ -2,10 +2,33 @@
 <robot xmlns:xacro="http://www.ros.org/wiki/xacro">
     <!-- ROS CONTROL GAZEBO PLUGIN -->
-    <xacro:macro name="ros_control" params="prefix publish_bf">
+    <xacro:macro name="ros_control" params="ros_distro">
         <gazebo>
-            <plugin name="gz_ros2_control::GazeboSimROS2ControlPlugin" filename="gz_ros2_control-system">
-                <parameters>$(find rb_theron_description)/config/rb_theron_gz_ros2_controller.yaml</parameters>
-            </plugin>
+            <xacro:if value="${ros_distro == 'humble'}">
+                <plugin name="ign_ros2_control::IgnitionROS2ControlPlugin" filename="libign_ros2_control-system.so">
+                    <parameters>$(find rb_theron_description)/config/rb_theron_gz_ros2_controller.yaml</parameters>
+                </plugin>
+            </xacro:if>
+            <xacro:unless value="${ros_distro == 'humble'}">
+                <plugin name="gz_ros2_control::GazeboSimROS2ControlPlugin" filename="gz_ros2_control-system">
+                    <parameters>$(find rb_theron_description)/config/rb_theron_gz_ros2_controller.yaml</parameters>
+                </plugin>
+            </xacro:unless>
         </gazebo>
+    </xacro:macro>
+    <xacro:macro name="gazebo_sensor_plugins" params="ros_distro">
+        <gazebo>
+            <xacro:if value="${ros_distro == 'humble'}">
+                <plugin name="ignition::gazebo::systems::Imu" filename="libignition-gazebo-imu-system.so"></plugin>
+                <plugin name="ignition::gazebo::systems::Sensors" filename="libignition-gazebo-sensors-system.so">
+                    <render_engine>ogre2</render_engine>
+                </plugin>
+            </xacro:if>
+            <xacro:unless value="${ros_distro == 'humble'}">
+                <plugin name="gz::sim::systems::Imu" filename="libgz-sim-imu-system"></plugin>
+                <plugin name="gz::sim::systems::Sensors" filename="libgz-sim-sensors-system.so">
+                    <render_engine>ogre2</render_engine>
+                </plugin>
+            </xacro:unless>
+		</gazebo>
     </xacro:macro>
     <xacro:macro name="gazebo_colors" params="prefix">

File: src/ros2/robot_description/rb_theron_common/rb_theron_description/urdf/door_opening_mechanism/arm_variations/rotating_arm.urdf.xacro (robot description, xacro)
@@ -6,5 +6,5 @@
                 izz="${m*(x*x+y*y)/12}" />
     </xacro:macro>
-    <xacro:macro name="rotating_arm" params="prefix parent ros2_control_hardware_type *origin arm_length">
+    <xacro:macro name="rotating_arm" params="prefix parent ros2_control_hardware_type ros_distro *origin arm_length">
         <xacro:basic_joint
             parent="${prefix}${parent}"
@@ -21,4 +21,5 @@
             port="0"
             direction="0"
+            ros_distro="${ros_distro}"
             link_name="${prefix}door_opening_mechanism_link_rotating_arm"
             link_origin_x="0.0"
@@ -55,5 +56,6 @@
             prefix="${prefix}"
             parent="${prefix}door_opening_mechanism_link_gripper_adapter"
-            ros2_control_hardware_type="${ros2_control_hardware_type}">
+            ros2_control_hardware_type="${ros2_control_hardware_type}"
+            ros_distro="${ros_distro}">
             <origin xyz="0.020 0.0 0.0" rpy="0 0 0"/>
         </xacro:freely_rotating_hook>

File: src/ros2/robot_description/rb_theron_common/rb_theron_description/urdf/door_opening_mechanism/arm_variations/tilting_arm.urdf.xacro (robot description, xacro)
@@ -6,5 +6,5 @@
                 izz="${m*(x*x+y*y)/12}" />
     </xacro:macro>
-    <xacro:macro name="tilting_arm" params="prefix parent ros2_control_hardware_type *origin">
+    <xacro:macro name="tilting_arm" params="prefix parent ros2_control_hardware_type ros_distro *origin">
         <xacro:basic_joint
             parent="${prefix}${parent}"
@@ -19,4 +19,7 @@
             friction="0.3"
             ros2_control_hardware_type="${ros2_control_hardware_type}"
+            port="0"
+            direction="0"
+            ros_distro="ros_distro"
             link_name="${prefix}door_opening_mechanism_link_tilting_hook"
             link_origin_x="0.0"

File: src/ros2/robot_description/rb_theron_common/rb_theron_description/urdf/door_opening_mechanism/basic_elements/basic_joint.urdf.xacro (robot description, xacro)
@@ -5,5 +5,5 @@
         <inertia ixx="${m*(y*y+z*z)/12}" ixy = "0" ixz = "0" iyy="${m*(x*x+z*z)/12}" iyz = "0" izz="${m*(x*x+y*y)/12}" />
     </xacro:macro>
-    <xacro:macro name="basic_joint" params="parent joint_name joint_type axis_x axis_y axis_z lower_limit upper_limit damping friction ros2_control_hardware_type port direction link_name link_origin_x link_origin_y link_origin_z m x y z r g b *origin">
+    <xacro:macro name="basic_joint" params="parent joint_name joint_type axis_x axis_y axis_z lower_limit upper_limit damping friction ros2_control_hardware_type port direction ros_distro link_name link_origin_x link_origin_y link_origin_z m x y z r g b *origin">
         <joint name="${joint_name}" type="${joint_type}">
             <axis xyz="${axis_x} ${axis_y} ${axis_z}" />
@@ -21,5 +21,10 @@
                 </xacro:if>
                 <xacro:if value="${ros2_control_hardware_type == 'gz_ros2_control'}">
-                    <plugin>gz_ros2_control/GazeboSimSystem</plugin>
+                    <xacro:if value="${ros_distro == 'humble'}">
+                        <plugin>ign_ros2_control/IgnitionSystem</plugin>
+                    </xacro:if>
+                    <xacro:unless value="${ros_distro == 'humble'}">
+                        <plugin>gz_ros2_control/GazeboSimSystem</plugin>
+                    </xacro:unless>
                 </xacro:if>
                 <xacro:if value="${ros2_control_hardware_type == 'dryve_d1'}">

File: src/ros2/robot_description/rb_theron_common/rb_theron_description/urdf/door_opening_mechanism/components/freely_rotating_hook.urdf.xacro (robot description, xacro)
@@ -1,5 +1,5 @@
 <?xml version="1.0"?>
 <robot name="freely_rotating_hook" xmlns:xacro="http://www.ros.org/wiki/xacro">
-    <xacro:macro name="freely_rotating_hook" params="prefix parent ros2_control_hardware_type *origin">
+    <xacro:macro name="freely_rotating_hook" params="prefix parent ros2_control_hardware_type ros_distro *origin">
         <!-- Please mind: This joint is actually passive, but in order to help moveit plan the trajectory we make it active -->
         <xacro:basic_joint
@@ -17,4 +17,5 @@
             port="0"
             direction="0"
+            ros_distro="${ros_distro}"
             link_name="${prefix}door_opening_mechanism_link_freely_rotating_hook"
             link_origin_x="0.0"

File: src/ros2/robot_description/rb_theron_common/rb_theron_description/urdf/door_opening_mechanism/door_opening_mechanism.urdf.xacro (robot description, xacro)
@@ -6,5 +6,5 @@
                 izz="${m*(x*x+y*y)/12}" />
     </xacro:macro>
-    <xacro:macro name="door_opening_mechanism" params="prefix parent ros2_control_hardware_type *origin hq">
+    <xacro:macro name="door_opening_mechanism" params="prefix parent ros2_control_hardware_type ros_distro *origin hq">
         <!-- Element imports -->
         <xacro:include filename="$(find rb_theron_description)/urdf/door_opening_mechanism/components/alu_profile.urdf.xacro" />
@@ -71,4 +71,5 @@
             port="3502"
             direction="1"
+            ros_distro="${ros_distro}"
             link_name="${prefix}door_opening_mechanism_link_y_axis_slide"
             link_origin_x="0.0"
@@ -98,4 +99,5 @@
             port="3503"
             direction="-1"
+            ros_distro="${ros_distro}"
             link_name="${prefix}door_opening_mechanism_link_x_axis_slide"
             link_origin_x="0.0"
@@ -135,4 +137,5 @@
             parent="${prefix}door_opening_mechanism_link_x_slide_screwing"
             ros2_control_hardware_type="${ros2_control_hardware_type}"
+            ros_distro="${ros_distro}"
             arm_length="0.3" >
             <origin xyz="0.05 -0.025 0" rpy="0 0 1.57079632679"/>

File: src/ros2/robot_description/rb_theron_common/rb_theron_description/urdf/drawer/drawer.urdf.xacro (robot description, xacro)
@@ -15,5 +15,5 @@
     <xacro:property name="drawer_offset_y" value="0.0" />
     <xacro:property name="drawer_offset_z" value="0.0" />
-    <xacro:macro name="drawer" params="prefix suffix parent *origin ros2_control_hardware_type drawer_size_z">
+    <xacro:macro name="drawer" params="prefix suffix parent *origin ros2_control_hardware_type ros_distro drawer_size_z">
         <link name="${prefix}drawer_${suffix}">
             <inertial>
@@ -55,5 +55,10 @@
                 </xacro:if>
                 <xacro:if value="${ros2_control_hardware_type == 'gz_ros2_control'}">
-                    <plugin>gz_ros2_control/GazeboSimSystem</plugin>
+                    <xacro:if value="${ros_distro == 'humble'}">
+                        <plugin>ign_ros2_control/IgnitionSystem</plugin>
+                    </xacro:if>
+                    <xacro:unless value="${ros_distro == 'humble'}">
+                        <plugin>gz_ros2_control/GazeboSimSystem</plugin>
+                    </xacro:unless>
                 </xacro:if>
                 <xacro:if value="${ros2_control_hardware_type == 'dryve_d1'}">

File: src/ros2/robot_description/rb_theron_common/rb_theron_description/urdf/wheels/castor.urdf.xacro (robot description, xacro)
@@ -18,5 +18,5 @@
               izz="${m*r*r/2}" />
   </xacro:macro>
-  <xacro:macro name="caster" params="prefix parent ros2_control_hardware_type *origin hq">
+  <xacro:macro name="caster" params="prefix parent ros2_control_hardware_type ros_distro *origin hq">
     <!--CASTER SUPPORT -->
     <joint name="${prefix}joint_support" type="continuous">
@@ -36,5 +36,10 @@
         </xacro:if>
         <xacro:if value="${ros2_control_hardware_type == 'gz_ros2_control'}">
-          <plugin>gz_ros2_control/GazeboSimSystem</plugin>
+          <xacro:if value="${ros_distro == 'humble'}">
+            <plugin>ign_ros2_control/IgnitionSystem</plugin>
+          </xacro:if>
+          <xacro:unless value="${ros_distro == 'humble'}">
+            <plugin>gz_ros2_control/GazeboSimSystem</plugin>
+          </xacro:unless>
         </xacro:if>
         <xacro:if value="${ros2_control_hardware_type == 'dryve_d1'}">
@@ -79,9 +84,10 @@
       parent="${prefix}support"
       ros2_control_hardware_type="${ros2_control_hardware_type}"
+      ros_distro="${ros_distro}"
       hq="${hq}">
       <origin xyz="${caster_wheel_offset_x} ${caster_wheel_offset_y} ${caster_wheel_offset_z}" rpy="0 0 0"/>
     </xacro:caster_wheel>
   </xacro:macro>
-  <xacro:macro name="caster_wheel" params="prefix parent *origin ros2_control_hardware_type hq">
+  <xacro:macro name="caster_wheel" params="prefix parent *origin ros2_control_hardware_type ros_distro hq">
     <joint name="${prefix}joint_wheel" type="continuous">
       <parent link="${parent}"/>
@@ -99,6 +105,11 @@
 				</xacro:if>
 				<xacro:if value="${ros2_control_hardware_type == 'gz_ros2_control'}">
-					<plugin>gz_ros2_control/GazeboSimSystem</plugin>
-				</xacro:if>
+          <xacro:if value="${ros_distro == 'humble'}">
+            <plugin>ign_ros2_control/IgnitionSystem</plugin>
+          </xacro:if>
+          <xacro:unless value="${ros_distro == 'humble'}">
+            <plugin>gz_ros2_control/GazeboSimSystem</plugin>
+          </xacro:unless>
+        </xacro:if>
 				<xacro:if value="${ros2_control_hardware_type == 'dryve_d1'}">
 					<plugin>mock_components/GenericSystem</plugin>

File: src/ros2/robot_description/rb_theron_common/rb_theron_description/urdf/wheels/rubber_wheel.transmission.xacro (robot description, xacro)
@@ -2,5 +2,5 @@
 <robot xmlns:xacro="http://www.ros.org/wiki/xacro">
     <!-- Rubber wheel transmission -->
-    <xacro:macro name="rubber_wheel_transmission" params="prefix ros2_control_hardware_type">
+    <xacro:macro name="rubber_wheel_transmission" params="prefix ros2_control_hardware_type ros_distro">
     <!-- Transmission is important to link the joints and the controller (see rb_theron_control/config/rb_theron_control.yaml)-->
         <transmission name="${prefix}_wheel_joint_trans">
@@ -36,6 +36,11 @@
 				</xacro:if>
 				<xacro:if value="${ros2_control_hardware_type == 'gz_ros2_control'}">
-					<plugin>gz_ros2_control/GazeboSimSystem</plugin>
-				</xacro:if>
+                    <xacro:if value="${ros_distro == 'humble'}">
+                        <plugin>ign_ros2_control/IgnitionSystem</plugin>
+                    </xacro:if>
+                    <xacro:unless value="${ros_distro == 'humble'}">
+                        <plugin>gz_ros2_control/GazeboSimSystem</plugin>
+                    </xacro:unless>
+                </xacro:if>
 				<xacro:if value="${ros2_control_hardware_type == 'dryve_d1'}">
 					<plugin>mock_components/GenericSystem</plugin>

File: src/ros2/robot_description/rb_theron_common/rb_theron_description/urdf/wheels/rubber_wheel.urdf.xacro (robot description, xacro)
@@ -13,5 +13,5 @@
         <inertia ixx="${m*(3*r*r+h*h)/12}" ixy = "0" ixz = "0" iyy="${m*(3*r*r+h*h)/12}" iyz = "0" izz="${m*r*r/2}" />
     </xacro:macro>
-    <xacro:macro name="rubber_wheel" params="prefix parent *origin reflect ros2_control_hardware_type hq">
+    <xacro:macro name="rubber_wheel" params="prefix parent *origin reflect ros2_control_hardware_type ros_distro hq">
         <!--WHEEL TIRE -->
         <joint name="${prefix}_wheel_joint" type="continuous">
@@ -44,5 +44,9 @@
             </inertial>
         </link>
-        <xacro:rubber_wheel_transmission prefix="${prefix}" ros2_control_hardware_type="${ros2_control_hardware_type}" />
+        <xacro:rubber_wheel_transmission
+            prefix="${prefix}"
+            ros2_control_hardware_type="${ros2_control_hardware_type}"
+            ros_distro="${ros_distro}"
+        />
         <xacro:rubber_wheel_gazebo prefix="${prefix}" />
     </xacro:macro>

File: src/ros2/robot_description/rb_theron_common/rb_theron_description/urdf/wheels/rubber_wheel_125.urdf.xacro (robot description, xacro)
@@ -12,5 +12,5 @@
         <inertia ixx="${m*(3*r*r+h*h)/12}" ixy = "0" ixz = "0" iyy="${m*(3*r*r+h*h)/12}" iyz = "0" izz="${m*r*r/2}" />
     </xacro:macro>
-    <xacro:macro name="rubber_wheel" params="prefix parent *origin reflect ros2_control_hardware_type hq">
+    <xacro:macro name="rubber_wheel" params="prefix parent *origin reflect ros2_control_hardware_type ros_distro hq">
         <!--WHEEL TIRE -->
         <joint name="${prefix}_wheel_joint" type="continuous">
@@ -43,5 +43,9 @@
             </inertial>
         </link>
-        <xacro:rubber_wheel_transmission prefix="${prefix}" ros2_control_hardware_type="${ros2_control_hardware_type}" />
+        <xacro:rubber_wheel_transmission
+            prefix="${prefix}"
+            ros2_control_hardware_type="${ros2_control_hardware_type}"
+            ros_distro="${ros_distro}"
+        />
         <xacro:rubber_wheel_gazebo prefix="${prefix}" />
     </xacro:macro>

File: src/ros2/robot_description/rb_theron_common/rb_theron_description/urdf/wheels/rubber_wheel_150.urdf.xacro (robot description, xacro)
@@ -13,5 +13,5 @@
         <inertia ixx="${m*(3*r*r+h*h)/12}" ixy = "0" ixz = "0" iyy="${m*(3*r*r+h*h)/12}" iyz = "0" izz="${m*r*r/2}" />
     </xacro:macro>
-    <xacro:macro name="rubber_wheel" params="prefix parent *origin ros2_control_hardware_type hq">
+    <xacro:macro name="rubber_wheel" params="prefix parent *origin ros2_control_hardware_type ros_distro hq">
         <!--WHEEL TIRE -->
         <joint name="${prefix}_wheel_joint" type="continuous">
@@ -57,5 +57,9 @@
             </visual>
         </link>
-        <xacro:rubber_wheel_transmission prefix="${prefix}" ros2_control_hardware_type="${ros2_control_hardware_type}" />
+        <xacro:rubber_wheel_transmission
+            prefix="${prefix}"
+            ros2_control_hardware_type="${ros2_control_hardware_type}"
+            ros_distro="${ros_distro}"
+        />
         <xacro:rubber_wheel_gazebo prefix="${prefix}" />
     </xacro:macro>

File: src/ros2/robot_description/robotnik_sensors/urdf/imu_hector_plugin.urdf.xacro (robot description, xacro)
@@ -104,10 +104,4 @@
 			</sensor>
 		</gazebo>
-		<gazebo>
-			<plugin
-				filename="libgz-sim-imu-system"
-				name="gz::sim::systems::Imu">
-			</plugin>
-		</gazebo>
 	</xacro:macro>
 </robot>
