Commit message: chore: small refinements in xacros to handle warnings

File: src/ros2/robot_description/rb_theron_common/rb_theron_description/robots/rb_theron.urdf.xacro (robot description, xacro)
@@ -90,5 +90,20 @@
 	<xacro:arg name="front_oak_d_pitch" default="0.0" />
 	<xacro:arg name="front_oak_d_yaw" default="0.0" />
-	<xacro:depthai_camera prefix="$(arg prefix)front_top_oak_d_camera" parent="$(arg prefix)base_link" publish_bf="${publish_bf}" robot_name="${robot_name}" prefix_topic="front_top_oak_d_camera" camera_model = "$(arg front_oak_d_camera_model)" base_frame = "$(arg front_oak_d_base_frame)" cam_pos_x = "$(arg front_oak_d_pos_x)" cam_pos_y = "$(arg front_oak_d_pos_y)" cam_pos_z = "$(arg front_oak_d_pos_z)" cam_roll = "$(arg front_oak_d_roll)" cam_pitch = "$(arg front_oak_d_pitch)" cam_yaw = "$(arg front_oak_d_yaw)"/>
+	<xacro:depthai_camera
+		prefix="$(arg prefix)front_top_oak_d_camera"
+		parent="$(arg prefix)base_link"
+		publish_bf="${publish_bf}"
+		robot_name="${robot_name}"
+		prefix_topic="front_top_oak_d_camera"
+		camera_model="$(arg front_oak_d_camera_model)"
+		base_frame="$(arg front_oak_d_base_frame)"
+		cam_pos_x="$(arg front_oak_d_pos_x)"
+		cam_pos_y="$(arg front_oak_d_pos_y)"
+		cam_pos_z="$(arg front_oak_d_pos_z)"
+		cam_roll="$(arg front_oak_d_roll)"
+		cam_pitch="$(arg front_oak_d_pitch)"
+		cam_yaw="$(arg front_oak_d_yaw)"
+		hq="${hq}">
+	</xacro:depthai_camera>
 	<!-- ROBAST Module Cage -->
 	<xacro:include filename="$(find rb_theron_description)/urdf/module_cage/module_cage.urdf.xacro" />

File: src/ros2/robot_description/rb_theron_common/rb_theron_description/urdf/wheels/rubber_wheel_150.urdf.xacro (robot description, xacro)
@@ -51,9 +51,15 @@
         <link name="${prefix}_wheel_tire_link">
             <visual>
-        <origin xyz="0 0 0" rpy="${M_PI/2} 0 0" />
+                <origin xyz="0 0 0" rpy="${M_PI/2} 0 0" />
                 <geometry>
                     <cylinder length="${wheel_height + 0.001}" radius="${wheel_radius * 0.92}" />
                 </geometry>
             </visual>
+            <collision>
+                <origin xyz="0 0 0" rpy="${M_PI/2} 0 0" />
+                <geometry>
+                    <cylinder length="${wheel_height + 0.001}" radius="${wheel_radius * 0.92}" />
+                </geometry>
+            </collision>
         </link>
         <xacro:rubber_wheel_transmission

File: src/ros2/robot_description/robotnik_sensors/urdf/depthai_macro.urdf.xacro (robot description, xacro)
@@ -3,5 +3,5 @@
 <xacro:macro name="depthai_camera" params="prefix parent publish_bf robot_name prefix_topic camera_model base_frame
                                            cam_pos_x cam_pos_y cam_pos_z
-                                           cam_roll cam_pitch cam_yaw
+                                           cam_roll cam_pitch cam_yaw hq
                                            r:=0.8 g:=0.8 b:=0.8 a:=0.8">
     <xacro:if value="${publish_bf}">
@@ -38,5 +38,11 @@
             <origin xyz="0 0 0" rpy="0 0 0"/>
             <geometry>
+              <xacro:if value="${hq}">
                 <mesh filename="$(find robotnik_sensors)/meshes/${model}.stl" />
+              </xacro:if>
+              <xacro:unless value="${hq}">
+                <!-- Please mind that this only a extremly rough estimation -->
+                <box size="0.100 0.025 0.025"/>
+              </xacro:unless>
             </geometry>
             <material name="mat">
@@ -44,4 +50,16 @@
             </material>
         </visual>
+        <collision>
+            <origin xyz="0 0 0" rpy="0 0 0"/>
+            <geometry>
+              <xacro:if value="${hq}">
+                <mesh filename="$(find robotnik_sensors)/meshes/${model}.stl" />
+              </xacro:if>
+              <xacro:unless value="${hq}">
+                <!-- Please mind that this only a extremly rough estimation -->
+                <box size="0.100 0.025 0.025"/>
+              </xacro:unless>
+            </geometry>
+        </collision>
     </link>
     <joint name="${prefix}_model_origin_joint" type="fixed">

Commit message: simulation adjustments for multi robot
simulation adjustments for multi robot

File: src/ros2/robot_description/rb_theron_common/rb_theron_description/robots/rb_theron.urdf.xacro (robot description, xacro)
@@ -35,4 +35,5 @@
     <xacro:arg name="ros2_control_hardware_type" default="mock_components" />
 	<xacro:arg name="ros_distro" default="humble" />
+	<xacro:arg name="namespace" default="" />
 	<!-- *************** -->
 	<!-- Robots Elements -->
@@ -169,5 +170,5 @@
 	</xacro:door_opening_mechanism>
 	<!-- Gazebo plugins -->
-	<xacro:ros_control ros_distro="$(arg ros_distro)"/>
+	<xacro:ros_control ros_distro="$(arg ros_distro)" namespace= "$(arg namespace)"/>
 	<xacro:gazebo_sensor_plugins ros_distro="$(arg ros_distro)"/>
 </robot>

File: src/ros2/robot_description/rb_theron_common/rb_theron_description/urdf/common.gazebo.xacro (robot description, xacro)
@@ -2,9 +2,12 @@
 <robot xmlns:xacro="http://www.ros.org/wiki/xacro">
     <!-- ROS CONTROL GAZEBO PLUGIN -->
-    <xacro:macro name="ros_control" params="ros_distro">
+    <xacro:macro name="ros_control" params="ros_distro namespace" >
         <gazebo>
             <xacro:if value="${ros_distro == 'humble'}">
                 <plugin name="ign_ros2_control::IgnitionROS2ControlPlugin" filename="libign_ros2_control-system.so">
                     <parameters>$(find rb_theron_description)/config/rb_theron_gz_ros2_controller.yaml</parameters>
+                    <ros>
+                        <namespace>${namespace}</namespace>
+                    </ros>
                 </plugin>
             </xacro:if>

Commit message: added a namespace in front of the robot topics if the robot name was changed from outside of the xacro

File: src/ros2/robot_description/rb_theron_common/rb_theron_description/robots/rb_theron.urdf.xacro (robot description, xacro)
@@ -18,6 +18,4 @@
 	<!-- Flag to determine if the base_footprint should be published or not -->
 	<xacro:property name="publish_bf" value="true"/>
-	<!-- This name should match the "-name" argument we need to declare when spawing the robot into ign gazebo -->
-	<xacro:property name="robot_name" value="rb_theron"/>
 	<!-- Wheel parameters -->
 	<!--xacro:property name="wheel_offset_x" value="0" />
@@ -26,5 +24,8 @@
 	<!-- Flag to select the high or low quality model -->
 	<xacro:property name="hq" value="false" />
+	<!-- This name should match the "-name" argument we need to declare when spawing the robot into ign gazebo -->
+	<xacro:arg name="robot_name" default="rb_theron"/>
 	<xacro:arg name="prefix" default=""/>
+	<xacro:arg name="use_gazebo_sensor_plugins" default="true"/>
 	<!-- <xacro:arg name="gpu" default="true"/> -->
 	<!-- ros2_control_hardware_type:
@@ -53,12 +54,12 @@
 	<!-- TODO: Should be sensor_intel_d435, but this one isn't migrated to ros2 yet -->
 	<!-- TODO: Moved 0.01 in x, otherwise the camera is still inside the robot -->
-	<xacro:sensor_r430 prefix="$(arg prefix)front_realsense_camera" parent="$(arg prefix)base_link" publish_bf="${publish_bf}" robot_name="${robot_name}" prefix_topic="front_realsense_camera" hq="${hq}">
+	<xacro:sensor_r430 prefix="$(arg prefix)front_realsense_camera" parent="$(arg prefix)base_link" publish_bf="${publish_bf}" robot_name="$(arg robot_name)" prefix_topic="front_realsense_camera" hq="${hq}">
 		<origin xyz="0.3305 0.0 0.1468" rpy="0 0 0"/>
 	</xacro:sensor_r430>
-	<xacro:sensor_r430 prefix="$(arg prefix)back_realsense_camera" parent="$(arg prefix)base_link" publish_bf="${publish_bf}" robot_name="${robot_name}" prefix_topic="back_realsense_camera" hq="${hq}">
+	<xacro:sensor_r430 prefix="$(arg prefix)back_realsense_camera" parent="$(arg prefix)base_link" publish_bf="${publish_bf}" robot_name="$(arg robot_name)" prefix_topic="back_realsense_camera" hq="${hq}">
 		<origin xyz="-0.3305 0.0 0.1468" rpy="0 0 3.1416"/>
 	</xacro:sensor_r430>
 	<!--Added back top realsense camera because running YOLO network on depthai camera in simulation reduces Real Time Factor (RTF)-->
-	<xacro:sensor_r430 prefix="$(arg prefix)back_top_realsense_camera" parent="$(arg prefix)base_link" publish_bf="${publish_bf}" robot_name="${robot_name}" prefix_topic="back_top_realsense_camera" hq="${hq}">
+	<xacro:sensor_r430 prefix="$(arg prefix)back_top_realsense_camera" parent="$(arg prefix)base_link" publish_bf="${publish_bf}" robot_name="$(arg robot_name)" prefix_topic="back_top_realsense_camera" hq="${hq}">
 		<origin xyz="-0.3305 0.0 1.1468" rpy="0 0 3.1416"/>
 	</xacro:sensor_r430>
@@ -67,8 +68,8 @@
 		<origin xyz="0.3305 0.0 0.1898" rpy="0 0 0"/>
 	</xacro:sensor_orbbec_astra -->
-	<xacro:sensor_imu_hector prefix="$(arg prefix)imu" parent="$(arg prefix)base_link">
+	<xacro:sensor_imu_hector prefix="$(arg prefix)imu" parent="$(arg prefix)base_link" robot_name="$(arg robot_name)">
 		<origin xyz="-0.1975 0.0 0.1598" rpy="0 0 0"/>
 	</xacro:sensor_imu_hector>
-	<xacro:sensor_sick_nanoscan3 prefix="$(arg prefix)front_laser" parent="$(arg prefix)base_link" publish_bf="${publish_bf}" robot_name="${robot_name}" prefix_topic="front_laser" hq="${hq}" min_angle="-1.9507619" max_angle="1.9507619" gpu="true">
+	<xacro:sensor_sick_nanoscan3 prefix="$(arg prefix)front_laser" parent="$(arg prefix)base_link" publish_bf="${publish_bf}" robot_name="$(arg robot_name)" prefix_topic="front_laser" hq="${hq}" min_angle="-1.9507619" max_angle="1.9507619" gpu="true">
 		<origin xyz="0.250 0.0 0.1643" rpy="0 3.1416 3.1416"/>
 	</xacro:sensor_sick_nanoscan3>
@@ -76,5 +77,5 @@
 		<origin xyz="0.214 0.0 0.275" rpy="-1.57079632679 0 -0.23"/>
 	</xacro:sensor_rs_lidar_16>-->
-	<xacro:sensor_rs_bpearl prefix="$(arg prefix)top_laser" parent="$(arg prefix)base_link" publish_bf="${publish_bf}" robot_name="${robot_name}" prefix_topic="top_laser" hq="${hq}" range_min="0.1" range_max="90" hfov="360" samples="1800" vfov="90.0" lasers="32" fps="10" gpu="false">
+	<xacro:sensor_rs_bpearl prefix="$(arg prefix)top_laser" parent="$(arg prefix)base_link" publish_bf="${publish_bf}" robot_name="$(arg robot_name)" prefix_topic="top_laser" hq="${hq}" range_min="0.1" range_max="90" hfov="360" samples="1800" vfov="90.0" lasers="32" fps="10" gpu="false">
 		<origin xyz="0.3 -0.175 1.165" rpy="-1.570796326795 0 -1.570796326795"/>
 		<!-- positions of the b-pearl based on solid: xyz="0.333 -0.180 1.194" rpy="-1.570796326795 0 -1.570796326795" -->
@@ -95,5 +96,5 @@
 		parent="$(arg prefix)base_link"
 		publish_bf="${publish_bf}"
-		robot_name="${robot_name}"
+		robot_name="$(arg robot_name)"
 		prefix_topic="front_top_oak_d_camera"
 		camera_model="$(arg front_oak_d_camera_model)"
@@ -171,4 +172,6 @@
 	<!-- Gazebo plugins -->
 	<xacro:ros_control ros_distro="$(arg ros_distro)" namespace= "$(arg namespace)"/>
-	<xacro:gazebo_sensor_plugins ros_distro="$(arg ros_distro)"/>
+	<xacro:if value="$(arg use_gazebo_sensor_plugins)">
+		<xacro:gazebo_sensor_plugins ros_distro="$(arg ros_distro)"/>
+	</xacro:if>
 </robot>

File: src/ros2/robot_description/robotnik_sensors/urdf/depthai_macro.urdf.xacro (robot description, xacro)
@@ -5,4 +5,10 @@
                                            cam_roll cam_pitch cam_yaw hq
                                            r:=0.8 g:=0.8 b:=0.8 a:=0.8">
+    <xacro:if value="${robot_name=='rb_theron'}">
+      <xacro:property name="robot_namespace" value="" />
+    </xacro:if>
+    <xacro:unless value="${robot_name=='rb_theron'}">
+			<xacro:property name="robot_namespace" value="${robot_name}/"/>
+		</xacro:unless>
     <xacro:if value="${publish_bf}">
 			<xacro:property name="sensor_link_name" value="${robot_name}/base_footprint/${prefix}" />
@@ -122,5 +128,5 @@
     <gazebo reference="${base_frame}">
       <sensor name="${prefix}_rgb_camera_optical_frame" type="camera">
-				<topic>${prefix_topic}/color</topic>
+				<topic>${robot_namespace}${prefix_topic}/color</topic>
         <camera name="oak-d">
             <horizontal_fov>1.2112585008840648</horizontal_fov>
@@ -142,5 +148,5 @@
       </sensor>
       <sensor name="${prefix}_right_camera_optical_frame" type="depth">
-        <topic>${prefix_topic}/${prefix}/depth</topic>
+        <topic>${robot_namespace}${prefix_topic}/depth</topic>
         <camera name="oak-d">
           <horizontal_fov>${85.2*M_PI/180.0}</horizontal_fov>

File: src/ros2/robot_description/robotnik_sensors/urdf/imu_hector_plugin.urdf.xacro (robot description, xacro)
@@ -1,5 +1,11 @@
 <?xml version="1.0"?>
 <robot name="sensor_imu" xmlns:xacro="http://wiki.ros.org/xacro">
-	<xacro:macro name="sensor_imu_hector" params="prefix topic:='imu/data' parent *origin">
+	<xacro:macro name="sensor_imu_hector" params="prefix robot_name topic:='imu/data' parent *origin">
+		<xacro:if value="${robot_name=='rb_theron'}">
+      		<xacro:property name="robot_namespace" value="" />
+    	</xacro:if>
+    	<xacro:unless value="${robot_name=='rb_theron'}">
+			<xacro:property name="robot_namespace" value="${robot_name}/"/>
+		</xacro:unless>
 		<xacro:if value="${publish_bf}">
 			<xacro:property name="sensor_link_name" value="${robot_name}/base_footprint/${prefix}_link" />
@@ -39,5 +45,5 @@
 				<update_rate>40</update_rate>
 				<visualize>true</visualize>
-				<topic>imu/data</topic>
+				<topic>${robot_namespace}imu/data</topic>
 				<imu>
 					<!-- <orientation>

File: src/ros2/robot_description/robotnik_sensors/urdf/intel_r430.urdf.xacro (robot description, xacro)
@@ -20,4 +20,10 @@
   <xacro:property name="r430_cam_depth_pz" value="0.0"/>
   <xacro:macro name="sensor_r430" params="prefix parent publish_bf robot_name prefix_topic:='front_rgbd_camera' hq *origin">
+  <xacro:if value="${robot_name=='rb_theron'}">
+    <xacro:property name="robot_namespace" value="" />
+  </xacro:if>
+  <xacro:unless value="${robot_name=='rb_theron'}">
+		<xacro:property name="robot_namespace" value="${robot_name}/"/>
+	</xacro:unless>
     <xacro:if value="${publish_bf}">
 			<xacro:property name="sensor_link_name" value="${robot_name}/base_footprint/${prefix}" />
@@ -125,5 +131,5 @@
     <gazebo reference="${prefix}_link">
       <sensor name="${prefix}_color_link" type="camera">
-				<topic>${prefix_topic}/color</topic>
+				<topic>${robot_namespace}${prefix_topic}/color</topic>
         <camera name="r430">
             <horizontal_fov>1.2112585008840648</horizontal_fov>
@@ -148,5 +154,5 @@
       </sensor>
       <sensor name="${prefix}_ired1" type="camera">
-      <topic>${prefix_topic}/${prefix}/ired1</topic>
+      <topic>${robot_namespace}${prefix_topic}/ired1</topic>
         <camera name="r430">
           <horizontal_fov>${91.2*M_PI/180.0}</horizontal_fov>
@@ -171,5 +177,5 @@
       </sensor>
       <sensor name="${prefix}_ired2" type="camera">
-        <topic>${prefix_topic}/${prefix}/ired2</topic>
+        <topic>${robot_namespace}${prefix_topic}/ired2</topic>
         <camera name="r430">
           <horizontal_fov>1.4870205226991688</horizontal_fov>
@@ -194,5 +200,5 @@
       </sensor>
       <sensor name="${prefix}_depth_link" type="depth">
-        <topic>${prefix_topic}/${prefix}/depth</topic>
+        <topic>${robot_namespace}${prefix_topic}/depth</topic>
         <camera name="r430">
           <horizontal_fov>${91.2*M_PI/180.0}</horizontal_fov>

File: src/ros2/robot_description/robotnik_sensors/urdf/rs_bpearl.urdf.xacro (robot description, xacro)
@@ -9,4 +9,10 @@
 			<xacro:property name="sensor_link_name" value="${robot_name}/base_link/${prefix}_link" />
 		</xacro:unless>
+    <xacro:if value="${robot_name=='rb_theron'}">
+      <xacro:property name="robot_namespace" value="" />
+    </xacro:if>
+    <xacro:unless value="${robot_name=='rb_theron'}">
+		  <xacro:property name="robot_namespace" value="${robot_name}/"/>
+	  </xacro:unless>
     <joint name="${prefix}_base_joint" type="fixed">
       <xacro:insert_block name="origin" />
@@ -74,5 +80,5 @@
       <sensor name='${prefix}_link' type='gpu_lidar'>
         <visualize>true</visualize>
-        <topic>bpearl_laser/scan</topic>
+        <topic>${robot_namespace}bpearl_laser/scan</topic>
         <update_rate>${fps}</update_rate>
         <ray>

File: src/ros2/robot_description/robotnik_sensors/urdf/sick_nanoscan3.urdf.xacro (robot description, xacro)
@@ -9,4 +9,10 @@
 			<xacro:property name="sensor_link_name" value="${robot_name}/base_link/${prefix}_link" />
 		</xacro:unless>
+		<xacro:if value="${robot_name=='rb_theron'}">
+      		<xacro:property name="robot_namespace" value="" />
+    	</xacro:if>
+    	<xacro:unless value="${robot_name=='rb_theron'}">
+			<xacro:property name="robot_namespace" value="${robot_name}/"/>
+	  	</xacro:unless>
 		<joint name="${prefix}_base_joint" type="fixed">
 			<xacro:insert_block name="origin" />
@@ -60,5 +66,5 @@
 			</xacro:unless>
 			<sensor type="${ray_type}" name="${prefix}_link">
-				<topic>${prefix_topic}/scan</topic>
+				<topic>${robot_namespace}/${prefix_topic}/scan</topic>
 				<always_on>1</always_on>
     				<visualize>false</visualize>
