Commit message: links and joint placed with the robot prefix

File: src/ros2/robot_description/rb_theron_common/rb_theron_description/robots/rb_theron.urdf.xacro (robot description, xacro)
@@ -108,7 +108,13 @@
 		hq="${hq}">
 	</xacro:depthai_camera>
+	<xacro:if value="${'$(arg robot_name)' == 'rb_theron'}">
+      <xacro:property name="robot_namespace" value="" />
+    </xacro:if>
+    <xacro:unless value="${'$(arg robot_name)' == 'rb_theron'}">
+		  <xacro:property name="robot_namespace" value="$(arg robot_name)/"/>
+	  </xacro:unless>
 	<!-- ROBAST Module Cage -->
 	<xacro:include filename="$(find rb_theron_description)/urdf/module_cage/module_cage.urdf.xacro" />
-	<xacro:module_cage prefix="$(arg prefix)" parent="$(arg prefix)base_link" hq="${hq}">
+	<xacro:module_cage prefix="${robot_namespace}$(arg prefix)" parent="$(arg prefix)base_link" hq="${hq}">
 		<origin xyz="-0.15 0.0 0.725" rpy="0 0 0"/>
 	</xacro:module_cage>

File: src/ros2/robot_description/robotnik_sensors/urdf/depthai_macro.urdf.xacro (robot description, xacro)
@@ -12,8 +12,8 @@
 		</xacro:unless>
     <xacro:if value="${publish_bf}">
-			<xacro:property name="sensor_link_name" value="${robot_name}/base_footprint/${prefix}" />
+			<xacro:property name="sensor_link_name" value="${robot_namespace}base_footprint/${prefix}" />
 		</xacro:if>
 		<xacro:unless value="${publish_bf}">
-			<xacro:property name="sensor_link_name" value="${robot_name}/base_link/${prefix}" />
+			<xacro:property name="sensor_link_name" value="${robot_namespace}base_link/${prefix}" />
 		</xacro:unless>
     <xacro:property name="M_PI"     value="3.1415926535897931" />
@@ -33,12 +33,12 @@
     </xacro:if>
     <!-- base_link of the sensor-->
-    <link name="${base_frame}"/>
+    <link name="${robot_namespace}${base_frame}"/>
     <joint name="${prefix}_center_joint" type="fixed">
         <parent link="${parent}"/>
-        <child link="${base_frame}"/>
+        <child link="${robot_namespace}${base_frame}"/>
         <origin xyz="${cam_pos_x} ${cam_pos_y} ${cam_pos_z}" rpy="${cam_roll} ${cam_pitch} ${cam_yaw}" />
     </joint>
     <!-- device Center -->
-    <link name="${prefix}_model_origin">
+    <link name="${robot_namespace}${prefix}_model_origin">
         <visual>
             <origin xyz="0 0 0" rpy="0 0 0"/>
@@ -69,56 +69,56 @@
         </collision>
     </link>
-    <joint name="${prefix}_model_origin_joint" type="fixed">
-        <parent link="${base_frame}"/>
-        <child link="${prefix}_model_origin"/>
+    <joint name="${robot_namespace}${prefix}_model_origin_joint" type="fixed">
+        <parent link="${robot_namespace}${base_frame}"/>
+        <child link="${robot_namespace}${prefix}_model_origin"/>
         <origin xyz="0 0 0" rpy="1.5708 0 1.5708" />
     </joint>
     <!-- IMU -->
     <xacro:if value="${has_imu}">
-        <link name="${prefix}_imu_frame" />
-        <joint name="${prefix}_imu_joint" type="fixed">
-            <parent link="${base_frame}"/>
-            <child link="${prefix}_imu_frame"/>
+        <link name="${robot_namespace}${prefix}_imu_frame" />
+        <joint name="${robot_namespace}${prefix}_imu_joint" type="fixed">
+            <parent link="${robot_namespace}${base_frame}"/>
+            <child link="${robot_namespace}${prefix}_imu_frame"/>
             <origin xyz="${imu_offset_x} ${imu_offset_y} ${imu_offset_z}" rpy="${imu_r} ${imu_p} ${imu_y}" />
         </joint>
     </xacro:if>
     <!-- RGB Camera -->
-    <link name="${prefix}_rgb_camera_frame" />
-    <joint name="${prefix}_rgb_camera_joint" type="fixed">
-        <parent link="${base_frame}"/>
-        <child link="${prefix}_rgb_camera_frame"/>
+    <link name="${robot_namespace}${prefix}_rgb_camera_frame" />
+    <joint name="${robot_namespace}${prefix}_rgb_camera_joint" type="fixed">
+        <parent link="${robot_namespace}${base_frame}"/>
+        <child link="${robot_namespace}${prefix}_rgb_camera_frame"/>
         <origin xyz="0 0 0" rpy="0 0 0" />
     </joint>
-    <link name="${sensor_link_name}_rgb_camera_optical_frame"/>
-    <joint name="${prefix}_rgb_camera_optical_joint" type="fixed">
+    <link name="${robot_namespace}${sensor_link_name}_rgb_camera_optical_frame"/>
+    <joint name="${robot_namespace}${prefix}_rgb_camera_optical_joint" type="fixed">
         <origin xyz="0 0 0" rpy="-${M_PI/2} 0.0 -${M_PI/2}"/>
-        <parent link="${prefix}_rgb_camera_frame"/>
-        <child link="${sensor_link_name}_rgb_camera_optical_frame"/>
+        <parent link="${robot_namespace}${prefix}_rgb_camera_frame"/>
+        <child link="${robot_namespace}${sensor_link_name}_rgb_camera_optical_frame"/>
     </joint>
     <!-- Left Camera -->
-    <link name="${prefix}_left_camera_frame" />
-    <joint name="${prefix}_left_camera_joint" type="fixed">
-        <parent link="${base_frame}"/>
-        <child link="${prefix}_left_camera_frame"/>
+    <link name="${robot_namespace}${prefix}_left_camera_frame" />
+    <joint name="${robot_namespace}${prefix}_left_camera_joint" type="fixed">
+        <parent link="${robot_namespace}${base_frame}"/>
+        <child link="${robot_namespace}${prefix}_left_camera_frame"/>
         <origin xyz="0 ${baseline/2} 0" rpy="0 0 0" />
     </joint>
-    <link name="${prefix}_left_camera_optical_frame"/>
-    <joint name="${prefix}_left_camera_optical_joint" type="fixed">
+    <link name="${robot_namespace}${prefix}_left_camera_optical_frame"/>
+    <joint name="${robot_namespace}${prefix}_left_camera_optical_joint" type="fixed">
         <origin xyz="0 0 0" rpy="-${M_PI/2} 0.0 -${M_PI/2}"/>
-        <parent link="${prefix}_left_camera_frame"/>
-        <child link="${prefix}_left_camera_optical_frame"/>
+        <parent link="${robot_namespace}${prefix}_left_camera_frame"/>
+        <child link="${robot_namespace}${prefix}_left_camera_optical_frame"/>
     </joint>
     <!-- right Camera -->
-    <link name="${prefix}_right_camera_frame" />
-    <joint name="${prefix}_right_camera_joint" type="fixed">
-        <parent link="${base_frame}"/>
-        <child link="${prefix}_right_camera_frame"/>
+    <link name="${robot_namespace}${prefix}_right_camera_frame" />
+    <joint name="${robot_namespace}${prefix}_right_camera_joint" type="fixed">
+        <parent link="${robot_namespace}${base_frame}"/>
+        <child link="${robot_namespace}${prefix}_right_camera_frame"/>
         <origin xyz="0 -${baseline/2} 0" rpy="0 0 0" />
     </joint>
-    <link name="${sensor_link_name}_right_camera_optical_frame"/>
-    <joint name="${prefix}_right_camera_optical_joint" type="fixed">
+    <link name="${robot_namespace}${sensor_link_name}_right_camera_optical_frame"/>
+    <joint name="${robot_namespace}${prefix}_right_camera_optical_joint" type="fixed">
         <origin xyz="0 0 0" rpy="0 0 0"/>
-        <parent link="${prefix}_right_camera_frame"/>
-        <child link="${sensor_link_name}_right_camera_optical_frame"/>
+        <parent link="${robot_namespace}${prefix}_right_camera_frame"/>
+        <child link="${robot_namespace}${sensor_link_name}_right_camera_optical_frame"/>
     </joint>
     <xacro:sensor_depthai_gazebo/>
@@ -126,5 +126,5 @@
   <xacro:macro name="sensor_depthai_gazebo">
     <!-- gazebo reference="${prefix}_rgb_base_link" -->
-    <gazebo reference="${base_frame}">
+    <gazebo reference="${robot_namespace}${base_frame}">
       <sensor name="${prefix}_rgb_camera_optical_frame" type="camera">
 				<topic>${robot_namespace}${prefix_topic}/color</topic>

File: src/ros2/robot_description/robotnik_sensors/urdf/intel_r430.urdf.xacro (robot description, xacro)
@@ -27,8 +27,8 @@
 	</xacro:unless>
     <xacro:if value="${publish_bf}">
-			<xacro:property name="sensor_link_name" value="${robot_name}/base_footprint/${prefix}" />
+			<xacro:property name="sensor_link_name" value="${robot_namespace}base_footprint/${prefix}" />
 		</xacro:if>
 		<xacro:unless value="${publish_bf}">
-			<xacro:property name="sensor_link_name" value="${robot_name}/base_link/${prefix}" />
+			<xacro:property name="sensor_link_name" value="${robot_namespace}base_link/${prefix}" />
 		</xacro:unless>
     <!-- camera body, with origin at bottom screw mount -->
@@ -36,7 +36,7 @@
       <xacro:insert_block name="origin" />
       <parent link="${parent}"/>
-      <child link="${prefix}_link" />
-    </joint>
-    <link name="${prefix}_link">
+      <child link="${robot_namespace}${prefix}_link" />
+    </joint>
+    <link name="${robot_namespace}${prefix}_link">
       <visual>
         <!-- origin xyz="0 ${-r430_cam_mount_from_center_offset} ${r430_cam_height/2}" rpy="${M_PI/2} 0 ${M_PI/2}"/ -->
@@ -69,59 +69,59 @@
     <joint name="${prefix}_camera_depth_joint" type="fixed">
       <origin xyz="${r430_cam_depth_px} ${r430_cam_depth_py} ${r430_cam_depth_pz}" rpy="0 0 0"/>
-      <parent link="${prefix}_link"/>
-      <child link="${prefix}_camera_depth_frame" />
-    </joint>
-    <link name="${prefix}_camera_depth_frame"/>
-    <joint name="${prefix}_camera_depth_optical_joint" type="fixed">
+      <parent link="${robot_namespace}${prefix}_link"/>
+      <child link="${robot_namespace}${prefix}_camera_depth_frame" />
+    </joint>
+    <link name="${robot_namespace}${prefix}_camera_depth_frame"/>
+    <joint name="${robot_namespace}${prefix}_camera_depth_optical_joint" type="fixed">
       <origin xyz="0 0 0" rpy="0 0 0" />
-      <parent link="${prefix}_camera_depth_frame" />
+      <parent link="${robot_namespace}${prefix}_camera_depth_frame" />
       <child link="${sensor_link_name}_depth_link" />
     </joint>
     <link name="${sensor_link_name}_depth_link"/>
-    <joint name="${prefix}_camera_color_joint" type="fixed">
-      <origin xyz="0 0 0" rpy="${-M_PI/2} 0 ${-M_PI/2}" />
-      <parent link="${prefix}_camera_depth_frame" />
+    <joint name="${robot_namespace}${prefix}_camera_color_joint" type="fixed">
+      <origin xyz="0 0 0" rpy="${-M_PI/2} 0 ${-M_PI/2}" />
+      <parent link="${robot_namespace}${prefix}_camera_depth_frame" />
       <child link="${sensor_link_name}_color_link" />
     </joint>
     <link name="${sensor_link_name}_color_link"/>
     <!-- camera left IR joints and links -->
-    <joint name="${prefix}_camera_left_ir_joint" type="fixed">
+    <joint name="${robot_namespace}${prefix}_camera_left_ir_joint" type="fixed">
       <origin xyz="0 ${r430_cam_depth_to_left_ir_offset} 0" rpy="0 0 0" />
-      <parent link="${prefix}_camera_depth_frame" />
-      <child link="${prefix}_camera_left_ir_frame" />
-    </joint>
-    <link name="${prefix}_camera_left_ir_frame"/>
-    <joint name="${prefix}_camera_left_ir_optical_joint" type="fixed">
-      <origin xyz="0 0 0" rpy="${-M_PI/2} 0 ${-M_PI/2}" />
-      <parent link="${prefix}_camera_left_ir_frame" />
-      <child link="${prefix}_camera_left_ir_optical_frame" />
-    </joint>
-    <link name="${prefix}_camera_left_ir_optical_frame"/>
+      <parent link="${robot_namespace}${prefix}_camera_depth_frame" />
+      <child link="${robot_namespace}${prefix}_camera_left_ir_frame" />
+    </joint>
+    <link name="${robot_namespace}${prefix}_camera_left_ir_frame"/>
+    <joint name="${robot_namespace}${prefix}_camera_left_ir_optical_joint" type="fixed">
+      <origin xyz="0 0 0" rpy="${-M_PI/2} 0 ${-M_PI/2}" />
+      <parent link="${robot_namespace}${prefix}_camera_left_ir_frame" />
+      <child link="${robot_namespace}${prefix}_camera_left_ir_optical_frame" />
+    </joint>
+    <link name="${robot_namespace}${prefix}_camera_left_ir_optical_frame"/>
     <!-- camera right IR joints and links -->
-    <joint name="${prefix}_camera_right_ir_joint" type="fixed">
+    <joint name="${robot_namespace}${prefix}_camera_right_ir_joint" type="fixed">
       <origin xyz="0 ${r430_cam_depth_to_right_ir_offset} 0" rpy="0 0 0" />
-      <parent link="${prefix}_camera_depth_frame" />
-      <child link="${prefix}_camera_right_ir_frame" />
-    </joint>
-    <link name="${prefix}_camera_right_ir_frame"/>
-    <joint name="${prefix}_camera_right_ir_optical_joint" type="fixed">
-      <origin xyz="0 0 0" rpy="${-M_PI/2} 0 ${-M_PI/2}" />
-      <parent link="${prefix}_camera_right_ir_frame" />
-      <child link="${prefix}_camera_right_ir_optical_frame" />
-    </joint>
-    <link name="${prefix}_camera_right_ir_optical_frame"/>
+      <parent link="${robot_namespace}${prefix}_camera_depth_frame" />
+      <child link="${robot_namespace}${prefix}_camera_right_ir_frame" />
+    </joint>
+    <link name="${robot_namespace}${prefix}_camera_right_ir_frame"/>
+    <joint name="${robot_namespace}${prefix}_camera_right_ir_optical_joint" type="fixed">
+      <origin xyz="0 0 0" rpy="${-M_PI/2} 0 ${-M_PI/2}" />
+      <parent link="${robot_namespace}${prefix}_camera_right_ir_frame" />
+      <child link="${robot_namespace}${prefix}_camera_right_ir_optical_frame" />
+    </joint>
+    <link name="${robot_namespace}${prefix}_camera_right_ir_optical_frame"/>
     <!-- camera fisheye joints and links -->
-    <joint name="${prefix}_camera_fisheye_joint" type="fixed">
+    <joint name="${robot_namespace}${prefix}_camera_fisheye_joint" type="fixed">
       <origin xyz="0 ${r430_cam_depth_to_fisheye_offset} 0" rpy="0 0 0" />
-      <parent link="${prefix}_camera_depth_frame" />
-      <child link="${prefix}_camera_fisheye_frame" />
-    </joint>
-    <link name="${prefix}_camera_fisheye_frame"/>
-    <joint name="${prefix}_camera_fisheye_optical_joint" type="fixed">
-      <origin xyz="0 0 0" rpy="${-M_PI/2} 0 ${-M_PI/2}" />
-      <parent link="${prefix}_camera_fisheye_frame" />
-      <child link="${prefix}_camera_fisheye_optical_frame" />
-    </joint>
-    <link name="${prefix}_camera_fisheye_optical_frame"/>
+      <parent link="${robot_namespace}${prefix}_camera_depth_frame" />
+      <child link="${robot_namespace}${prefix}_camera_fisheye_frame" />
+    </joint>
+    <link name="${robot_namespace}${prefix}_camera_fisheye_frame"/>
+    <joint name="${robot_namespace}${prefix}_camera_fisheye_optical_joint" type="fixed">
+      <origin xyz="0 0 0" rpy="${-M_PI/2} 0 ${-M_PI/2}" />
+      <parent link="${robot_namespace}${prefix}_camera_fisheye_frame" />
+      <child link="${robot_namespace}${prefix}_camera_fisheye_optical_frame" />
+    </joint>
+    <link name="${robot_namespace}${prefix}_camera_fisheye_optical_frame"/>
     <!-- RGBD sensor for simulation, same as Kinect -->
     <xacro:sensor_r430_gazebo/>

File: src/ros2/robot_description/robotnik_sensors/urdf/rs_bpearl.urdf.xacro (robot description, xacro)
@@ -3,10 +3,4 @@
   <xacro:property name="M_PI" value="3.1415926535897931" />
   <xacro:macro name="sensor_rs_bpearl" params="prefix parent publish_bf robot_name prefix_topic hq *origin range_min range_max hfov samples vfov lasers fps gpu:=true">
-    <xacro:if value="${publish_bf}">
-			<xacro:property name="sensor_link_name" value="${robot_name}/base_footprint/${prefix}_link" />
-		</xacro:if>
-		<xacro:unless value="${publish_bf}">
-			<xacro:property name="sensor_link_name" value="${robot_name}/base_link/${prefix}_link" />
-		</xacro:unless>
     <xacro:if value="${robot_name=='rb_theron'}">
       <xacro:property name="robot_namespace" value="" />
@@ -15,10 +9,16 @@
 		  <xacro:property name="robot_namespace" value="${robot_name}/"/>
 	  </xacro:unless>
-    <joint name="${prefix}_base_joint" type="fixed">
+    <xacro:if value="${publish_bf}">
+			<xacro:property name="sensor_link_name" value="${robot_namespace}base_footprint/${prefix}_link" />
+		</xacro:if>
+		<xacro:unless value="${publish_bf}">
+			<xacro:property name="sensor_link_name" value="${robot_namespace}base_link/${prefix}_link" />
+		</xacro:unless>
+    <joint name="${robot_namespace}${prefix}_base_joint" type="fixed">
       <xacro:insert_block name="origin" />
       <parent link="${parent}"/>
-      <child link="${prefix}_base_link" />
+      <child link="${robot_namespace}${prefix}_base_link" />
     </joint>
-    <link name="${prefix}_base_link">
+    <link name="${robot_namespace}${prefix}_base_link">
       <visual>
         <!-- origin xyz="0 0 0" rpy="0 0 1.5708"/ -->
@@ -51,5 +51,5 @@
     </link>
     <joint name="${prefix}_joint" type="fixed">
-      <parent link="${prefix}_base_link"/>
+      <parent link="${robot_namespace}${prefix}_base_link"/>
       <child link="${sensor_link_name}"/>
       <origin xyz="0 0 0.09427" rpy="0 0 0"/>

File: src/ros2/robot_description/robotnik_sensors/urdf/sick_nanoscan3.urdf.xacro (robot description, xacro)
@@ -3,10 +3,4 @@
 	xmlns:xacro="http://wiki.ros.org/xacro">
 	<xacro:macro name="sensor_sick_nanoscan3" params="prefix parent publish_bf robot_name prefix_topic:='front_laser' hq *origin max_angle:=2.3998 min_angle:=-2.3998 gpu:=^|false">
-		<xacro:if value="${publish_bf}">
-			<xacro:property name="sensor_link_name" value="${robot_name}/base_footprint/${prefix}_link" />
-		</xacro:if>
-		<xacro:unless value="${publish_bf}">
-			<xacro:property name="sensor_link_name" value="${robot_name}/base_link/${prefix}_link" />
-		</xacro:unless>
 		<xacro:if value="${robot_name=='rb_theron'}">
       		<xacro:property name="robot_namespace" value="" />
@@ -15,10 +9,16 @@
 			<xacro:property name="robot_namespace" value="${robot_name}/"/>
 	  	</xacro:unless>
-		<joint name="${prefix}_base_joint" type="fixed">
+		<xacro:if value="${publish_bf}">
+			<xacro:property name="sensor_link_name" value="${robot_namespace}base_footprint/${prefix}_link" />
+		</xacro:if>
+		<xacro:unless value="${publish_bf}">
+			<xacro:property name="sensor_link_name" value="${robot_namespace}/base_link/${prefix}_link" />
+		</xacro:unless>
+		<joint name="${robot_namespace}${prefix}_base_joint" type="fixed">
 			<xacro:insert_block name="origin" />
 			<parent link="${parent}"/>
-			<child link="${prefix}_base_link"/>
+			<child link="${robot_namespace}${prefix}_base_link"/>
 		</joint>
-		<link name="${prefix}_base_link">
+		<link name="${robot_namespace}${prefix}_base_link">
 			<collision>
 				<origin xyz="0 0 0" rpy="0 0 0"/>
@@ -48,10 +48,10 @@
 			</inertial>
 		</link>
-		<joint name="${prefix}_joint" type="fixed">
-			<parent link="${prefix}_base_link"/>
-			<child link="${sensor_link_name}"/>
+		<joint name="${robot_namespace}${prefix}_joint" type="fixed">
+			<parent link="${robot_namespace}${prefix}_base_link"/>
+			<child link="${robot_namespace}${sensor_link_name}"/>
 			<origin xyz="0.0 0 0.0505" rpy="0 0 0"/>
 		</joint>
-		<link name="${sensor_link_name}" />
+		<link name="${robot_namespace}${sensor_link_name}" />
 		<!-- Sick sensor sensor for simulation -->
 		<xacro:sensor_sick_nanoscan3_gazebo />
