Commit message: arm  tf with prefixes

File: src/ros2/robot_description/rb_theron_common/rb_theron_description/robots/rb_theron.urdf.xacro (robot description, xacro)
@@ -170,4 +170,5 @@
 	<xacro:door_opening_mechanism
 	    prefix="$(arg prefix)"
+		robot_name="${robot_namespace}"
 		parent="$(arg prefix)base_link"
 		ros2_control_hardware_type="$(arg ros2_control_hardware_type)"

File: src/ros2/robot_description/rb_theron_common/rb_theron_description/urdf/door_opening_mechanism/arm_variations/rotating_arm.urdf.xacro (robot description, xacro)
@@ -6,8 +6,8 @@
                 izz="${m*(x*x+y*y)/12}" />
     </xacro:macro>
-    <xacro:macro name="rotating_arm" params="prefix parent ros2_control_hardware_type ros_distro *origin arm_length">
+    <xacro:macro name="rotating_arm" params="prefix parent robot_name ros2_control_hardware_type ros_distro *origin arm_length">
         <xacro:basic_joint
             parent="${prefix}${parent}"
-            joint_name="${prefix}door_opening_mechanism_joint_rotating_arm"
+            joint_name="${robot_name}${prefix}door_opening_mechanism_joint_rotating_arm"
             joint_type="revolute"
             axis_x="1"
@@ -23,5 +23,5 @@
             direction="0"
             ros_distro="${ros_distro}"
-            link_name="${prefix}door_opening_mechanism_link_rotating_arm"
+            link_name="${robot_name}${prefix}door_opening_mechanism_link_rotating_arm"
             link_origin_x="0.0"
             link_origin_y="0.0"
@@ -40,7 +40,7 @@
         path planning -->
         <xacro:basic_box
-            parent="${prefix}door_opening_mechanism_link_rotating_arm"
-            joint_name="${prefix}door_opening_mechanism_joint_gripper_adapter"
-            link_name="${prefix}door_opening_mechanism_link_gripper_adapter"
+            parent="${robot_name}${prefix}door_opening_mechanism_link_rotating_arm"
+            joint_name="${robot_name}${prefix}door_opening_mechanism_joint_gripper_adapter"
+            link_name="${robot_name}${prefix}door_opening_mechanism_link_gripper_adapter"
             m="0.1"
             x="0.01"
@@ -56,5 +56,6 @@
         <xacro:freely_rotating_hook
             prefix="${prefix}"
-            parent="${prefix}door_opening_mechanism_link_gripper_adapter"
+            parent="${robot_name}${prefix}door_opening_mechanism_link_gripper_adapter"
+            robot_name="${robot_name}"
             ros2_control_hardware_type="${ros2_control_hardware_type}"
             ros_distro="${ros_distro}">

File: src/ros2/robot_description/rb_theron_common/rb_theron_description/urdf/door_opening_mechanism/components/freely_rotating_hook.urdf.xacro (robot description, xacro)
@@ -1,9 +1,9 @@
 <?xml version="1.0"?>
 <robot name="freely_rotating_hook" xmlns:xacro="http://www.ros.org/wiki/xacro">
-    <xacro:macro name="freely_rotating_hook" params="prefix parent ros2_control_hardware_type ros_distro *origin">
+    <xacro:macro name="freely_rotating_hook" params="prefix parent robot_name ros2_control_hardware_type ros_distro *origin">
         <!-- Please mind: This joint is actually passive, but in order to help moveit plan the trajectory we make it active -->
         <xacro:basic_joint
             parent="${prefix}${parent}"
-            joint_name="${prefix}door_opening_mechanism_joint_freely_rotating_hook"
+            joint_name="${robot_name}${prefix}door_opening_mechanism_joint_freely_rotating_hook"
             joint_type="revolute"
             axis_x="1"
@@ -19,5 +19,5 @@
             direction="0"
             ros_distro="${ros_distro}"
-            link_name="${prefix}door_opening_mechanism_link_freely_rotating_hook"
+            link_name="${robot_name}${prefix}door_opening_mechanism_link_freely_rotating_hook"
             link_origin_x="0.0"
             link_origin_y="0.0"
@@ -34,5 +34,5 @@
         </xacro:basic_joint>
         <xacro:include filename="$(find rb_theron_description)/urdf/door_opening_mechanism/components/hook.urdf.xacro" />
-        <xacro:hook prefix="${prefix}" suffix="" parent="${prefix}door_opening_mechanism_link_freely_rotating_hook" r="1" g="0" b="1">
+        <xacro:hook prefix="${prefix}" suffix="" robot_name="${robot_name}" parent="${robot_name}${prefix}door_opening_mechanism_link_freely_rotating_hook" r="1" g="0" b="1">
             <origin xyz="0.01 0.0 0.0" rpy="0 0 -1.57079632679"/>
         </xacro:hook>

File: src/ros2/robot_description/rb_theron_common/rb_theron_description/urdf/door_opening_mechanism/components/hook.urdf.xacro (robot description, xacro)
@@ -6,5 +6,5 @@
                 izz="${m*(x*x+y*y)/12}" />
     </xacro:macro>
-    <xacro:macro name="hook" params="prefix suffix parent *origin r g b">
+    <xacro:macro name="hook" params="prefix suffix parent robot_name *origin r g b">
     <xacro:include filename="$(find rb_theron_description)/urdf/door_opening_mechanism/basic_elements/basic_box.urdf.xacro" />
     <xacro:basic_box

File: src/ros2/robot_description/rb_theron_common/rb_theron_description/urdf/door_opening_mechanism/door_opening_mechanism.urdf.xacro (robot description, xacro)
@@ -6,5 +6,5 @@
                 izz="${m*(x*x+y*y)/12}" />
     </xacro:macro>
-    <xacro:macro name="door_opening_mechanism" params="prefix parent ros2_control_hardware_type ros_distro *origin hq">
+    <xacro:macro name="door_opening_mechanism" params="prefix parent robot_name ros2_control_hardware_type ros_distro *origin hq">
         <!-- Element imports -->
         <xacro:include filename="$(find rb_theron_description)/urdf/door_opening_mechanism/components/alu_profile.urdf.xacro" />
@@ -16,8 +16,8 @@
         therefore steering of the rb_theron becomes impossible. -->
         <!-- Base link -->
-        <xacro:property name="door_opening_mechanism_base_link" value="${prefix}door_opening_mechanism_base_link" />
+        <xacro:property name="door_opening_mechanism_base_link" value="${robot_name}${prefix}door_opening_mechanism_base_link" />
         <xacro:basic_box
             parent="${parent}"
-            joint_name="${prefix}door_opening_mechanism_joint"
+            joint_name="${robot_name}${prefix}door_opening_mechanism_joint"
             link_name="${door_opening_mechanism_base_link}"
             m="0.001"
@@ -31,14 +31,14 @@
         </xacro:basic_box>
         <!-- Aluprofile frame -->
-        <xacro:alu_profile prefix="${prefix}" suffix="bottom" parent="${door_opening_mechanism_base_link}" x="0.03" y="0.03" z="0.46" r="0.1" g="0.1" b="0.1" >
+        <xacro:alu_profile prefix="${robot_name}${prefix}" suffix="bottom" parent="${door_opening_mechanism_base_link}" x="0.03" y="0.03" z="0.46" r="0.1" g="0.1" b="0.1" >
             <origin xyz="0 0 0" rpy="1.57079632679 0 0"/>
         </xacro:alu_profile>
-        <xacro:alu_profile prefix="${prefix}" suffix="left" parent="${door_opening_mechanism_base_link}" x="0.03" y="0.03" z="1.0" r="0.1" g="0.1" b="0.1" >
+        <xacro:alu_profile prefix="${robot_name}${prefix}" suffix="left" parent="${door_opening_mechanism_base_link}" x="0.03" y="0.03" z="1.0" r="0.1" g="0.1" b="0.1" >
             <origin xyz="0 -0.245 0.515" rpy="0 0 0"/>
         </xacro:alu_profile>
-        <xacro:alu_profile prefix="${prefix}" suffix="right" parent="${door_opening_mechanism_base_link}" x="0.03" y="0.03" z="1.0" r="0.1" g="0.1" b="0.1" >
+        <xacro:alu_profile prefix="${robot_name}${prefix}" suffix="right" parent="${door_opening_mechanism_base_link}" x="0.03" y="0.03" z="1.0" r="0.1" g="0.1" b="0.1" >
             <origin xyz="0 +0.245 0.515" rpy="0 0 0"/>
         </xacro:alu_profile>
-        <xacro:alu_profile prefix="${prefix}" suffix="top" parent="${door_opening_mechanism_base_link}" x="0.03" y="0.03" z="0.52" r="0.1" g="0.1" b="0.1" >
+        <xacro:alu_profile prefix="${robot_name}${prefix}" suffix="top" parent="${door_opening_mechanism_base_link}" x="0.03" y="0.03" z="0.52" r="0.1" g="0.1" b="0.1" >
             <origin xyz="0 0 1.03" rpy="1.57079632679 0 0"/>
         </xacro:alu_profile>
@@ -46,6 +46,6 @@
         <xacro:basic_box
             parent="${door_opening_mechanism_base_link}"
-            joint_name="${prefix}door_opening_mechanism_joint_y_axis_rail"
-            link_name="${prefix}door_opening_mechanism_link_y_axis_rail"
+            joint_name="${robot_name}${prefix}door_opening_mechanism_joint_y_axis_rail"
+            link_name="${robot_name}${prefix}door_opening_mechanism_link_y_axis_rail"
             m="2.64"
             x="0.06"
@@ -58,6 +58,6 @@
         </xacro:basic_box>
         <xacro:basic_joint
-            parent="${prefix}alu_profile_link_right"
-            joint_name="${prefix}door_opening_mechanism_joint_y_axis_slide"
+            parent="${robot_name}${prefix}alu_profile_link_right"
+            joint_name="${robot_name}${prefix}door_opening_mechanism_joint_y_axis_slide"
             joint_type="prismatic"
             axis_x="0"
@@ -73,5 +73,5 @@
             direction="1"
             ros_distro="${ros_distro}"
-            link_name="${prefix}door_opening_mechanism_link_y_axis_slide"
+            link_name="${robot_name}${prefix}door_opening_mechanism_link_y_axis_slide"
             link_origin_x="0.0"
             link_origin_y="0.0"
@@ -87,6 +87,6 @@
         </xacro:basic_joint>
         <xacro:basic_joint
-            parent="${prefix}door_opening_mechanism_link_y_axis_slide"
-            joint_name="${prefix}door_opening_mechanism_joint_x_axis_slide"
+            parent="${robot_name}${prefix}door_opening_mechanism_link_y_axis_slide"
+            joint_name="${robot_name}${prefix}door_opening_mechanism_joint_x_axis_slide"
             joint_type="prismatic"
             axis_x="0"
@@ -102,5 +102,5 @@
             direction="-1"
             ros_distro="${ros_distro}"
-            link_name="${prefix}door_opening_mechanism_link_x_axis_slide"
+            link_name="${robot_name}${prefix}door_opening_mechanism_link_x_axis_slide"
             link_origin_x="0.0"
             link_origin_y="0.0"
@@ -116,7 +116,7 @@
         </xacro:basic_joint>
         <xacro:basic_box
-            parent="${prefix}door_opening_mechanism_link_x_axis_slide"
-            joint_name="${prefix}door_opening_mechanism_joint_x_axis_slide_screwing"
-            link_name="${prefix}door_opening_mechanism_link_x_slide_screwing"
+            parent="${robot_name}${prefix}door_opening_mechanism_link_x_axis_slide"
+            joint_name="${robot_name}${prefix}door_opening_mechanism_joint_x_axis_slide_screwing"
+            link_name="${robot_name}${prefix}door_opening_mechanism_link_x_slide_screwing"
             m="1"
             x="0.073"
@@ -137,5 +137,6 @@
         <xacro:rotating_arm
             prefix="${prefix}"
-            parent="${prefix}door_opening_mechanism_link_x_slide_screwing"
+            parent="${robot_name}${prefix}door_opening_mechanism_link_x_slide_screwing"
+            robot_name="${robot_name}"
             ros2_control_hardware_type="${ros2_control_hardware_type}"
             ros_distro="${ros_distro}"

Commit message: feat: model the base movement as a prismatic joint between base_footprint and base_link

File: src/ros2/robot_description/rb_theron_common/rb_theron_description/robots/rb_theron.urdf.xacro (robot description, xacro)
@@ -37,4 +37,6 @@
     <xacro:arg name="ros2_control_hardware_type" default="mock_components" />
 	<xacro:arg name="ros_distro" default="humble" />
+	<!-- Whether the position joint should be modeled as a prismatic joint or just as a fixed joint -->
+	<xacro:arg name="model_position_joint" default="false" />
 	<!-- *************** -->
 	<!-- Robots Elements -->
@@ -46,5 +48,6 @@
 	  publish_bf="${publish_bf}"
 	  ros2_control_hardware_type="$(arg ros2_control_hardware_type)"
-	  ros_distro="$(arg ros_distro)">
+	  ros_distro="$(arg ros_distro)"
+	  model_position_joint="$(arg model_position_joint)">
 	</xacro:rb_theron_base>
 	<!-- Gazebo ros control pluggins -->

File: src/ros2/robot_description/rb_theron_common/rb_theron_description/robots/rb_theron_base.urdf.xacro (robot description, xacro)
@@ -20,6 +20,11 @@
   <!-- Robots Elements -->
   <!-- *************** -->
-  <xacro:macro name="rb_theron_base" params="prefix hq publish_bf ros2_control_hardware_type ros_distro">
-    <xacro:theron_base prefix="${prefix}" publish_bf="${publish_bf}" hq="${hq}" />
+  <xacro:macro name="rb_theron_base" params="prefix hq publish_bf ros2_control_hardware_type ros_distro model_position_joint">
+    <xacro:theron_base
+      prefix="${prefix}"
+      publish_bf="${publish_bf}"
+      model_position_joint="${model_position_joint}"
+      hq="${hq}"
+    />
     <xacro:gazebo_colors prefix="${prefix}"/>
     <!-- WHEELS -->

File: src/ros2/robot_description/rb_theron_common/rb_theron_description/urdf/bases/theron_base.urdf.xacro (robot description, xacro)
@@ -6,22 +6,7 @@
               izz="${m*(x*x+y*y)/12}" />
   </xacro:macro>
-  <xacro:macro name="theron_base" params="prefix publish_bf hq">
+  <xacro:macro name="theron_base" params="prefix publish_bf model_position_joint hq">
     <xacro:property name="PI" value="3.1415926535897931"/>
     <!-- xacro:property name="wheel_width" value="0.150" / -->
-    <!-- This is the joint we configured with Henning. We might not need it as a planar joint with 3 DOFs. It might be enough
-    to configure this joint as a prismatic joint with 1 DOF as we do only need to drive strictly forwards and backwards
-    during the door opening process -->
-    <!-- <ros2_control name="position_ros2_control" type="system">
-      <hardware>
-          <plugin>fake_components/GenericSystem</plugin>
-      </hardware>
-      <joint name="position" type="planar">
-          <param name="initial_position">0.0 0.0 0.0</param>
-          <command_interface name="position" />
-          <command_interface name="velocity" />
-          <state_interface name="position"/>
-          <state_interface name="velocity"/>
-      </joint>
-    </ros2_control> -->
     <!-- BASE FOOTPRINT -->
     <xacro:if value="${publish_bf}">
@@ -40,9 +25,33 @@
         </collision>
       </link>
-      <joint name="${prefix}base_footprint_joint" type="fixed">
-        <origin xyz="0 0 ${wheel_radius - wheel_offset_z}" rpy="0 0 0" />
-        <parent link="${prefix}base_footprint"/>
-        <child link="${prefix}base_link" />
-      </joint>
+      <xacro:if value="${model_position_joint}">
+        <joint name="position" type="prismatic">
+          <axis xyz="1 0 0" />
+          <origin xyz="0 0 ${wheel_radius - wheel_offset_z}" rpy="0 0 0" />
+          <parent link="${prefix}base_footprint"/>
+          <child link="${prefix}base_link"/>
+          <limit lower="-1" upper="1" effort="1000" velocity="100" />
+          <!-- <dynamics damping="${damping}" friction="${friction}"/> -->
+        </joint>
+        <ros2_control name="position_ros2_control" type="system">
+          <hardware>
+              <plugin>fake_components/GenericSystem</plugin>
+          </hardware>
+          <joint name="position" type="prismatic">
+              <param name="initial_position">0.0</param>
+              <command_interface name="position" />
+              <command_interface name="velocity" />
+              <state_interface name="position"/>
+              <state_interface name="velocity"/>
+          </joint>
+        </ros2_control>
+      </xacro:if>
+      <xacro:unless value="${model_position_joint}">
+        <joint name="${prefix}base_footprint_joint" type="fixed">
+          <origin xyz="0 0 ${wheel_radius - wheel_offset_z}" rpy="0 0 0" />
+          <parent link="${prefix}base_footprint"/>
+          <child link="${prefix}base_link"/>
+        </joint>
+      </xacro:unless>
     </xacro:if>
     <!-- BASE_LINK -->

Commit message: feat(WIP): adds first draft for ros2_control plugin for linear_base_movement

File: src/ros2/robot_description/rb_theron_common/rb_theron_description/robots/rb_theron.urdf.xacro (robot description, xacro)
@@ -36,4 +36,5 @@
 	-->
     <xacro:arg name="ros2_control_hardware_type" default="mock_components" />
+	<xacro:arg name="ros2_control_hardware_type_positon_joint" default="mock_components" />
 	<xacro:arg name="ros_distro" default="humble" />
 	<!-- Whether the position joint should be modeled as a prismatic joint or just as a fixed joint -->
@@ -48,4 +49,5 @@
 	  publish_bf="${publish_bf}"
 	  ros2_control_hardware_type="$(arg ros2_control_hardware_type)"
+	  ros2_control_hardware_type_positon_joint="$(arg ros2_control_hardware_type_positon_joint)"
 	  ros_distro="$(arg ros_distro)"
 	  model_position_joint="$(arg model_position_joint)">

File: src/ros2/robot_description/rb_theron_common/rb_theron_description/robots/rb_theron_base.urdf.xacro (robot description, xacro)
@@ -20,9 +20,19 @@
   <!-- Robots Elements -->
   <!-- *************** -->
-  <xacro:macro name="rb_theron_base" params="prefix hq publish_bf ros2_control_hardware_type ros_distro model_position_joint">
+  <xacro:macro
+    name="rb_theron_base"
+    params="
+      prefix
+      hq
+      publish_bf
+      ros2_control_hardware_type
+      ros2_control_hardware_type_positon_joint
+      ros_distro
+      model_position_joint">
     <xacro:theron_base
       prefix="${prefix}"
       publish_bf="${publish_bf}"
       model_position_joint="${model_position_joint}"
+      ros2_control_hardware_type_positon_joint="${ros2_control_hardware_type_positon_joint}"
       hq="${hq}"
     />

File: src/ros2/robot_description/rb_theron_common/rb_theron_description/urdf/bases/theron_base.urdf.xacro (robot description, xacro)
@@ -6,5 +6,5 @@
               izz="${m*(x*x+y*y)/12}" />
   </xacro:macro>
-  <xacro:macro name="theron_base" params="prefix publish_bf model_position_joint hq">
+  <xacro:macro name="theron_base" params="prefix publish_bf model_position_joint ros2_control_hardware_type_positon_joint hq">
     <xacro:property name="PI" value="3.1415926535897931"/>
     <!-- xacro:property name="wheel_width" value="0.150" / -->
@@ -27,5 +27,5 @@
       <xacro:if value="${model_position_joint}">
         <joint name="position" type="prismatic">
-          <axis xyz="1 0 0" />
+          <axis xyz="-1 0 0" />
           <origin xyz="0 0 ${wheel_radius - wheel_offset_z}" rpy="0 0 0" />
           <parent link="${prefix}base_footprint"/>
@@ -36,5 +36,11 @@
         <ros2_control name="position_ros2_control" type="system">
           <hardware>
-              <plugin>fake_components/GenericSystem</plugin>
+            <xacro:if value="${ros2_control_hardware_type_positon_joint == 'mock_components'}">
+              <plugin>mock_components/GenericSystem</plugin>
+              <param name="calculate_dynamics">true</param>
+            </xacro:if>
+            <xacro:if value="${ros2_control_hardware_type_positon_joint == 'linear_base_movement'}">
+              <plugin>ros2_control_plugin_linear_base_movement/LinearBaseMovementSystemHardware</plugin>
+            </xacro:if>
           </hardware>
           <joint name="position" type="prismatic">
