Commit message: fix: sensor_base_frame for sensor data generated from gazebo sensor plugins

File: src/ros2/robot_description/rb_theron_common/rb_theron_description/robots/rb_theron.urdf.xacro (robot description, xacro)
@@ -40,4 +40,17 @@
 	<!-- Whether the position joint should be modeled as a prismatic joint or just as a fixed joint -->
 	<xacro:arg name="model_position_joint" default="false" />
+	<!-- If we model the position joint, the sensors need be placed in the base_link frame,
+	otherwise they should be placed in the base_footprint frame -->
+	<xacro:if value="$(arg model_position_joint)">
+		<xacro:property name="sensor_base_frame" value="base_link" />
+	</xacro:if>
+	<xacro:unless value="$(arg model_position_joint)">
+		<xacro:if value="${publish_bf}">
+			<xacro:property name="sensor_base_frame" value="base_footprint" />
+		</xacro:if>
+		<xacro:unless value="${publish_bf}">
+			<xacro:property name="sensor_base_frame" value="base_link" />
+		</xacro:unless>
+	</xacro:unless>
 	<!-- *************** -->
 	<!-- Robots Elements -->
@@ -59,12 +72,12 @@
 	<!-- TODO: Should be sensor_intel_d435, but this one isn't migrated to ros2 yet -->
 	<!-- TODO: Moved 0.01 in x, otherwise the camera is still inside the robot -->
-	<xacro:sensor_r430 prefix="$(arg prefix)front_realsense_camera" parent="$(arg prefix)base_link" publish_bf="${publish_bf}" robot_name="${robot_name}" prefix_topic="front_realsense_camera" hq="${hq}">
+	<xacro:sensor_r430 prefix="$(arg prefix)front_realsense_camera" parent="$(arg prefix)base_link" sensor_base_frame="${sensor_base_frame}" robot_name="${robot_name}" prefix_topic="front_realsense_camera" hq="${hq}">
 		<origin xyz="0.3305 0.0 0.1468" rpy="0 0 0"/>
 	</xacro:sensor_r430>
-	<xacro:sensor_r430 prefix="$(arg prefix)back_realsense_camera" parent="$(arg prefix)base_link" publish_bf="${publish_bf}" robot_name="${robot_name}" prefix_topic="back_realsense_camera" hq="${hq}">
+	<xacro:sensor_r430 prefix="$(arg prefix)back_realsense_camera" parent="$(arg prefix)base_link" sensor_base_frame="${sensor_base_frame}" robot_name="${robot_name}" prefix_topic="back_realsense_camera" hq="${hq}">
 		<origin xyz="-0.3305 0.0 0.1468" rpy="0 0 3.1416"/>
 	</xacro:sensor_r430>
 	<!--Added back top realsense camera because running YOLO network on depthai camera in simulation reduces Real Time Factor (RTF)-->
-	<xacro:sensor_r430 prefix="$(arg prefix)back_top_realsense_camera" parent="$(arg prefix)base_link" publish_bf="${publish_bf}" robot_name="${robot_name}" prefix_topic="back_top_realsense_camera" hq="${hq}">
+	<xacro:sensor_r430 prefix="$(arg prefix)back_top_realsense_camera" parent="$(arg prefix)base_link" sensor_base_frame="${sensor_base_frame}" robot_name="${robot_name}" prefix_topic="back_top_realsense_camera" hq="${hq}">
 		<origin xyz="-0.3305 0.0 1.1468" rpy="0 0 3.1416"/>
 	</xacro:sensor_r430>
@@ -73,8 +86,8 @@
 		<origin xyz="0.3305 0.0 0.1898" rpy="0 0 0"/>
 	</xacro:sensor_orbbec_astra -->
-	<xacro:sensor_imu_hector prefix="$(arg prefix)imu" parent="$(arg prefix)base_link">
+	<xacro:sensor_imu_hector prefix="$(arg prefix)imu" parent="$(arg prefix)base_link" sensor_base_frame="${sensor_base_frame}">
 		<origin xyz="-0.1975 0.0 0.1598" rpy="0 0 0"/>
 	</xacro:sensor_imu_hector>
-	<xacro:sensor_sick_nanoscan3 prefix="$(arg prefix)front_laser" parent="$(arg prefix)base_link" publish_bf="${publish_bf}" robot_name="${robot_name}" prefix_topic="front_laser" hq="${hq}" min_angle="-1.9507619" max_angle="1.9507619" gpu="true">
+	<xacro:sensor_sick_nanoscan3 prefix="$(arg prefix)front_laser" parent="$(arg prefix)base_link" sensor_base_frame="${sensor_base_frame}" robot_name="${robot_name}" prefix_topic="front_laser" hq="${hq}" min_angle="-1.9507619" max_angle="1.9507619" gpu="true">
 		<origin xyz="0.250 0.0 0.1643" rpy="0 3.1416 3.1416"/>
 	</xacro:sensor_sick_nanoscan3>
@@ -82,5 +95,5 @@
 		<origin xyz="0.214 0.0 0.275" rpy="-1.57079632679 0 -0.23"/>
 	</xacro:sensor_rs_lidar_16>-->
-	<xacro:sensor_rs_bpearl prefix="$(arg prefix)top_laser" parent="$(arg prefix)base_link" publish_bf="${publish_bf}" robot_name="${robot_name}" prefix_topic="top_laser" hq="${hq}" range_min="0.1" range_max="90" hfov="360" samples="1800" vfov="90.0" lasers="32" fps="10" gpu="false">
+	<xacro:sensor_rs_bpearl prefix="$(arg prefix)top_laser" parent="$(arg prefix)base_link" sensor_base_frame="${sensor_base_frame}" robot_name="${robot_name}" prefix_topic="top_laser" hq="${hq}" range_min="0.1" range_max="90" hfov="360" samples="1800" vfov="90.0" lasers="32" fps="10" gpu="false">
 		<origin xyz="0.3 -0.175 1.165" rpy="-1.570796326795 0 -1.570796326795"/>
 		<!-- positions of the b-pearl based on solid: xyz="0.333 -0.180 1.194" rpy="-1.570796326795 0 -1.570796326795" -->
@@ -100,5 +113,5 @@
 		prefix="$(arg prefix)front_top_oak_d_camera"
 		parent="$(arg prefix)base_link"
-		publish_bf="${publish_bf}"
+		sensor_base_frame="${sensor_base_frame}"
 		robot_name="${robot_name}"
 		prefix_topic="front_top_oak_d_camera"

File: src/ros2/robot_description/robotnik_sensors/urdf/depthai_macro.urdf.xacro (robot description, xacro)
@@ -1,14 +1,9 @@
 <?xml version="1.0"?>
 <robot name="depthai_camera" xmlns:xacro="http://ros.org/wiki/xacro">
-<xacro:macro name="depthai_camera" params="prefix parent publish_bf robot_name prefix_topic camera_model base_frame
+<xacro:macro name="depthai_camera" params="prefix parent sensor_base_frame robot_name prefix_topic camera_model base_frame
                                            cam_pos_x cam_pos_y cam_pos_z
                                            cam_roll cam_pitch cam_yaw hq
                                            r:=0.8 g:=0.8 b:=0.8 a:=0.8">
-    <xacro:if value="${publish_bf}">
-			<xacro:property name="sensor_link_name" value="${robot_name}/base_footprint/${prefix}" />
-		</xacro:if>
-		<xacro:unless value="${publish_bf}">
-			<xacro:property name="sensor_link_name" value="${robot_name}/base_link/${prefix}" />
-		</xacro:unless>
+    <xacro:property name="sensor_link_name" value="${robot_name}/${sensor_base_frame}/${prefix}" />
     <xacro:property name="M_PI"     value="3.1415926535897931" />
     <xacro:property name="model"    value="${camera_model}" />

File: src/ros2/robot_description/robotnik_sensors/urdf/imu_hector_plugin.urdf.xacro (robot description, xacro)
@@ -1,11 +1,6 @@
 <?xml version="1.0"?>
 <robot name="sensor_imu" xmlns:xacro="http://wiki.ros.org/xacro">
-	<xacro:macro name="sensor_imu_hector" params="prefix topic:='imu/data' parent *origin">
-		<xacro:if value="${publish_bf}">
-			<xacro:property name="sensor_link_name" value="${robot_name}/base_footprint/${prefix}_link" />
-		</xacro:if>
-		<xacro:unless value="${publish_bf}">
-			<xacro:property name="sensor_link_name" value="${robot_name}/base_link/${prefix}_link" />
-		</xacro:unless>
+	<xacro:macro name="sensor_imu_hector" params="prefix topic:='imu/data' parent sensor_base_frame *origin">
+		<xacro:property name="sensor_link_name" value="${robot_name}/${sensor_base_frame}/${prefix}_link" />
 		<joint name="${prefix}_joint" type="fixed">
 			<axis xyz="1 0 0"/>

File: src/ros2/robot_description/robotnik_sensors/urdf/intel_r430.urdf.xacro (robot description, xacro)
@@ -19,11 +19,6 @@
   <xacro:property name="r430_cam_depth_py" value="-0.0115"/>
   <xacro:property name="r430_cam_depth_pz" value="0.0"/>
-  <xacro:macro name="sensor_r430" params="prefix parent publish_bf robot_name prefix_topic:='front_rgbd_camera' hq *origin">
-    <xacro:if value="${publish_bf}">
-			<xacro:property name="sensor_link_name" value="${robot_name}/base_footprint/${prefix}" />
-		</xacro:if>
-		<xacro:unless value="${publish_bf}">
-			<xacro:property name="sensor_link_name" value="${robot_name}/base_link/${prefix}" />
-		</xacro:unless>
+  <xacro:macro name="sensor_r430" params="prefix parent sensor_base_frame robot_name prefix_topic:='front_rgbd_camera' hq *origin">
+    <xacro:property name="sensor_link_name" value="${robot_name}/${sensor_base_frame}/${prefix}" />
     <!-- camera body, with origin at bottom screw mount -->
     <joint name="${prefix}_camera_joint" type="fixed">

File: src/ros2/robot_description/robotnik_sensors/urdf/rs_bpearl.urdf.xacro (robot description, xacro)
@@ -2,11 +2,6 @@
 <robot name="sensor_rs_bpearl" xmlns:xacro="http://wiki.ros.org/xacro">
   <xacro:property name="M_PI" value="3.1415926535897931" />
-  <xacro:macro name="sensor_rs_bpearl" params="prefix parent publish_bf robot_name prefix_topic hq *origin range_min range_max hfov samples vfov lasers fps gpu:=true">
-    <xacro:if value="${publish_bf}">
-			<xacro:property name="sensor_link_name" value="${robot_name}/base_footprint/${prefix}_link" />
-		</xacro:if>
-		<xacro:unless value="${publish_bf}">
-			<xacro:property name="sensor_link_name" value="${robot_name}/base_link/${prefix}_link" />
-		</xacro:unless>
+  <xacro:macro name="sensor_rs_bpearl" params="prefix parent sensor_base_frame robot_name prefix_topic hq *origin range_min range_max hfov samples vfov lasers fps gpu:=true">
+    <xacro:property name="sensor_link_name" value="${robot_name}/${sensor_base_frame}/${prefix}_link" />
     <joint name="${prefix}_base_joint" type="fixed">
       <xacro:insert_block name="origin" />

File: src/ros2/robot_description/robotnik_sensors/urdf/sick_nanoscan3.urdf.xacro (robot description, xacro)
@@ -2,11 +2,6 @@
 <robot name="sensor_sick_nanoscan3"
 	xmlns:xacro="http://wiki.ros.org/xacro">
-	<xacro:macro name="sensor_sick_nanoscan3" params="prefix parent publish_bf robot_name prefix_topic:='front_laser' hq *origin max_angle:=2.3998 min_angle:=-2.3998 gpu:=^|false">
-		<xacro:if value="${publish_bf}">
-			<xacro:property name="sensor_link_name" value="${robot_name}/base_footprint/${prefix}_link" />
-		</xacro:if>
-		<xacro:unless value="${publish_bf}">
-			<xacro:property name="sensor_link_name" value="${robot_name}/base_link/${prefix}_link" />
-		</xacro:unless>
+	<xacro:macro name="sensor_sick_nanoscan3" params="prefix parent sensor_base_frame robot_name prefix_topic:='front_laser' hq *origin max_angle:=2.3998 min_angle:=-2.3998 gpu:=^|false">
+		<xacro:property name="sensor_link_name" value="${robot_name}/${sensor_base_frame}/${prefix}_link" />
 		<joint name="${prefix}_base_joint" type="fixed">
 			<xacro:insert_block name="origin" />

Commit message: feat: changes parent of `door_opening_mechanism` in dependency of ros2_control_hardware_type

File: src/ros2/robot_description/rb_theron_common/rb_theron_description/robots/rb_theron.urdf.xacro (robot description, xacro)
@@ -180,7 +180,14 @@
 	<!-- ROBAST Door Opening Mechanism -->
 	<xacro:include filename="$(find rb_theron_description)/urdf/door_opening_mechanism/door_opening_mechanism.urdf.xacro" />
+	<xacro:property name="ros2_control_hardware_type" value="$(arg ros2_control_hardware_type)" />
+	<xacro:if value="${ros2_control_hardware_type == 'dryve_d1'}">
+		<xacro:property name="door_opening_mechanism_parent" value="$(arg prefix)robot_base_link" />
+	</xacro:if>
+	<xacro:unless value="${ros2_control_hardware_type == 'dryve_d1'}">
+		<xacro:property name="door_opening_mechanism_parent" value="$(arg prefix)base_link" />
+	</xacro:unless>
 	<xacro:door_opening_mechanism
 	    prefix="$(arg prefix)"
-		parent="$(arg prefix)base_link"
+		parent="${door_opening_mechanism_parent}"
 		ros2_control_hardware_type="$(arg ros2_control_hardware_type)"
 		ros_distro="$(arg ros_distro)"

Commit message: fix: adds `robot_name` argument to `sensor_imu_hector` macro

File: src/ros2/robot_description/rb_theron_common/rb_theron_description/robots/rb_theron.urdf.xacro (robot description, xacro)
@@ -86,5 +86,5 @@
 		<origin xyz="0.3305 0.0 0.1898" rpy="0 0 0"/>
 	</xacro:sensor_orbbec_astra -->
-	<xacro:sensor_imu_hector prefix="$(arg prefix)imu" parent="$(arg prefix)base_link" sensor_base_frame="${sensor_base_frame}">
+	<xacro:sensor_imu_hector prefix="$(arg prefix)imu" parent="$(arg prefix)base_link" sensor_base_frame="${sensor_base_frame}" robot_name="${robot_name}">
 		<origin xyz="-0.1975 0.0 0.1598" rpy="0 0 0"/>
 	</xacro:sensor_imu_hector>

File: src/ros2/robot_description/robotnik_sensors/urdf/imu_hector_plugin.urdf.xacro (robot description, xacro)
@@ -1,5 +1,5 @@
 <?xml version="1.0"?>
 <robot name="sensor_imu" xmlns:xacro="http://wiki.ros.org/xacro">
-	<xacro:macro name="sensor_imu_hector" params="prefix topic:='imu/data' parent sensor_base_frame *origin">
+	<xacro:macro name="sensor_imu_hector" params="prefix topic:='imu/data' parent sensor_base_frame robot_name *origin">
 		<xacro:property name="sensor_link_name" value="${robot_name}/${sensor_base_frame}/${prefix}_link" />
 		<joint name="${prefix}_joint" type="fixed">

Commit message: fix: take base_link as parent for the door_opening_mechanism again

File: src/ros2/robot_description/rb_theron_common/rb_theron_description/robots/rb_theron.urdf.xacro (robot description, xacro)
@@ -180,14 +180,7 @@
 	<!-- ROBAST Door Opening Mechanism -->
 	<xacro:include filename="$(find rb_theron_description)/urdf/door_opening_mechanism/door_opening_mechanism.urdf.xacro" />
-	<xacro:property name="ros2_control_hardware_type" value="$(arg ros2_control_hardware_type)" />
-	<xacro:if value="${ros2_control_hardware_type == 'dryve_d1'}">
-		<xacro:property name="door_opening_mechanism_parent" value="$(arg prefix)robot_base_link" />
-	</xacro:if>
-	<xacro:unless value="${ros2_control_hardware_type == 'dryve_d1'}">
-		<xacro:property name="door_opening_mechanism_parent" value="$(arg prefix)base_link" />
-	</xacro:unless>
 	<xacro:door_opening_mechanism
 	    prefix="$(arg prefix)"
-		parent="${door_opening_mechanism_parent}"
+		parent="$(arg prefix)base_link"
 		ros2_control_hardware_type="$(arg ros2_control_hardware_type)"
 		ros_distro="$(arg ros_distro)"

File: src/ros2/robot_description/rb_theron_common/rb_theron_description/robots/rb_theron_arm.urdf.xacro (robot description, xacro)
@@ -48,14 +48,7 @@
 	<!-- ROBAST Door Opening Mechanism -->
 	<xacro:include filename="$(find rb_theron_description)/urdf/door_opening_mechanism/door_opening_mechanism.urdf.xacro" />
-	<xacro:property name="ros2_control_hardware_type" value="$(arg ros2_control_hardware_type)" />
-	<xacro:if value="${ros2_control_hardware_type == 'dryve_d1'}">
-		<xacro:property name="door_opening_mechanism_parent" value="$(arg prefix)robot_base_link" />
-	</xacro:if>
-	<xacro:unless value="${ros2_control_hardware_type == 'dryve_d1'}">
-		<xacro:property name="door_opening_mechanism_parent" value="$(arg prefix)base_link" />
-	</xacro:unless>
 	<xacro:door_opening_mechanism
 	    prefix="$(arg prefix)"
-		parent="${door_opening_mechanism_parent}"
+		parent="$(arg prefix)base_link"
 		ros2_control_hardware_type="$(arg ros2_control_hardware_type)"
 		ros_distro="$(arg ros_distro)"

Commit message: feat: disable door_opening_mechanism for normal robot simulation

File: src/ros2/robot_description/rb_theron_common/rb_theron_description/robots/rb_theron.urdf.xacro (robot description, xacro)
@@ -179,13 +179,16 @@
 	</xacro:drawer>
 	<!-- ROBAST Door Opening Mechanism -->
-	<xacro:include filename="$(find rb_theron_description)/urdf/door_opening_mechanism/door_opening_mechanism.urdf.xacro" />
-	<xacro:door_opening_mechanism
-	    prefix="$(arg prefix)"
-		parent="$(arg prefix)base_link"
-		ros2_control_hardware_type="$(arg ros2_control_hardware_type)"
-		ros_distro="$(arg ros_distro)"
-		hq="${hq}">
-		<origin xyz="-0.3 0 0.225" rpy="0 0 0"/>
-	</xacro:door_opening_mechanism>
+	<!-- The door opening mechanism should NOT be included when used for normal navigation simulations. -->
+	<xacro:if value="$(arg model_position_joint)">
+		<xacro:include filename="$(find rb_theron_description)/urdf/door_opening_mechanism/door_opening_mechanism.urdf.xacro" />
+		<xacro:door_opening_mechanism
+			prefix="$(arg prefix)"
+			parent="$(arg prefix)base_link"
+			ros2_control_hardware_type="$(arg ros2_control_hardware_type)"
+			ros_distro="$(arg ros_distro)"
+			hq="${hq}">
+			<origin xyz="-0.3 0 0.225" rpy="0 0 0"/>
+		</xacro:door_opening_mechanism>
+	</xacro:if>
 	<!-- Gazebo plugins -->
 	<xacro:ros_control ros_distro="$(arg ros_distro)"/>
