Commit message: feat: introduce linear mobile base movement with new ros2_controller (RE-1902) (#102)
This PR relates to RE-1902. It includes:
- a new hardware_interface ros2_control_base_movement for moving the robot base in a linear motion forwards and backwards in real life (inherits from the SystemInterface)
- a new hardware_interface gz_ros2_control_base_movement for moving the robot base in a linear motion forwards and backwards in Gazebo resp. Ignition (inherits from the GazeboSimSystemInterface resp. IgnitionSystemInterface)
- a new ros2_controller mobile_base_controller (inherits from the ChainableControllerInterface) which generates cmd_vel commands out the planed linear motions it receives
- updating the door_opening_mechanism.urdf to our current setup
- the option to add a newly introduced position_joint to the /tf tree, which is responsible for planing the linear base movement and is placed between the base_link and the base_footprint. Therefore it is important to keep this in a separate namespace like /arm/tf to not disturb the normal navigation.
- a new launch_manager package, which can contain nodes, that help with launching nodes in the right order. At a first helper node this PR introduces the rosout_listener which exits after it received a certain trigger msg on the /rosout topic

Furthermore:
- integrating endstops, which was originally formulated in RE-1960
- replaces hard coded ros distro by value of env var ROS_DISTRO
- a lot of formatting "fixes" to get green tests for flake8 and pep257 in the moveit docker container
- some renamings

File: src/ros2/robot_description/rb_theron_common/rb_theron_description/robots/rb_theron.urdf.xacro (robot description, xacro)
@@ -36,5 +36,21 @@
 	-->
     <xacro:arg name="ros2_control_hardware_type" default="mock_components" />
+	<xacro:arg name="ros2_control_hardware_type_positon_joint" default="mock_components" />
 	<xacro:arg name="ros_distro" default="humble" />
+	<!-- Whether the position joint should be modeled as a prismatic joint or just as a fixed joint -->
+	<xacro:arg name="model_position_joint" default="false" />
+	<!-- If we model the position joint, the sensors need be placed in the base_link frame,
+	otherwise they should be placed in the base_footprint frame -->
+	<xacro:if value="$(arg model_position_joint)">
+		<xacro:property name="sensor_base_frame" value="base_link" />
+	</xacro:if>
+	<xacro:unless value="$(arg model_position_joint)">
+		<xacro:if value="${publish_bf}">
+			<xacro:property name="sensor_base_frame" value="base_footprint" />
+		</xacro:if>
+		<xacro:unless value="${publish_bf}">
+			<xacro:property name="sensor_base_frame" value="base_link" />
+		</xacro:unless>
+	</xacro:unless>
 	<!-- *************** -->
 	<!-- Robots Elements -->
@@ -46,5 +62,7 @@
 	  publish_bf="${publish_bf}"
 	  ros2_control_hardware_type="$(arg ros2_control_hardware_type)"
-	  ros_distro="$(arg ros_distro)">
+	  ros2_control_hardware_type_positon_joint="$(arg ros2_control_hardware_type_positon_joint)"
+	  ros_distro="$(arg ros_distro)"
+	  model_position_joint="$(arg model_position_joint)">
 	</xacro:rb_theron_base>
 	<!-- Gazebo ros control pluggins -->
@@ -54,12 +72,12 @@
 	<!-- TODO: Should be sensor_intel_d435, but this one isn't migrated to ros2 yet -->
 	<!-- TODO: Moved 0.01 in x, otherwise the camera is still inside the robot -->
-	<xacro:sensor_r430 prefix="$(arg prefix)front_realsense_camera" parent="$(arg prefix)base_link" publish_bf="${publish_bf}" robot_name="${robot_name}" prefix_topic="front_realsense_camera" hq="${hq}">
+	<xacro:sensor_r430 prefix="$(arg prefix)front_realsense_camera" parent="$(arg prefix)base_link" sensor_base_frame="${sensor_base_frame}" robot_name="${robot_name}" prefix_topic="front_realsense_camera" hq="${hq}">
 		<origin xyz="0.3305 0.0 0.1468" rpy="0 0 0"/>
 	</xacro:sensor_r430>
-	<xacro:sensor_r430 prefix="$(arg prefix)back_realsense_camera" parent="$(arg prefix)base_link" publish_bf="${publish_bf}" robot_name="${robot_name}" prefix_topic="back_realsense_camera" hq="${hq}">
+	<xacro:sensor_r430 prefix="$(arg prefix)back_realsense_camera" parent="$(arg prefix)base_link" sensor_base_frame="${sensor_base_frame}" robot_name="${robot_name}" prefix_topic="back_realsense_camera" hq="${hq}">
 		<origin xyz="-0.3305 0.0 0.1468" rpy="0 0 3.1416"/>
 	</xacro:sensor_r430>
 	<!--Added back top realsense camera because running YOLO network on depthai camera in simulation reduces Real Time Factor (RTF)-->
-	<xacro:sensor_r430 prefix="$(arg prefix)back_top_realsense_camera" parent="$(arg prefix)base_link" publish_bf="${publish_bf}" robot_name="${robot_name}" prefix_topic="back_top_realsense_camera" hq="${hq}">
+	<xacro:sensor_r430 prefix="$(arg prefix)back_top_realsense_camera" parent="$(arg prefix)base_link" sensor_base_frame="${sensor_base_frame}" robot_name="${robot_name}" prefix_topic="back_top_realsense_camera" hq="${hq}">
 		<origin xyz="-0.3305 0.0 1.1468" rpy="0 0 3.1416"/>
 	</xacro:sensor_r430>
@@ -68,8 +86,8 @@
 		<origin xyz="0.3305 0.0 0.1898" rpy="0 0 0"/>
 	</xacro:sensor_orbbec_astra -->
-	<xacro:sensor_imu_hector prefix="$(arg prefix)imu" parent="$(arg prefix)base_link">
+	<xacro:sensor_imu_hector prefix="$(arg prefix)imu" parent="$(arg prefix)base_link" sensor_base_frame="${sensor_base_frame}" robot_name="${robot_name}">
 		<origin xyz="-0.1975 0.0 0.1598" rpy="0 0 0"/>
 	</xacro:sensor_imu_hector>
-	<xacro:sensor_sick_nanoscan3 prefix="$(arg prefix)front_laser" parent="$(arg prefix)base_link" publish_bf="${publish_bf}" robot_name="${robot_name}" prefix_topic="front_laser" hq="${hq}" min_angle="-1.9507619" max_angle="1.9507619" gpu="true">
+	<xacro:sensor_sick_nanoscan3 prefix="$(arg prefix)front_laser" parent="$(arg prefix)base_link" sensor_base_frame="${sensor_base_frame}" robot_name="${robot_name}" prefix_topic="front_laser" hq="${hq}" min_angle="-1.9507619" max_angle="1.9507619" gpu="true">
 		<origin xyz="0.250 0.0 0.1643" rpy="0 3.1416 3.1416"/>
 	</xacro:sensor_sick_nanoscan3>
@@ -77,5 +95,5 @@
 		<origin xyz="0.214 0.0 0.275" rpy="-1.57079632679 0 -0.23"/>
 	</xacro:sensor_rs_lidar_16>-->
-	<xacro:sensor_rs_bpearl prefix="$(arg prefix)top_laser" parent="$(arg prefix)base_link" publish_bf="${publish_bf}" robot_name="${robot_name}" prefix_topic="top_laser" hq="${hq}" range_min="0.1" range_max="90" hfov="360" samples="1800" vfov="90.0" lasers="32" fps="10" gpu="false">
+	<xacro:sensor_rs_bpearl prefix="$(arg prefix)top_laser" parent="$(arg prefix)base_link" sensor_base_frame="${sensor_base_frame}" robot_name="${robot_name}" prefix_topic="top_laser" hq="${hq}" range_min="0.1" range_max="90" hfov="360" samples="1800" vfov="90.0" lasers="32" fps="10" gpu="false">
 		<origin xyz="0.3 -0.175 1.165" rpy="-1.570796326795 0 -1.570796326795"/>
 		<!-- positions of the b-pearl based on solid: xyz="0.333 -0.180 1.194" rpy="-1.570796326795 0 -1.570796326795" -->
@@ -95,5 +113,5 @@
 		prefix="$(arg prefix)front_top_oak_d_camera"
 		parent="$(arg prefix)base_link"
-		publish_bf="${publish_bf}"
+		sensor_base_frame="${sensor_base_frame}"
 		robot_name="${robot_name}"
 		prefix_topic="front_top_oak_d_camera"
@@ -161,13 +179,16 @@
 	</xacro:drawer>
 	<!-- ROBAST Door Opening Mechanism -->
-	<xacro:include filename="$(find rb_theron_description)/urdf/door_opening_mechanism/door_opening_mechanism.urdf.xacro" />
-	<xacro:door_opening_mechanism
-	    prefix="$(arg prefix)"
-		parent="$(arg prefix)base_link"
-		ros2_control_hardware_type="$(arg ros2_control_hardware_type)"
-		ros_distro="$(arg ros_distro)"
-		hq="${hq}">
-		<origin xyz="-0.3 0 0.225" rpy="0 0 0"/>
-	</xacro:door_opening_mechanism>
+	<!-- The door opening mechanism should NOT be included when used for normal navigation simulations. -->
+	<xacro:if value="$(arg model_position_joint)">
+		<xacro:include filename="$(find rb_theron_description)/urdf/door_opening_mechanism/door_opening_mechanism.urdf.xacro" />
+		<xacro:door_opening_mechanism
+			prefix="$(arg prefix)"
+			parent="$(arg prefix)base_link"
+			ros2_control_hardware_type="$(arg ros2_control_hardware_type)"
+			ros_distro="$(arg ros_distro)"
+			hq="${hq}">
+			<origin xyz="-0.3 0 0.225" rpy="0 0 0"/>
+		</xacro:door_opening_mechanism>
+	</xacro:if>
 	<!-- Gazebo plugins -->
 	<xacro:ros_control ros_distro="$(arg ros_distro)"/>

File: src/ros2/robot_description/rb_theron_common/rb_theron_description/urdf/bases/theron_base.urdf.xacro (robot description, xacro)
@@ -6,22 +6,7 @@
               izz="${m*(x*x+y*y)/12}" />
   </xacro:macro>
-  <xacro:macro name="theron_base" params="prefix publish_bf hq">
+  <xacro:macro name="theron_base" params="prefix publish_bf model_position_joint ros2_control_hardware_type_positon_joint hq">
     <xacro:property name="PI" value="3.1415926535897931"/>
     <!-- xacro:property name="wheel_width" value="0.150" / -->
-    <!-- This is the joint we configured with Henning. We might not need it as a planar joint with 3 DOFs. It might be enough
-    to configure this joint as a prismatic joint with 1 DOF as we do only need to drive strictly forwards and backwards
-    during the door opening process -->
-    <!-- <ros2_control name="position_ros2_control" type="system">
-      <hardware>
-          <plugin>fake_components/GenericSystem</plugin>
-      </hardware>
-      <joint name="position" type="planar">
-          <param name="initial_position">0.0 0.0 0.0</param>
-          <command_interface name="position" />
-          <command_interface name="velocity" />
-          <state_interface name="position"/>
-          <state_interface name="velocity"/>
-      </joint>
-    </ros2_control> -->
     <!-- BASE FOOTPRINT -->
     <xacro:if value="${publish_bf}">
@@ -40,9 +25,71 @@
         </collision>
       </link>
-      <joint name="${prefix}base_footprint_joint" type="fixed">
-        <origin xyz="0 0 ${wheel_radius - wheel_offset_z}" rpy="0 0 0" />
-        <parent link="${prefix}base_footprint"/>
-        <child link="${prefix}base_link" />
-      </joint>
+      <xacro:if value="${model_position_joint}">
+        <joint name="${prefix}base_footprint_joint" type="fixed">
+          <origin xyz="0 0 ${wheel_radius - wheel_offset_z}" rpy="0 0 0" />
+          <parent link="${prefix}base_footprint"/>
+          <child link="${prefix}position_link"/>
+        </joint>
+        <link name="${prefix}position_link">
+          <inertial>
+            <mass value="0.01" />
+            <origin xyz="0.0 0.0 0.0" />
+            <xacro:solid_cuboid_inertia m="0.01" w="0.001" h="0.001" d="0.001" />
+          </inertial>
+          <visual>
+            <origin xyz="0 0 0.01" rpy="0 0 0" />
+            <geometry>
+              <box size="0.001 0.001 0.001" />
+            </geometry>
+          </visual>
+          <collision>
+            <origin xyz="0 0 0.01" rpy="0 0 0" />
+            <geometry>
+              <box size="0.001 0.001 0.001" />
+            </geometry>
+          </collision>
+        </link>
+        <joint name="position_joint" type="prismatic">
+          <axis xyz="-1 0 0" />
+          <origin xyz="0 0 0" rpy="0 0 0" />
+          <parent link="${prefix}position_link"/>
+          <child link="${prefix}base_link"/>
+          <limit lower="-1" upper="1" effort="1000" velocity="100" />
+          <!-- <dynamics damping="${damping}" friction="${friction}"/> -->
+        </joint>
+        <ros2_control name="position_ros2_control" type="system">
+          <hardware>
+            <xacro:if value="${ros2_control_hardware_type_positon_joint == 'mock_components'}">
+              <plugin>mock_components/GenericSystem</plugin>
+              <param name="calculate_dynamics">true</param>
+            </xacro:if>
+            <xacro:if value="${ros2_control_hardware_type_positon_joint == 'gz_ros2_control'}">
+              <xacro:if value="${ros_distro == 'humble'}">
+                <plugin>ign_ros2_control_base_movement/IgnBaseMovementSystemHardware</plugin>
+              </xacro:if>
+              <xacro:unless value="${ros_distro == 'humble'}">
+                <plugin>gz_ros2_control_base_movement/GzBaseMovementSystemHardware</plugin>
+              </xacro:unless>
+            </xacro:if>
+            <xacro:if value="${ros2_control_hardware_type_positon_joint == 'real_life'}">
+              <plugin>ros2_control_base_movement/BaseMovementSystemHardware</plugin>
+            </xacro:if>
+          </hardware>
+          <joint name="position_joint" type="prismatic">
+              <param name="initial_position">0.0</param>
+              <command_interface name="position" />
+              <command_interface name="velocity" />
+              <state_interface name="position"/>
+              <state_interface name="velocity"/>
+          </joint>
+        </ros2_control>
+      </xacro:if>
+      <xacro:unless value="${model_position_joint}">
+        <joint name="${prefix}base_footprint_joint" type="fixed">
+          <origin xyz="0 0 ${wheel_radius - wheel_offset_z}" rpy="0 0 0" />
+          <parent link="${prefix}base_footprint"/>
+          <child link="${prefix}base_link"/>
+        </joint>
+      </xacro:unless>
     </xacro:if>
     <!-- BASE_LINK -->

File: src/ros2/robot_description/rb_theron_common/rb_theron_description/urdf/door_opening_mechanism/arm_variations/rotating_arm.urdf.xacro (robot description, xacro)
@@ -29,6 +29,6 @@
             link_origin_z="${arm_length/2}"
             m="0.2"
-            x="0.03"
-            y="0.03"
+            x="0.02"
+            y="0.05"
             z="${arm_length}"
             r="0"
@@ -51,5 +51,5 @@
             g="1"
             b="0">
-            <origin xyz="0.020 0.0 ${arm_length-0.015}" rpy="0 0 0"/>
+            <origin xyz="-0.015 0.0 ${arm_length-0.015}" rpy="0 3.14159265359 0"/>
         </xacro:basic_box>
         <!-- Gripper -->
@@ -57,5 +57,5 @@
         <xacro:freely_rotating_hook
             prefix="${prefix}"
-            parent="${prefix}door_opening_mechanism_link_gripper_adapter"
+            parent="door_opening_mechanism_link_gripper_adapter"
             ros2_control_hardware_type="${ros2_control_hardware_type}"
             ros_distro="${ros_distro}">

File: src/ros2/robot_description/rb_theron_common/rb_theron_description/urdf/door_opening_mechanism/door_opening_mechanism.urdf.xacro (robot description, xacro)
@@ -64,6 +64,6 @@
             axis_y="0"
             axis_z="1"
-            lower_limit="-0.05"
-            upper_limit="0.25"
+            lower_limit="-0.015"
+            upper_limit="0.40"
             damping="0.1"
             friction="0.3"
@@ -79,7 +79,7 @@
             link_origin_z="0.0"
             m="2.64"
-            x="0.06"
+            x="0.045"
             y="0.55"
-            z="0.06"
+            z="0.108"
             r="1"
             g="0"
@@ -94,6 +94,6 @@
             axis_y="0"
             axis_z="1"
-            lower_limit="-0.175"
-            upper_limit="0.20"
+            lower_limit="-0.01"
+            upper_limit="0.30"
             damping="0.1"
             friction="0.3"
@@ -111,26 +111,26 @@
             x="0.065"
             y="0.015"
-            z="0.175"
+            z="0.10"
             r="1"
             g="1"
             b="1">
-            <origin xyz="-0.04 0 0" rpy="1.57079632679 4.71238898038 0"/>
+            <origin xyz="-0.032 0.15 0" rpy="1.57079632679 4.71238898038 0"/>
         </xacro:basic_joint>
         <xacro:basic_box
             parent="${prefix}door_opening_mechanism_link_x_axis_slide"
-            joint_name="${prefix}door_opening_mechanism_joint_x_axis_slide_screwing"
-            link_name="${prefix}door_opening_mechanism_link_x_slide_screwing"
+            joint_name="${prefix}door_opening_mechanism_rotating_arm_mounting_plate_joint"
+            link_name="${prefix}door_opening_mechanism_rotating_arm_mounting_plate_link"
             m="1"
-            x="0.073"
-            y="0.015"
-            z="0.175"
+            x="0.145"
+            y="0.05"
+            z="0.05"
             r="1"
             g="1"
             b="1">
-            <origin xyz="0.038 -0.027 0" rpy="0 0 1.57079632679"/>
+            <origin xyz="0 0.033 0" rpy="0 0 0"/>
         </xacro:basic_box>
         <!-- Tilting arm -->
         <!-- <xacro:include filename="$(find rb_theron_description)/urdf/door_opening_mechanism/arm_variations/tilting_arm.urdf.xacro" />
-        <xacro:tilting_arm prefix="${prefix}" parent="${prefix}door_opening_mechanism_link_x_slide_screwing" >
+        <xacro:tilting_arm prefix="${prefix}" parent="${prefix}door_opening_mechanism_rotating_arm_mounting_plate_link" >
             <origin xyz="0 -0.025 0" rpy="0 1.57079632679 0"/>
         </xacro:tilting_arm> -->
@@ -139,9 +139,9 @@
         <xacro:rotating_arm
             prefix="${prefix}"
-            parent="${prefix}door_opening_mechanism_link_x_slide_screwing"
+            parent="door_opening_mechanism_rotating_arm_mounting_plate_link"
             ros2_control_hardware_type="${ros2_control_hardware_type}"
             ros_distro="${ros_distro}"
             arm_length="0.3" >
-            <origin xyz="0.05 -0.025 0" rpy="0 0 1.57079632679"/>
+            <origin xyz="-0.083 0 0" rpy="3.14159265359 0 0"/>
         </xacro:rotating_arm>
     </xacro:macro>

File: src/ros2/robot_description/robotnik_sensors/urdf/imu_hector_plugin.urdf.xacro (robot description, xacro)
@@ -1,11 +1,6 @@
 <?xml version="1.0"?>
 <robot name="sensor_imu" xmlns:xacro="http://wiki.ros.org/xacro">
-	<xacro:macro name="sensor_imu_hector" params="prefix topic:='imu/data' parent *origin">
-		<xacro:if value="${publish_bf}">
-			<xacro:property name="sensor_link_name" value="${robot_name}/base_footprint/${prefix}_link" />
-		</xacro:if>
-		<xacro:unless value="${publish_bf}">
-			<xacro:property name="sensor_link_name" value="${robot_name}/base_link/${prefix}_link" />
-		</xacro:unless>
+	<xacro:macro name="sensor_imu_hector" params="prefix topic:='imu/data' parent sensor_base_frame robot_name *origin">
+		<xacro:property name="sensor_link_name" value="${robot_name}/${sensor_base_frame}/${prefix}_link" />
 		<joint name="${prefix}_joint" type="fixed">
 			<axis xyz="1 0 0"/>

Commit message: changed rtabmap params

File: src/ros2/robot_description/rb_theron_common/rb_theron_description/robots/rb_theron.urdf.xacro (robot description, xacro)
@@ -102,4 +102,10 @@
 		<origin xyz="-0.250 0.0 0.1643" rpy="0 3.1416 0"/>
 	</xacro:sensor_sick_nanoscan3> -->
+	<!-- <xacro:stereolabs_zed2 prefix="$(arg prefix)zed_camera" parent="$(arg prefix)base_link" prefix_topic="zed_camera" >
+		<origin xyz="0.317 -0.197 1.3044" rpy="-0.0 0.0 -3.1416"/>
+	</xacro:stereolabs_zed2> -->
+	<xacro:sensor_r430 prefix="$(arg prefix)front_top_realsense_camera" parent="$(arg prefix)base_link" sensor_base_frame="${sensor_base_frame}" robot_name="${robot_name}" prefix_topic="back_top_realsense_camera" hq="${hq}">
+		<origin xyz="0.317 -0.197 1.3044" rpy="0 0 0"/>
+	</xacro:sensor_r430>
 	<!-- <xacro:arg name="front_zed_camera_model" default="zed2" />
 	<xacro:arg name="front_zed_base_frame" default="zed-2i-base-frame" />
@@ -125,5 +131,5 @@
 		cam_yaw="$(arg front_oak_d_yaw)">
 	</xacro:zed2> -->
-	<xacro:arg name="front_oak_d_camera_model" default="OAK-D-S2" />
+	<!-- <xacro:arg name="front_oak_d_camera_model" default="OAK-D-S2" />
 	<xacro:arg name="front_oak_d_base_frame" default="oak-d-s2-usb-base-frame" />
 	<xacro:arg name="front_oak_d_pos_x" default="0.317" />
@@ -148,5 +154,5 @@
 		cam_yaw="$(arg front_oak_d_yaw)"
 		hq="${hq}">
-	</xacro:depthai_camera>
+	</xacro:depthai_camera> -->
 	<!-- ROBAST Module Cage -->
 	<xacro:include filename="$(find rb_theron_description)/urdf/module_cage/module_cage.urdf.xacro" />
