Commit message: remove old gayebo plugings from zed camera

File: src/ros2/robot_description/rb_theron_common/rb_theron_description/robots/rb_theron.urdf.xacro (robot description, xacro)
@@ -102,10 +102,10 @@
 		<origin xyz="-0.250 0.0 0.1643" rpy="0 3.1416 0"/>
 	</xacro:sensor_sick_nanoscan3> -->
-	<!-- <xacro:stereolabs_zed2 prefix="$(arg prefix)zed_camera" parent="$(arg prefix)base_link" prefix_topic="zed_camera" >
+	<xacro:stereolabs_zed2 prefix="$(arg prefix)zed_camera" parent="$(arg prefix)base_link" sensor_base_frame="${sensor_base_frame}" robot_name="${robot_name}" prefix_topic="zed_camera" >
 		<origin xyz="0.317 -0.197 1.3044" rpy="-0.0 0.0 -3.1416"/>
-	</xacro:stereolabs_zed2> -->
-	<xacro:sensor_r430 prefix="$(arg prefix)front_top_realsense_camera" parent="$(arg prefix)base_link" sensor_base_frame="${sensor_base_frame}" robot_name="${robot_name}" prefix_topic="back_top_realsense_camera" hq="${hq}">
+	</xacro:stereolabs_zed2>
+	<!-- <xacro:sensor_r430 prefix="$(arg prefix)front_top_realsense_camera" parent="$(arg prefix)base_link" sensor_base_frame="${sensor_base_frame}" robot_name="${robot_name}" prefix_topic="back_top_realsense_camera" hq="${hq}">
 		<origin xyz="0.317 -0.197 1.3044" rpy="0 0 0"/>
-	</xacro:sensor_r430>
+	</xacro:sensor_r430> -->
 	<!-- <xacro:arg name="front_zed_camera_model" default="zed2" />
 	<xacro:arg name="front_zed_base_frame" default="zed-2i-base-frame" />

File: src/ros2/robot_description/robotnik_sensors/urdf/zed2.urdf.xacro (robot description, xacro)
@@ -1,65 +1,45 @@
 <?xml version="1.0"?>
 <robot xmlns:xacro="http://wiki.ros.org/xacro">
-  <xacro:macro name="depth_camera"
-    params="prefix fps baseline hfov width height format near far  prefix_topic:='zed_node'">
-    <gazebo reference="${prefix}_base_link">
-      <visual>
-        <material>
-          <ambient>0.35 0.35 0.35 1.0</ambient>
-          <diffuse>0.350754 0.350754 0.350754 1.0</diffuse>
-          <specular>0.308273 0.3508273 0.3508273 1.0</specular>
-          <emissive>0.0 0.0 0.0 0.0</emissive>
-        </material>
-      </visual>
-      <sensor type="depth" name="depth_camera">
-        <update_rate>${fps}</update_rate>
-        <camera>
-          <horizontal_fov>${hfov}</horizontal_fov>
+  <xacro:macro name="depth_camera">
+      <gazebo reference="${prefix}_link">
+        <sensor type="camera" name="${prefix}_right_link">
+          <update_rate>10.0</update_rate>
+          <always_on>true</always_on>
+          <ignition_frame_id>camera_link_optical</ignition_frame_id>
+          <pose>0 -0.12 0 0 0 0</pose>
+          <topic>${prefix_topic}/right/image_raw</topic>
+          <horizontal_fov>1.3962634</horizontal_fov>
           <image>
-            <width>${width}</width>
-            <height>${height}</height>
-            <format>${format}</format>
+              <width>1024</width>
+              <height>1024</height>
+              <format>R8G8B8</format>
           </image>
           <clip>
-            <near>${near}</near>
-            <far>${far}</far>
+              <near>0.02</near>
+              <far>300</far>
           </clip>
-          <noise>
-            <type>gaussian</type>
-            <mean>0.0</mean>
-            <stddev>0.007</stddev>
-          </noise>
-        </camera>
-        <plugin name="camera_plugin" filename="libgazebo_ros_openni_kinect.so">
-          <baseline>${baseline}</baseline>
-          <alwaysOn>true</alwaysOn>
-          <!-- Keep this zero, update_rate in the parent <sensor> tag
-            will control the frame rate. -->
-          <updateRate>0.0</updateRate>
-          <cameraName>${prefix_topic}</cameraName>
-          <imageTopicName> rgb/image_raw</imageTopicName>
-          <cameraInfoTopicName>rgb/camera_info</cameraInfoTopicName>
-          <depthImageTopicName>depth/image_raw</depthImageTopicName>
-          <depthImageCameraInfoTopicName>depth/camera_info</depthImageCameraInfoTopicName>
-          <pointCloudTopicName>depth/points</pointCloudTopicName>
-          <frameName>/${prefix}_depth_optical_frame</frameName>
-          <pointCloudCutoff>${near}</pointCloudCutoff>
-          <pointCloudCutoffMax>${far}</pointCloudCutoffMax>
-          <distortionK1>0</distortionK1>
-          <distortionK2>0</distortionK2>
-          <distortionK3>0</distortionK3>
-          <distortionT1>0</distortionT1>
-          <distortionT2>0</distortionT2>
-          <CxPrime>0</CxPrime>
-          <Cx>0</Cx>
-          <Cy>0</Cy>
-          <focalLength>0</focalLength>
-          <hackBaseline>0</hackBaseline>
-        </plugin>
-      </sensor>
-    </gazebo>
+        </sensor>
+          <sensor type="camera" name="${prefix}_left_link">
+          <topic>${prefix_topic}/left/image_raw</topic>
+          <update_rate>10.0</update_rate>
+          <always_on>true</always_on>
+          <ignition_frame_id>camera_link_optical</ignition_frame_id>
+          <pose>0 0 0 0 0 0</pose>
+          <horizontal_fov>1.3962634</horizontal_fov>
+          <image>
+              <width>1024</width>
+              <height>1024</height>
+              <format>R8G8B8</format>
+          </image>
+          <clip>
+              <near>0.02</near>
+              <far>300</far>
+          </clip>
+        </sensor>
+        </gazebo>
   </xacro:macro>
   <xacro:macro name="stereolabs_zed2"
-    params="prefix:=zed parent *origin model:=zed format:=R8G8B8 near:=0.5 far:=30  prefix_topic:=zed_node">
+    params="prefix parent sensor_base_frame robot_name *origin model:=zed format:=R8G8B8 near:=0.5 far:=30  prefix_topic:=zed_node">
+    <xacro:property name="sensor_link_name" value="${robot_name}/${sensor_base_frame}/${prefix}" />
     <xacro:if value="${model == 'zed'}">
         <xacro:property name="baseline" value="0.12" />
@@ -125,10 +105,10 @@
     <link name="${prefix}_right_camera_optical_frame"/>
     <!-- Depth image-->
-    <joint name="${prefix}_depth_joint" type="fixed">
+    <!-- <joint name="${prefix}_depth_joint" type="fixed">
       <origin xyz="0.0 0.0 0.0" rpy="0.0 0.0 0.0" />
       <parent link="${prefix}_base_link" />
       <child link="${prefix}_depth_frame" />
-    </joint>
-    <link name="${prefix}_depth_frame"/>
+    </joint> -->
+    <!-- <link name="${prefix}_depth_frame"/>
     <joint name="${prefix}_depth_optical_joint" type="fixed">
       <origin xyz="0.0 0.0 0.0" rpy="${-M_PI/2} 0.0 ${-M_PI/2}" />
@@ -136,18 +116,7 @@
       <child link="${prefix}_depth_optical_frame" />
     </joint>
-    <link name="${prefix}_depth_optical_frame"/>
-      <xacro:depth_camera
-        prefix="${prefix}"
-        hfov="1.2217"
-        baseline="${baseline}"
-        fps="30"
-        width="1280"
-        height="720"
-        format="${format}"
-        near="${near}"
-        far="${far}"
-        prefix_topic="${prefix_topic}"
-        />
-  </xacro:macro>
+    <link name="${prefix}_depth_optical_frame"/> -->
+      <xacro:depth_camera/>
+    </xacro:macro>
   <xacro:macro name="sensor_zed2" params="prefix:=zed2 parent *origin model:=zed2  prefix_topic:=zed_node" >
     <stereolabs_zed2 prefix="${prefix}" parent="${parent}" model="${model}" prefix_topic="${prefix_topic}">

Commit message: update the sim

File: src/ros2/robot_description/rb_theron_common/rb_theron_description/robots/rb_theron.urdf.xacro (robot description, xacro)
@@ -82,4 +82,7 @@
 		<origin xyz="-0.3305 0.0 1.1468" rpy="0 0 3.1416"/>
 	</xacro:sensor_r430>
+	<!-- <xacro:sensor_r430 prefix="$(arg prefix)front_top_realsense_camera" parent="$(arg prefix)base_link" sensor_base_frame="${sensor_base_frame}" robot_name="${robot_name}" prefix_topic="front_top_realsense_camera" hq="${hq}">
+		<origin xyz="0.317 -0.197 1.3044" rpy="0 0 -3.1416"/>
+	</xacro:sensor_r430> -->
 	<!-- TODO: Moved 0.01 in x, otherwise the camera is still inside the robot -->
 	<!--xacro:sensor_orbbec_astra prefix="$(arg prefix)front_rgbd_camera" parent="$(arg prefix)base_link" prefix_topic="front_rgbd_camera">
@@ -103,56 +106,6 @@
 	</xacro:sensor_sick_nanoscan3> -->
 	<xacro:stereolabs_zed2 prefix="$(arg prefix)zed_camera" parent="$(arg prefix)base_link" sensor_base_frame="${sensor_base_frame}" robot_name="${robot_name}" prefix_topic="zed_camera" >
-		<origin xyz="0.317 -0.197 1.3044" rpy="-0.0 0.0 -3.1416"/>
+		<origin xyz="0.317 -0.197 1.3044" rpy="-0 0 -3.1416"/>
 	</xacro:stereolabs_zed2>
-	<!-- <xacro:sensor_r430 prefix="$(arg prefix)front_top_realsense_camera" parent="$(arg prefix)base_link" sensor_base_frame="${sensor_base_frame}" robot_name="${robot_name}" prefix_topic="back_top_realsense_camera" hq="${hq}">
-		<origin xyz="0.317 -0.197 1.3044" rpy="0 0 0"/>
-	</xacro:sensor_r430> -->
-	<!-- <xacro:arg name="front_zed_camera_model" default="zed2" />
-	<xacro:arg name="front_zed_base_frame" default="zed-2i-base-frame" />
-	<xacro:arg name="front_oak_d_pos_x" default="0.317" />
-	<xacro:arg name="front_oak_d_pos_y" default="-0.197" />
-	<xacro:arg name="front_oak_d_pos_z" default="1.3044" />
-	<xacro:arg name="front_oak_d_roll" default="0.0" />
-	<xacro:arg name="front_oak_d_pitch" default="0.0" />
-	<xacro:arg name="front_oak_d_yaw" default="0.0" />
-	<xacro:zed2
-		prefix="$(arg prefix)front_top_zed_camera"
-		parent="$(arg prefix)base_link"
-		sensor_base_frame="${sensor_base_frame}"
-		base_frame="$(arg front_oak_d_base_frame)"
-		robot_name="${robot_name}"
-		prefix_topic="front_top_zed_camera"
-		model="$(arg front_oak_d_camera_model)"
-		cam_pos_x="$(arg front_oak_d_pos_x)"
-		cam_pos_y="$(arg front_oak_d_pos_y)"
-		cam_pos_z="$(arg front_oak_d_pos_z)"
-		cam_roll="$(arg front_oak_d_roll)"
-		cam_pitch="$(arg front_oak_d_pitch)"
-		cam_yaw="$(arg front_oak_d_yaw)">
-	</xacro:zed2> -->
-	<!-- <xacro:arg name="front_oak_d_camera_model" default="OAK-D-S2" />
-	<xacro:arg name="front_oak_d_base_frame" default="oak-d-s2-usb-base-frame" />
-	<xacro:arg name="front_oak_d_pos_x" default="0.317" />
-	<xacro:arg name="front_oak_d_pos_y" default="-0.197" />
-	<xacro:arg name="front_oak_d_pos_z" default="1.3044" />
-	<xacro:arg name="front_oak_d_roll" default="0.0" />
-	<xacro:arg name="front_oak_d_pitch" default="0.0" />
-	<xacro:arg name="front_oak_d_yaw" default="0.0" />
-	<xacro:depthai_camera
-		prefix="$(arg prefix)front_top_oak_d_camera"
-		parent="$(arg prefix)base_link"
-		sensor_base_frame="${sensor_base_frame}"
-		robot_name="${robot_name}"
-		prefix_topic="front_top_oak_d_camera"
-		camera_model="$(arg front_oak_d_camera_model)"
-		base_frame="$(arg front_oak_d_base_frame)"
-		cam_pos_x="$(arg front_oak_d_pos_x)"
-		cam_pos_y="$(arg front_oak_d_pos_y)"
-		cam_pos_z="$(arg front_oak_d_pos_z)"
-		cam_roll="$(arg front_oak_d_roll)"
-		cam_pitch="$(arg front_oak_d_pitch)"
-		cam_yaw="$(arg front_oak_d_yaw)"
-		hq="${hq}">
-	</xacro:depthai_camera> -->
 	<!-- ROBAST Module Cage -->
 	<xacro:include filename="$(find rb_theron_description)/urdf/module_cage/module_cage.urdf.xacro" />

File: src/ros2/robot_description/robotnik_sensors/urdf/zed2.urdf.xacro (robot description, xacro)
@@ -1,54 +1,8 @@
 <?xml version="1.0"?>
 <robot xmlns:xacro="http://wiki.ros.org/xacro">
-  <xacro:macro name="depth_camera">
-      <gazebo reference="${prefix}_link">
-        <sensor type="camera" name="${prefix}_right_link">
-          <update_rate>10.0</update_rate>
-          <always_on>true</always_on>
-          <ignition_frame_id>camera_link_optical</ignition_frame_id>
-          <pose>0 -0.12 0 0 0 0</pose>
-          <topic>${prefix_topic}/right/image_raw</topic>
-          <horizontal_fov>1.3962634</horizontal_fov>
-          <image>
-              <width>1024</width>
-              <height>1024</height>
-              <format>R8G8B8</format>
-          </image>
-          <clip>
-              <near>0.02</near>
-              <far>300</far>
-          </clip>
-        </sensor>
-          <sensor type="camera" name="${prefix}_left_link">
-          <topic>${prefix_topic}/left/image_raw</topic>
-          <update_rate>10.0</update_rate>
-          <always_on>true</always_on>
-          <ignition_frame_id>camera_link_optical</ignition_frame_id>
-          <pose>0 0 0 0 0 0</pose>
-          <horizontal_fov>1.3962634</horizontal_fov>
-          <image>
-              <width>1024</width>
-              <height>1024</height>
-              <format>R8G8B8</format>
-          </image>
-          <clip>
-              <near>0.02</near>
-              <far>300</far>
-          </clip>
-        </sensor>
-        </gazebo>
-  </xacro:macro>
   <xacro:macro name="stereolabs_zed2"
-    params="prefix parent sensor_base_frame robot_name *origin model:=zed format:=R8G8B8 near:=0.5 far:=30  prefix_topic:=zed_node">
+    params="prefix parent sensor_base_frame robot_name *origin prefix_topic">
     <xacro:property name="sensor_link_name" value="${robot_name}/${sensor_base_frame}/${prefix}" />
-    <xacro:if value="${model == 'zed'}">
-        <xacro:property name="baseline" value="0.12" />
-    </xacro:if>
-    <xacro:if value="${model == 'zedm'}">
-        <xacro:property name="baseline" value="0.06" />
-    </xacro:if>
-    <xacro:if value="${model == 'zed2'}">
-        <xacro:property name="baseline" value="0.12" />
-    </xacro:if>
+    <!-- <xacro:property name="baseline" value="0.12" /> -->
     <joint name="${prefix}_base_joint" type="fixed">
       <xacro:insert_block name="origin" />
@@ -60,14 +14,15 @@
         <origin xyz="0 0 0" rpy="0 0 0"/>
         <geometry>
-          <mesh filename="$(find robotnik_sensors)/meshes/${model}.stl"/>
+          <mesh filename="$(find robotnik_sensors)/meshes/zed2.stl"/>
+          <box size="0.025 0.100 0.025 "/>
         </geometry>
-        <material name="light_zed_grey">
-          <color rgba="0.35 0.35 0.35 1"/>
+        <material name="aluminium">
+          <color rgba="0.5 0.5 0.5 1"/>
         </material>
       </visual>
       <collision>
-        <origin xyz="0.0 0.0 0.0" rpy="0 0 0" />
+        <origin xyz="0 0 0" rpy="0 0 0" />
         <geometry>
-          <mesh filename="$(find robotnik_sensors)/meshes/${model}.stl" />
+        <box size="0.025 0.100 0.025 "/>
         </geometry>
       </collision>
@@ -75,10 +30,10 @@
         <mass value="0.135" />
         <origin xyz="0 0 0" />
-        <xacro:solid_cuboid_inertia m="0.135" w="0.033" h="0.175" d="0.03" />
+        <xacro:solid_cuboid_inertia m="0.1" w="0.025" h="0.09" d="0.025" />
       </inertial>
     </link>
    <!-- Left camera -->
     <joint name="${prefix}_camera_left_joint" type="fixed">
-      <origin xyz="0.0 0.06 0.0" rpy="0.0 0.0 0.0" />
+      <origin xyz="0 0.0115 0" rpy="0 0 0" />
       <parent link="${prefix}_base_link" />
       <child link="${prefix}_left_camera_frame" />
@@ -86,12 +41,12 @@
     <link name="${prefix}_left_camera_frame"/>
     <joint name="${prefix}_camera_left_optical_joint" type="fixed">
-      <origin xyz="0.0 0.0 0.0" rpy="${-M_PI/2} 0.0 ${-M_PI/2}" />
+      <origin xyz="0 0 0" rpy="${-M_PI/2} 0 ${-M_PI/2}" />
       <parent link="${prefix}_left_camera_frame" />
-      <child link="${prefix}_left_camera_optical_frame" />
+      <child link="${sensor_link_name}_left_camera_optical_frame" />
     </joint>
-    <link name="${prefix}_left_camera_optical_frame"/>
+    <link name="${sensor_link_name}_left_camera_optical_frame"/>
     <!-- Right camera-->
     <joint name="${prefix}_camera_right_joint" type="fixed">
-      <origin xyz="0.0 -0.06 0.0" rpy="0.0 0.0 0.0" />
+      <origin xyz="0 -0.06 0" rpy="0 0 0" />
       <parent link="${prefix}_base_link" />
       <child link="${prefix}_right_camera_frame" />
@@ -99,9 +54,9 @@
     <link name="${prefix}_right_camera_frame"/>
     <joint name="${prefix}_camera_right_optical_joint" type="fixed">
-      <origin xyz="0.0 0 0.0" rpy="${-M_PI/2} 0.0 ${-M_PI/2}" />
+      <origin xyz="0 0 0" rpy="${-M_PI/2} 0.0 ${-M_PI/2}" />
       <parent link="${prefix}_right_camera_frame" />
-      <child link="${prefix}_right_camera_optical_frame" />
+      <child link="${sensor_link_name}_right_camera_optical_frame" />
     </joint>
-    <link name="${prefix}_right_camera_optical_frame"/>
+    <link name="${sensor_link_name}_right_camera_optical_frame"/>
     <!-- Depth image-->
     <!-- <joint name="${prefix}_depth_joint" type="fixed">
@@ -117,10 +72,47 @@
     </joint>
     <link name="${prefix}_depth_optical_frame"/> -->
-      <xacro:depth_camera/>
-    </xacro:macro>
-  <xacro:macro name="sensor_zed2" params="prefix:=zed2 parent *origin model:=zed2  prefix_topic:=zed_node" >
-    <stereolabs_zed2 prefix="${prefix}" parent="${parent}" model="${model}" prefix_topic="${prefix_topic}">
-      <xacro:insert_block name="origin" />
-    </stereolabs_zed2>
+    <xacro:depth_camera/>
+  </xacro:macro>
+  <xacro:macro name="depth_camera">
+      <gazebo reference="${prefix}_link">
+        <sensor name="${prefix}_right_link" type="camera" >
+          <topic>zed/right/image_raw</topic>
+          <camera name="zed">
+            <horizontal_fov>1.3962634</horizontal_fov>
+            <!-- <pose>0 -0.12 0 0 0 0</pose> -->
+            <image>
+                <width>640</width>
+                <height>480</height>
+                <format>RGB_INT8</format>
+            </image>
+            <clip>
+                <near>0.02</near>
+                <far>300</far>
+            </clip>
+            </camera>
+          <always_on>true</always_on>
+          <update_rate>10</update_rate>
+          <visualize>1</visualize>
+        </sensor>
+          <sensor name="${prefix}_left_link" type="camera" >
+          <topic>zed/left/image_raw</topic>
+          <camera>
+          <!-- <pose>0 0 0 0 0 0</pose> -->
+          <horizontal_fov>1.3962634</horizontal_fov>
+          <image>
+              <width>640</width>
+              <height>480</height>
+              <format>RGB_INT8</format>
+          </image>
+          <clip>
+              <near>0.02</near>
+              <far>300</far>
+          </clip>
+          </camera>
+          <update_rate>10.0</update_rate>
+          <always_on>true</always_on>
+          <visualize>1</visualize>
+        </sensor>
+        </gazebo>
   </xacro:macro>
 </robot>
