Commit message: feat: first draft for planar base support for rb_theron

File: src/ros2/robot_description/rb_theron_common/rb_theron_description/robots/rb_theron.urdf.xacro (robot description, xacro)
@@ -38,19 +38,20 @@
 	<xacro:arg name="ros2_control_hardware_type_positon_joint" default="mock_components" />
 	<xacro:arg name="ros_distro" default="humble" />
-	<!-- Whether the position joint should be modeled as a prismatic joint or just as a fixed joint -->
-	<xacro:arg name="model_position_joint" default="false" />
+	<!-- Whether the position joint should be modeled as a fixed joint, a prismatic joint or a planar joint -->
+	<xacro:arg name="model_position_joint" default="fixed" />
+	<xacro:property name="model_position_joint_prop" value="$(arg model_position_joint)"/>
 	<!-- If we model the position joint, the sensors need be placed in the base_link frame,
 	otherwise they should be placed in the base_footprint frame -->
-	<xacro:if value="$(arg model_position_joint)">
-		<xacro:property name="sensor_base_frame" value="base_link" />
+	<xacro:if value="${model_position_joint_prop == 'prismatic' or model_position_joint_prop == 'planar'}">
+		<xacro:property name="sensor_base_frame" value="base_link"/>
 	</xacro:if>
-	<xacro:unless value="$(arg model_position_joint)">
-		<xacro:if value="${publish_bf}">
-			<xacro:property name="sensor_base_frame" value="base_footprint" />
+	<xacro:if value="${model_position_joint_prop == 'prismatic'}">
+		<xacro:if value="$(arg publish_bf)">
+			<xacro:property name="sensor_base_frame" value="base_footprint"/>
 		</xacro:if>
-		<xacro:unless value="${publish_bf}">
-			<xacro:property name="sensor_base_frame" value="base_link" />
+		<xacro:unless value="$(arg publish_bf)">
+			<xacro:property name="sensor_base_frame" value="base_link"/>
 		</xacro:unless>
-	</xacro:unless>
+	</xacro:if>
 	<!-- *************** -->
 	<!-- Robots Elements -->
@@ -180,5 +181,5 @@
 	<!-- ROBAST Door Opening Mechanism -->
 	<!-- The door opening mechanism should NOT be included when used for normal navigation simulations. -->
-	<xacro:if value="$(arg model_position_joint)">
+	<xacro:if value="${model_position_joint_prop == 'prismatic' or model_position_joint_prop == 'planar'}">
 		<xacro:include filename="$(find rb_theron_description)/urdf/door_opening_mechanism/door_opening_mechanism.urdf.xacro" />
 		<xacro:door_opening_mechanism
@@ -216,5 +217,5 @@
 	</xacro:if>
 	<!-- Gazebo plugins -->
-	<xacro:ros_control ros_distro="$(arg ros_distro)"/>
+	<xacro:ros_control ros_distro="$(arg ros_distro)" model_position_joint="$(arg model_position_joint)"/>
 	<xacro:gazebo_sensor_plugins ros_distro="$(arg ros_distro)"/>
 </robot>

File: src/ros2/robot_description/rb_theron_common/rb_theron_description/urdf/bases/theron_base.urdf.xacro (robot description, xacro)
@@ -25,5 +25,5 @@
         </collision>
       </link>
-      <xacro:if value="${model_position_joint}">
+      <xacro:if value="${model_position_joint == 'prismatic'}">
         <joint name="${prefix}base_footprint_joint" type="fixed">
           <origin xyz="0 0 ${wheel_radius - wheel_offset_z}" rpy="0 0 0" />
@@ -85,5 +85,36 @@
         </ros2_control>
       </xacro:if>
-      <xacro:unless value="${model_position_joint}">
+      <xacro:if value="${model_position_joint == 'planar'}">
+        <link name="odom">
+          <inertial>
+            <mass value="0.01" />
+            <origin xyz="0.0 0.0 0.0" />
+            <xacro:solid_cuboid_inertia m="0.01" w="0.001" h="0.001" d="0.001" />
+          </inertial>
+          <visual>
+            <origin xyz="0 0 0.01" rpy="0 0 0" />
+            <geometry>
+              <box size="0.001 0.001 0.001" />
+            </geometry>
+          </visual>
+          <collision>
+            <origin xyz="0 0 0.01" rpy="0 0 0" />
+            <geometry>
+              <box size="0.001 0.001 0.001" />
+            </geometry>
+          </collision>
+        </link>
+        <joint name="position" type="planar">
+          <origin rpy="0 0 0" xyz="0 0 0"/>
+          <parent link="odom"/>
+          <child link="${prefix}base_footprint"/>
+        </joint>
+        <!-- <joint name="position" type="prismatic">
+          <axis xyz="-1 0 0" />
+          <origin rpy="0 0 0" xyz="0 0 0"/>
+          <parent link="odom"/>
+          <child link="${prefix}base_footprint"/>
+          <limit lower="-1" upper="1" effort="1000" velocity="100" />
+        </joint>         -->
         <joint name="${prefix}base_footprint_joint" type="fixed">
           <origin xyz="0 0 ${wheel_radius - wheel_offset_z}" rpy="0 0 0" />
@@ -91,5 +122,61 @@
           <child link="${prefix}base_link"/>
         </joint>
-      </xacro:unless>
+        <ros2_control name="position_ros2_control" type="system">
+          <hardware>
+            <xacro:if value="${ros2_control_hardware_type_positon_joint == 'mock_components'}">
+              <plugin>mock_components/GenericSystem</plugin>
+              <param name="calculate_dynamics">true</param>
+            </xacro:if>
+            <xacro:if value="${ros2_control_hardware_type_positon_joint == 'gz_ros2_control'}">
+              <xacro:if value="${ros_distro == 'humble'}">
+                <plugin>ign_ros2_control_base_movement/IgnBaseMovementSystemHardware</plugin>
+              </xacro:if>
+              <xacro:unless value="${ros_distro == 'humble'}">
+                <plugin>gz_ros2_control_base_movement/GzBaseMovementSystemHardware</plugin>
+              </xacro:unless>
+            </xacro:if>
+            <xacro:if value="${ros2_control_hardware_type_positon_joint == 'real_life'}">
+              <plugin>ros2_control_base_movement/BaseMovementSystemHardware</plugin>
+            </xacro:if>
+          </hardware>
+          <!-- Virtual position joint for supporting MoveIt's planar joint type in joint trajectories -->
+          <joint name="position/x">
+            <param name="initial_position">0.0</param>
+            <command_interface name="velocity" />
+            <state_interface name="position"/>
+            <state_interface name="velocity"/>
+          </joint>
+          <joint name="position/y">
+            <param name="initial_position">0.0</param>
+            <command_interface name="velocity" />
+            <state_interface name="position"/>
+            <state_interface name="velocity"/>
+          </joint>
+          <joint name="position/theta">
+            <param name="initial_position">0.0</param>
+            <command_interface name="velocity" />
+            <state_interface name="position"/>
+            <state_interface name="velocity"/>
+          </joint>
+          <!-- Wheel joints used for diff drive controller support -->
+          <joint name="joint_left_wheel">
+            <command_interface name="velocity"/>
+            <state_interface name="position"/>
+            <state_interface name="velocity"/>
+          </joint>
+          <joint name="joint_right_wheel">
+            <command_interface name="velocity"/>
+            <state_interface name="position"/>
+            <state_interface name="velocity"/>
+          </joint>
+        </ros2_control>
+      </xacro:if>
+      <xacro:if value="${model_position_joint == 'fixed'}">
+        <joint name="${prefix}base_footprint_joint" type="fixed">
+          <origin xyz="0 0 ${wheel_radius - wheel_offset_z}" rpy="0 0 0" />
+          <parent link="${prefix}base_footprint"/>
+          <child link="${prefix}base_link"/>
+        </joint>
+      </xacro:if>
     </xacro:if>
     <!-- BASE_LINK -->

File: src/ros2/robot_description/rb_theron_common/rb_theron_description/urdf/common.gazebo.xacro (robot description, xacro)
@@ -2,15 +2,29 @@
 <robot xmlns:xacro="http://www.ros.org/wiki/xacro">
     <!-- ROS CONTROL GAZEBO PLUGIN -->
-    <xacro:macro name="ros_control" params="ros_distro">
+    <xacro:macro name="ros_control" params="ros_distro model_position_joint">
         <gazebo>
             <xacro:if value="${ros_distro == 'humble'}">
-                <plugin name="ign_ros2_control::IgnitionROS2ControlPlugin" filename="libign_ros2_control-system.so">
-                    <parameters>$(find rb_theron_description)/config/rb_theron_gz_ros2_controller.yaml</parameters>
-                </plugin>
+                <xacro:if value="${model_position_joint == 'fixed' or model_position_joint == 'prismatic'}">
+                    <plugin name="ign_ros2_control::IgnitionROS2ControlPlugin" filename="libign_ros2_control-system.so">
+                        <parameters>$(find rb_theron_description)/config/rb_theron_gz_ros2_controller.yaml</parameters>
+                    </plugin>
+                </xacro:if>
+                <xacro:if value="${model_position_joint == 'planar'}">
+                    <plugin name="ign_ros2_control::IgnitionROS2ControlPlugin" filename="libign_ros2_control-system.so">
+                        <parameters>$(find rb_theron_description)/config/rb_theron_planar_base_gz_ros2_control.yaml</parameters>
+                    </plugin>
+                </xacro:if>
             </xacro:if>
             <xacro:unless value="${ros_distro == 'humble'}">
-                <plugin name="gz_ros2_control::GazeboSimROS2ControlPlugin" filename="gz_ros2_control-system">
-                    <parameters>$(find rb_theron_description)/config/rb_theron_gz_ros2_controller.yaml</parameters>
-                </plugin>
+                <xacro:if value="${model_position_joint == 'fixed' or model_position_joint == 'prismatic'}">
+                    <plugin name="gz_ros2_control::GazeboSimROS2ControlPlugin" filename="gz_ros2_control-system">
+                        <parameters>$(find rb_theron_description)/config/rb_theron_gz_ros2_controller.yaml</parameters>
+                    </plugin>
+                </xacro:if>
+                <xacro:if value="${model_position_joint == 'planar'}">
+                    <plugin name="gz_ros2_control::GazeboSimROS2ControlPlugin" filename="gz_ros2_control-system">
+                        <parameters>$(find rb_theron_description)/config/rb_theron_planar_base_gz_ros2_control.yaml</parameters>
+                    </plugin>
+                </xacro:if>
             </xacro:unless>
         </gazebo>

Commit message: fix: some minor issues due to latest restructure of `model_position_joint`

File: src/ros2/robot_description/rb_theron_common/rb_theron_description/robots/rb_theron.urdf.xacro (robot description, xacro)
@@ -46,5 +46,5 @@
 		<xacro:property name="sensor_base_frame" value="base_link"/>
 	</xacro:if>
-	<xacro:if value="${model_position_joint_prop == 'prismatic'}">
+	<xacro:if value="${model_position_joint_prop == 'fixed'}">
 		<xacro:if value="${publish_bf}">
 			<xacro:property name="sensor_base_frame" value="base_footprint"/>

File: src/ros2/robot_description/rb_theron_common/rb_theron_description/robots/rb_theron_arm.urdf.xacro (robot description, xacro)
@@ -23,11 +23,12 @@
 	<xacro:arg name="ros_distro" default="humble" />
 	<!-- Whether the position joint should be modeled as a prismatic joint or just as a fixed joint -->
-	<xacro:arg name="model_position_joint" default="false" />
+	<xacro:arg name="model_position_joint" default="fixed" />
+	<xacro:property name="model_position_joint_prop" value="$(arg model_position_joint)"/>
 	<!-- If we model the position joint, the sensors need be placed in the base_link frame,
 	otherwise they should be placed in the base_footprint frame -->
-	<xacro:if value="$(arg model_position_joint)">
+	<xacro:if value="${model_position_joint_prop == 'prismatic'}">
 		<xacro:property name="sensor_base_frame" value="base_link" />
 	</xacro:if>
-	<xacro:unless value="$(arg model_position_joint)">
+	<xacro:if value="${model_position_joint_prop == 'fixed'}">
 		<xacro:if value="${publish_bf}">
 			<xacro:property name="sensor_base_frame" value="base_footprint" />
@@ -36,5 +37,5 @@
 			<xacro:property name="sensor_base_frame" value="base_link" />
 		</xacro:unless>
-	</xacro:unless>
+	</xacro:if>
     <xacro:include filename="$(find rb_theron_description)/urdf/bases/theron_base.urdf.xacro" />
     <xacro:include filename="$(find rb_theron_description)/urdf/inertia.urdf.xacro" />

Commit message: feat: first attempt to get door opening mechanism running in parallel with nav

File: src/ros2/robot_description/rb_theron_common/rb_theron_description/robots/rb_theron.urdf.xacro (robot description, xacro)
@@ -38,20 +38,15 @@
 	<xacro:arg name="ros2_control_hardware_type_positon_joint" default="mock_components" />
 	<xacro:arg name="ros_distro" default="humble" />
+	<!-- Whether the robot should have a door opening mechanism -->
+	<xacro:arg name="model_door_opening_mechanism" default="false" />
 	<!-- Whether the position joint should be modeled as a fixed joint, a prismatic joint or a planar joint -->
 	<xacro:arg name="model_position_joint" default="fixed" />
 	<xacro:property name="model_position_joint_prop" value="$(arg model_position_joint)"/>
-	<!-- If we model the position joint, the sensors need be placed in the base_link frame,
-	otherwise they should be placed in the base_footprint frame -->
-	<xacro:if value="${model_position_joint_prop == 'prismatic' or model_position_joint_prop == 'planar'}">
+	<xacro:if value="${publish_bf}">
+		<xacro:property name="sensor_base_frame" value="base_footprint"/>
+	</xacro:if>
+	<xacro:unless value="${publish_bf}">
 		<xacro:property name="sensor_base_frame" value="base_link"/>
-	</xacro:if>
-	<xacro:if value="${model_position_joint_prop == 'fixed'}">
-		<xacro:if value="${publish_bf}">
-			<xacro:property name="sensor_base_frame" value="base_footprint"/>
-		</xacro:if>
-		<xacro:unless value="${publish_bf}">
-			<xacro:property name="sensor_base_frame" value="base_link"/>
-		</xacro:unless>
-	</xacro:if>
+	</xacro:unless>
 	<!-- *************** -->
 	<!-- Robots Elements -->
@@ -65,5 +60,6 @@
 	  ros2_control_hardware_type_positon_joint="$(arg ros2_control_hardware_type_positon_joint)"
 	  ros_distro="$(arg ros_distro)"
-	  model_position_joint="$(arg model_position_joint)">
+	  model_position_joint="$(arg model_position_joint)"
+	  model_door_opening_mechanism="$(arg model_door_opening_mechanism)">
 	</xacro:rb_theron_base>
 	<!-- Gazebo ros control pluggins -->
@@ -181,5 +177,5 @@
 	<!-- ROBAST Door Opening Mechanism -->
 	<!-- The door opening mechanism should NOT be included when used for normal navigation simulations. -->
-	<xacro:if value="${model_position_joint_prop == 'prismatic' or model_position_joint_prop == 'planar'}">
+	<xacro:if value="$(arg model_door_opening_mechanism)">
 		<xacro:include filename="$(find rb_theron_description)/urdf/door_opening_mechanism/door_opening_mechanism.urdf.xacro" />
 		<xacro:door_opening_mechanism

File: src/ros2/robot_description/rb_theron_common/rb_theron_description/robots/rb_theron_base.urdf.xacro (robot description, xacro)
@@ -29,9 +29,11 @@
       ros2_control_hardware_type_positon_joint
       ros_distro
-      model_position_joint">
+      model_position_joint
+      model_door_opening_mechanism">
     <xacro:theron_base
       prefix="${prefix}"
       publish_bf="${publish_bf}"
       model_position_joint="${model_position_joint}"
+      model_door_opening_mechanism="${model_door_opening_mechanism}"
       ros2_control_hardware_type_positon_joint="${ros2_control_hardware_type_positon_joint}"
       hq="${hq}"

File: src/ros2/robot_description/rb_theron_common/rb_theron_description/urdf/bases/theron_base.urdf.xacro (robot description, xacro)
@@ -6,5 +6,5 @@
               izz="${m*(x*x+y*y)/12}" />
   </xacro:macro>
-  <xacro:macro name="theron_base" params="prefix publish_bf model_position_joint ros2_control_hardware_type_positon_joint hq">
+  <xacro:macro name="theron_base" params="prefix publish_bf model_position_joint model_door_opening_mechanism ros2_control_hardware_type_positon_joint hq">
     <xacro:property name="PI" value="3.1415926535897931"/>
     <!-- xacro:property name="wheel_width" value="0.150" / -->
@@ -25,67 +25,15 @@
         </collision>
       </link>
+      <!-- Prismatic position joint -->
       <xacro:if value="${model_position_joint == 'prismatic'}">
-        <joint name="${prefix}base_footprint_joint" type="fixed">
-          <origin xyz="0 0 ${wheel_radius - wheel_offset_z}" rpy="0 0 0" />
-          <parent link="${prefix}base_footprint"/>
-          <child link="${prefix}position_link"/>
-        </joint>
-        <link name="${prefix}position_link">
-          <inertial>
-            <mass value="0.01" />
-            <origin xyz="0.0 0.0 0.0" />
-            <xacro:solid_cuboid_inertia m="0.01" w="0.001" h="0.001" d="0.001" />
-          </inertial>
-          <visual>
-            <origin xyz="0 0 0.01" rpy="0 0 0" />
-            <geometry>
-              <box size="0.001 0.001 0.001" />
-            </geometry>
-          </visual>
-          <collision>
-            <origin xyz="0 0 0.01" rpy="0 0 0" />
-            <geometry>
-              <box size="0.001 0.001 0.001" />
-            </geometry>
-          </collision>
-        </link>
         <joint name="position_joint" type="prismatic">
           <axis xyz="-1 0 0" />
           <origin xyz="0 0 0" rpy="0 0 0" />
-          <parent link="${prefix}position_link"/>
+          <parent link="base_footprint"/>
           <child link="${prefix}base_link"/>
           <limit lower="-1" upper="1" effort="1000" velocity="100" />
-          <!-- <dynamics damping="${damping}" friction="${friction}"/> -->
-        </joint>
-        <ros2_control name="position_ros2_control" type="system">
-          <hardware>
-            <xacro:if value="${ros2_control_hardware_type_positon_joint == 'mock_components'}">
-              <plugin>mock_components/GenericSystem</plugin>
-              <param name="calculate_dynamics">true</param>
-            </xacro:if>
-            <xacro:if value="${ros2_control_hardware_type_positon_joint == 'gz_ros2_control'}">
-              <xacro:if value="${ros_distro == 'humble'}">
-                <plugin>ign_ros2_control_base_movement/IgnBaseMovementSystemHardware</plugin>
-                <param name="odom_topic">/diff_drive_base_controller/odom</param>
-              </xacro:if>
-              <xacro:unless value="${ros_distro == 'humble'}">
-                <plugin>gz_ros2_control_base_movement/GzBaseMovementSystemHardware</plugin>
-                <param name="odom_topic">/diff_drive_base_controller/odom</param>
-              </xacro:unless>
-            </xacro:if>
-            <xacro:if value="${ros2_control_hardware_type_positon_joint == 'real_life'}">
-              <plugin>ros2_control_base_movement/BaseMovementSystemHardware</plugin>
-              <param name="odom_topic">/diff_drive_base_controller/odom</param>
-            </xacro:if>
-          </hardware>
-          <joint name="position_joint" type="prismatic">
-              <param name="initial_position">0.0</param>
-              <command_interface name="position" />
-              <command_interface name="velocity" />
-              <state_interface name="position"/>
-              <state_interface name="velocity"/>
-          </joint>
-        </ros2_control>
-      </xacro:if>
+        </joint>
+      </xacro:if>
+      <!-- Planar position joint -->
       <xacro:if value="${model_position_joint == 'planar'}">
         <link name="odom">
@@ -175,4 +123,5 @@
         </ros2_control>
       </xacro:if>
+      <!-- Fixed position joint -->
       <xacro:if value="${model_position_joint == 'fixed'}">
         <joint name="${prefix}base_footprint_joint" type="fixed">
@@ -181,4 +130,41 @@
           <child link="${prefix}base_link"/>
         </joint>
+      </xacro:if>
+      <xacro:if value="${model_door_opening_mechanism}">
+        <ros2_control name="position_ros2_control" type="system">
+          <hardware>
+            <xacro:if value="${ros2_control_hardware_type_positon_joint == 'mock_components'}">
+              <plugin>mock_components/GenericSystem</plugin>
+              <param name="calculate_dynamics">true</param>
+            </xacro:if>
+            <xacro:if value="${ros2_control_hardware_type_positon_joint == 'gz_ros2_control'}">
+              <xacro:if value="${ros_distro == 'humble'}">
+                <plugin>ign_ros2_control_base_movement/IgnBaseMovementSystemHardware</plugin>
+                <param name="odom_topic">/diff_drive_base_controller/odom</param>
+                <param name="enable_state_feedback">false</param>
+                <param name="reset_position_state_after_each_trajectory">true</param>
+              </xacro:if>
+              <xacro:unless value="${ros_distro == 'humble'}">
+                <plugin>gz_ros2_control_base_movement/GzBaseMovementSystemHardware</plugin>
+                <param name="odom_topic">/diff_drive_base_controller/odom</param>
+                <param name="enable_state_feedback">false</param>
+                <param name="reset_position_state_after_each_trajectory">true</param>
+              </xacro:unless>
+            </xacro:if>
+            <xacro:if value="${ros2_control_hardware_type_positon_joint == 'real_life'}">
+              <plugin>ros2_control_base_movement/BaseMovementSystemHardware</plugin>
+              <param name="odom_topic">/diff_drive_base_controller/odom</param>
+              <param name="enable_state_feedback">false</param>
+              <param name="reset_position_state_after_each_trajectory">true</param>
+            </xacro:if>
+          </hardware>
+          <joint name="position_joint" type="prismatic">
+              <param name="initial_position">0.0</param>
+              <command_interface name="position" />
+              <command_interface name="velocity" />
+              <state_interface name="position"/>
+              <state_interface name="velocity"/>
+          </joint>
+        </ros2_control>
       </xacro:if>
     </xacro:if>
