Commit message: refactor: renames `model_position_joint` to `position_joint_type`

File: src/ros2/robot_description/rb_theron_common/rb_theron_description/robots/rb_theron.urdf.xacro (robot description, xacro)
@@ -45,5 +45,5 @@
 	<xacro:arg name="model_door_opening_mechanism" default="false" />
 	<!-- Whether the position joint should be modeled as a fixed joint, a prismatic joint or a planar joint -->
-	<xacro:arg name="model_position_joint" default="fixed" />
+	<xacro:arg name="position_joint_type" default="fixed" />
 	<xacro:if value="${publish_bf}">
 		<xacro:property name="sensor_base_frame" value="base_footprint"/>
@@ -63,5 +63,5 @@
 	  ros2_control_hardware_type_positon_joint="$(arg ros2_control_hardware_type_positon_joint)"
 	  ros_distro="$(arg ros_distro)"
-	  model_position_joint="$(arg model_position_joint)"
+	  position_joint_type="$(arg position_joint_type)"
 	  model_door_opening_mechanism="$(arg model_door_opening_mechanism)">
 	</xacro:rb_theron_base>
@@ -220,5 +220,5 @@
 	</xacro:if>
 	<!-- Gazebo plugins -->
-	<xacro:ros_control ros_distro="$(arg ros_distro)" model_position_joint="$(arg model_position_joint)"/>
+	<xacro:ros_control ros_distro="$(arg ros_distro)" position_joint_type="$(arg position_joint_type)"/>
 	<xacro:gazebo_sensor_plugins ros_distro="$(arg ros_distro)"/>
 </robot>

File: src/ros2/robot_description/rb_theron_common/rb_theron_description/robots/rb_theron_base.urdf.xacro (robot description, xacro)
@@ -29,10 +29,10 @@
       ros2_control_hardware_type_positon_joint
       ros_distro
-      model_position_joint
+      position_joint_type
       model_door_opening_mechanism">
     <xacro:theron_base
       prefix="${prefix}"
       publish_bf="${publish_bf}"
-      model_position_joint="${model_position_joint}"
+      position_joint_type="${position_joint_type}"
       model_door_opening_mechanism="${model_door_opening_mechanism}"
       ros2_control_hardware_type_positon_joint="${ros2_control_hardware_type_positon_joint}"

File: src/ros2/robot_description/rb_theron_common/rb_theron_description/urdf/bases/theron_base.urdf.xacro (robot description, xacro)
@@ -6,5 +6,5 @@
               izz="${m*(x*x+y*y)/12}" />
   </xacro:macro>
-  <xacro:macro name="theron_base" params="prefix publish_bf model_position_joint model_door_opening_mechanism ros2_control_hardware_type_positon_joint hq">
+  <xacro:macro name="theron_base" params="prefix publish_bf position_joint_type model_door_opening_mechanism ros2_control_hardware_type_positon_joint hq">
     <xacro:property name="PI" value="3.1415926535897931"/>
     <!-- xacro:property name="wheel_width" value="0.150" / -->
@@ -26,5 +26,5 @@
       </link>
       <!-- Prismatic position joint -->
-      <xacro:if value="${model_position_joint == 'prismatic'}">
+      <xacro:if value="${position_joint_type == 'prismatic'}">
         <joint name="position_joint" type="prismatic">
           <axis xyz="-1 0 0" />
@@ -36,5 +36,5 @@
       </xacro:if>
       <!-- Planar position joint -->
-      <xacro:if value="${model_position_joint == 'planar'}">
+      <xacro:if value="${position_joint_type == 'planar'}">
         <link name="${prefix}odom">
           <inertial>
@@ -124,5 +124,5 @@
       </xacro:if>
       <!-- Fixed position joint -->
-      <xacro:if value="${model_position_joint == 'fixed'}">
+      <xacro:if value="${position_joint_type == 'fixed'}">
         <joint name="${prefix}base_footprint_joint" type="fixed">
           <origin xyz="0 0 ${wheel_radius - wheel_offset_z}" rpy="0 0 0" />

Commit message: feat: state feedback for `prismatic` position joint and first steps for `planar_joint` support (RE-2124) (#150)
This PR belongs to RE-2124 and RE-2244 contains:
- first steps to support modeling our base as planar joint
- new moveit_pro config rb_theron_planar_base_config which was adopted from the Picknik Stretch example
- state feedback for mobile base modeled as state prismatic joint (RE-2244)

File: src/ros2/robot_description/rb_theron_common/rb_theron_description/robots/rb_theron.urdf.xacro (robot description, xacro)
@@ -38,19 +38,20 @@
 	<xacro:arg name="ros2_control_hardware_type_positon_joint" default="mock_components" />
 	<xacro:arg name="ros_distro" default="humble" />
-	<!-- Whether the position joint should be modeled as a prismatic joint or just as a fixed joint -->
-	<xacro:arg name="model_position_joint" default="false" />
+	<!-- Whether the position joint should be modeled as a fixed joint, a prismatic joint or a planar joint -->
+	<xacro:arg name="position_joint_type" default="fixed" />
+	<xacro:property name="position_joint_type_prop" value="$(arg position_joint_type)"/>
 	<!-- If we model the position joint, the sensors need be placed in the base_link frame,
 	otherwise they should be placed in the base_footprint frame -->
-	<xacro:if value="$(arg model_position_joint)">
-		<xacro:property name="sensor_base_frame" value="base_link" />
+	<xacro:if value="${position_joint_type_prop == 'prismatic' or position_joint_type_prop == 'planar'}">
+		<xacro:property name="sensor_base_frame" value="base_link"/>
 	</xacro:if>
-	<xacro:unless value="$(arg model_position_joint)">
+	<xacro:if value="${position_joint_type_prop == 'fixed'}">
 		<xacro:if value="${publish_bf}">
-			<xacro:property name="sensor_base_frame" value="base_footprint" />
+			<xacro:property name="sensor_base_frame" value="base_footprint"/>
 		</xacro:if>
 		<xacro:unless value="${publish_bf}">
-			<xacro:property name="sensor_base_frame" value="base_link" />
+			<xacro:property name="sensor_base_frame" value="base_link"/>
 		</xacro:unless>
-	</xacro:unless>
+	</xacro:if>
 	<!-- *************** -->
 	<!-- Robots Elements -->
@@ -64,5 +65,5 @@
 	  ros2_control_hardware_type_positon_joint="$(arg ros2_control_hardware_type_positon_joint)"
 	  ros_distro="$(arg ros_distro)"
-	  model_position_joint="$(arg model_position_joint)">
+	  position_joint_type="$(arg position_joint_type)">
 	</xacro:rb_theron_base>
 	<!-- Gazebo ros control pluggins -->
@@ -180,5 +181,5 @@
 	<!-- ROBAST Door Opening Mechanism -->
 	<!-- The door opening mechanism should NOT be included when used for normal navigation simulations. -->
-	<xacro:if value="$(arg model_position_joint)">
+	<xacro:if value="${position_joint_type_prop == 'prismatic' or position_joint_type_prop == 'planar'}">
 		<xacro:include filename="$(find rb_theron_description)/urdf/door_opening_mechanism/door_opening_mechanism.urdf.xacro" />
 		<xacro:door_opening_mechanism
@@ -216,5 +217,5 @@
 	</xacro:if>
 	<!-- Gazebo plugins -->
-	<xacro:ros_control ros_distro="$(arg ros_distro)"/>
+	<xacro:ros_control ros_distro="$(arg ros_distro)" position_joint_type="$(arg position_joint_type)"/>
 	<xacro:gazebo_sensor_plugins ros_distro="$(arg ros_distro)"/>
 </robot>

File: src/ros2/robot_description/rb_theron_common/rb_theron_description/robots/rb_theron_arm.urdf.xacro (robot description, xacro)
@@ -23,11 +23,12 @@
 	<xacro:arg name="ros_distro" default="humble" />
 	<!-- Whether the position joint should be modeled as a prismatic joint or just as a fixed joint -->
-	<xacro:arg name="model_position_joint" default="false" />
+	<xacro:arg name="position_joint_type" default="fixed" />
+	<xacro:property name="position_joint_type_prop" value="$(arg position_joint_type)"/>
 	<!-- If we model the position joint, the sensors need be placed in the base_link frame,
 	otherwise they should be placed in the base_footprint frame -->
-	<xacro:if value="$(arg model_position_joint)">
+	<xacro:if value="${position_joint_type_prop == 'prismatic'}">
 		<xacro:property name="sensor_base_frame" value="base_link" />
 	</xacro:if>
-	<xacro:unless value="$(arg model_position_joint)">
+	<xacro:if value="${position_joint_type_prop == 'fixed'}">
 		<xacro:if value="${publish_bf}">
 			<xacro:property name="sensor_base_frame" value="base_footprint" />
@@ -36,5 +37,5 @@
 			<xacro:property name="sensor_base_frame" value="base_link" />
 		</xacro:unless>
-	</xacro:unless>
+	</xacro:if>
     <xacro:include filename="$(find rb_theron_description)/urdf/bases/theron_base.urdf.xacro" />
     <xacro:include filename="$(find rb_theron_description)/urdf/inertia.urdf.xacro" />
@@ -42,5 +43,5 @@
       prefix="$(arg prefix)"
       publish_bf="${publish_bf}"
-      model_position_joint="$(arg model_position_joint)"
+      position_joint_type="$(arg position_joint_type)"
       ros2_control_hardware_type_positon_joint="$(arg ros2_control_hardware_type_positon_joint)"
       hq="${hq}"

File: src/ros2/robot_description/rb_theron_common/rb_theron_description/urdf/bases/theron_base.urdf.xacro (robot description, xacro)
@@ -6,5 +6,5 @@
               izz="${m*(x*x+y*y)/12}" />
   </xacro:macro>
-  <xacro:macro name="theron_base" params="prefix publish_bf model_position_joint ros2_control_hardware_type_positon_joint hq">
+  <xacro:macro name="theron_base" params="prefix publish_bf position_joint_type ros2_control_hardware_type_positon_joint hq">
     <xacro:property name="PI" value="3.1415926535897931"/>
     <!-- xacro:property name="wheel_width" value="0.150" / -->
@@ -25,5 +25,5 @@
         </collision>
       </link>
-      <xacro:if value="${model_position_joint}">
+      <xacro:if value="${position_joint_type == 'prismatic'}">
         <joint name="${prefix}base_footprint_joint" type="fixed">
           <origin xyz="0 0 ${wheel_radius - wheel_offset_z}" rpy="0 0 0" />
@@ -67,11 +67,14 @@
               <xacro:if value="${ros_distro == 'humble'}">
                 <plugin>ign_ros2_control_base_movement/IgnBaseMovementSystemHardware</plugin>
+                <param name="odom_topic">/diff_drive_base_controller/odom</param>
               </xacro:if>
               <xacro:unless value="${ros_distro == 'humble'}">
                 <plugin>gz_ros2_control_base_movement/GzBaseMovementSystemHardware</plugin>
+                <param name="odom_topic">/diff_drive_base_controller/odom</param>
               </xacro:unless>
             </xacro:if>
             <xacro:if value="${ros2_control_hardware_type_positon_joint == 'real_life'}">
               <plugin>ros2_control_base_movement/BaseMovementSystemHardware</plugin>
+              <param name="odom_topic">/diff_drive_base_controller/odom</param>
             </xacro:if>
           </hardware>
@@ -85,5 +88,36 @@
         </ros2_control>
       </xacro:if>
-      <xacro:unless value="${model_position_joint}">
+      <xacro:if value="${position_joint_type == 'planar'}">
+        <link name="odom">
+          <inertial>
+            <mass value="0.01" />
+            <origin xyz="0.0 0.0 0.0" />
+            <xacro:solid_cuboid_inertia m="0.01" w="0.001" h="0.001" d="0.001" />
+          </inertial>
+          <visual>
+            <origin xyz="0 0 0.01" rpy="0 0 0" />
+            <geometry>
+              <box size="0.001 0.001 0.001" />
+            </geometry>
+          </visual>
+          <collision>
+            <origin xyz="0 0 0.01" rpy="0 0 0" />
+            <geometry>
+              <box size="0.001 0.001 0.001" />
+            </geometry>
+          </collision>
+        </link>
+        <joint name="position" type="planar">
+          <origin rpy="0 0 0" xyz="0 0 0"/>
+          <parent link="odom"/>
+          <child link="${prefix}base_footprint"/>
+        </joint>
+        <!-- <joint name="position" type="prismatic">
+          <axis xyz="-1 0 0" />
+          <origin rpy="0 0 0" xyz="0 0 0"/>
+          <parent link="odom"/>
+          <child link="${prefix}base_footprint"/>
+          <limit lower="-1" upper="1" effort="1000" velocity="100" />
+        </joint>         -->
         <joint name="${prefix}base_footprint_joint" type="fixed">
           <origin xyz="0 0 ${wheel_radius - wheel_offset_z}" rpy="0 0 0" />
@@ -91,5 +125,61 @@
           <child link="${prefix}base_link"/>
         </joint>
-      </xacro:unless>
+        <ros2_control name="position_ros2_control" type="system">
+          <hardware>
+            <xacro:if value="${ros2_control_hardware_type_positon_joint == 'mock_components'}">
+              <plugin>mock_components/GenericSystem</plugin>
+              <param name="calculate_dynamics">true</param>
+            </xacro:if>
+            <xacro:if value="${ros2_control_hardware_type_positon_joint == 'gz_ros2_control'}">
+              <xacro:if value="${ros_distro == 'humble'}">
+                <plugin>ign_ros2_control_base_movement/IgnBaseMovementSystemHardware</plugin>
+              </xacro:if>
+              <xacro:unless value="${ros_distro == 'humble'}">
+                <plugin>gz_ros2_control_base_movement/GzBaseMovementSystemHardware</plugin>
+              </xacro:unless>
+            </xacro:if>
+            <xacro:if value="${ros2_control_hardware_type_positon_joint == 'real_life'}">
+              <plugin>ros2_control_base_movement/BaseMovementSystemHardware</plugin>
+            </xacro:if>
+          </hardware>
+          <!-- Virtual position joint for supporting MoveIt's planar joint type in joint trajectories -->
+          <joint name="position/x">
+            <param name="initial_position">0.0</param>
+            <command_interface name="velocity" />
+            <state_interface name="position"/>
+            <state_interface name="velocity"/>
+          </joint>
+          <joint name="position/y">
+            <param name="initial_position">0.0</param>
+            <command_interface name="velocity" />
+            <state_interface name="position"/>
+            <state_interface name="velocity"/>
+          </joint>
+          <joint name="position/theta">
+            <param name="initial_position">0.0</param>
+            <command_interface name="velocity" />
+            <state_interface name="position"/>
+            <state_interface name="velocity"/>
+          </joint>
+          <!-- Wheel joints used for diff drive controller support -->
+          <joint name="joint_left_wheel">
+            <command_interface name="velocity"/>
+            <state_interface name="position"/>
+            <state_interface name="velocity"/>
+          </joint>
+          <joint name="joint_right_wheel">
+            <command_interface name="velocity"/>
+            <state_interface name="position"/>
+            <state_interface name="velocity"/>
+          </joint>
+        </ros2_control>
+      </xacro:if>
+      <xacro:if value="${position_joint_type == 'fixed'}">
+        <joint name="${prefix}base_footprint_joint" type="fixed">
+          <origin xyz="0 0 ${wheel_radius - wheel_offset_z}" rpy="0 0 0" />
+          <parent link="${prefix}base_footprint"/>
+          <child link="${prefix}base_link"/>
+        </joint>
+      </xacro:if>
     </xacro:if>
     <!-- BASE_LINK -->

File: src/ros2/robot_description/rb_theron_common/rb_theron_description/urdf/common.gazebo.xacro (robot description, xacro)
@@ -2,15 +2,29 @@
 <robot xmlns:xacro="http://www.ros.org/wiki/xacro">
     <!-- ROS CONTROL GAZEBO PLUGIN -->
-    <xacro:macro name="ros_control" params="ros_distro">
+    <xacro:macro name="ros_control" params="ros_distro position_joint_type">
         <gazebo>
             <xacro:if value="${ros_distro == 'humble'}">
-                <plugin name="ign_ros2_control::IgnitionROS2ControlPlugin" filename="libign_ros2_control-system.so">
-                    <parameters>$(find rb_theron_description)/config/rb_theron_gz_ros2_controller.yaml</parameters>
-                </plugin>
+                <xacro:if value="${position_joint_type == 'fixed' or position_joint_type == 'prismatic'}">
+                    <plugin name="ign_ros2_control::IgnitionROS2ControlPlugin" filename="libign_ros2_control-system.so">
+                        <parameters>$(find rb_theron_description)/config/rb_theron_gz_ros2_controller.yaml</parameters>
+                    </plugin>
+                </xacro:if>
+                <xacro:if value="${position_joint_type == 'planar'}">
+                    <plugin name="ign_ros2_control::IgnitionROS2ControlPlugin" filename="libign_ros2_control-system.so">
+                        <parameters>$(find rb_theron_description)/config/rb_theron_planar_base_gz_ros2_control.yaml</parameters>
+                    </plugin>
+                </xacro:if>
             </xacro:if>
             <xacro:unless value="${ros_distro == 'humble'}">
-                <plugin name="gz_ros2_control::GazeboSimROS2ControlPlugin" filename="gz_ros2_control-system">
-                    <parameters>$(find rb_theron_description)/config/rb_theron_gz_ros2_controller.yaml</parameters>
-                </plugin>
+                <xacro:if value="${position_joint_type == 'fixed' or position_joint_type == 'prismatic'}">
+                    <plugin name="gz_ros2_control::GazeboSimROS2ControlPlugin" filename="gz_ros2_control-system">
+                        <parameters>$(find rb_theron_description)/config/rb_theron_gz_ros2_controller.yaml</parameters>
+                    </plugin>
+                </xacro:if>
+                <xacro:if value="${position_joint_type == 'planar'}">
+                    <plugin name="gz_ros2_control::GazeboSimROS2ControlPlugin" filename="gz_ros2_control-system">
+                        <parameters>$(find rb_theron_description)/config/rb_theron_planar_base_gz_ros2_control.yaml</parameters>
+                    </plugin>
+                </xacro:if>
             </xacro:unless>
         </gazebo>

Commit message: starting to add zed to sim

File: src/ros2/robot_description/rb_theron_common/rb_theron_description/robots/rb_theron.urdf.xacro (robot description, xacro)
@@ -69,4 +69,11 @@
 	<!-- <xacro:ros_control/> -->
 	<xacro:gazebo_colors prefix="$(arg prefix)"/>
+	<!--Zed added more or less manually TODO why robot everywhere-->
+	<xacro:stereolabs_zed2 prefix="$(arg prefix)zed2" parent="base_link" model="zed2" near="0.3" far="20">
+	    <origin
+		xyz="0.27 0 1.43"
+		rpy="0 0.416 0"
+		/>
+  	</xacro:stereolabs_zed2>
 	<!-- SENSORS  DEBUGG-->
 	<!-- TODO: Should be sensor_intel_d435, but this one isn't migrated to ros2 yet -->

File: src/ros2/robot_description/robotnik_sensors/urdf/zed2.urdf.xacro (robot description, xacro)
@@ -3,4 +3,48 @@
   <xacro:macro name="depth_camera"
     params="prefix fps baseline hfov width height format near far  prefix_topic:='zed_node'">
+    <gazebo reference="${base_frame}">
+      <sensor name="${prefix}_rgb_camera_optical_frame" type="camera">
+				<topic>${prefix_topic}/color</topic>
+        <camera name="oak-d">
+            <horizontal_fov>1.2112585008840648</horizontal_fov>
+            <image>
+                <width>640</width>
+                <height>480</height>
+                <format>RGB_INT8</format>
+            </image>
+            <clip>
+                <near>0.1</near>
+                <far>100</far>
+            </clip>
+              <noise>
+                <type>gaussian</type>
+                <mean>0.0</mean>
+                <stddev>0.007</stddev>
+            </noise>
+        </camera>
+      </sensor>
+      <sensor name="${prefix}_right_camera_optical_frame" type="depth">
+        <topic>${prefix_topic}/${prefix}/depth</topic>
+        <camera name="oak-d">
+          <horizontal_fov>${85.2*M_PI/180.0}</horizontal_fov>
+          <image>
+            <width>640</width>
+            <height>480</height>
+          </image>
+          <clip>
+            <near>0.3</near>
+            <far>10.0</far>
+          </clip>
+          <noise>
+            <type>gaussian</type>
+            <mean>0.0</mean>
+            <stddev>0.010</stddev>
+          </noise>
+        </camera>
+        <always_on>1</always_on>
+        <update_rate>15</update_rate>
+        <visualize>1</visualize>
+      </sensor>
+    </gazebo>
     <gazebo reference="${prefix}_base_link">
       <visual>

Commit message: Revert "starting to add zed to sim"
This reverts commit 90022a9de8b11e99963ce31af8f18a033210885d.

File: src/ros2/robot_description/rb_theron_common/rb_theron_description/robots/rb_theron.urdf.xacro (robot description, xacro)
@@ -70,11 +70,4 @@
 	<!-- <xacro:ros_control/> -->
 	<xacro:gazebo_colors prefix="$(arg prefix)"/>
-	<!--Zed added more or less manually TODO why robot everywhere-->
-	<xacro:stereolabs_zed2 prefix="$(arg prefix)zed2" parent="base_link" model="zed2" near="0.3" far="20">
-	    <origin
-		xyz="0.27 0 1.43"
-		rpy="0 0.416 0"
-		/>
-  	</xacro:stereolabs_zed2>
 	<!-- SENSORS  DEBUGG-->
 	<!-- TODO: Should be sensor_intel_d435, but this one isn't migrated to ros2 yet -->

File: src/ros2/robot_description/robotnik_sensors/urdf/zed2.urdf.xacro (robot description, xacro)
@@ -3,48 +3,4 @@
   <xacro:macro name="depth_camera"
     params="prefix fps baseline hfov width height format near far  prefix_topic:='zed_node'">
-    <gazebo reference="${base_frame}">
-      <sensor name="${prefix}_rgb_camera_optical_frame" type="camera">
-				<topic>${prefix_topic}/color</topic>
-        <camera name="oak-d">
-            <horizontal_fov>1.2112585008840648</horizontal_fov>
-            <image>
-                <width>640</width>
-                <height>480</height>
-                <format>RGB_INT8</format>
-            </image>
-            <clip>
-                <near>0.1</near>
-                <far>100</far>
-            </clip>
-              <noise>
-                <type>gaussian</type>
-                <mean>0.0</mean>
-                <stddev>0.007</stddev>
-            </noise>
-        </camera>
-      </sensor>
-      <sensor name="${prefix}_right_camera_optical_frame" type="depth">
-        <topic>${prefix_topic}/${prefix}/depth</topic>
-        <camera name="oak-d">
-          <horizontal_fov>${85.2*M_PI/180.0}</horizontal_fov>
-          <image>
-            <width>640</width>
-            <height>480</height>
-          </image>
-          <clip>
-            <near>0.3</near>
-            <far>10.0</far>
-          </clip>
-          <noise>
-            <type>gaussian</type>
-            <mean>0.0</mean>
-            <stddev>0.010</stddev>
-          </noise>
-        </camera>
-        <always_on>1</always_on>
-        <update_rate>15</update_rate>
-        <visualize>1</visualize>
-      </sensor>
-    </gazebo>
     <gazebo reference="${prefix}_base_link">
       <visual>
