Commit message: changed sim sensor setup to match reality again

File: src/ros2/robot_description/rb_theron_common/rb_theron_description/robots/rb_theron.urdf.xacro (robot description, xacro)
@@ -93,38 +93,10 @@
 		<origin xyz="0.250 0.0 0.1643" rpy="0 3.1416 3.1416"/>
 	</xacro:sensor_sick_nanoscan3>
-	<!--<xacro:sensor_rs_lidar_16 prefix="$(arg prefix)top_laser" parent="$(arg prefix)base_link" prefix_topic="top_laser" min_angle="-3.1416" max_angle="3.1416">
-		<origin xyz="0.214 0.0 0.275" rpy="-1.57079632679 0 -0.23"/>
-	</xacro:sensor_rs_lidar_16>-->
-	<xacro:sensor_rs_bpearl prefix="$(arg prefix)top_laser" parent="$(arg prefix)base_link" sensor_base_frame="${sensor_base_frame}" robot_name="${robot_name}" prefix_topic="top_laser" hq="${hq}" range_min="0.1" range_max="90" hfov="360" samples="1800" vfov="90.0" lasers="32" fps="10" gpu="false">
-		<origin xyz="0.3 -0.175 1.165" rpy="-1.570796326795 0 -1.570796326795"/>
-		<!-- positions of the b-pearl based on solid: xyz="0.333 -0.180 1.194" rpy="-1.570796326795 0 -1.570796326795" -->
-	</xacro:sensor_rs_bpearl>
+	<xacro:sensor_zed2 prefix="$(arg prefix)zed" parent="$(arg prefix)base_link" sensor_base_frame="${sensor_base_frame}" robot_name="${robot_name}" prefix_topic="zed2" hq="${hq}">
+		<origin xyz="0.27 0 1.43" rpy="0 0.416 0"/>
+  	</xacro:sensor_zed2>
 	<!-- <xacro:sensor_sick_nanoscan3 prefix="$(arg prefix)back_laser" parent="$(arg prefix)base_link" prefix_topic="back_laser" min_angle="-1.8107619" max_angle="1.8107619">
 		<origin xyz="-0.250 0.0 0.1643" rpy="0 3.1416 0"/>
 	</xacro:sensor_sick_nanoscan3> -->
-	<xacro:arg name="front_oak_d_camera_model" default="OAK-D-S2" />
-	<xacro:arg name="front_oak_d_base_frame" default="oak-d-s2-usb-base--frame" />
-	<xacro:arg name="front_oak_d_pos_x" default="0.317" />
-	<xacro:arg name="front_oak_d_pos_y" default="-0.197" />
-	<xacro:arg name="front_oak_d_pos_z" default="1.3044" />
-	<xacro:arg name="front_oak_d_roll" default="0.0" />
-	<xacro:arg name="front_oak_d_pitch" default="0.0" />
-	<xacro:arg name="front_oak_d_yaw" default="0.0" />
-	<xacro:depthai_camera
-		prefix="$(arg prefix)front_top_oak_d_camera"
-		parent="$(arg prefix)base_link"
-		sensor_base_frame="${sensor_base_frame}"
-		robot_name="${robot_name}"
-		prefix_topic="front_top_oak_d_camera"
-		camera_model="$(arg front_oak_d_camera_model)"
-		base_frame="$(arg front_oak_d_base_frame)"
-		cam_pos_x="$(arg front_oak_d_pos_x)"
-		cam_pos_y="$(arg front_oak_d_pos_y)"
-		cam_pos_z="$(arg front_oak_d_pos_z)"
-		cam_roll="$(arg front_oak_d_roll)"
-		cam_pitch="$(arg front_oak_d_pitch)"
-		cam_yaw="$(arg front_oak_d_yaw)"
-		hq="${hq}">
-	</xacro:depthai_camera>
 	<!-- ROBAST Module Cage -->
 	<xacro:include filename="$(find rb_theron_description)/urdf/module_cage/module_cage.urdf.xacro" />

File: src/ros2/robot_description/robotnik_sensors/urdf/zed2.urdf.xacro (robot description, xacro)
@@ -1,4 +1,4 @@
 <?xml version="1.0"?>
-<robot xmlns:xacro="http://wiki.ros.org/xacro">
+<robot name="sensor_zed2" xmlns:xacro="http://wiki.ros.org/xacro">
   <xacro:macro name="depth_camera"
     params="prefix fps baseline hfov width height format near far  prefix_topic:='zed_node'">
@@ -12,16 +12,35 @@
         </material>
       </visual>
-      <sensor type="depth" name="depth_camera">
-        <update_rate>${fps}</update_rate>
-        <camera>
-          <horizontal_fov>${hfov}</horizontal_fov>
+      <sensor name="${prefix}_rgb_camera_optical_frame" type="camera">
+				<topic>${prefix_topic}/color</topic>
+        <camera name="zed2">
+            <horizontal_fov>1.2217</horizontal_fov>
+            <image>
+                <width>1280</width>
+                <height>720</height>
+                <format>RGB_INT8</format>
+            </image>
+            <clip>
+                <near>0.1</near>
+                <far>100</far>
+            </clip>
+              <noise>
+                <type>gaussian</type>
+                <mean>0.0</mean>
+                <stddev>0.007</stddev>
+            </noise>
+        </camera>
+      </sensor>
+      <sensor name="${prefix}_right_camera_optical_frame" type="depth">
+        <topic>${prefix_topic}/${prefix}/depth</topic>
+        <camera name="zed2">
+          <horizontal_fov>${85.2*M_PI/180.0}</horizontal_fov>
           <image>
-            <width>${width}</width>
-            <height>${height}</height>
-            <format>${format}</format>
+            <width>1280</width>
+            <height>720</height>
           </image>
           <clip>
-            <near>${near}</near>
-            <far>${far}</far>
+            <near>0.3</near>
+            <far>10.0</far>
           </clip>
           <noise>
@@ -31,30 +50,7 @@
           </noise>
         </camera>
-        <plugin name="camera_plugin" filename="libgazebo_ros_openni_kinect.so">
-          <baseline>${baseline}</baseline>
-          <alwaysOn>true</alwaysOn>
-          <!-- Keep this zero, update_rate in the parent <sensor> tag
-            will control the frame rate. -->
-          <updateRate>0.0</updateRate>
-          <cameraName>${prefix_topic}</cameraName>
-          <imageTopicName> rgb/image_raw</imageTopicName>
-          <cameraInfoTopicName>rgb/camera_info</cameraInfoTopicName>
-          <depthImageTopicName>depth/image_raw</depthImageTopicName>
-          <depthImageCameraInfoTopicName>depth/camera_info</depthImageCameraInfoTopicName>
-          <pointCloudTopicName>depth/points</pointCloudTopicName>
-          <frameName>/${prefix}_depth_optical_frame</frameName>
-          <pointCloudCutoff>${near}</pointCloudCutoff>
-          <pointCloudCutoffMax>${far}</pointCloudCutoffMax>
-          <distortionK1>0</distortionK1>
-          <distortionK2>0</distortionK2>
-          <distortionK3>0</distortionK3>
-          <distortionT1>0</distortionT1>
-          <distortionT2>0</distortionT2>
-          <CxPrime>0</CxPrime>
-          <Cx>0</Cx>
-          <Cy>0</Cy>
-          <focalLength>0</focalLength>
-          <hackBaseline>0</hackBaseline>
-        </plugin>
+        <always_on>1</always_on>
+        <update_rate>10</update_rate>
+        <visualize>1</visualize>
       </sensor>
     </gazebo>
@@ -150,8 +146,8 @@
         />
   </xacro:macro>
-  <xacro:macro name="sensor_zed2" params="prefix:=zed2 parent *origin model:=zed2  prefix_topic:=zed_node" >
-    <stereolabs_zed2 prefix="${prefix}" parent="${parent}" model="${model}" prefix_topic="${prefix_topic}">
+  <xacro:macro name="sensor_zed2" params="prefix:=zed2 parent sensor_base_frame robot_name hq *origin model:=zed2  prefix_topic:=zed_node" >
+    <xacro:stereolabs_zed2 prefix="${prefix}" parent="${parent}" model="${model}" prefix_topic="${prefix_topic}">
       <xacro:insert_block name="origin" />
-    </stereolabs_zed2>
+    </xacro:stereolabs_zed2>
   </xacro:macro>
 </robot>

Commit message: removed unused parameters

File: src/ros2/robot_description/rb_theron_common/rb_theron_description/robots/rb_theron.urdf.xacro (robot description, xacro)
@@ -93,5 +93,5 @@
 		<origin xyz="0.250 0.0 0.1643" rpy="0 3.1416 3.1416"/>
 	</xacro:sensor_sick_nanoscan3>
-	<xacro:sensor_zed2 prefix="$(arg prefix)zed" parent="$(arg prefix)base_link" sensor_base_frame="${sensor_base_frame}" robot_name="${robot_name}" prefix_topic="zed2" hq="${hq}">
+	<xacro:sensor_zed2 prefix="$(arg prefix)zed" parent="$(arg prefix)base_link" prefix_topic="zed2">
 		<origin xyz="0.27 0 1.43" rpy="0 0.416 0"/>
   	</xacro:sensor_zed2>

File: src/ros2/robot_description/robotnik_sensors/urdf/zed2.urdf.xacro (robot description, xacro)
@@ -148,5 +148,5 @@
         />
   </xacro:macro>
-  <xacro:macro name="sensor_zed2" params="prefix:=zed2 parent sensor_base_frame robot_name hq *origin model:=zed2  prefix_topic:=zed_node" >
+  <xacro:macro name="sensor_zed2" params="prefix:=zed2 parent *origin model:=zed2 prefix_topic:=zed_node" >
     <xacro:stereolabs_zed2 prefix="${prefix}" parent="${parent}" model="${model}" prefix_topic="${prefix_topic}">
       <xacro:insert_block name="origin" />

Commit message: feat: - added 2nd laser to sim - added a ported version of the ros1 package ira_laser_tools - configured a laser merge - added the merged lasers to slam

File: src/ros2/robot_description/rb_theron_common/rb_theron_description/robots/rb_theron.urdf.xacro (robot description, xacro)
@@ -22,4 +22,6 @@
 	<!-- This name should match the "-name" argument we need to declare when spawing the robot into ign gazebo -->
 	<xacro:property name="robot_name" value="rb_theron"/>
+	<xacro:arg name="robot_type" default="cura"/>
+	<xacro:property name="robot_type_prop" value="$(arg robot_type)"/>
 	<!-- Wheel parameters -->
 	<!--xacro:property name="wheel_offset_x" value="0" />
@@ -90,7 +92,17 @@
 		<origin xyz="-0.1975 0.0 0.1598" rpy="0 0 0"/>
 	</xacro:sensor_imu_hector>
-	<xacro:sensor_sick_nanoscan3 prefix="$(arg prefix)front_laser" parent="$(arg prefix)base_link" sensor_base_frame="${sensor_base_frame}" robot_name="${robot_name}" prefix_topic="front_laser" hq="${hq}" min_angle="-1.9507619" max_angle="1.9507619" gpu="true">
-		<origin xyz="0.250 0.0 0.1643" rpy="0 3.1416 3.1416"/>
-	</xacro:sensor_sick_nanoscan3>
+	<xacro:if value="${robot_type_prop == 'cura'}">
+		<xacro:sensor_sick_nanoscan3 prefix="$(arg prefix)front_laser" parent="$(arg prefix)base_link" sensor_base_frame="${sensor_base_frame}" robot_name="${robot_name}" prefix_topic="front_laser" hq="${hq}" min_angle="-2.356" max_angle="2.356" gpu="true">
+			<origin xyz="0.2675 -0.215 0.1613" rpy="0 -3.1416 2.3562"/>
+		</xacro:sensor_sick_nanoscan3>
+		<xacro:sensor_sick_nanoscan3 prefix="$(arg prefix)rear_laser" parent="$(arg prefix)base_link" sensor_base_frame="${sensor_base_frame}" robot_name="${robot_name}" prefix_topic="rear_laser" hq="${hq}" min_angle="-2.356" max_angle="2.356" gpu="true">
+			<origin xyz="-0.2675 0.215 0.1613" rpy="0 -3.1416 -0.7854"/>
+		</xacro:sensor_sick_nanoscan3>
+	</xacro:if>
+	<xacro:unless value="${robot_type_prop == 'cura'}">
+		<xacro:sensor_sick_nanoscan3 prefix="$(arg prefix)front_laser" parent="$(arg prefix)base_link" sensor_base_frame="${sensor_base_frame}" robot_name="${robot_name}" prefix_topic="front_laser" hq="${hq}" min_angle="-1.9507619" max_angle="1.9507619" gpu="true">
+			<origin xyz="0.250 0.0 0.1643" rpy="0 3.1416 3.1416"/>
+		</xacro:sensor_sick_nanoscan3>
+	</xacro:unless>
 	<!--<xacro:sensor_rs_lidar_16 prefix="$(arg prefix)top_laser" parent="$(arg prefix)base_link" prefix_topic="top_laser" min_angle="-3.1416" max_angle="3.1416">
 		<origin xyz="0.214 0.0 0.275" rpy="-1.57079632679 0 -0.23"/>

File: src/ros2/robot_description/rb_theron_common/rb_theron_description/urdf/bases/theron_base.urdf.xacro (robot description, xacro)
@@ -146,5 +146,5 @@
           <joint name="position/x">
             <param name="initial_position">0.0</param>
-            <command_interface name="velocity" />
+            <command_interface name="velocity"/>
             <state_interface name="position"/>
             <state_interface name="velocity"/>
