Commit message: Adding again door_opening_mechanism_joint_x_axis_slide and door_opening_mechanism_joint_tilting_hook

File: src/ros2/simulation/moveit2_ressources/moveit2_door_opening_mechanism/config/rb_theron.ros2_control.xacro (robot description, xacro)
@@ -15,4 +15,18 @@
                 <state_interface name="velocity"/>
             </joint>
+            <joint name="door_opening_mechanism_joint_x_axis_slide">
+                <command_interface name="position"/>
+                <state_interface name="position">
+                  <param name="initial_value">${initial_positions['door_opening_mechanism_joint_x_axis_slide']}</param>
+                </state_interface>
+                <state_interface name="velocity"/>
+            </joint>
+            <joint name="door_opening_mechanism_joint_tilting_hook">
+                <command_interface name="position"/>
+                <state_interface name="position">
+                  <param name="initial_value">${initial_positions['door_opening_mechanism_joint_tilting_hook']}</param>
+                </state_interface>
+                <state_interface name="velocity"/>
+            </joint>
         </ros2_control>
     </xacro:macro>
