Commit message: Plugins gazebo -> ignition for rb_theron

File: src/ros2/robot_description/rb_theron_common/rb_theron_description/urdf/common.gazebo.xacro (robot description, xacro)
@@ -7,45 +7,17 @@
 				<parameters>$(find rb_theron_description)/config/rb_theron_controller.yaml</parameters>
 			</plugin> -->
-			<plugin name="joint_state" filename="libgazebo_ros_joint_state_publisher.so">
-				<ros>
-					<remapping>~/out:=joint_states</remapping>
-				</ros>
-				<alwaysOn>1</alwaysOn>
-				<update_rate>30</update_rate>
-				<joint_name>$(arg prefix)leftjoint_rsupport</joint_name>
-				<joint_name>$(arg prefix)rightjoint_rsupport</joint_name>
-				<joint_name>$(arg prefix)left_wheel_joint</joint_name>
-				<joint_name>$(arg prefix)right_wheel_joint</joint_name>
-				<joint_name>$(arg prefix)leftcastorjoint_support</joint_name>
-				<joint_name>$(arg prefix)rightcastorjoint_support</joint_name>
-				<joint_name>$(arg prefix)leftcastorjoint_wheel</joint_name>
-				<joint_name>$(arg prefix)rightcastorjoint_wheel</joint_name>
-				<joint_name>$(arg prefix)leftjoint_support</joint_name>
-				<joint_name>$(arg prefix)rightjoint_support</joint_name>
-				<joint_name>$(arg prefix)leftjoint_wheel</joint_name>
-				<joint_name>$(arg prefix)rightjoint_wheel</joint_name>
-				<joint_name>top_drawer_joint</joint_name>
+			<plugin
+				filename="gz-sim-joint-state-publisher-system"
+				name="gz::sim::systems::JointStatePublisher">
 			</plugin>
-			<plugin name="diff_drive" filename="libgazebo_ros_diff_drive.so">
-				<alwaysOn>1</alwaysOn>
-				<update_rate>30</update_rate>
-				<!-- wheels -->
+			<plugin
+				filename="libgz-sim-diff-drive-system.so"
+				name="gz::sim::systems::DiffDrive">
 				<left_joint>$(arg prefix)left_wheel_joint</left_joint>
 				<right_joint>$(arg prefix)right_wheel_joint</right_joint>
-				<!-- kinematics -->
 				<wheel_separation>0.5032</wheel_separation>
-				<wheel_diameter>0.1524</wheel_diameter>
-				<!-- limits -->
-				<max_wheel_torque>20</max_wheel_torque>
-				<max_wheel_acceleration>2.5</max_wheel_acceleration>
-				<command_topic>cmd_vel</command_topic>
-				<!-- output -->
-				<publish_odom>true</publish_odom>
-				<publish_odom_tf>true</publish_odom_tf>
-				<publish_wheel_tf>false</publish_wheel_tf>
-				<odometry_topic>odom</odometry_topic>
-				<odometry_frame>$(arg prefix)odom</odometry_frame>
-				<!-- <base_frame>$(arg prefix)base_footprint</base_frame> -->
-    				<robot_base_frame>$(arg prefix)base_footprint</robot_base_frame>
+				<wheel_radius>0.0762</wheel_radius>
+				<odom_publish_frequency>30</odom_publish_frequency>
+				<topic>cmd_vel</topic>
 			</plugin>
 		</gazebo>

File: src/ros2/robot_description/robotnik_sensors/urdf/imu_hector_plugin.urdf.xacro (robot description, xacro)
@@ -29,24 +29,10 @@
 	  </link>
 	  <gazebo>
-	    <plugin name="${prefix}_controller" filename="libhector_gazebo_ros_imu.so">
-	       <alwaysOn>true</alwaysOn>
-	       <topicName>${topic}</topicName>
-		   <serviceName>${prefix}imu/service</serviceName>
-		   <bodyName>${prefix}_link</bodyName>
-		   <frameId>${prefix}_link</frameId>
-	       <updateRate>50.0</updateRate>
-	       <gaussianNoise>0.00</gaussianNoise>
-           <yawOffset>0.0</yawOffset>
-           <yawDrift>0.0</yawDrift>
-           <yawGaussianNoise>0.0</yawGaussianNoise>
-           <!-- angular velocities parameters -->
-           <rateOffset>0.0 0.0 0.0</rateOffset>
-           <rateDrift>0.0 0.0 0.0</rateDrift>
-           <rateGaussianNoise>0.0 0.0 0.0</rateGaussianNoise>
-           <!-- linear accelerations parameters -->
-           <accelOffset>0.0 0.0 0.0</accelOffset>
-           <accelDrift>0.0 0.0 0.0</accelDrift>
-           <accelGaussianNoise>0.0 0.0 0.0</accelGaussianNoise>
-	    </plugin>
+		<plugin name="gz::sim::systems::Imu" filename="libgz-sim-imu-system.so">
+			<always_on>1</always_on>
+			<update_rate>50</update_rate>
+			<topic>${topic}</topic>
+			<visualize>true</visualize>
+		</plugin>
 	  </gazebo>
   </xacro:macro>

File: src/ros2/robot_description/robotnik_sensors/urdf/sick_nanoscan3.urdf.xacro (robot description, xacro)
@@ -49,13 +49,15 @@
 			<xacro:if value="${gpu}">
 				<xacro:property name="ray_type" value="gpu_ray" />
-				<xacro:property name="plugin_lib" value="libgazebo_ros_ray_sensor.so" />
+				<xacro:property name="plugin_lib" value="libgz-sim-sensors-system.so" />
 			</xacro:if>
 			<xacro:unless value="${gpu}">
 				<xacro:property name="ray_type" value="ray" />
-				<xacro:property name="plugin_lib" value="libgazebo_ros_ray_sensor.so" />
+				<xacro:property name="plugin_lib" value="libgz-sim-sensors-system.so" />
 			</xacro:unless>
 			<sensor type="${ray_type}" name="${prefix}_sensor">
-				<pose>0 0 0 0 0 0</pose>
-				<visualize>false</visualize>
+				<pose relative_to='${prefix}_link'>0 0 0 0 0 0</pose>
+				<topic>${prefix_topic}/scan</topic>
+				<always_on>1</always_on>
+    				<visualize>true</visualize>
 				<update_rate>12.5</update_rate>
 				<ray>
@@ -67,4 +69,10 @@
 							<max_angle>${max_angle}</max_angle>
 						</horizontal>
+						<vertical>
+							<samples>1</samples>
+							<resolution>0.01</resolution> <!-- TODO: CHECK IF THIS VALUE IS CORRECT -->
+							<min_angle>0</min_angle>
+							<max_angle>0</max_angle>
+						</vertical>
 					</scan>
 					<range>
@@ -79,11 +87,6 @@
 					</noise>
 				</ray>
-				<plugin name="${prefix}_controller" filename="${plugin_lib}">
-					<ros>
-						<remapping>~/out:=${prefix_topic}/scan</remapping>
-					</ros>
-					<frame_name>${prefix}_link</frame_name>
-					<output_type>sensor_msgs/LaserScan</output_type>
-					<!-- if not global (leading /) sets the current namespace as a prefix (/ns/name_laser_link) -->
+				<plugin name="gz::sim::systems::Sensors" filename="${plugin_lib}">
+					<render_engine>ogre2</render_engine>
 				</plugin>
 			</sensor>

Commit message: Adding ign_ros2_control and changing garden->fortress because ign_ros2_control does not yet support garden

File: src/ros2/robot_description/rb_theron_common/rb_theron_description/urdf/common.gazebo.xacro (robot description, xacro)
@@ -8,10 +8,10 @@
 			</plugin> -->
 			<plugin
-				filename="gz-sim-joint-state-publisher-system"
-				name="gz::sim::systems::JointStatePublisher">
+				filename="libignition-gazebo-joint-state-publisher-system"
+				name="ignition::gazebo::systems::JointStatePublisher">
 			</plugin>
 			<plugin
-				filename="libgz-sim-diff-drive-system.so"
-				name="gz::sim::systems::DiffDrive">
+				filename="libignition-gazebo-diff-drive-system.so"
+				name="ignition::gazebo::systems::DiffDrive">
 				<left_joint>$(arg prefix)left_wheel_joint</left_joint>
 				<right_joint>$(arg prefix)right_wheel_joint</right_joint>

File: src/ros2/robot_description/robotnik_sensors/urdf/imu_hector_plugin.urdf.xacro (robot description, xacro)
@@ -29,5 +29,5 @@
 	  </link>
 	  <gazebo>
-		<plugin name="gz::sim::systems::Imu" filename="libgz-sim-imu-system.so">
+		<plugin name="ignition::gazebo::systems::Imu" filename="libignition-gazebo-imu-system.so">
 			<always_on>1</always_on>
 			<update_rate>50</update_rate>

File: src/ros2/robot_description/robotnik_sensors/urdf/sick_nanoscan3.urdf.xacro (robot description, xacro)
@@ -55,9 +55,9 @@
 			<xacro:if value="${gpu}">
 				<xacro:property name="ray_type" value="gpu_ray" />
-				<xacro:property name="plugin_lib" value="gz-sim-sensors-system" />
+				<xacro:property name="plugin_lib" value="libignition-gazebo-sensors-system.so" />
 			</xacro:if>
 			<xacro:unless value="${gpu}">
 				<xacro:property name="ray_type" value="ray" />
-				<xacro:property name="plugin_lib" value="gz-sim-sensors-system" />
+				<xacro:property name="plugin_lib" value="libignition-gazebo-sensors-system.so" />
 			</xacro:unless>
 			<sensor type="${ray_type}" name="${prefix}_link">
@@ -93,5 +93,5 @@
 					</noise>
 				</ray>
-				<plugin name="gz::sim::systems::Sensors" filename="${plugin_lib}">
+				<plugin name="ignition::gazebo::systems::Sensors" filename="${plugin_lib}">
 					<render_engine>ogre2</render_engine>
 				</plugin>

Commit message: Disabling odom->base_footprint tf by diffdrive plugin and adding sensor plugin for IMU so we can use robot_localization

File: src/ros2/robot_description/rb_theron_common/rb_theron_description/urdf/common.gazebo.xacro (robot description, xacro)
@@ -21,4 +21,7 @@
 				<topic>cmd_vel</topic>
 				<frame_id>$(arg prefix)odom</frame_id>
+				<!-- There is no possiblity (as far as I know) to disable tf publishing of odom->base, so if you
+				don't want the tf to be published, you can just dump it into a different topic -->
+				<tf_topic>tf_dump</tf_topic>
 				<xacro:if value="${publish_bf}">
 					<child_frame_id>$(arg prefix)base_footprint</child_frame_id>

File: src/ros2/robot_description/robotnik_sensors/urdf/imu_hector_plugin.urdf.xacro (robot description, xacro)
@@ -1,39 +1,51 @@
 <?xml version="1.0"?>
 <robot name="sensor_imu" xmlns:xacro="http://wiki.ros.org/xacro">
-  <xacro:macro name="sensor_imu_hector" params="prefix topic:='imu/data' parent *origin">
-	  <joint name="${prefix}_joint" type="fixed">
-	      <axis xyz="1 0 0"/>
-	      <!--origin xyz="0 0 0.2825"/-->
-	      <xacro:insert_block name="origin"/>
-	      <parent link="${parent}"/>
-	      <child link="${prefix}_link"/>
-	  </joint>
-	  <link name="${prefix}_link">
-	      <inertial>
-			<origin xyz="0.0 0 0.01" rpy="0 0 0" />
-			<mass value="0.05" />
-			<xacro:solid_cuboid_inertia m="0.05" w="0.02" h="0.02" d="0.02" />
-		  </inertial>
-	      <visual>
-	        <origin rpy="0 0 0" xyz="0 0 0"/>
-	        <geometry>
-	          <box size="0.001 0.001 0.001"/>
-	        </geometry>
-	      </visual>
-	      <collision>
-	        <origin rpy="0 0 0" xyz="0 0 0"/>
-	        <geometry>
-	          <box size=".001 .001 .001"/>
-	        </geometry>
-	      </collision>
-	  </link>
-	  <gazebo>
-		<plugin name="gz::sim::systems::Imu" filename="libgz-sim-imu-system.so">
-			<always_on>1</always_on>
-			<update_rate>50</update_rate>
-			<topic>${topic}</topic>
-			<visualize>true</visualize>
-		</plugin>
-	  </gazebo>
-  </xacro:macro>
+	<xacro:macro name="sensor_imu_hector" params="prefix topic:='imu/data' parent *origin">
+		<xacro:if value="${publish_bf}">
+			<xacro:property name="sensor_link_name" value="${robot_name}/base_footprint/${prefix}_link" />
+		</xacro:if>
+		<xacro:unless value="${publish_bf}">
+			<xacro:property name="sensor_link_name" value="${robot_name}/base_link/${prefix}_link" />
+		</xacro:unless>
+		<joint name="${prefix}_joint" type="fixed">
+			<axis xyz="1 0 0"/>
+			<!--origin xyz="0 0 0.2825"/-->
+			<xacro:insert_block name="origin"/>
+			<parent link="${parent}"/>
+			<child link="${sensor_link_name}"/>
+		</joint>
+		<link name="${sensor_link_name}">
+			<inertial>
+				<origin xyz="0.0 0 0.01" rpy="0 0 0" />
+				<mass value="0.05" />
+				<xacro:solid_cuboid_inertia m="0.05" w="0.02" h="0.02" d="0.02" />
+			</inertial>
+			<visual>
+				<origin rpy="0 0 0" xyz="0 0 0"/>
+				<geometry>
+					<box size="0.001 0.001 0.001"/>
+				</geometry>
+			</visual>
+			<collision>
+				<origin rpy="0 0 0" xyz="0 0 0"/>
+				<geometry>
+					<box size=".001 .001 .001"/>
+				</geometry>
+			</collision>
+		</link>
+		<gazebo reference="${sensor_link_name}">
+			<sensor name="${prefix}_link" type="imu">
+				<always_on>1</always_on>
+				<update_rate>40</update_rate>
+				<visualize>true</visualize>
+				<topic>imu/data</topic>
+			</sensor>
+		</gazebo>
+		<gazebo>
+			<plugin
+				filename="libgz-sim-imu-system"
+				name="gz::sim::systems::Imu">
+			</plugin>
+		</gazebo>
+	</xacro:macro>
 </robot>
