Commit message: reactor: reorganize xacros for door_opening_mechanism to facilitate introduction of new mechanism

File: src/ros2/robot_description/rb_theron_common/rb_theron_description/urdf/door_opening_mechanism/components/crossbar_with_double_hook.urdf.xacro (robot description, xacro)
@@ -1,10 +1,10 @@
 <?xml version="1.0"?>
-<robot name="door_opening_gripper" xmlns:xacro="http://www.ros.org/wiki/xacro">
-    <xacro:macro name="door_opening_gripper" params="prefix parent *origin">
-        <xacro:include filename="$(find rb_theron_description)/urdf/door_opening_mechanism/alu_profile.urdf.xacro" />
+<robot name="crossbar_with_double_hook" xmlns:xacro="http://www.ros.org/wiki/xacro">
+    <xacro:macro name="crossbar_with_double_hook" params="prefix parent *origin">
+        <xacro:include filename="$(find rb_theron_description)/urdf/door_opening_mechanism/components/alu_profile.urdf.xacro" />
         <xacro:alu_profile prefix="${prefix}" suffix="gripper" parent="${parent}" x="0.03" y="0.03" z="0.3" r="0" g="1" b="0">
             <xacro:insert_block name="origin" />
         </xacro:alu_profile>
-        <xacro:include filename="$(find rb_theron_description)/urdf/door_opening_mechanism/hook.urdf.xacro" />
+        <xacro:include filename="$(find rb_theron_description)/urdf/door_opening_mechanism/components/hook.urdf.xacro" />
         <xacro:hook prefix="${prefix}" suffix="left_hook" parent="${prefix}alu_profile_link_gripper" r="0" g="0" b="1">
             <origin xyz="-0.045 -0.01 0.13" rpy="0 0 0"/>

File: src/ros2/robot_description/rb_theron_common/rb_theron_description/urdf/door_opening_mechanism/components/hook.urdf.xacro (robot description, xacro)
@@ -7,5 +7,5 @@
     </xacro:macro>
     <xacro:macro name="hook" params="prefix suffix parent *origin r g b">
-    <xacro:include filename="$(find rb_theron_description)/urdf/door_opening_mechanism/basic_box.urdf.xacro" />
+    <xacro:include filename="$(find rb_theron_description)/urdf/door_opening_mechanism/basic_elements/basic_box.urdf.xacro" />
     <xacro:basic_box
         parent="${prefix}${parent}"

File: src/ros2/robot_description/rb_theron_common/rb_theron_description/urdf/door_opening_mechanism/door_opening_mechanism.urdf.xacro (robot description, xacro)
@@ -8,7 +8,7 @@
     <xacro:macro name="door_opening_mechanism" params="prefix parent *origin hq">
         <!-- Element imports -->
-        <xacro:include filename="$(find rb_theron_description)/urdf/door_opening_mechanism/alu_profile.urdf.xacro" />
-        <xacro:include filename="$(find rb_theron_description)/urdf/door_opening_mechanism/basic_box.urdf.xacro" />
-        <xacro:include filename="$(find rb_theron_description)/urdf/door_opening_mechanism/basic_joint.urdf.xacro" />
+        <xacro:include filename="$(find rb_theron_description)/urdf/door_opening_mechanism/components/alu_profile.urdf.xacro" />
+        <xacro:include filename="$(find rb_theron_description)/urdf/door_opening_mechanism/basic_elements/basic_box.urdf.xacro" />
+        <xacro:include filename="$(find rb_theron_description)/urdf/door_opening_mechanism/basic_elements/basic_joint.urdf.xacro" />
         <!-- Please mind: We might need to set the settings for the mass extremly low, because there
         is an issue, that if there is too much load on the theron base, it would be able to drive
@@ -124,37 +124,9 @@
             <origin xyz="0.038 -0.027 0" rpy="0 0 1.57079632679"/>
         </xacro:basic_box>
-        <xacro:basic_joint
-            parent="${prefix}door_opening_mechanism_link_x_slide_screwing"
-            joint_name="${prefix}door_opening_mechanism_joint_tilting_hook"
-            joint_type="revolute"
-            axis_x="1"
-            axis_y="0"
-            axis_z="0"
-            lower_limit="-0.02"
-            upper_limit="1.6"
-            damping="0.1"
-            friction="0.3"
-            p_gain="500"
-            i_gain="1000"
-            d_gain="10"
-            link_name="${prefix}door_opening_mechanism_link_tilting_hook"
-            link_origin_x="0.0"
-            link_origin_y="0.0"
-            link_origin_z="0.1"
-            m="0.2"
-            x="0.03"
-            y="0.03"
-            z="0.2"
-            r="0"
-            g="1"
-            b="0">
-            <!-- The default value for roll can be changed from 0 to pi/2 to position the arm upwards to get it out of the way -->
+        <!-- Tilting arm -->
+        <xacro:include filename="$(find rb_theron_description)/urdf/door_opening_mechanism/arm_variations/tilting_arm.urdf.xacro" />
+        <xacro:tilting_arm prefix="${prefix}" parent="${prefix}door_opening_mechanism_link_x_slide_screwing" >
             <origin xyz="0 -0.025 0" rpy="0 1.57079632679 0"/>
-        </xacro:basic_joint>
-        <!-- Gripper -->
-        <xacro:include filename="$(find rb_theron_description)/urdf/door_opening_mechanism/door_opening_gripper.urdf.xacro" />
-        <xacro:door_opening_gripper prefix="${prefix}" parent="${prefix}door_opening_mechanism_link_tilting_hook" >
-            <origin xyz="0 0 0.215" rpy="0 1.57079632679 0"/>
-        </xacro:door_opening_gripper>
+        </xacro:tilting_arm>
     </xacro:macro>
 </robot>
