Commit message: feat: adds freely_rotating_hook as active joint in order to help moveit in path planning (in theory)

File: src/ros2/moveit2_resources/moveit_door_opening_mechanism_rotating_arm_config/config/rb_theron.ros2_control.xacro (robot description, xacro)
@@ -29,4 +29,11 @@
                 <state_interface name="velocity"/>
             </joint>
+            <joint name="door_opening_mechanism_joint_freely_rotating_hook">
+                <command_interface name="position"/>
+                <state_interface name="position">
+                  <param name="initial_value">${initial_positions['door_opening_mechanism_joint_freely_rotating_hook']}</param>
+                </state_interface>
+                <state_interface name="velocity"/>
+            </joint>
         </ros2_control>
     </xacro:macro>

File: src/ros2/robot_description/rb_theron_common/rb_theron_description/urdf/door_opening_mechanism/components/freely_rotating_hook.urdf.xacro (robot description, xacro)
@@ -2,15 +2,16 @@
 <robot name="freely_rotating_hook" xmlns:xacro="http://www.ros.org/wiki/xacro">
     <xacro:macro name="freely_rotating_hook" params="prefix parent *origin">
+        <!-- Please mind: This joint is actually passive, but in order to help moveit plan the trajectory we make it active -->
         <xacro:basic_joint
             parent="${prefix}${parent}"
             joint_name="${prefix}door_opening_mechanism_joint_freely_rotating_hook"
-            joint_type="continuous"
+            joint_type="revolute"
             axis_x="1"
             axis_y="0"
             axis_z="0"
-            lower_limit="0"
-            upper_limit="3.141"
-            damping="0.01"
-            friction="0.01"
+            lower_limit="0.0"
+            upper_limit="3.14"
+            damping="0.05"
+            friction="0.1"
             p_gain="500"
             i_gain="1000"
