Commit message: fix: door_opening_mechanism_joint_tilting_hook -> door_opening_mechanism_joint_rotating_arm

File: src/ros2/robot_description/rb_theron_common/rb_theron_description/ros2_control/door_opening_mechanism.ros2_control.xacro (robot description, xacro)
@@ -33,5 +33,5 @@
         <state_interface name="velocity"/>
       </joint>
-      <joint name="${prefix}door_opening_mechanism_joint_tilting_hook">
+      <joint name="${prefix}door_opening_mechanism_joint_rotating_arm">
         <command_interface name="position">
           <param name="min">-1</param>

Commit message: feat: adds door_opening_mechanism_joint_freely_rotating_hook as controllable arm for now

File: src/ros2/robot_description/rb_theron_common/rb_theron_description/ros2_control/door_opening_mechanism.ros2_control.xacro (robot description, xacro)
@@ -11,10 +11,10 @@
       <joint name="${prefix}door_opening_mechanism_joint_y_axis_slide">
         <command_interface name="position">
-          <param name="min">-1</param>
-          <param name="max">1</param>
+          <param name="min">-5</param>
+          <param name="max">5</param>
         </command_interface>
         <command_interface name="velocity">
-          <param name="min">-1</param>
-          <param name="max">1</param>
+          <param name="min">-5</param>
+          <param name="max">5</param>
         </command_interface>
         <state_interface name="position"/>
@@ -23,10 +23,10 @@
       <joint name="${prefix}door_opening_mechanism_joint_x_axis_slide">
         <command_interface name="position">
-          <param name="min">-1</param>
-          <param name="max">1</param>
+          <param name="min">-5</param>
+          <param name="max">5</param>
         </command_interface>
         <command_interface name="velocity">
-          <param name="min">-1</param>
-          <param name="max">1</param>
+          <param name="min">-5</param>
+          <param name="max">5</param>
         </command_interface>
         <state_interface name="position"/>
@@ -45,4 +45,16 @@
         <state_interface name="velocity"/>
       </joint>
+      <joint name="${prefix}door_opening_mechanism_joint_freely_rotating_hook">
+        <command_interface name="position">
+          <param name="min">-1</param>
+          <param name="max">1</param>
+        </command_interface>
+        <command_interface name="velocity">
+          <param name="min">-1</param>
+          <param name="max">1</param>
+        </command_interface>
+        <state_interface name="position"/>
+        <state_interface name="velocity"/>
+      </joint>
     </ros2_control>
   </xacro:macro>
