Commit message: feat: executing trajectories in rviz works now

File: src/ros2/moveit/moveit_resources/moveit_door_opening_mechanism_rotating_arm_config/config/rb_theron.ros2_control.xacro (robot description, xacro)
@@ -1,40 +1,40 @@
 <?xml version="1.0"?>
 <robot xmlns:xacro="http://www.ros.org/wiki/xacro">
-    <xacro:macro name="rb_theron_ros2_control" params="name initial_positions_file">
-        <xacro:property name="initial_positions" value="${load_yaml(initial_positions_file)['initial_positions']}"/>
-        <ros2_control name="${name}" type="system">
-            <hardware>
-                <!-- By default, set up controllers for simulation. This won't work on real hardware -->
-                <plugin>mock_components/GenericSystem</plugin>
-            </hardware>
-            <joint name="door_opening_mechanism_joint_y_axis_slide">
-                <command_interface name="position"/>
-                <state_interface name="position">
-                  <param name="initial_value">${initial_positions['door_opening_mechanism_joint_y_axis_slide']}</param>
-                </state_interface>
-                <state_interface name="velocity"/>
-            </joint>
-            <joint name="door_opening_mechanism_joint_x_axis_slide">
-                <command_interface name="position"/>
-                <state_interface name="position">
-                  <param name="initial_value">${initial_positions['door_opening_mechanism_joint_x_axis_slide']}</param>
-                </state_interface>
-                <state_interface name="velocity"/>
-            </joint>
-            <joint name="door_opening_mechanism_joint_rotating_arm">
-                <command_interface name="position"/>
-                <state_interface name="position">
-                  <param name="initial_value">${initial_positions['door_opening_mechanism_joint_rotating_arm']}</param>
-                </state_interface>
-                <state_interface name="velocity"/>
-            </joint>
-            <joint name="door_opening_mechanism_joint_freely_rotating_hook">
-                <command_interface name="position"/>
-                <state_interface name="position">
-                  <param name="initial_value">${initial_positions['door_opening_mechanism_joint_freely_rotating_hook']}</param>
-                </state_interface>
-                <state_interface name="velocity"/>
-            </joint>
-        </ros2_control>
-    </xacro:macro>
+  <xacro:macro name="rb_theron_ros2_control" params="name initial_positions_file ros2_control_hardware_type">
+    <xacro:property name="initial_positions" value="${load_yaml(initial_positions_file)['initial_positions']}"/>
+    <ros2_control name="${name}" type="system">
+      <hardware>
+        <xacro:if value="${ros2_control_hardware_type == 'mock_components'}">
+            <plugin>mock_components/GenericSystem</plugin>
+        </xacro:if>
+        <xacro:if value="${ros2_control_hardware_type == 'dryve_d1'}">
+          <plugin>ros2_control_plugin_door_opening_mechanism/DoorOpeningMechanismSystemPositionOnlyHardware</plugin>
+          <!-- TODO@Jacob: Remove these params? -->
+          <param name="example_param_hw_start_duration_sec">0</param>
+          <param name="example_param_hw_stop_duration_sec">3.0</param>
+          <param name="example_param_hw_slowdown">100</param>
+        </xacro:if>
+      </hardware>
+      <joint name="door_opening_mechanism_joint_y_axis_slide">
+        <command_interface name="position"/>
+        <state_interface name="position"/>
+        <state_interface name="velocity"/>
+      </joint>
+      <joint name="door_opening_mechanism_joint_x_axis_slide">
+        <command_interface name="position"/>
+        <state_interface name="position"/>
+        <state_interface name="velocity"/>
+      </joint>
+      <joint name="door_opening_mechanism_joint_rotating_arm">
+        <command_interface name="position"/>
+        <state_interface name="position"/>
+        <state_interface name="velocity"/>
+      </joint>
+      <joint name="door_opening_mechanism_joint_freely_rotating_hook">
+        <command_interface name="position"/>
+        <state_interface name="position"/>
+        <state_interface name="velocity"/>
+      </joint>
+    </ros2_control>
+  </xacro:macro>
 </robot>

File: src/ros2/moveit/moveit_resources/moveit_door_opening_mechanism_rotating_arm_config/config/rb_theron.urdf.xacro (robot description, xacro)
@@ -2,8 +2,12 @@
 <robot xmlns:xacro="http://www.ros.org/wiki/xacro" name="rb_theron">
     <xacro:arg name="initial_positions_file" default="initial_positions.yaml" />
+    <!-- TODO: How do I pass a parameter to this xacro from a launch file? -->
+    <!-- Maybe like robotnik did here:
+    https://github.com/RobotnikAutomation/rb_theron_sim/blob/humble/rb_theron_gazebo/launch/description.launch.py -->
+    <xacro:arg name="ros2_control_hardware_type" default="mock_components" />
     <!-- Import rb_theron urdf file -->
     <xacro:include filename="$(find rb_theron_description)/robots/rb_theron.urdf.xacro" />
     <!-- Import control_xacro -->
     <xacro:include filename="rb_theron.ros2_control.xacro" />
-    <xacro:rb_theron_ros2_control name="FakeSystem" initial_positions_file="$(arg initial_positions_file)"/>
+    <xacro:rb_theron_ros2_control name="FakeSystem" initial_positions_file="$(arg initial_positions_file)" ros2_control_hardware_type="$(arg ros2_control_hardware_type)"/>
 </robot>

File: src/ros2/robot_description/rb_theron_common/rb_theron_description/robots/rb_theron.urdf.xacro (robot description, xacro)
@@ -12,6 +12,4 @@
 	<!-- Import Gazebo Stuff -->
 	<xacro:include filename="$(find rb_theron_description)/urdf/common.gazebo.xacro" />
-	<!-- Import Door opening mechanism ros2_control description -->
-  	<xacro:include filename="$(find rb_theron_description)/ros2_control/door_opening_mechanism.ros2_control.xacro" />
 	<!-- ***************** -->
 	<!-- Global parameters -->
@@ -114,5 +112,3 @@
 	<!-- Gazebo ros control pluggins -->
 	<xacro:ros_control prefix="$(arg prefix)" publish_bf="${publish_bf}"/>
-    <!-- ros2_control for the door_opening_mechanism -->
-	<xacro:ros2_control_door_opening_mechanism name="Door_opening_mechanism" prefix="$(arg prefix)"/>
 </robot>
