Commit message: feat: joints are now controlled only by ros2_control. gz_ros2_control is not fully working yet

File: src/ros2/moveit/moveit_resources/moveit_door_opening_mechanism_rotating_arm_config/config/rb_theron.ros2_control.xacro (robot description, xacro)
@@ -2,36 +2,4 @@
 <robot xmlns:xacro="http://www.ros.org/wiki/xacro">
   <xacro:macro name="rb_theron_ros2_control" params="name initial_positions_file ros2_control_hardware_type">
-    <xacro:property name="initial_positions" value="${load_yaml(initial_positions_file)['initial_positions']}"/>
-    <ros2_control name="${name}" type="system">
-      <hardware>
-        <xacro:if value="${ros2_control_hardware_type == 'mock_components'}">
-            <plugin>mock_components/GenericSystem</plugin>
-            <param name="calculate_dynamics">true</param>
-        </xacro:if>
-        <xacro:if value="${ros2_control_hardware_type == 'dryve_d1'}">
-          <plugin>ros2_control_plugin_door_opening_mechanism/DoorOpeningMechanismSystemHardware</plugin>
-        </xacro:if>
-      </hardware>
-      <joint name="door_opening_mechanism_joint_y_axis_slide">
-        <command_interface name="velocity"/>
-        <state_interface name="position"/>
-        <state_interface name="velocity"/>
-      </joint>
-      <joint name="door_opening_mechanism_joint_x_axis_slide">
-        <command_interface name="velocity"/>
-        <state_interface name="position"/>
-        <state_interface name="velocity"/>
-      </joint>
-      <joint name="door_opening_mechanism_joint_rotating_arm">
-        <command_interface name="velocity"/>
-        <state_interface name="position"/>
-        <state_interface name="velocity"/>
-      </joint>
-      <joint name="door_opening_mechanism_joint_freely_rotating_hook">
-        <command_interface name="velocity"/>
-        <state_interface name="position"/>
-        <state_interface name="velocity"/>
-      </joint>
-    </ros2_control>
   </xacro:macro>
 </robot>

File: src/ros2/robot_description/rb_theron_common/rb_theron_description/robots/rb_theron.urdf.xacro (robot description, xacro)
@@ -28,9 +28,20 @@
 	<xacro:arg name="prefix" default=""/>
 	<!-- <xacro:arg name="gpu" default="true"/> -->
+	<!-- ros2_control_hardware_type:
+		mock_components = ros2_control only in rviz
+		gz_ros2_control = ros2_control in gazebo
+		dryve_d1 = ros2_control only in real life
+	-->
+    <xacro:arg name="ros2_control_hardware_type" default="mock_components" />
 	<!-- *************** -->
 	<!-- Robots Elements -->
 	<!-- *************** -->
 	<!-- base with wheels -->
-	<xacro:rb_theron_base prefix="$(arg prefix)" hq="${hq}" publish_bf="${publish_bf}" />
+	<xacro:rb_theron_base
+	  prefix="$(arg prefix)"
+	  hq="${hq}"
+	  publish_bf="${publish_bf}"
+	  ros2_control_hardware_type="$(arg ros2_control_hardware_type)">
+	</xacro:rb_theron_base>
 	<!-- Gazebo ros control pluggins -->
 	<!-- <xacro:ros_control/> -->
@@ -90,22 +101,51 @@
 	<!-- ROBAST Drawer -->
 	<xacro:include filename="$(find rb_theron_description)/urdf/drawer/drawer.urdf.xacro" />
-	<xacro:drawer prefix="$(arg prefix)" suffix="5" parent="$(arg prefix)base_link" drawer_size_z="0.28">
+	<xacro:drawer
+	    prefix="$(arg prefix)"
+		suffix="5"
+		parent="$(arg prefix)base_link"
+		ros2_control_hardware_type="$(arg ros2_control_hardware_type)"
+		drawer_size_z="0.28">
 		<origin xyz="0.125 0.0 0.42" rpy="0 0 0"/>
 	</xacro:drawer>
-	<xacro:drawer prefix="$(arg prefix)" suffix="4" parent="$(arg prefix)base_link" drawer_size_z="0.18">
+	<xacro:drawer
+	    prefix="$(arg prefix)"
+		suffix="4"
+		parent="$(arg prefix)base_link"
+		ros2_control_hardware_type="$(arg ros2_control_hardware_type)"
+		drawer_size_z="0.18">
 		<origin xyz="0.125 0.0 0.67" rpy="0 0 0"/>
 	</xacro:drawer>
-	<xacro:drawer prefix="$(arg prefix)" suffix="3" parent="$(arg prefix)base_link" drawer_size_z="0.08">
+	<xacro:drawer
+	    prefix="$(arg prefix)"
+		suffix="3"
+		parent="$(arg prefix)base_link"
+		ros2_control_hardware_type="$(arg ros2_control_hardware_type)"
+		drawer_size_z="0.08">
 		<origin xyz="0.125 0.0 0.82" rpy="0 0 0"/>
 	</xacro:drawer>
-	<xacro:drawer prefix="$(arg prefix)" suffix="2" parent="$(arg prefix)base_link" drawer_size_z="0.08">
+	<xacro:drawer
+		prefix="$(arg prefix)"
+		suffix="2"
+		parent="$(arg prefix)base_link"
+		ros2_control_hardware_type="$(arg ros2_control_hardware_type)"
+		drawer_size_z="0.08">
 		<origin xyz="0.125 0.0 0.92" rpy="0 0 0"/>
 	</xacro:drawer>
-	<xacro:drawer prefix="$(arg prefix)" suffix="1" parent="$(arg prefix)base_link" drawer_size_z="0.08">
+	<xacro:drawer
+		prefix="$(arg prefix)"
+		suffix="1"
+		parent="$(arg prefix)base_link"
+		ros2_control_hardware_type="$(arg ros2_control_hardware_type)"
+		drawer_size_z="0.08">
 		<origin xyz="0.125 0.0 1.02" rpy="0 0 0"/>
 	</xacro:drawer>
 	<!-- ROBAST Door Opening Mechanism -->
 	<xacro:include filename="$(find rb_theron_description)/urdf/door_opening_mechanism/door_opening_mechanism.urdf.xacro" />
-	<xacro:door_opening_mechanism prefix="$(arg prefix)" parent="$(arg prefix)base_link" hq="${hq}">
+	<xacro:door_opening_mechanism
+	    prefix="$(arg prefix)"
+		parent="$(arg prefix)base_link"
+		ros2_control_hardware_type="$(arg ros2_control_hardware_type)"
+		hq="${hq}">
 		<origin xyz="-0.3 0 0.225" rpy="0 0 0"/>
 	</xacro:door_opening_mechanism>

File: src/ros2/robot_description/rb_theron_common/rb_theron_description/robots/rb_theron_base.urdf.xacro (robot description, xacro)
@@ -20,25 +20,49 @@
   <!-- Robots Elements -->
   <!-- *************** -->
-  <xacro:macro name="rb_theron_base" params="prefix hq publish_bf">
+  <xacro:macro name="rb_theron_base" params="prefix hq publish_bf ros2_control_hardware_type">
     <xacro:theron_base prefix="${prefix}" publish_bf="${publish_bf}" hq="${hq}" />
     <xacro:gazebo_colors prefix="${prefix}"/>
     <!-- WHEELS -->
-    <xacro:rubber_wheel prefix="${prefix}right" parent="${prefix}base_link" hq="${hq}">
+    <xacro:rubber_wheel
+      prefix="${prefix}right"
+      parent="${prefix}base_link"
+      ros2_control_hardware_type="${ros2_control_hardware_type}"
+      hq="${hq}">
       <origin xyz="${wheel_offset_x} ${-wheel_offset_y} ${wheel_offset_z}" rpy="0 0 0"/>
     </xacro:rubber_wheel>
-    <xacro:rubber_wheel prefix="${prefix}left" parent="${prefix}base_link" hq="${hq}">
+    <xacro:rubber_wheel
+      prefix="${prefix}left"
+      parent="${prefix}base_link"
+      ros2_control_hardware_type="${ros2_control_hardware_type}"
+      hq="${hq}">
       <origin xyz="${wheel_offset_x} ${wheel_offset_y} ${wheel_offset_z}" rpy="0 0 0"/>
     </xacro:rubber_wheel>
     <!-- CASTORS WHEELS -->
-    <xacro:caster prefix="${prefix}front_left" parent="${prefix}base_link" hq="${hq}">
+    <xacro:caster
+      prefix="${prefix}front_left"
+      parent="${prefix}base_link"
+      ros2_control_hardware_type="${ros2_control_hardware_type}"
+      hq="${hq}">
       <origin xyz="0.235 0.1825 0.046" rpy="0 0 0"/>
     </xacro:caster>
-    <xacro:caster prefix="${prefix}front_right" parent="${prefix}base_link" hq="${hq}">
+    <xacro:caster
+      prefix="${prefix}front_right"
+      parent="${prefix}base_link"
+      ros2_control_hardware_type="${ros2_control_hardware_type}"
+      hq="${hq}">
       <origin xyz="0.235 -0.1825 0.046" rpy="0 0 0"/>
     </xacro:caster>
-    <xacro:caster prefix="${prefix}rear_left" parent="${prefix}base_link" hq="${hq}">
+    <xacro:caster
+      prefix="${prefix}rear_left"
+      parent="${prefix}base_link"
+      ros2_control_hardware_type="${ros2_control_hardware_type}"
+      hq="${hq}">
       <origin xyz="-0.235 0.1825 0.046" rpy="0 0 0"/>
     </xacro:caster>
-    <xacro:caster prefix="${prefix}rear_right" parent="${prefix}base_link" hq="${hq}">
+    <xacro:caster
+      prefix="${prefix}rear_right"
+      parent="${prefix}base_link"
+      ros2_control_hardware_type="${ros2_control_hardware_type}"
+      hq="${hq}">
       <origin xyz="-0.235 -0.1825 0.046" rpy="0 0 0"/>
     </xacro:caster>

File: src/ros2/robot_description/rb_theron_common/rb_theron_description/urdf/common.gazebo.xacro (robot description, xacro)
@@ -4,43 +4,6 @@
     <xacro:macro name="ros_control" params="prefix publish_bf">
         <gazebo>
-            <!-- <plugin filename="libgazebo_ros2_control.so" name="gazebo_ros2_control">
-				<parameters>$(find rb_theron_description)/config/rb_theron_controller.yaml</parameters>
-			</plugin> -->
-            <plugin filename="libgz-sim-joint-state-publisher-system" name="gz::sim::systems::JointStatePublisher">
-                <joint_name>rightjoint_rsupport</joint_name>
-                <joint_name>leftjoint_rsupport</joint_name>
-                <joint_name>right_wheel_joint</joint_name>
-                <joint_name>left_wheel_joint</joint_name>
-                <joint_name>rightcastorjoint_support</joint_name>
-                <joint_name>leftcastorjoint_support</joint_name>
-                <joint_name>rightjoint_wheel</joint_name>
-                <joint_name>leftjoint_wheel</joint_name>
-                <joint_name>rightcastorjoint_wheel</joint_name>
-                <joint_name>leftcastorjoint_wheel</joint_name>
-                <joint_name>rightjoint_support</joint_name>
-                <joint_name>leftjoint_support</joint_name>
-                <joint_name>drawer_1_joint</joint_name>
-                <joint_name>drawer_2_joint</joint_name>
-                <joint_name>drawer_3_joint</joint_name>
-                <joint_name>drawer_4_joint</joint_name>
-                <joint_name>drawer_5_joint</joint_name>
-            </plugin>
-            <plugin filename="libgz-sim-diff-drive-system.so" name="gz::sim::systems::DiffDrive">
-                <left_joint>$(arg prefix)left_wheel_joint</left_joint>
-                <right_joint>$(arg prefix)right_wheel_joint</right_joint>
-                <wheel_separation>0.5032</wheel_separation>
-                <wheel_radius>0.0762</wheel_radius>
-                <odom_publish_frequency>30</odom_publish_frequency>
-                <topic>cmd_vel</topic>
-                <frame_id>$(arg prefix)odom</frame_id>
-                <!-- There is no possiblity (as far as I know) to disable tf publishing of odom->base, so if you
-				don't want the tf to be published, you can just dump it into a different topic -->
-                <tf_topic>tf_dump</tf_topic>
-                <xacro:if value="${publish_bf}">
-                    <child_frame_id>$(arg prefix)base_footprint</child_frame_id>
-                </xacro:if>
-                <xacro:unless value="${publish_bf}">
-                    <child_frame_id>$(arg prefix)base_link</child_frame_id>
-                </xacro:unless>
+            <plugin name="gz_ros2_control::GazeboSimROS2ControlPlugin" filename="gz_ros2_control-system">
+                <parameters>$(find rb_theron_description)/config/rb_theron_gz_ros2_controller.yaml</parameters>
             </plugin>
         </gazebo>

File: src/ros2/robot_description/rb_theron_common/rb_theron_description/urdf/door_opening_mechanism/arm_variations/rotating_arm.urdf.xacro (robot description, xacro)
@@ -6,5 +6,5 @@
                 izz="${m*(x*x+z*z)/12}" />
     </xacro:macro>
-    <xacro:macro name="rotating_arm" params="prefix parent *origin arm_length">
+    <xacro:macro name="rotating_arm" params="prefix parent ros2_control_hardware_type *origin arm_length">
         <xacro:basic_joint
             parent="${prefix}${parent}"
@@ -18,7 +18,5 @@
             damping="0.1"
             friction="0.3"
-            p_gain="500"
-            i_gain="1000"
-            d_gain="10"
+            ros2_control_hardware_type="${ros2_control_hardware_type}"
             link_name="${prefix}door_opening_mechanism_link_rotating_arm"
             link_origin_x="0.0"
@@ -52,5 +50,8 @@
         <!-- Gripper -->
         <xacro:include filename="$(find rb_theron_description)/urdf/door_opening_mechanism/components/freely_rotating_hook.urdf.xacro" />
-        <xacro:freely_rotating_hook prefix="${prefix}" parent="${prefix}door_opening_mechanism_link_gripper_adapter">
+        <xacro:freely_rotating_hook
+            prefix="${prefix}"
+            parent="${prefix}door_opening_mechanism_link_gripper_adapter"
+            ros2_control_hardware_type="${ros2_control_hardware_type}">
             <origin xyz="0.020 0.0 0.0" rpy="0 0 0"/>
         </xacro:freely_rotating_hook>

File: src/ros2/robot_description/rb_theron_common/rb_theron_description/urdf/door_opening_mechanism/arm_variations/tilting_arm.urdf.xacro (robot description, xacro)
@@ -6,5 +6,5 @@
                 izz="${m*(x*x+z*z)/12}" />
     </xacro:macro>
-    <xacro:macro name="tilting_arm" params="prefix parent *origin">
+    <xacro:macro name="tilting_arm" params="prefix parent ros2_control_hardware_type *origin">
         <xacro:basic_joint
             parent="${prefix}${parent}"
@@ -18,7 +18,5 @@
             damping="0.1"
             friction="0.3"
-            p_gain="500"
-            i_gain="1000"
-            d_gain="10"
+            ros2_control_hardware_type="${ros2_control_hardware_type}"
             link_name="${prefix}door_opening_mechanism_link_tilting_hook"
             link_origin_x="0.0"

File: src/ros2/robot_description/rb_theron_common/rb_theron_description/urdf/door_opening_mechanism/basic_elements/basic_joint.urdf.xacro (robot description, xacro)
@@ -6,5 +6,5 @@
                 izz="${m*(x*x+z*z)/12}" />
     </xacro:macro>
-    <xacro:macro name="basic_joint" params="parent joint_name joint_type axis_x axis_y axis_z lower_limit upper_limit damping friction p_gain i_gain d_gain link_name link_origin_x link_origin_y link_origin_z m x y z r g b *origin">
+    <xacro:macro name="basic_joint" params="parent joint_name joint_type axis_x axis_y axis_z lower_limit upper_limit damping friction ros2_control_hardware_type link_name link_origin_x link_origin_y link_origin_z m x y z r g b *origin">
     <joint name="${joint_name}" type="${joint_type}" >
         <axis xyz="${axis_x} ${axis_y} ${axis_z}" />
@@ -15,16 +15,26 @@
         <xacro:insert_block name="origin" />
     </joint>
-    <gazebo>
-        <plugin filename="libgz-sim-joint-position-controller-system.so" name="gz::sim::systems::JointPositionController">
-            <joint_name>${joint_name}</joint_name>
-            <p_gain>${p_gain}</p_gain>
-            <i_gain>${i_gain}</i_gain>
-            <d_gain>${d_gain}</d_gain>
-            <i_max>200</i_max>
-            <i_min>-200</i_min>
-            <cmd_max>1000</cmd_max>
-            <cmd_min>-1000</cmd_min>
-        </plugin>
-    </gazebo>
+    <ros2_control name="${joint_name}_ros2_control" type="system">
+        <hardware>
+            <xacro:if value="${ros2_control_hardware_type == 'mock_components'}">
+                <plugin>mock_components/GenericSystem</plugin>
+                <param name="calculate_dynamics">true</param>
+            </xacro:if>
+            <xacro:if value="${ros2_control_hardware_type == 'gz_ros2_control'}">
+                <plugin>gz_ros2_control/GazeboSimSystem</plugin>
+            </xacro:if>
+            <xacro:if value="${ros2_control_hardware_type == 'dryve_d1'}">
+                <plugin>ros2_control_plugin_door_opening_mechanism/DoorOpeningMechanismSystemHardware</plugin>
+            </xacro:if>
+        </hardware>
+        <joint name="${joint_name}">
+            <command_interface name="velocity">
+                <param name="min">-10</param>
+                <param name="max">10</param>
+            </command_interface>
+            <state_interface name="position"/>
+            <state_interface name="velocity"/>
+        </joint>
+    </ros2_control>
     <link name="${link_name}">
         <inertial>

File: src/ros2/robot_description/rb_theron_common/rb_theron_description/urdf/door_opening_mechanism/components/freely_rotating_hook.urdf.xacro (robot description, xacro)
@@ -1,5 +1,5 @@
 <?xml version="1.0"?>
 <robot name="freely_rotating_hook" xmlns:xacro="http://www.ros.org/wiki/xacro">
-    <xacro:macro name="freely_rotating_hook" params="prefix parent *origin">
+    <xacro:macro name="freely_rotating_hook" params="prefix parent ros2_control_hardware_type *origin">
         <!-- Please mind: This joint is actually passive, but in order to help moveit plan the trajectory we make it active -->
         <xacro:basic_joint
@@ -14,7 +14,5 @@
             damping="0.05"
             friction="0.1"
-            p_gain="500"
-            i_gain="1000"
-            d_gain="10"
+            ros2_control_hardware_type="${ros2_control_hardware_type}"
             link_name="${prefix}door_opening_mechanism_link_freely_rotating_hook"
             link_origin_x="0.0"

File: src/ros2/robot_description/rb_theron_common/rb_theron_description/urdf/door_opening_mechanism/door_opening_mechanism.urdf.xacro (robot description, xacro)
@@ -6,5 +6,5 @@
                 izz="${m*(x*x+z*z)/12}" />
     </xacro:macro>
-    <xacro:macro name="door_opening_mechanism" params="prefix parent *origin hq">
+    <xacro:macro name="door_opening_mechanism" params="prefix parent ros2_control_hardware_type *origin hq">
         <!-- Element imports -->
         <xacro:include filename="$(find rb_theron_description)/urdf/door_opening_mechanism/components/alu_profile.urdf.xacro" />
@@ -68,7 +68,5 @@
             damping="0.1"
             friction="0.3"
-            p_gain="50000"
-            i_gain="1000"
-            d_gain="5000"
+            ros2_control_hardware_type="${ros2_control_hardware_type}"
             link_name="${prefix}door_opening_mechanism_link_y_axis_slide"
             link_origin_x="0.0"
@@ -95,7 +93,5 @@
             damping="0.1"
             friction="0.3"
-            p_gain="50000"
-            i_gain="100"
-            d_gain="5000"
+            ros2_control_hardware_type="${ros2_control_hardware_type}"
             link_name="${prefix}door_opening_mechanism_link_x_axis_slide"
             link_origin_x="0.0"
@@ -131,5 +127,9 @@
         <!-- Rotating arm -->
         <xacro:include filename="$(find rb_theron_description)/urdf/door_opening_mechanism/arm_variations/rotating_arm.urdf.xacro" />
-        <xacro:rotating_arm prefix="${prefix}" parent="${prefix}door_opening_mechanism_link_x_slide_screwing" arm_length="0.3" >
+        <xacro:rotating_arm
+            prefix="${prefix}"
+            parent="${prefix}door_opening_mechanism_link_x_slide_screwing"
+            ros2_control_hardware_type="${ros2_control_hardware_type}"
+            arm_length="0.3" >
             <origin xyz="0.05 -0.025 0" rpy="0 0 1.57079632679"/>
         </xacro:rotating_arm>

File: src/ros2/robot_description/rb_theron_common/rb_theron_description/urdf/drawer/drawer.urdf.xacro (robot description, xacro)
@@ -15,5 +15,5 @@
     <xacro:property name="drawer_offset_y" value="0.0" />
     <xacro:property name="drawer_offset_z" value="0.0" />
-    <xacro:macro name="drawer" params="prefix suffix parent *origin drawer_size_z">
+    <xacro:macro name="drawer" params="prefix suffix parent *origin ros2_control_hardware_type drawer_size_z">
         <link name="${prefix}drawer_${suffix}">
             <inertial>
@@ -48,14 +48,27 @@
             <limit lower="0.0" upper="${0.95*drawer_size_y}" effort="100" velocity="100" />
         </joint>
-        <gazebo>
-            <plugin filename="libgz-sim-joint-position-controller-system.so" name="gz::sim::systems::JointPositionController">
-                <joint_name>${prefix}drawer_${suffix}_joint</joint_name>
-                <p_gain>50000.0</p_gain>
-                <i_gain>100</i_gain>
-                <d_gain>1000</d_gain>
-                <i_max>200</i_max>
-                <i_min>-200</i_min>
-            </plugin>
-        </gazebo>
+        <ros2_control name="${prefix}drawer_${suffix}_ros2_control" type="system">
+            <hardware>
+                <xacro:if value="${ros2_control_hardware_type == 'mock_components'}">
+                    <plugin>mock_components/GenericSystem</plugin>
+                    <param name="calculate_dynamics">true</param>
+                </xacro:if>
+                <xacro:if value="${ros2_control_hardware_type == 'gz_ros2_control'}">
+                    <plugin>gz_ros2_control/GazeboSimSystem</plugin>
+                </xacro:if>
+                <xacro:if value="${ros2_control_hardware_type == 'dryve_d1'}">
+                    <plugin>mock_components/GenericSystem</plugin>
+                    <param name="calculate_dynamics">true</param>
+                </xacro:if>
+            </hardware>
+            <joint name="${prefix}drawer_${suffix}_joint">
+                <command_interface name="velocity">
+                    <param name="min">-10</param>
+                    <param name="max">10</param>
+                </command_interface>
+                <state_interface name="position"/>
+                <state_interface name="velocity"/>
+            </joint>
+        </ros2_control>
     </xacro:macro>
 </robot>
