Commit message: feat: joints are now controlled only by ros2_control. gz_ros2_control is not fully working yet

File: src/ros2/robot_description/rb_theron_common/rb_theron_description/urdf/wheels/castor.urdf.xacro (robot description, xacro)
@@ -18,7 +18,7 @@
               izz="${m*r*r/2}" />
   </xacro:macro>
-  <xacro:macro name="caster" params="prefix parent *origin hq">
-  <!--CASTER SUPPORT -->
-  <joint name="${prefix}joint_support" type="continuous">
+  <xacro:macro name="caster" params="prefix parent ros2_control_hardware_type *origin hq">
+    <!--CASTER SUPPORT -->
+    <joint name="${prefix}joint_support" type="continuous">
       <parent link="${parent}"/>
       <child link="${prefix}support"/>
@@ -29,4 +29,23 @@
       <dynamics damping="0" friction="0.01"/>
     </joint>
+    <ros2_control name="${prefix}joint_support_ros2_control" type="system">
+      <hardware>
+        <xacro:if value="${ros2_control_hardware_type == 'mock_components'}">
+          <plugin>mock_components/GenericSystem</plugin>
+         <param name="calculate_dynamics">true</param>
+        </xacro:if>
+        <xacro:if value="${ros2_control_hardware_type == 'gz_ros2_control'}">
+          <plugin>gz_ros2_control/GazeboSimSystem</plugin>
+        </xacro:if>
+        <xacro:if value="${ros2_control_hardware_type == 'dryve_d1'}">
+          <plugin>mock_components/GenericSystem</plugin>
+          <param name="calculate_dynamics">true</param>
+        </xacro:if>
+      </hardware>
+      <joint name="${prefix}joint_support">
+        <state_interface name="position"/>
+        <state_interface name="velocity"/>
+      </joint>
+    </ros2_control>
     <link name="${prefix}support">
       <visual>
@@ -54,19 +73,42 @@
       </inertial>
     </link>
-  <!--CASTER WHEEL -->
-  <!-- xacro:caster_wheel prefix="${prefix}" parent="${prefix}support" hq="${hq}" -->
-  <xacro:caster_wheel prefix="${prefix}" parent="${prefix}support" hq="${hq}">
-    <origin xyz="${caster_wheel_offset_x} ${caster_wheel_offset_y} ${caster_wheel_offset_z}" rpy="0 0 0"/>
-   </xacro:caster_wheel>
- </xacro:macro>
- <xacro:macro name="caster_wheel" params="prefix parent *origin hq">
-     <joint name="${prefix}joint_wheel" type="continuous">
-       <parent link="${parent}"/>
-       <child link="${prefix}wheel"/>
-       <xacro:insert_block name="origin" />
-       <axis xyz="0 1 0" rpy="0 0 0" />
-       <limit effort="100" velocity="100"/>
-       <joint_properties damping="0.1" friction="0.1"/>
+    <!--CASTER WHEEL -->
+    <!-- xacro:caster_wheel prefix="${prefix}" parent="${prefix}support" hq="${hq}" -->
+    <xacro:caster_wheel
+      prefix="${prefix}"
+      parent="${prefix}support"
+      ros2_control_hardware_type="${ros2_control_hardware_type}"
+      hq="${hq}">
+      <origin xyz="${caster_wheel_offset_x} ${caster_wheel_offset_y} ${caster_wheel_offset_z}" rpy="0 0 0"/>
+    </xacro:caster_wheel>
+  </xacro:macro>
+  <xacro:macro name="caster_wheel" params="prefix parent *origin ros2_control_hardware_type hq">
+    <joint name="${prefix}joint_wheel" type="continuous">
+      <parent link="${parent}"/>
+      <child link="${prefix}wheel"/>
+      <xacro:insert_block name="origin" />
+      <axis xyz="0 1 0" rpy="0 0 0" />
+      <limit effort="100" velocity="100"/>
+      <joint_properties damping="0.1" friction="0.1"/>
     </joint>
+    <ros2_control name="${prefix}joint_wheel_ros2_control" type="system">
+      <hardware>
+				<xacro:if value="${ros2_control_hardware_type == 'mock_components'}">
+					<plugin>mock_components/GenericSystem</plugin>
+					<param name="calculate_dynamics">true</param>
+				</xacro:if>
+				<xacro:if value="${ros2_control_hardware_type == 'gz_ros2_control'}">
+					<plugin>gz_ros2_control/GazeboSimSystem</plugin>
+				</xacro:if>
+				<xacro:if value="${ros2_control_hardware_type == 'dryve_d1'}">
+					<plugin>mock_components/GenericSystem</plugin>
+					<param name="calculate_dynamics">true</param>
+				</xacro:if>
+			</hardware>
+      <joint name="${prefix}joint_wheel">
+        <state_interface name="position"/>
+        <state_interface name="velocity"/>
+      </joint>
+    </ros2_control>
     <link name="${prefix}wheel">
       <visual>

File: src/ros2/robot_description/rb_theron_common/rb_theron_description/urdf/wheels/rubber_wheel.transmission.xacro (robot description, xacro)
@@ -2,5 +2,5 @@
 <robot xmlns:xacro="http://www.ros.org/wiki/xacro">
     <!-- Rubber wheel transmission -->
-    <xacro:macro name="rubber_wheel_transmission" params="prefix">
+    <xacro:macro name="rubber_wheel_transmission" params="prefix ros2_control_hardware_type">
     <!-- Transmission is important to link the joints and the controller (see rb_theron_control/config/rb_theron_control.yaml)-->
         <transmission name="${prefix}_wheel_joint_trans">
@@ -31,5 +31,15 @@
 			</hardware> -->
 			<hardware>
-				<plugin>fake_components/GenericSystem</plugin>
+				<xacro:if value="${ros2_control_hardware_type == 'mock_components'}">
+					<plugin>mock_components/GenericSystem</plugin>
+					<param name="calculate_dynamics">true</param>
+				</xacro:if>
+				<xacro:if value="${ros2_control_hardware_type == 'gz_ros2_control'}">
+					<plugin>gz_ros2_control/GazeboSimSystem</plugin>
+				</xacro:if>
+				<xacro:if value="${ros2_control_hardware_type == 'dryve_d1'}">
+					<plugin>mock_components/GenericSystem</plugin>
+					<param name="calculate_dynamics">true</param>
+				</xacro:if>
 			</hardware>
 			<joint name="${prefix}_wheel_joint">

File: src/ros2/robot_description/rb_theron_common/rb_theron_description/urdf/wheels/rubber_wheel.urdf.xacro (robot description, xacro)
@@ -13,5 +13,5 @@
         <inertia ixx="${m*(3*r*r+h*h)/12}" ixy = "0" ixz = "0" iyy="${m*(3*r*r+h*h)/12}" iyz = "0" izz="${m*r*r/2}" />
     </xacro:macro>
-    <xacro:macro name="rubber_wheel" params="prefix parent *origin reflect hq">
+    <xacro:macro name="rubber_wheel" params="prefix parent *origin reflect ros2_control_hardware_type hq">
         <!--WHEEL TIRE -->
         <joint name="${prefix}_wheel_joint" type="continuous">
@@ -44,5 +44,5 @@
             </inertial>
         </link>
-        <xacro:rubber_wheel_transmission prefix="${prefix}" />
+        <xacro:rubber_wheel_transmission prefix="${prefix}" ros2_control_hardware_type="${ros2_control_hardware_type}" />
         <xacro:rubber_wheel_gazebo prefix="${prefix}" />
     </xacro:macro>

File: src/ros2/robot_description/rb_theron_common/rb_theron_description/urdf/wheels/rubber_wheel_125.urdf.xacro (robot description, xacro)
@@ -12,5 +12,5 @@
         <inertia ixx="${m*(3*r*r+h*h)/12}" ixy = "0" ixz = "0" iyy="${m*(3*r*r+h*h)/12}" iyz = "0" izz="${m*r*r/2}" />
     </xacro:macro>
-    <xacro:macro name="rubber_wheel" params="prefix parent *origin reflect hq">
+    <xacro:macro name="rubber_wheel" params="prefix parent *origin reflect ros2_control_hardware_type hq">
         <!--WHEEL TIRE -->
         <joint name="${prefix}_wheel_joint" type="continuous">
@@ -43,5 +43,5 @@
             </inertial>
         </link>
-        <xacro:rubber_wheel_transmission prefix="${prefix}" />
+        <xacro:rubber_wheel_transmission prefix="${prefix}" ros2_control_hardware_type="${ros2_control_hardware_type}" />
         <xacro:rubber_wheel_gazebo prefix="${prefix}" />
     </xacro:macro>

File: src/ros2/robot_description/rb_theron_common/rb_theron_description/urdf/wheels/rubber_wheel_150.urdf.xacro (robot description, xacro)
@@ -13,5 +13,5 @@
         <inertia ixx="${m*(3*r*r+h*h)/12}" ixy = "0" ixz = "0" iyy="${m*(3*r*r+h*h)/12}" iyz = "0" izz="${m*r*r/2}" />
     </xacro:macro>
-    <xacro:macro name="rubber_wheel" params="prefix parent *origin hq">
+    <xacro:macro name="rubber_wheel" params="prefix parent *origin ros2_control_hardware_type hq">
         <!--WHEEL TIRE -->
         <joint name="${prefix}_wheel_joint" type="continuous">
@@ -57,5 +57,5 @@
             </visual>
         </link>
-        <xacro:rubber_wheel_transmission prefix="${prefix}" />
+        <xacro:rubber_wheel_transmission prefix="${prefix}" ros2_control_hardware_type="${ros2_control_hardware_type}" />
         <xacro:rubber_wheel_gazebo prefix="${prefix}" />
     </xacro:macro>
