Commit message: Adding JointPositionController plugin - but drawer joint still cant be controlled via set_joint_state topic

File: src/ros2/robot_description/rb_theron_common/rb_theron_description/urdf/drawer/drawer.urdf.xacro (robot description, xacro)
@@ -46,14 +46,12 @@
                 <limit lower="0.0" upper="${0.95*drawer_size_y}" effort="100" velocity="100" />
         </joint>
-        <transmission name="${prefix}_drawer_joint">
-                <type>transmission_interface/SimpleTransmission</type>
-                <joint name="top_drawer_joint">
-                        <hardwareInterface>hardware_interface/EffortJointInterface</hardwareInterface>
-                </joint>
-                <actuator name="${prefix}_drawer_joint_motor">
-                        <mechanicalReduction>1</mechanicalReduction>
-                        <motorTorqueConstant>1</motorTorqueConstant>
-                </actuator>
-        </transmission>
+        <plugin filename="ignition-gazebo-joint-position-controller-system" name="ignition::gazebo::systems::JointPositionController">
+                <joint_name>top_drawer_joint</joint_name>
+                <p_gain>50000.0</p_gain>
+                <i_gain>100</i_gain>
+                <d_gain>1000</d_gain>
+                <i_max>200</i_max>
+                <i_min>-200</i_min>
+        </plugin>
 </xacro:macro>
 </robot>

Commit message: Fixing the problem that the driving wheels sometimes lose contact to the ground - not a perfect solution, but works for now

File: src/ros2/robot_description/rb_theron_common/rb_theron_description/urdf/drawer/drawer.urdf.xacro (robot description, xacro)
@@ -11,5 +11,5 @@
       it would be able to drive properly, because this makes some of the wheels lose contact to the ground and
       therefore steering of the rb_theron becomes impossible -->
-    <xacro:property name="drawer_mass" value="0.1" />
+    <xacro:property name="drawer_mass" value="1.0" />
     <xacro:property name="drawer_offset_x" value="0.0" />
     <xacro:property name="drawer_offset_y" value="0.0" />

File: src/ros2/robot_description/rb_theron_common/rb_theron_description/urdf/rocker/mcq_prototype_rocker.urdf.xacro (robot description, xacro)
@@ -28,6 +28,12 @@
       <xacro:insert_block name="origin" />
       <axis xyz="0 1 0" rpy="0 0 ${M_PI}" />
-      <limit lower="-0.5" upper="0.5" effort="100" velocity="100"/>
-      <joint_properties damping="0.1" friction="0.1"/>
+      <!-- The upper limit should actually be something around 0.5.
+      Setting the upper limit to -0.01 makes the robot rocker wheels lose contact on one side,
+      so that only 4 robot wheels have contact to ground.
+      Otherwise the robot would not be able to drive properly, because the rocker wheels some times
+      make the driving wheels lose contact to the ground and therefore steering of the rb_theron
+      becomes impossible -->
+      <limit lower="-0.5" upper="-0.01" effort="100" velocity="100"/>
+      <dynamics damping="0.1" friction="0.1"/>
 	</joint>
 	<link name="${prefix}rsupport">
@@ -112,5 +118,5 @@
 			</joint>
 		</ros2_control>
-    <xacro:property name="wheel_offset_x" value="-0.1175" />
+    <xacro:property name="wheel_offset_x" value="-0.175" />
     <xacro:if value="${reflect}">
          <xacro:property name="wheel_offset_y" value="-0.079" />

Commit message: feat: first draft to add drawer_bridge_simulation back together with ros2_control

File: src/ros2/robot_description/rb_theron_common/rb_theron_description/urdf/drawer/drawer.urdf.xacro (robot description, xacro)
@@ -46,5 +46,5 @@
             <child link="${prefix}drawer_${suffix}" />
             <xacro:insert_block name="origin" />
-            <limit lower="0.0" upper="${0.95*drawer_size_y}" effort="100" velocity="100" />
+            <limit lower="0.0" upper="${0.95*drawer_size_y}" effort="1000" velocity="100" />
         </joint>
         <ros2_control name="${prefix}drawer_${suffix}_ros2_control" type="system">
@@ -63,5 +63,5 @@
             </hardware>
             <joint name="${prefix}drawer_${suffix}_joint">
-                <command_interface name="velocity">
+                <command_interface name="position">
                     <param name="min">-10</param>
                     <param name="max">10</param>

Commit message: fix: drawers can now be moved in gazebo with the drawer_bridge_simulation node

File: src/ros2/robot_description/rb_theron_common/rb_theron_description/urdf/drawer/drawer.urdf.xacro (robot description, xacro)
@@ -46,5 +46,5 @@
             <child link="${prefix}drawer_${suffix}" />
             <xacro:insert_block name="origin" />
-            <limit lower="0.0" upper="${0.95*drawer_size_y}" effort="1000" velocity="100" />
+            <limit lower="-0.01" upper="${0.95*drawer_size_y}" effort="1000" velocity="100" />
         </joint>
         <ros2_control name="${prefix}drawer_${suffix}_ros2_control" type="system">
@@ -64,6 +64,6 @@
             <joint name="${prefix}drawer_${suffix}_joint">
                 <command_interface name="position">
-                    <param name="min">-10</param>
-                    <param name="max">10</param>
+                    <param name="min">-0.01</param>
+                    <param name="max">${0.95*drawer_size_y}</param>
                 </command_interface>
                 <state_interface name="position"/>
