Commit message: fix: increases effort for basic joint

File: src/ros2/robot_description/rb_theron_common/rb_theron_description/urdf/door_opening_mechanism/basic_elements/basic_joint.urdf.xacro (robot description, xacro)
@@ -11,5 +11,5 @@
         <parent link="${parent}" />
         <child link="${link_name}" />
-        <limit lower="${lower_limit}" upper="${upper_limit}" effort="100" velocity="100" />
+        <limit lower="${lower_limit}" upper="${upper_limit}" effort="1000" velocity="100" />
         <dynamics damping="${damping}" friction="${friction}"/>
         <xacro:insert_block name="origin" />

Commit message: fix: removes doubled tag </xacro:macro>

File: src/ros2/robot_description/rb_theron_common/rb_theron_description/urdf/door_opening_mechanism/basic_elements/basic_joint.urdf.xacro (robot description, xacro)
@@ -35,5 +35,4 @@
             b
             *origin">
-    </xacro:macro>
     <joint name="${joint_name}" type="${joint_type}">
         <axis xyz="${axis_x} ${axis_y} ${axis_z}" />
