Commit message: feat: adds gripper adapter to rotating arm in order to exclude the freely rotating hook from moveit chain

File: src/ros2/robot_description/rb_theron_common/rb_theron_description/urdf/door_opening_mechanism/arm_variations/rotating_arm.urdf.xacro (robot description, xacro)
@@ -34,8 +34,24 @@
             <xacro:insert_block name="origin" />
         </xacro:basic_joint>
+        <!-- Adapter for Gripper -->
+        <!-- Please mind: We need this link as end effector for moveit in order to not include the freely rotating hook into
+        path planning -->
+        <xacro:basic_box
+            parent="${prefix}door_opening_mechanism_link_rotating_arm"
+            joint_name="${prefix}door_opening_mechanism_joint_gripper_adapter"
+            link_name="${prefix}door_opening_mechanism_link_gripper_adapter"
+            m="0.1"
+            x="0.01"
+            y="0.03"
+            z="0.03"
+            r="0"
+            g="1"
+            b="0">
+            <origin xyz="0.020 0.0 ${arm_length-0.015}" rpy="0 0 0"/>
+        </xacro:basic_box>
         <!-- Gripper -->
         <xacro:include filename="$(find rb_theron_description)/urdf/door_opening_mechanism/components/freely_rotating_hook.urdf.xacro" />
-        <xacro:freely_rotating_hook prefix="${prefix}" parent="${prefix}door_opening_mechanism_link_rotating_arm">
-            <origin xyz="0.030 0.0 ${arm_length-0.015}" rpy="0 0 0"/>
+        <xacro:freely_rotating_hook prefix="${prefix}" parent="${prefix}door_opening_mechanism_link_gripper_adapter">
+            <origin xyz="0.020 0.0 0.0" rpy="0 0 0"/>
         </xacro:freely_rotating_hook>
     </xacro:macro>

File: src/ros2/robot_description/rb_theron_common/rb_theron_description/urdf/door_opening_mechanism/components/freely_rotating_hook.urdf.xacro (robot description, xacro)
@@ -28,4 +28,5 @@
             b="1">
             <xacro:insert_block name="origin" />
+            <!-- <origin xyz="-0.026 0.02 0" rpy="0 0 0"/> -->
         </xacro:basic_joint>
         <xacro:include filename="$(find rb_theron_description)/urdf/door_opening_mechanism/components/hook.urdf.xacro" />

Commit message: feat: ros2_control plugin for door_opening_mechanism is now a bit more general and takes params for a port and direction

File: src/ros2/robot_description/rb_theron_common/rb_theron_description/urdf/door_opening_mechanism/arm_variations/rotating_arm.urdf.xacro (robot description, xacro)
@@ -19,4 +19,6 @@
             friction="0.3"
             ros2_control_hardware_type="${ros2_control_hardware_type}"
+            port="0"
+            direction="0"
             link_name="${prefix}door_opening_mechanism_link_rotating_arm"
             link_origin_x="0.0"

File: src/ros2/robot_description/rb_theron_common/rb_theron_description/urdf/door_opening_mechanism/basic_elements/basic_joint.urdf.xacro (robot description, xacro)
@@ -1,69 +1,77 @@
 <?xml version="1.0"?>
-<robot name="basic_joint" xmlns:xacro="http://www.ros.org/wiki/xacro">
+<robot name="basic_joint"
+    xmlns:xacro="http://www.ros.org/wiki/xacro">
     <xacro:macro name="box_inertia_robot" params="m x y z">
-        <inertia  ixx="${m*(y*y+z*z)/12}" ixy = "0" ixz = "0"
-                iyy="${m*(x*x+z*z)/12}" iyz = "0"
-                izz="${m*(x*x+y*y)/12}" />
+        <inertia ixx="${m*(y*y+z*z)/12}" ixy = "0" ixz = "0" iyy="${m*(x*x+z*z)/12}" iyz = "0" izz="${m*(x*x+y*y)/12}" />
     </xacro:macro>
-    <xacro:macro name="basic_joint" params="parent joint_name joint_type axis_x axis_y axis_z lower_limit upper_limit damping friction ros2_control_hardware_type link_name link_origin_x link_origin_y link_origin_z m x y z r g b *origin">
-    <joint name="${joint_name}" type="${joint_type}" >
-        <axis xyz="${axis_x} ${axis_y} ${axis_z}" />
-        <parent link="${parent}" />
-        <child link="${link_name}" />
-        <limit lower="${lower_limit}" upper="${upper_limit}" effort="1000" velocity="100" />
-        <dynamics damping="${damping}" friction="${friction}"/>
-        <xacro:insert_block name="origin" />
-    </joint>
-    <ros2_control name="${joint_name}_ros2_control" type="system">
-        <hardware>
-            <xacro:if value="${ros2_control_hardware_type == 'mock_components'}">
-                <plugin>mock_components/GenericSystem</plugin>
-                <param name="calculate_dynamics">true</param>
-            </xacro:if>
-            <xacro:if value="${ros2_control_hardware_type == 'gz_ros2_control'}">
-                <plugin>gz_ros2_control/GazeboSimSystem</plugin>
-            </xacro:if>
-            <xacro:if value="${ros2_control_hardware_type == 'dryve_d1'}">
-                <plugin>ros2_control_plugin_door_opening_mechanism/DoorOpeningMechanismSystemHardware</plugin>
-            </xacro:if>
-        </hardware>
-        <joint name="${joint_name}">
-            <command_interface name="velocity">
-                <param name="min">-10</param>
-                <param name="max">10</param>
-            </command_interface>
-            <state_interface name="position"/>
-            <state_interface name="velocity"/>
+    <xacro:macro name="basic_joint" params="parent joint_name joint_type axis_x axis_y axis_z lower_limit upper_limit damping friction ros2_control_hardware_type port direction link_name link_origin_x link_origin_y link_origin_z m x y z r g b *origin">
+        <joint name="${joint_name}" type="${joint_type}">
+            <axis xyz="${axis_x} ${axis_y} ${axis_z}" />
+            <parent link="${parent}" />
+            <child link="${link_name}" />
+            <limit lower="${lower_limit}" upper="${upper_limit}" effort="1000" velocity="100" />
+            <dynamics damping="${damping}" friction="${friction}"/>
+            <xacro:insert_block name="origin" />
         </joint>
-    </ros2_control>
-    <link name="${link_name}">
-        <inertial>
-            <origin xyz="${link_origin_x} ${link_origin_y} ${link_origin_z}" />
-            <mass value="${m}" />
-            <xacro:box_inertia_robot m="${m}" x="${x}" y="${y}" z="${z}"/>
-        </inertial>
-        <visual>
-            <origin xyz="${link_origin_x} ${link_origin_y} ${link_origin_z}" />
-            <geometry>
-                <box size="${x} ${y} ${z}"/>
-            </geometry>
-        </visual>
-        <collision>
-            <origin xyz="${link_origin_x} ${link_origin_y} ${link_origin_z}" />
-            <geometry>
-                <box size="${x} ${y} ${z}"/>
-            </geometry>
-        </collision>
-    </link>
-    <gazebo reference="${link_name}">
-        <visual>
-            <material>
-                <!-- RGBA -->
-                <ambient>${r} ${g} ${b} 1</ambient>
-                <diffuse>${r} ${g} ${b} 1</diffuse>
-                <specular>${r} ${g} ${b} 1</specular>
-            </material>
-        </visual>
-    </gazebo>
+        <ros2_control name="${joint_name}_ros2_control" type="system">
+            <hardware>
+                <xacro:if value="${ros2_control_hardware_type == 'mock_components'}">
+                    <plugin>mock_components/GenericSystem</plugin>
+                    <param name="calculate_dynamics">true</param>
+                </xacro:if>
+                <xacro:if value="${ros2_control_hardware_type == 'gz_ros2_control'}">
+                    <plugin>gz_ros2_control/GazeboSimSystem</plugin>
+                </xacro:if>
+                <xacro:if value="${ros2_control_hardware_type == 'dryve_d1'}">
+                    <!-- if the value for the port is zero, there is no dryve_d1 for this joint yet so we mock it -->
+                    <xacro:if value="${port == 0}">
+                        <plugin>mock_components/GenericSystem</plugin>
+                        <param name="calculate_dynamics">true</param>
+                    </xacro:if>
+                    <xacro:unless value="${port == 0}">
+                        <plugin>ros2_control_plugin_door_opening_mechanism/DoorOpeningMechanismSystemHardware</plugin>
+                        <param name="port">${port}</param>
+                        <param name="direction">${direction}</param>
+                    </xacro:unless>
+                </xacro:if>
+            </hardware>
+            <joint name="${joint_name}">
+                <command_interface name="velocity">
+                    <param name="min">-10</param>
+                    <param name="max">10</param>
+                </command_interface>
+                <state_interface name="position"/>
+                <state_interface name="velocity"/>
+            </joint>
+        </ros2_control>
+        <link name="${link_name}">
+            <inertial>
+                <origin xyz="${link_origin_x} ${link_origin_y} ${link_origin_z}" />
+                <mass value="${m}" />
+                <xacro:box_inertia_robot m="${m}" x="${x}" y="${y}" z="${z}"/>
+            </inertial>
+            <visual>
+                <origin xyz="${link_origin_x} ${link_origin_y} ${link_origin_z}" />
+                <geometry>
+                    <box size="${x} ${y} ${z}"/>
+                </geometry>
+            </visual>
+            <collision>
+                <origin xyz="${link_origin_x} ${link_origin_y} ${link_origin_z}" />
+                <geometry>
+                    <box size="${x} ${y} ${z}"/>
+                </geometry>
+            </collision>
+        </link>
+        <gazebo reference="${link_name}">
+            <visual>
+                <material>
+                    <!-- RGBA -->
+                    <ambient>${r} ${g} ${b} 1</ambient>
+                    <diffuse>${r} ${g} ${b} 1</diffuse>
+                    <specular>${r} ${g} ${b} 1</specular>
+                </material>
+            </visual>
+        </gazebo>
     </xacro:macro>
 </robot>

File: src/ros2/robot_description/rb_theron_common/rb_theron_description/urdf/door_opening_mechanism/components/freely_rotating_hook.urdf.xacro (robot description, xacro)
@@ -15,4 +15,6 @@
             friction="0.1"
             ros2_control_hardware_type="${ros2_control_hardware_type}"
+            port="0"
+            direction="0"
             link_name="${prefix}door_opening_mechanism_link_freely_rotating_hook"
             link_origin_x="0.0"

File: src/ros2/robot_description/rb_theron_common/rb_theron_description/urdf/door_opening_mechanism/door_opening_mechanism.urdf.xacro (robot description, xacro)
@@ -69,4 +69,6 @@
             friction="0.3"
             ros2_control_hardware_type="${ros2_control_hardware_type}"
+            port="3502"
+            direction="1"
             link_name="${prefix}door_opening_mechanism_link_y_axis_slide"
             link_origin_x="0.0"
@@ -94,4 +96,6 @@
             friction="0.3"
             ros2_control_hardware_type="${ros2_control_hardware_type}"
+            port="3503"
+            direction="-1"
             link_name="${prefix}door_opening_mechanism_link_x_axis_slide"
             link_origin_x="0.0"

Commit message: feat: set a individual ip for each dryve d1 motor control as we need this for running it on the robot

File: src/ros2/robot_description/rb_theron_common/rb_theron_description/urdf/door_opening_mechanism/arm_variations/rotating_arm.urdf.xacro (robot description, xacro)
@@ -19,4 +19,5 @@
             friction="0.3"
             ros2_control_hardware_type="${ros2_control_hardware_type}"
+            ip_address="192.168.0.12"
             port="0"
             direction="0"

File: src/ros2/robot_description/rb_theron_common/rb_theron_description/urdf/door_opening_mechanism/basic_elements/basic_joint.urdf.xacro (robot description, xacro)
@@ -5,78 +5,109 @@
         <inertia ixx="${m*(y*y+z*z)/12}" ixy = "0" ixz = "0" iyy="${m*(x*x+z*z)/12}" iyz = "0" izz="${m*(x*x+y*y)/12}" />
     </xacro:macro>
-    <xacro:macro name="basic_joint" params="parent joint_name joint_type axis_x axis_y axis_z lower_limit upper_limit damping friction ros2_control_hardware_type port direction ros_distro link_name link_origin_x link_origin_y link_origin_z m x y z r g b *origin">
-        <joint name="${joint_name}" type="${joint_type}">
-            <axis xyz="${axis_x} ${axis_y} ${axis_z}" />
-            <parent link="${parent}" />
-            <child link="${link_name}" />
-            <limit lower="${lower_limit}" upper="${upper_limit}" effort="1000" velocity="100" />
-            <dynamics damping="${damping}" friction="${friction}"/>
-            <xacro:insert_block name="origin" />
-        </joint>
-        <ros2_control name="${joint_name}_ros2_control" type="system">
-            <hardware>
-                <xacro:if value="${ros2_control_hardware_type == 'mock_components'}">
+    <xacro:macro
+        name="basic_joint"
+        params="
+            parent
+            joint_name
+            joint_type
+            axis_x
+            axis_y
+            axis_z
+            lower_limit
+            upper_limit
+            damping
+            friction
+            ros2_control_hardware_type
+            ip_address
+            port
+            direction
+            ros_distro
+            link_name
+            link_origin_x
+            link_origin_y
+            link_origin_z
+            m
+            x
+            y
+            z
+            r
+            g
+            b
+            *origin">
+    </xacro:macro>
+    <joint name="${joint_name}" type="${joint_type}">
+        <axis xyz="${axis_x} ${axis_y} ${axis_z}" />
+        <parent link="${parent}" />
+        <child link="${link_name}" />
+        <limit lower="${lower_limit}" upper="${upper_limit}" effort="1000" velocity="100" />
+        <dynamics damping="${damping}" friction="${friction}"/>
+        <xacro:insert_block name="origin" />
+    </joint>
+    <ros2_control name="${joint_name}_ros2_control" type="system">
+        <hardware>
+            <xacro:if value="${ros2_control_hardware_type == 'mock_components'}">
+                <plugin>mock_components/GenericSystem</plugin>
+                <param name="calculate_dynamics">true</param>
+            </xacro:if>
+            <xacro:if value="${ros2_control_hardware_type == 'gz_ros2_control'}">
+                <xacro:if value="${ros_distro == 'humble'}">
+                    <plugin>ign_ros2_control/IgnitionSystem</plugin>
+                </xacro:if>
+                <xacro:unless value="${ros_distro == 'humble'}">
+                    <plugin>gz_ros2_control/GazeboSimSystem</plugin>
+                </xacro:unless>
+            </xacro:if>
+            <xacro:if value="${ros2_control_hardware_type == 'dryve_d1'}">
+                <!-- if the value for the port is zero, there is no dryve_d1 for this joint yet so we mock it -->
+                <xacro:if value="${port == 0}">
                     <plugin>mock_components/GenericSystem</plugin>
                     <param name="calculate_dynamics">true</param>
                 </xacro:if>
-                <xacro:if value="${ros2_control_hardware_type == 'gz_ros2_control'}">
-                    <xacro:if value="${ros_distro == 'humble'}">
-                        <plugin>ign_ros2_control/IgnitionSystem</plugin>
-                    </xacro:if>
-                    <xacro:unless value="${ros_distro == 'humble'}">
-                        <plugin>gz_ros2_control/GazeboSimSystem</plugin>
-                    </xacro:unless>
-                </xacro:if>
-                <xacro:if value="${ros2_control_hardware_type == 'dryve_d1'}">
-                    <!-- if the value for the port is zero, there is no dryve_d1 for this joint yet so we mock it -->
-                    <xacro:if value="${port == 0}">
-                        <plugin>mock_components/GenericSystem</plugin>
-                        <param name="calculate_dynamics">true</param>
-                    </xacro:if>
-                    <xacro:unless value="${port == 0}">
-                        <plugin>ros2_control_plugin_door_opening_mechanism/DoorOpeningMechanismSystemHardware</plugin>
-                        <param name="port">${port}</param>
-                        <param name="direction">${direction}</param>
-                    </xacro:unless>
-                </xacro:if>
-            </hardware>
-            <joint name="${joint_name}">
-                <command_interface name="velocity">
-                    <param name="min">-10</param>
-                    <param name="max">10</param>
-                </command_interface>
-                <state_interface name="position"/>
-                <state_interface name="velocity"/>
-            </joint>
-        </ros2_control>
-        <link name="${link_name}">
-            <inertial>
-                <origin xyz="${link_origin_x} ${link_origin_y} ${link_origin_z}" />
-                <mass value="${m}" />
-                <xacro:box_inertia_robot m="${m}" x="${x}" y="${y}" z="${z}"/>
-            </inertial>
-            <visual>
-                <origin xyz="${link_origin_x} ${link_origin_y} ${link_origin_z}" />
-                <geometry>
-                    <box size="${x} ${y} ${z}"/>
-                </geometry>
-            </visual>
-            <collision>
-                <origin xyz="${link_origin_x} ${link_origin_y} ${link_origin_z}" />
-                <geometry>
-                    <box size="${x} ${y} ${z}"/>
-                </geometry>
-            </collision>
-        </link>
-        <gazebo reference="${link_name}">
-            <visual>
-                <material>
-                    <!-- RGBA -->
-                    <ambient>${r} ${g} ${b} 1</ambient>
-                    <diffuse>${r} ${g} ${b} 1</diffuse>
-                    <specular>${r} ${g} ${b} 1</specular>
-                </material>
-            </visual>
-        </gazebo>
-    </xacro:macro>
+                <xacro:unless value="${port == 0}">
+                    <plugin>ros2_control_plugin_door_opening_mechanism/DoorOpeningMechanismSystemHardware</plugin>
+                    <param name="ip_address">${ip_address}</param>
+                    <param name="port">${port}</param>
+                    <param name="direction">${direction}</param>
+                </xacro:unless>
+            </xacro:if>
+        </hardware>
+        <joint name="${joint_name}">
+            <command_interface name="velocity">
+                <param name="min">-10</param>
+                <param name="max">10</param>
+            </command_interface>
+            <state_interface name="position"/>
+            <state_interface name="velocity"/>
+        </joint>
+    </ros2_control>
+    <link name="${link_name}">
+        <inertial>
+            <origin xyz="${link_origin_x} ${link_origin_y} ${link_origin_z}" />
+            <mass value="${m}" />
+            <xacro:box_inertia_robot m="${m}" x="${x}" y="${y}" z="${z}"/>
+        </inertial>
+        <visual>
+            <origin xyz="${link_origin_x} ${link_origin_y} ${link_origin_z}" />
+            <geometry>
+                <box size="${x} ${y} ${z}"/>
+            </geometry>
+        </visual>
+        <collision>
+            <origin xyz="${link_origin_x} ${link_origin_y} ${link_origin_z}" />
+            <geometry>
+                <box size="${x} ${y} ${z}"/>
+            </geometry>
+        </collision>
+    </link>
+    <gazebo reference="${link_name}">
+        <visual>
+            <material>
+                <!-- RGBA -->
+                <ambient>${r} ${g} ${b} 1</ambient>
+                <diffuse>${r} ${g} ${b} 1</diffuse>
+                <specular>${r} ${g} ${b} 1</specular>
+            </material>
+        </visual>
+    </gazebo>
+</xacro:macro>
 </robot>

File: src/ros2/robot_description/rb_theron_common/rb_theron_description/urdf/door_opening_mechanism/components/freely_rotating_hook.urdf.xacro (robot description, xacro)
@@ -15,4 +15,5 @@
             friction="0.1"
             ros2_control_hardware_type="${ros2_control_hardware_type}"
+            ip_address="0"
             port="0"
             direction="0"

File: src/ros2/robot_description/rb_theron_common/rb_theron_description/urdf/door_opening_mechanism/door_opening_mechanism.urdf.xacro (robot description, xacro)
@@ -69,4 +69,5 @@
             friction="0.3"
             ros2_control_hardware_type="${ros2_control_hardware_type}"
+            ip_address="192.168.0.11"
             port="3502"
             direction="1"
@@ -97,4 +98,5 @@
             friction="0.3"
             ros2_control_hardware_type="${ros2_control_hardware_type}"
+            ip_address="192.168.0.53"
             port="3503"
             direction="-1"
