Commit message: refactor: adapts door_opening_mechanism to the latest hardware changes

File: src/ros2/robot_description/rb_theron_common/rb_theron_description/urdf/door_opening_mechanism/arm_variations/rotating_arm.urdf.xacro (robot description, xacro)
@@ -29,6 +29,6 @@
             link_origin_z="${arm_length/2}"
             m="0.2"
-            x="0.03"
-            y="0.03"
+            x="0.02"
+            y="0.05"
             z="${arm_length}"
             r="0"
@@ -51,5 +51,5 @@
             g="1"
             b="0">
-            <origin xyz="0.020 0.0 ${arm_length-0.015}" rpy="0 0 0"/>
+            <origin xyz="-0.015 0.0 ${arm_length-0.015}" rpy="0 3.14159265359 0"/>
         </xacro:basic_box>
         <!-- Gripper -->

File: src/ros2/robot_description/rb_theron_common/rb_theron_description/urdf/door_opening_mechanism/door_opening_mechanism.urdf.xacro (robot description, xacro)
@@ -64,6 +64,6 @@
             axis_y="0"
             axis_z="1"
-            lower_limit="-0.05"
-            upper_limit="0.25"
+            lower_limit="-0.01"
+            upper_limit="0.40"
             damping="0.1"
             friction="0.3"
@@ -79,7 +79,7 @@
             link_origin_z="0.0"
             m="2.64"
-            x="0.06"
+            x="0.045"
             y="0.55"
-            z="0.06"
+            z="0.108"
             r="1"
             g="0"
@@ -94,6 +94,6 @@
             axis_y="0"
             axis_z="1"
-            lower_limit="-0.175"
-            upper_limit="0.20"
+            lower_limit="-0.01"
+            upper_limit="0.30"
             damping="0.1"
             friction="0.3"
@@ -111,22 +111,22 @@
             x="0.065"
             y="0.015"
-            z="0.175"
+            z="0.10"
             r="1"
             g="1"
             b="1">
-            <origin xyz="-0.04 0 0" rpy="1.57079632679 4.71238898038 0"/>
+            <origin xyz="-0.032 0 0" rpy="1.57079632679 4.71238898038 0"/>
         </xacro:basic_joint>
         <xacro:basic_box
             parent="${prefix}door_opening_mechanism_link_x_axis_slide"
-            joint_name="${prefix}door_opening_mechanism_joint_x_axis_slide_screwing"
-            link_name="${prefix}door_opening_mechanism_link_x_slide_screwing"
+            joint_name="${prefix}door_opening_mechanism_rotating_arm_mounting_plate"
+            link_name="${prefix}door_opening_mechanism_rotating_arm_mounting_plate"
             m="1"
-            x="0.073"
-            y="0.015"
-            z="0.175"
+            x="0.145"
+            y="0.05"
+            z="0.05"
             r="1"
             g="1"
             b="1">
-            <origin xyz="0.038 -0.027 0" rpy="0 0 1.57079632679"/>
+            <origin xyz="0 0.033 0" rpy="0 0 0"/>
         </xacro:basic_box>
         <!-- Tilting arm -->
@@ -139,9 +139,9 @@
         <xacro:rotating_arm
             prefix="${prefix}"
-            parent="door_opening_mechanism_link_x_slide_screwing"
+            parent="door_opening_mechanism_rotating_arm_mounting_plate"
             ros2_control_hardware_type="${ros2_control_hardware_type}"
             ros_distro="${ros_distro}"
             arm_length="0.3" >
-            <origin xyz="0.05 -0.025 0" rpy="0 0 1.57079632679"/>
+            <origin xyz="-0.083 0 0" rpy="3.14159265359 0 0"/>
         </xacro:rotating_arm>
     </xacro:macro>

Commit message: chore: gently reduces size of hook

File: src/ros2/robot_description/rb_theron_common/rb_theron_description/urdf/door_opening_mechanism/arm_variations/rotating_arm.urdf.xacro (robot description, xacro)
@@ -60,5 +60,5 @@
             ros2_control_hardware_type="${ros2_control_hardware_type}"
             ros_distro="${ros_distro}">
-            <origin xyz="0.020 0.0 0.0" rpy="0 0 0"/>
+            <origin xyz="0.010 0.0 0.0" rpy="0 0 0"/>
         </xacro:freely_rotating_hook>
     </xacro:macro>

File: src/ros2/robot_description/rb_theron_common/rb_theron_description/urdf/door_opening_mechanism/components/freely_rotating_hook.urdf.xacro (robot description, xacro)
@@ -25,5 +25,5 @@
             link_origin_z="0.0"
             m="0.2"
-            x="0.03"
+            x="0.01"
             y="0.03"
             z="0.03"
@@ -36,5 +36,5 @@
         <xacro:include filename="$(find rb_theron_description)/urdf/door_opening_mechanism/components/hook.urdf.xacro" />
         <xacro:hook prefix="${prefix}" suffix="" parent="door_opening_mechanism_link_freely_rotating_hook" r="1" g="0" b="1">
-            <origin xyz="0.01 0.0 0.0" rpy="0 0 -1.57079632679"/>
+            <origin xyz="0.0 0.0 0.0" rpy="0 0 -1.57079632679"/>
         </xacro:hook>
     </xacro:macro>
