Commit message: adding collision to base_footprint

File: src/ros2/robot_description/rb_theron_common/rb_theron_description/urdf/bases/theron_base.urdf.xacro (robot description, xacro)
@@ -20,4 +20,10 @@
           </geometry>
         </visual>
+        <collision>
+          <origin xyz="0 0 0" rpy="0 0 0" />
+          <geometry>
+            <box size="0.001 0.001 0.001" />
+          </geometry>
+        </collision>
       </link>
       <joint name="${prefix}base_footprint_joint" type="fixed">

Commit message: Changing base link mass and inertia to enable all wheels contact to the ground

File: src/ros2/robot_description/rb_theron_common/rb_theron_description/urdf/bases/theron_base.urdf.xacro (robot description, xacro)
@@ -36,7 +36,7 @@
     <link name="${prefix}base_link">
       <inertial>
-        <mass value="50.0" />
-        <origin xyz="-0.120 0 0" />
-	    <xacro:box_inertia_robot m="50" x="0.700" y="0.600" z="0.350"/>
+        <mass value="45" />
+        <origin xyz="0.0 0.0 0.0" />
+	    <xacro:solid_cuboid_inertia m="45" w="0.3275" h="0.2775" d="0.1525" />
       </inertial>
       <visual>

Commit message: Changing base_link collision size to prevent collision with the supporting wheels

File: src/ros2/robot_description/rb_theron_common/rb_theron_description/urdf/bases/theron_base.urdf.xacro (robot description, xacro)
@@ -48,7 +48,7 @@
         </xacro:if>
         <xacro:unless value="${hq}">
-          <origin xyz="0 0 0.05" rpy="0 0 0" />
+          <origin xyz="0 0 0.105" rpy="0 0 0" />
           <geometry>
-            <box size="0.390 0.240 0.165"/>
+            <box size="0.390 0.240 0.140"/>
           </geometry>
         </xacro:unless>
@@ -58,7 +58,7 @@
       </visual>
       <collision>
-        <origin xyz="0 0 0.05" rpy="0 0 0 " />
+        <origin xyz="0 0 0.105" rpy="0 0 0 " />
         <geometry>
-          <box size="0.390 0.240 0.165"/>
+          <box size="0.390 0.240 0.140"/>
           <!-- <mesh filename="$(find rb_theron_description)/meshes/bases/theron_base.stl"/> -->
         </geometry>

Commit message: chore: reducing collision geometry just like visual geometry

File: src/ros2/robot_description/rb_theron_common/rb_theron_description/urdf/bases/theron_base.urdf.xacro (robot description, xacro)
@@ -58,5 +58,5 @@
         <origin xyz="0 0 0.105" rpy="0 0 0 " />
         <geometry>
-          <box size="0.390 0.240 0.165"/>
+          <box size="0.390 0.240 0.140"/>
           <!-- <mesh filename="(find rb_theron_description)/meshes/bases/theron_base.dae"/> -->
         </geometry>

Commit message: feat: adds position ros2_control interface

File: src/ros2/robot_description/rb_theron_common/rb_theron_description/urdf/bases/theron_base.urdf.xacro (robot description, xacro)
@@ -9,4 +9,15 @@
     <xacro:property name="PI" value="3.1415926535897931"/>
     <!-- xacro:property name="wheel_width" value="0.150" / -->
+    <ros2_control name="position_ros2_control" type="system">
+      <hardware>
+          <plugin>fake_components/GenericSystem</plugin>
+      </hardware>
+      <joint name="position">
+          <param name="initial_position">0.0 0.0 0.0</param>
+          <command_interface name="position" />
+          <state_interface name="position"/>
+          <state_interface name="velocity"/>
+      </joint>
+    </ros2_control>
     <!-- BASE FOOTPRINT -->
     <xacro:if value="${publish_bf}">

Commit message: chore: changes type for position to planar

File: src/ros2/robot_description/rb_theron_common/rb_theron_description/urdf/bases/theron_base.urdf.xacro (robot description, xacro)
@@ -13,5 +13,5 @@
           <plugin>fake_components/GenericSystem</plugin>
       </hardware>
-      <joint name="position">
+      <joint name="position" type="planar">
           <param name="initial_position">0.0 0.0 0.0</param>
           <command_interface name="position" />

Commit message: feat: adds position_link and the option to model_position_joint

File: src/ros2/robot_description/rb_theron_common/rb_theron_description/urdf/bases/theron_base.urdf.xacro (robot description, xacro)
@@ -26,8 +26,32 @@
       </link>
       <xacro:if value="${model_position_joint}">
+        <joint name="${prefix}base_footprint_joint" type="fixed">
+          <origin xyz="0 0 ${wheel_radius - wheel_offset_z}" rpy="0 0 0" />
+          <parent link="${prefix}base_footprint"/>
+          <child link="${prefix}position_link"/>
+        </joint>
+        <link name="${prefix}position_link">
+          <inertial>
+            <mass value="0.01" />
+            <origin xyz="0.0 0.0 0.0" />
+            <xacro:solid_cuboid_inertia m="0.01" w="0.001" h="0.001" d="0.001" />
+          </inertial>
+          <visual>
+            <origin xyz="0 0 0.01" rpy="0 0 0" />
+            <geometry>
+              <box size="0.001 0.001 0.001" />
+            </geometry>
+          </visual>
+          <collision>
+            <origin xyz="0 0 0.01" rpy="0 0 0" />
+            <geometry>
+              <box size="0.001 0.001 0.001" />
+            </geometry>
+          </collision>
+        </link>
         <joint name="position" type="prismatic">
           <axis xyz="-1 0 0" />
-          <origin xyz="0 0 ${wheel_radius - wheel_offset_z}" rpy="0 0 0" />
-          <parent link="${prefix}base_footprint"/>
+          <origin xyz="0 0 0" rpy="0 0 0" />
+          <parent link="${prefix}position_link"/>
           <child link="${prefix}base_link"/>
           <limit lower="-1" upper="1" effort="1000" velocity="100" />
@@ -40,6 +64,9 @@
               <param name="calculate_dynamics">true</param>
             </xacro:if>
-            <xacro:if value="${ros2_control_hardware_type_positon_joint == 'linear_base_movement'}">
-              <plugin>ros2_control_plugin_linear_base_movement/LinearBaseMovementSystemHardware</plugin>
+            <xacro:if value="${ros2_control_hardware_type_positon_joint == 'gz_ros2_control'}">
+              <plugin>gz_ros2_control_base_movement/BaseMovementSystemHardware</plugin>
+            </xacro:if>
+            <xacro:if value="${ros2_control_hardware_type_positon_joint == 'real_life'}">
+              <plugin>ros2_control_base_movement/BaseMovementSystemHardware</plugin>
             </xacro:if>
           </hardware>

Commit message: refactor: renames joint `position` to `position_joint`

File: src/ros2/robot_description/rb_theron_common/rb_theron_description/urdf/bases/theron_base.urdf.xacro (robot description, xacro)
@@ -50,5 +50,5 @@
           </collision>
         </link>
-        <joint name="position" type="prismatic">
+        <joint name="position_joint" type="prismatic">
           <axis xyz="-1 0 0" />
           <origin xyz="0 0 0" rpy="0 0 0" />
@@ -71,5 +71,5 @@
             </xacro:if>
           </hardware>
-          <joint name="position" type="prismatic">
+          <joint name="position_joint" type="prismatic">
               <param name="initial_position">0.0</param>
               <command_interface name="position" />

Commit message: refactor: moves `position_ros2_control` configs into separate file

File: src/ros2/robot_description/rb_theron_common/rb_theron_description/urdf/bases/theron_base.urdf.xacro (robot description, xacro)
@@ -132,39 +132,9 @@
       </xacro:if>
       <xacro:if value="${model_door_opening_mechanism}">
-        <ros2_control name="position_ros2_control" type="system">
-          <hardware>
-            <xacro:if value="${ros2_control_hardware_type_positon_joint == 'mock_components'}">
-              <plugin>mock_components/GenericSystem</plugin>
-              <param name="calculate_dynamics">true</param>
-            </xacro:if>
-            <xacro:if value="${ros2_control_hardware_type_positon_joint == 'gz_ros2_control'}">
-              <xacro:if value="${ros_distro == 'humble'}">
-                <plugin>ign_ros2_control_base_movement/IgnBaseMovementSystemHardware</plugin>
-                <param name="odom_topic">/diff_drive_base_controller/odom</param>
-                <param name="enable_state_feedback">false</param>
-                <param name="reset_position_state_after_each_trajectory">true</param>
-              </xacro:if>
-              <xacro:unless value="${ros_distro == 'humble'}">
-                <plugin>gz_ros2_control_base_movement/GzBaseMovementSystemHardware</plugin>
-                <param name="odom_topic">/diff_drive_base_controller/odom</param>
-                <param name="enable_state_feedback">false</param>
-                <param name="reset_position_state_after_each_trajectory">true</param>
-              </xacro:unless>
-            </xacro:if>
-            <xacro:if value="${ros2_control_hardware_type_positon_joint == 'real_life'}">
-              <plugin>ros2_control_base_movement/BaseMovementSystemHardware</plugin>
-              <param name="odom_topic">/diff_drive_base_controller/odom</param>
-              <param name="enable_state_feedback">false</param>
-              <param name="reset_position_state_after_each_trajectory">true</param>
-            </xacro:if>
-          </hardware>
-          <joint name="position_joint" type="prismatic">
-              <param name="initial_position">0.0</param>
-              <command_interface name="position" />
-              <command_interface name="velocity" />
-              <state_interface name="position"/>
-              <state_interface name="velocity"/>
-          </joint>
-        </ros2_control>
+        <xacro:include filename="$(find rb_theron_description)/urdf/door_opening_mechanism/ros2_control/position_ros2_control.urdf.xacro" />
+        <xacro:position_ros2_control
+            ros2_control_hardware_type_positon_joint="${ros2_control_hardware_type_positon_joint}"
+            ros_distro="${ros_distro}">
+        </xacro:position_ros2_control>
       </xacro:if>
     </xacro:if>

Commit message: fix: increase joint limit for `position_joint`

File: src/ros2/robot_description/rb_theron_common/rb_theron_description/urdf/bases/theron_base.urdf.xacro (robot description, xacro)
@@ -32,5 +32,5 @@
           <parent link="${prefix}base_footprint"/>
           <child link="${prefix}base_link"/>
-          <limit lower="-1" upper="1" effort="1000" velocity="100" />
+          <limit lower="-3.0" upper="3.0" effort="1000" velocity="100" />
         </joint>
       </xacro:if>
