Commit message: Update ZED camera launch configuration and Docker Compose file for Jetson bringup

File: bringups/jetson/zed_setup/zed_descr.urdf.xacro (robot description, xacro)
@@ -16,19 +16,26 @@
 -->
 <robot name="stereolabs_camera" xmlns:xacro="http://ros.org/wiki/xacro">
-  <xacro:arg name="camera_name"   default="zed" />
+  <xacro:arg name="camera_name"   default="robot/zed" />
   <xacro:arg name="camera_model"  default="zed" />
+  <xacro:arg name="custom_baseline"  default="0.0" />
+  <!-- If GNSS fusion is enabled the position of the antenna with respect to the camera mount point is required -->
+  <xacro:arg name="enable_gnss"   default="false" />
+  <xacro:arg name="gnss_x" default="0.0" />
+  <xacro:arg name="gnss_y" default="0.0" />
+  <xacro:arg name="gnss_z" default="0.0" />
   <xacro:include filename="$(find zed_wrapper)/urdf/zed_macro.urdf.xacro" />
-  <xacro:zed_camera name="$(arg camera_name)" model="$(arg camera_model)">
+  <xacro:zed_camera name="$(arg camera_name)" model="$(arg camera_model)" custom_baseline="$(arg custom_baseline)" enable_gnss="$(arg enable_gnss)">
+	    <origin xyz="$(arg gnss_x) $(arg gnss_y) $(arg gnss_z)" rpy="0 0 0"/>
   </xacro:zed_camera>
   <!-- Add a joint to connect the ZED Camera to the robot -->
-  <link name="robot_base_link"/>
+  <!-- <link name="robot/base_link"/> -->
   <!-- NO ZED Localization -> '$(arg camera_name)_camera_link' is a child of 'base_link' -->
-  <joint name="$(arg camera_name)_joint" type="fixed">
-    <parent link="robot_base_link"/>
+  <!-- <joint name="$(arg camera_name)_joint" type="fixed">
+    <parent link="robot/base_link"/>
     <child link="$(arg camera_name)_camera_link"/>
     <origin
-      xyz="0.341 -0.18 1.15"
-      rpy="3.14 0 0"
+      xyz="0.27 0 1.40"
+      rpy="0 0.436 0"
     />
-  </joint>
+  </joint> -->
 </robot>

Commit message: Update ZED camera launch file and Dockerfile for Jetson bringup

File: bringups/jetson/zed_setup/zed_descr.urdf.xacro (robot description, xacro)
@@ -16,18 +16,18 @@
 -->
 <robot name="stereolabs_camera" xmlns:xacro="http://ros.org/wiki/xacro">
-  <xacro:arg name="camera_name"   default="zed" />
-  <xacro:arg name="camera_model"  default="zed" />
+  <xacro:arg name="camera_name"   default="zed2" />
+  <xacro:arg name="camera_model"  default="zed2" />
   <xacro:include filename="$(find zed_wrapper)/urdf/zed_macro.urdf.xacro" />
   <xacro:zed_camera name="$(arg camera_name)" model="$(arg camera_model)">
   </xacro:zed_camera>
   <!-- Add a joint to connect the ZED Camera to the robot -->
-  <link name="robot_base_link"/>
+  <link name="robot/base_link"/>
   <!-- NO ZED Localization -> '$(arg camera_name)_camera_link' is a child of 'base_link' -->
   <joint name="$(arg camera_name)_joint" type="fixed">
-    <parent link="robot_base_link"/>
+    <parent link="robot/base_link"/>
     <child link="$(arg camera_name)_camera_link"/>
     <origin
-      xyz="0.341 -0.18 1.15"
-      rpy="3.14 0 0"
+      xyz="0.27 0 1.40"
+		  rpy="0 0.436 0"
     />
   </joint>

Commit message: serveral changes to fix the zed camera

File: bringups/jetson/zed_setup/zed_descr.urdf.xacro (robot description, xacro)
@@ -29,7 +29,7 @@
   </xacro:zed_camera>
   <!-- Add a joint to connect the ZED Camera to the robot -->
-  <!-- <link name="robot/base_link"/> -->
+  <link name="robot/base_link"/>
   <!-- NO ZED Localization -> '$(arg camera_name)_camera_link' is a child of 'base_link' -->
-  <!-- <joint name="$(arg camera_name)_joint" type="fixed">
+  <joint name="$(arg camera_name)_joint" type="fixed">
     <parent link="robot/base_link"/>
     <child link="$(arg camera_name)_camera_link"/>
@@ -38,4 +38,4 @@
       rpy="0 0.436 0"
     />
-  </joint> -->
+  </joint>
 </robot>
